File: ECAD/SCART_switcher/SCART_input.kicad_sch (KiCad schematic)
At the start: 10 parts, among them J1 SCART-F, Q1 BC847, Q2 BC847

Commit message: Update SCART_input.kicad_sch
Parts:
- added R13, R14, R15, R16: 75R, symbol Device:R
- added U1: THS7374, Package_SO:TSSOP-14_4.4x5mm_P0.65mm, symbol Amplifier_Video:THS7374
Connections:
- net +3.3V: now also U1.10 (V_{S+})
- net BLUE: now also R16.1, U1.4 (CH4_IN)
- net GND: now also R13.2, R14.2, R15.2, R16.2, U1.5 (GND)
- net GREEN: now also R15.1, U1.3 (CH3_IN)
- net RED: now also R14.1, U1.2 (CH2_IN)
- net VIDEO/RGB_SYNC: now also R13.1, U1.1 (CH1_IN)
Other:
- moved on the sheet: J1

Commit message: progressed ECAD
Parts:
- added C3: C_Small, symbol Device:C_Small
- added JP1: Jumper, Connector_PinHeader_2.54mm:PinHeader_1x03_P2.54mm_Vertical, symbol Jumper:Jumper_3_Open
- added R8: 3kR, symbol Device:R
- renumbered R16 to R1, R4 to R10, R6 to R11, R15 to R2, R14 to R3, R13 to R4, R1 to R5, R2 to R6, R3 to R7, R5 to R9
Connections:
- net GND: now also R8.2
- net VIDEO/RGB_SYNC: now also C3.1; no longer R4.1, U1.1 (CH1_IN)
- net at Q2.1 (B), R10.2: now also JP1.2 (C); no longer R9.1
- new net: C3.2, R4.1, U1.1 (CH1_IN)
- new net: JP1.3 (B), R8.1
- new net: JP1.1 (A), R9.1
Other:
- note added: "16:9 mode detect"
- note added: "Function detection and override"
- note added: "SCART input"
- note added: "Video/Audio signals buffer"
- note added: "force 4:3 mode"
- moved on the sheet: Q2, R1, R10, R11, R2, R3, R4, R9, U1

Commit message: progressed ecad
Parts:
- J1: footprint (none) -> SCART:SCART-F
Changed lines of the file:
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@@
       (effects (font (size 1.27 1.27)))
     )
-    (property "Footprint" "" (at 75.692 70.358 0)
+    (property "Footprint" "SCART:SCART-F" (at 75.692 70.358 0)
       (effects (font (size 1.27 1.27)) hide)
     )

Commit message: Progressed ECAD
Parts:
- removed C3: C_Small, symbol Device:C_Small
- added C3, C5, C6, C7: 0.1uC, symbol Device:C
- added C8: 100nC, Capacitor_SMD:C_0805_2012Metric_Pad1.18x1.45mm_HandSolder, symbol Device:C
- added R20, R21, R22, R23: 75R, Resistor_SMD:R_0805_2012Metric_Pad1.20x1.40mm_HandSolder, symbol Device:R
- C1: footprint (none) -> Capacitor_SMD:C_0805_2012Metric_Pad1.18x1.45mm_HandSolder
- R1, R10, R11, R2, R3, R4, R5, R6, R7, R8, R9: footprint (none) -> Resistor_SMD:R_0805_2012Metric_Pad1.20x1.40mm_HandSolder
Connections:
- net AUDIO_COM_GND is gone; now on net GND: J1.4 (P4)
- net BLANKING_GND is gone; now on net GND: J1.14 (P14)
- net BLUE_GND is gone; now on net GND: J1.5 (P5)
- net GREEN_GND is gone; now on net GND: J1.9 (P9)
- net RED_GND is gone; now on net GND: J1.13 (P13)
- net VIDEO_GND is gone; now on net GND: J1.18 (P18)
- net +3.3V: now also C8.1
- net BLUE: now also R2.1, C7.1, R20.2; no longer U1.4 (CH4_IN)
- net GND: now also C8.2
- net GREEN: now also C6.1, R21.2; no longer R2.1, U1.3 (CH3_IN)
- net RED: now also C5.1, R22.2; no longer U1.2 (CH2_IN)
- net VIDEO/RGB_SYNC: now also R4.1, C3.1, R23.2
- net at U1.1 (CH1_IN): now also C3.2; no longer R4.1
- net at U1.11 (CH4_OUT): now also R20.1
- net at U1.12 (CH3_OUT): now also R21.1
- net at U1.13 (CH2_OUT): now also R22.1
- net at U1.14 (CH1_OUT): now also R23.1
- net IN_DISABLE: now reaches U1.6 (DISABLE)
- new net: C5.2, U1.2 (CH2_IN)
- new net: C6.2, U1.3 (CH3_IN)
- new net: C7.2, U1.4 (CH4_IN)
Other:
- note added: "Video signals buffer"
- note removed: "Video/Audio signals buffer"
- moved on the sheet: C1, J1, JP1, Q1, Q2, R1, R10, R11, R2, R3, R4, R5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

Commit message: Progressed ECAD.
Parts:
- added C6: 100nC, Capacitor_SMD:C_0805_2012Metric_Pad1.18x1.45mm_HandSolder, symbol Device:C
- added Q1: BC847, Package_TO_SOT_SMD:SOT-23, symbol Transistor_BJT:BC847
- added R3: 50R, Resistor_SMD:R_0805_2012Metric_Pad1.20x1.40mm_HandSolder, symbol Device:R
- added R4: 25R, Resistor_SMD:R_0805_2012Metric_Pad1.20x1.40mm_HandSolder, symbol Device:R
- added R7: 4k7R, Resistor_SMD:R_0805_2012Metric_Pad1.20x1.40mm_HandSolder, symbol Device:R
- added U8: 74AHC1G08, symbol 74xGxx:74AHC1G08
- renumbered C3 to C1, C5 to C2, C6 to C3, C7 to C4, C8 to C5, C1 to C7, Q1 to Q2, Q2 to Q3, R21 to R10, R20 to R11, R5 to R12, R6 to R13, R7 to R14, R8 to R15, R10 to R16, R9 to R17, R11 to R18, R3 to R5, R4 to R6, R23 to R8, R22 to R9
Connections:
- net +3.3V: now also C6.1, R7.1, U8.5 (VCC)
- net BLANKING: now also R3.1, U8.4
- net GND: now also C6.2, Q1.2 (E), R4.2, U8.3 (GND)
- net IN_DISABLE renamed IN_ENABLE
- net IN_ENABLE: now also U8.1
- new net: Q1.3 (C), R7.2, U8.2
- new net: Q1.1 (B), R3.2, R4.1
Other:
- note added: "(*1)"
- note added: "(*1) Level 0: 0 V to +2 V (TV mode) Level 1A: +4,5 V to +7 V (AV mode, aspect ratio 16.9) Level 1B: +9,5 V to +12 V (AV mode)"
- note added: "(*2)"
- note added: "(*2) The input terminal FUNCTION of the voltage monitoring circuit has two outputs, FNC_IN1 and FNC_IN2, with voltages of 3.3V when the signal level input FUNCTION of the SCART interface is 0-2V (SCART off). When the functional selection control signal level is 4.5-7V (SCART on, 16:9), the voltage of the first output terminal FNC_IN1 is 0V, and the voltage of the second output terminal FNC_IN2 is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"
- note added: "(*3)"
- note added: "(*3) Level 0: 0 V to 0,4 V (Composite video mode) Level 1: +1 V to +3 V (RGB video mode)"
- note added: "Blanking signal buffer"
- note added: "Series equivalent to 75 ohms."
- note removed: "The input terminal FUNCTION of the voltage monitoring circuit has two outputs, FNC_IN1 and FNC_IN2, with voltages of 3.3V when the signal level input FUNCTION of the SCART interface is 0-2V (SCART off). When the functional selection control signal level is 4.5-7V (SCART on, 16:9), the voltage of the first output terminal FNC_IN1 is 0V, and the voltage of the second output terminal FNC_IN2 is 3.3V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"
- moved on the sheet: C1, C2, C3, C4, C5, J1, R1, R10, R11, R2, R5, R6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

Commit message: Progressed ECAD.
Parts:
- added C8: 100nC, Capacitor_SMD:C_0805_2012Metric_Pad1.18x1.45mm_HandSolder, symbol Device:C
- added U3: 74AHC1G00, symbol 74xGxx:74AHC1G00
- added U4: 74AHC1G02, symbol 74xGxx:74AHC1G02
- renumbered C7 to C6, C6 to C7
Connections:
- net +3.3V: now also C8.1, U3.5 (VCC), U4.5 (VCC)
- net FNC_IN1: now also U3.1, U4.1
- net FNC_IN2: now also U3.2, U4.2
- net GND: now also C8.2, U3.3 (GND), U4.3 (GND)
- new net IN_ACTIVE: U3.4
- new net VIDEO_4_3: U4.4
Other:
- note added: "(*4)"
- note added: "(*4) The IN_ACTIVE signal flags the existence of an active video source as function of FUNCTION signal voltage levels. FNC_IN1 FNC_IN2 IN_ACTIVE 0V 0V 3.3V 0V 3.3V 3.3V 3.3V 0V 3.3V 3.3V 3.3V 0V"
- note added: "(*5)"
- note added: "(*5) The VIDEO_4_3 signal flags whether the video source is configured in the 4:3 format as function of FUNCTION signal voltage levels. FNC_IN1 FNC_IN2 VIDEO_4_3 0V 0V 0V 0V 3.3V 3.3V 3.3V 0V 3.3V 3.3V 3.3V 3.3V"
- moved on the sheet: C6, C7, JP1, Q2, Q3, R12, R13, R14, R15, R16, R17, R18

Commit message: progressed ECAD
Other:
- note added: "(*5) The VIDEO_4_3 signal flags whether the video source is configured in the 4:3 format as function of FUNCTION signal voltage levels. FNC_IN1 FNC_IN2 VIDEO_4_3 0V 0V 3.3V 0V 3.3V 0V 3.3V 0V 0V 3.3V 3.3V 0V"
- note removed: "(*5) The VIDEO_4_3 signal flags whether the video source is configured in the 4:3 format as function of FUNCTION signal voltage levels. FNC_IN1 FNC_IN2 VIDEO_4_3 0V 0V 0V 0V 3.3V 3.3V 3.3V 0V 3.3V 3.3V 3.3V 3.3V"
Changed lines of the file:
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@@
     (effects (font (size 1.27 1.27)) (justify left bottom))
   )
-  (text "(*5)\nThe VIDEO_4_3 signal flags whether the video source is configured\nin the 4:3 format as function of FUNCTION signal voltage levels.\n\nFNC_IN1 FNC_IN2 VIDEO_4_3\n   0V      0V      0V\n   0V      3.3V    3.3V\n   3.3V    0V      3.3V\n   3.3V    3.3V    3.3V"
+  (text "(*5)\nThe VIDEO_4_3 signal flags whether the video source is configured\nin the 4:3 format as function of FUNCTION signal voltage levels.\n\nFNC_IN1 FNC_IN2 VIDEO_4_3\n   0V      0V      3.3V\n   0V      3.3V    0V\n   3.3V    0V      0V\n   3.3V    3.3V    0V"
     (at 111.76 96.52 0)
     (effects (font (size 1.27 1.27)) (justify left bottom))
@@
     )
   )
+  (symbol (lib_id "74xGxx:74AHC1G02") (at 224.79 130.81 0) (unit 1)
+    (in_bom yes) (on_board yes) (dnp no)
+    (property "Reference" "U4" (at 237.49 135.89 0)
+      (effects (font (size 1.27 1.27)))
+    )
+    (property "Value" "74AHC1G02" (at 237.49 133.35 0)
+      (effects (font (size 1.27 1.27)))
+    )
+    (property "Footprint" "" (at 224.79 130.81 0)
+      (effects (font (size 1.27 1.27)) hide)
+    )
+    (property "Datasheet" "http://www.ti.com/lit/sg/scyt129e/scyt129e.pdf" (at 224.79 130.81 0)
+      (effects (font (size 1.27 1.27)) hide)
+    )
+    (pin "1")
+    (pin "2")
+    (pin "3")
+    (pin "4")
+    (pin "5")
+    (instances
+      (project "SCART_switcher"
+        (path "/8cd08eb5-4755-4ef5-8eeb-77fd9974b180/6e53f4c9-ed59-4c5d-ac8d-a66f0d353ca7"
+          (reference "U4") (unit 1)
+        )
+        (path "/8cd08eb5-4755-4ef5-8eeb-77fd9974b180/8ea6db35-25d0-43bc-9de5-3ca23502dcdc"
+          (reference "U17") (unit 1)
+        )
+        (path "/8cd08eb5-4755-4ef5-8eeb-77fd9974b180/272a4677-3ef2-418e-abc5-b29f59e726f9"
+          (reference "U21") (unit 1)
+        )
+        (path "/8cd08eb5-4755-4ef5-8eeb-77fd9974b180/56b7edd2-65bf-4844-b6bd-3868b6562f83"
+          (reference "U25") (unit 1)
+        )
+        (path "/8cd08eb5-4755-4ef5-8eeb-77fd9974b180/a066fdde-5f40-4269-95c1-258d611fd7cb"
+          (reference "U29") (unit 1)
+        )
+        (path "/8cd08eb5-4755-4ef5-8eeb-77fd9974b180/ec158eb5-f3e0-409c-b64c-a90e3358941f"
+          (reference "U33") (unit 1)
+        )
+        (path "/8cd08eb5-4755-4ef5-8eeb-77fd9974b180/6c53b757-b2e6-4d60-b760-4a4a0f832c07"
+          (reference "U37") (unit 1)
+        )
+        (path "/8cd08eb5-4755-4ef5-8eeb-77fd9974b180/0223a704-ac47-44ed-9ba1-f418acceedb3"
+          (reference "U41") (unit 1)
+        )
+        (path "/8cd08eb5-4755-4ef5-8eeb-77fd9974b180/2ffa7ecd-d29d-4261-a577-43650ca26099"
+          (reference "U45") (unit 1)
+        )
+        (path "/8cd08eb5-4755-4ef5-8eeb-77fd9974b180/f71a1287-269d-4354-9179-cb80a7e1dbca"
+          (reference "U49") (unit 1)
+        )
+      )
+    )
+  )
   (symbol (lib_id "power:GND") (at 224.79 105.41 0) (unit 1)
     (in_bom yes) (on_board yes) (dnp no) (fields_autoplaced)
@@
         )
       )
-    )
-  )
-  (symbol (lib_id "74xGxx:74AHC1G02") (at 224.79 130.81 0) (unit 1)
-    (in_bom yes) (on_board yes) (dnp no)
-    (property "Reference" "U4" (at 236.22 135.89 0)
-      (effects (font (size 1.27 1.27)))
-    )
-    (property "Value" "74AHC1G02" (at 236.22 133.35 0)
-      (effects (font (size 1.27 1.27)))
-    )
-    (property "Footprint" "" (at 224.79 130.81 0)
-      (effects (font (size 1.27 1.27)) hide)
-    )
-    (property "Datasheet" "http://www.ti.com/lit/sg/scyt129e/scyt129e.pdf" (at 224.79 130.81 0)
-      (effects (font (size 1.27 1.27)) hide)
-    )
-    (pin "1")
-    (pin "2")
-    (pin "3")
-    (pin "4")
-    (pin "5")
-    (instances
-      (project "SCART_switcher"
-        (path "/8cd08eb5-4755-4ef5-8eeb-77fd9974b180/6e53f4c9-ed59-4c5d-ac8d-a66f0d353ca7"
-          (reference "U4") (unit 1)
-        )
-        (path "/8cd08eb5-4755-4ef5-8eeb-77fd9974b180/8ea6db35-25d0-43bc-9de5-3ca23502dcdc"
-          (reference "U17") (unit 1)
-        )
-        (path "/8cd08eb5-4755-4ef5-8eeb-77fd9974b180/272a4677-3ef2-418e-abc5-b29f59e726f9"
-          (reference "U21") (unit 1)
-        )
-        (path "/8cd08eb5-4755-4ef5-8eeb-77fd9974b180/56b7edd2-65bf-4844-b6bd-3868b6562f83"
-          (reference "U25") (unit 1)
-        )
-        (path "/8cd08eb5-4755-4ef5-8eeb-77fd9974b180/a066fdde-5f40-4269-95c1-258d611fd7cb"
-          (reference "U29") (unit 1)
-        )
-        (path "/8cd08eb5-4755-4ef5-8eeb-77fd9974b180/ec158eb5-f3e0-409c-b64c-a90e3358941f"
-          (reference "U33") (unit 1)
-        )
-        (path "/8cd08eb5-4755-4ef5-8eeb-77fd9974b180/6c53b757-b2e6-4d60-b760-4a4a0f832c07"
-          (reference "U37") (unit 1)
-        )
-        (path "/8cd08eb5-4755-4ef5-8eeb-77fd9974b180/0223a704-ac47-44ed-9ba1-f418acceedb3"
-          (reference "U41") (unit 1)
-        )
-        (path "/8cd08eb5-4755-4ef5-8eeb-77fd9974b180/2ffa7ecd-d29d-4261-a577-43650ca26099"
-          (reference "U45") (unit 1)
-        )
-        (path "/8cd08eb5-4755-4ef5-8eeb-77fd9974b180/f71a1287-269d-4354-9179-cb80a7e1dbca"
-          (reference "U49") (unit 1)
-        )
-      )

Commit message: progressed ecad
Other:
- note added: "(*1) Level 0: 0 V to +2 V (SCART off) Level 1A: +4,5 V to +7 V (SCART on, 16:9) Level 1B: +9,5 V to +12 V (SCART on)"
- note added: "(*2) The input terminal FUNCTION of the voltage monitoring circuit has two outputs, FNC_IN1 and FNC_IN2, with voltages of 3.3V when the signal level input FUNCTION of the SCART interface is 0 V to +2 V (SCART off). When the functional selection control signal level is +4,5 V to +7 V (SCART on, 16:9), the voltage of the first output terminal FNC_IN1 is 0V, and the voltage of the second output term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"
- note added: "tbd: incorrect"
- note removed: "(*1) Level 0: 0 V to +2 V (TV mode) Level 1A: +4,5 V to +7 V (AV mode, aspect ratio 16.9) Level 1B: +9,5 V to +12 V (AV mode)"
- note removed: "(*2) The input terminal FUNCTION of the voltage monitoring circuit has two outputs, FNC_IN1 and FNC_IN2, with voltages of 3.3V when the signal level input FUNCTION of the SCART interface is 0-2V (SCART off). When the functional selection control signal level is 4.5-7V (SCART on, 16:9), the voltage of the first output terminal FNC_IN1 is 0V, and the voltage of the second output terminal FNC_IN2 is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"
Changed lines of the file:
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@@
     (stroke (width 0) (type default))
   )
-  (wire (pts (xy 193.04 40.64) (xy 207.01 40.64))
+  (wire (pts (xy 195.58 40.64) (xy 207.01 40.64))
     (stroke (width 0) (type default))
   )
@@
   (wire (pts (xy 260.35 44.45) (xy 260.35 45.72))
     (stroke (width 0) (type default))
+  )
+  (text "tbd: incorrect" (at 119.38 114.3 0)
+    (effects (font (size 1.27 1.27)) (justify left bottom))
   )
   (text "(*1)" (at 91.44 68.58 0)
@@
     (effects (font (size 1.27 1.27)) (justify left bottom))
   )
-  (text "(*1)\nLevel 0: 0 V to +2 V (TV mode)\nLevel 1A: +4,5 V to +7 V (AV mode, aspect ratio 16.9)\nLevel 1B: +9,5 V to +12 V (AV mode)"
+  (text "(*1)\nLevel 0: 0 V to +2 V (SCART off)\nLevel 1A: +4,5 V to +7 V (SCART on, 16:9)\nLevel 1B: +9,5 V to +12 V (SCART on)"
     (at 111.76 21.59 0)
     (effects (font (size 1.27 1.27)) (justify left bottom))
@@
     (effects (font (size 1.27 1.27)) (justify left bottom))
   )
-  (text "(*2)\nThe input terminal FUNCTION of the voltage monitoring circuit has\ntwo outputs, FNC_IN1 and FNC_IN2, with voltages of 3.3V when\nthe signal level input FUNCTION of the SCART interface is 0-2V (SCART off).\nWhen the functional selection control signal level is 4.5-7V (SCART on, 16:9),\nthe voltage of the first output terminal FNC_IN1 is 0V,\nand the voltage of the second output terminal FNC_IN2 is 3.3V.\nWhen the functional selection control signal level is 9.5-12V (SCART on),\nthe voltages of both the first output terminal FNC_IN1\nand the second output terminal FNC_IN2 are 0V."
+  (text "(*2)\nThe input terminal FUNCTION of the voltage monitoring circuit has\ntwo outputs, FNC_IN1 and FNC_IN2, with voltages of 3.3V when\nthe signal level input FUNCTION of the SCART interface is 0 V to +2 V (SCART off).\nWhen the functional selection control signal level is +4,5 V to +7 V (SCART on, 16:9),\nthe voltage of the first output terminal FNC_IN1 is 0V,\nand the voltage of the second output terminal FNC_IN2 is 3.3V.\nWhen the functional selection control signal level is +9,5 V to +12 V (SCART on),\nthe voltages of both the first output terminal FNC_IN1\nand the second output terminal FNC_IN2 are 0V."
     (at 111.76 44.45 0)
     (effects (font (size 1.27 1.27)) (justify left bottom))
@@
     (effects (font (size 1.27 1.27)) (justify left bottom))
   )
-  (label "FUNCTION" (at 193.04 40.64 0) (fields_autoplaced)
+  (label "FUNCTION" (at 195.58 40.64 0) (fields_autoplaced)
     (effects (font (size 1.27 1.27)) (justify left bottom))
   )
