File: ECAD/SCART_switcher/priority_encoder.kicad_sch (KiCad schematic)
At the start: 8 parts, among them U2 74AHC1G04, U3 74AHC1G08, U4 74AHC1G04, U5 74AHC1G08, U6 74AHC1G04, U7 74AHC1G08, U8 74AHC1G08, U9 74AHC1G08

Commit message: Progressed ECAD
Parts:
- added C4: 2n2C, symbol Device:C
- added D1: BAS316, symbol Device:D
- added R18: 10kR, Resistor_SMD:R_0805_2012Metric_Pad1.20x1.40mm_HandSolder, symbol Device:R
- added R19: 2k2R, Resistor_SMD:R_0805_2012Metric_Pad1.20x1.40mm_HandSolder, symbol Device:R
- added U10: 74AHC1G14, symbol 74xGxx:74AHC1G14
Connections:
- net FNC_INA: now also D1.1 (K), R19.1
- new net: C4.1, D1.2 (A), R18.1, R19.2, U10.2
- new net GND: C4.2, R18.2, U10.3 (GND)
- new net INA_DIS: U10.4
Other:
- note added: "Dead time delay to allow for break before make input video selection."

Commit message: Progressed ECAD.
Parts:
- renumbered C4 to C14, R19 to R25, R18 to R26, U9 to U10, U10 to U11, U2 to U3, U6 to U5, U5 to U6, U3 to U8, U8 to U9
Connections:
- net INA_DIS: no longer names the net of U11.4

Commit message: Progressed ECAD.
Parts:
- renumbered C14 to C15, U8 to U10, U9 to U11, U10 to U12, U11 to U13, U3 to U5, U4 to U6, U5 to U7, U6 to U8, U7 to U9

Commit message: progressed ECAD
Changed lines of the file:
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@@
     (effects (font (size 1.27 1.27)) (justify right bottom))
   )
-  (hierarchical_label "FNC_IN3" (shape input) (at 33.02 54.61 180) (fields_autoplaced)
+  (hierarchical_label "IN3_ACTIVE" (shape input) (at 33.02 54.61 180) (fields_autoplaced)
     (effects (font (size 1.27 1.27)) (justify right))
   )
@@
     (effects (font (size 1.27 1.27)) (justify left))
   )
-  (hierarchical_label "FNC_IN8" (shape input) (at 33.0089 67.4096 180) (fields_autoplaced)
+  (hierarchical_label "IN8_ACTIVE" (shape input) (at 33.0089 67.4096 180) (fields_autoplaced)
     (effects (font (size 1.27 1.27)) (justify right))
   )
@@
     (effects (font (size 1.27 1.27)) (justify left))
   )
-  (hierarchical_label "FNC_IN7" (shape input) (at 33.02 64.77 180) (fields_autoplaced)
+  (hierarchical_label "IN7_ACTIVE" (shape input) (at 33.02 64.77 180) (fields_autoplaced)
     (effects (font (size 1.27 1.27)) (justify right))
   )
-  (hierarchical_label "FNC_IN5" (shape input) (at 33.02 59.69 180) (fields_autoplaced)
+  (hierarchical_label "IN5_ACTIVE" (shape input) (at 33.02 59.69 180) (fields_autoplaced)
     (effects (font (size 1.27 1.27)) (justify right))
   )
-  (hierarchical_label "FNC_IN10" (shape input) (at 33.02 72.39 180) (fields_autoplaced)
+  (hierarchical_label "IN10_ACTIVE" (shape input) (at 33.02 72.39 180) (fields_autoplaced)
     (effects (font (size 1.27 1.27)) (justify right))
   )
@@
     (effects (font (size 1.27 1.27)) (justify left))
   )
-  (hierarchical_label "FNC_IN1" (shape input) (at 33.02 49.53 180) (fields_autoplaced)
+  (hierarchical_label "IN1_ACTIVE" (shape input) (at 33.02 49.53 180) (fields_autoplaced)
     (effects (font (size 1.27 1.27)) (justify right))
   )
-  (hierarchical_label "FNC_IN6" (shape input) (at 33.02 62.23 180) (fields_autoplaced)
+  (hierarchical_label "IN6_ACTIVE" (shape input) (at 33.02 62.23 180) (fields_autoplaced)
     (effects (font (size 1.27 1.27)) (justify right))
   )
-  (hierarchical_label "FNC_IN2" (shape input) (at 33.02 52.07 180) (fields_autoplaced)
+  (hierarchical_label "IN2_ACTIVE" (shape input) (at 33.02 52.07 180) (fields_autoplaced)
     (effects (font (size 1.27 1.27)) (justify right))
   )
@@
     (effects (font (size 1.27 1.27)) (justify left))
   )
-  (hierarchical_label "FNC_IN9" (shape input) (at 33.02 69.85 180) (fields_autoplaced)
+  (hierarchical_label "IN9_ACTIVE" (shape input) (at 33.02 69.85 180) (fields_autoplaced)
     (effects (font (size 1.27 1.27)) (justify right))
   )
@@
     (effects (font (size 1.27 1.27)) (justify left))
   )
-  (hierarchical_label "FNC_IN4" (shape input) (at 33.02 57.15 180) (fields_autoplaced)
+  (hierarchical_label "IN4_ACTIVE" (shape input) (at 33.02 57.15 180) (fields_autoplaced)
     (effects (font (size 1.27 1.27)) (justify right))
   )

Commit message: progressed ecad
Changed lines of the file:
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@@
     (effects (font (size 1.27 1.27)) (justify right bottom))
+  )
+  (hierarchical_label "IN4_VIDEO_4_3" (shape input) (at 20.32 88.9 0) (fields_autoplaced)
+    (effects (font (size 1.27 1.27)) (justify left))
+  )
+  (hierarchical_label "IN3_VIDEO_4_3" (shape input) (at 20.32 85.09 0) (fields_autoplaced)
+    (effects (font (size 1.27 1.27)) (justify left))
   )
   (hierarchical_label "IN3_ACTIVE" (shape input) (at 33.02 54.61 180) (fields_autoplaced)
@@
   (hierarchical_label "IN8_ACTIVE" (shape input) (at 33.0089 67.4096 180) (fields_autoplaced)
     (effects (font (size 1.27 1.27)) (justify right))
+  )
+  (hierarchical_label "IN10_VIDEO_4_3" (shape input) (at 20.32 113.03 0) (fields_autoplaced)
+    (effects (font (size 1.27 1.27)) (justify left))
   )
   (hierarchical_label "IN8_ENABLE" (shape output) (at 257.81 88.9 0) (fields_autoplaced)
@@
     (effects (font (size 1.27 1.27)) (justify right))
   )
+  (hierarchical_label "IN6_VIDEO_4_3" (shape input) (at 20.2777 96.5495 0) (fields_autoplaced)
+    (effects (font (size 1.27 1.27)) (justify left))
+  )
   (hierarchical_label "IN9_ENABLE" (shape output) (at 257.81 91.44 0) (fields_autoplaced)
     (effects (font (size 1.27 1.27)) (justify left))
@@
     (effects (font (size 1.27 1.27)) (justify right))
   )
+  (hierarchical_label "IN2_VIDEO_4_3" (shape input) (at 20.32 81.28 0) (fields_autoplaced)
+    (effects (font (size 1.27 1.27)) (justify left))
+  )
+  (hierarchical_label "IN9_VIDEO_4_3" (shape input) (at 20.32 109.22 0) (fields_autoplaced)
+    (effects (font (size 1.27 1.27)) (justify left))
+  )
   (hierarchical_label "IN6_ACTIVE" (shape input) (at 33.02 62.23 180) (fields_autoplaced)
     (effects (font (size 1.27 1.27)) (justify right))
+  )
+  (hierarchical_label "IN1_VIDEO_4_3" (shape input) (at 20.32 78.74 0) (fields_autoplaced)
+    (effects (font (size 1.27 1.27)) (justify left))
+  )
+  (hierarchical_label "IN8_VIDEO_4_3" (shape input) (at 20.32 105.41 0) (fields_autoplaced)
+    (effects (font (size 1.27 1.27)) (justify left))
   )
   (hierarchical_label "IN2_ACTIVE" (shape input) (at 33.02 52.07 180) (fields_autoplaced)
     (effects (font (size 1.27 1.27)) (justify right))
   )
+  (hierarchical_label "OUT_ACTIVE" (shape output) (at 261.62 110.49 0) (fields_autoplaced)
+    (effects (font (size 1.27 1.27)) (justify left))
+  )
+  (hierarchical_label "IN7_VIDEO_4_3" (shape input) (at 20.32 100.33 0) (fields_autoplaced)
+    (effects (font (size 1.27 1.27)) (justify left))
+  )
   (hierarchical_label "IN7_ENABLE" (shape output) (at 257.81 86.36 0) (fields_autoplaced)
+    (effects (font (size 1.27 1.27)) (justify left))
+  )
+  (hierarchical_label "IN5_VIDEO_4_3" (shape input) (at 20.32 92.71 0) (fields_autoplaced)
     (effects (font (size 1.27 1.27)) (justify left))
   )
@@
     (effects (font (size 1.27 1.27)) (justify right))
   )
+  (hierarchical_label "VIDEO_4_3" (shape output) (at 261.62 105.41 0) (fields_autoplaced)
+    (effects (font (size 1.27 1.27)) (justify left))
+  )
   (hierarchical_label "IN3_ENABLE" (shape output) (at 210.82 106.68 0) (fields_autoplaced)

Commit message: progressed ecad
Connections:
- net FNC_INA renamed INA_EN
Changed lines of the file:
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@@
-    (effects (font (size 1.27 1.27)) (justify left bottom))
-  )
-  (label "FNC_INA" (at 119.634 31.496 0) (fields_autoplaced)
     (effects (font (size 1.27 1.27)) (justify left bottom))
   )
@@
     (effects (font (size 1.27 1.27)) (justify left))
   )
-  (hierarchical_label "IN3_ACTIVE" (shape input) (at 33.02 54.61 180) (fields_autoplaced)
+  (hierarchical_label "IN3_ACTIVE" (shape input) (at 116.84 102.87 180) (fields_autoplaced)
     (effects (font (size 1.27 1.27)) (justify right))
   )
@@
     (effects (font (size 1.27 1.27)) (justify left))
   )
-  (hierarchical_label "IN1_ACTIVE" (shape input) (at 33.02 49.53 180) (fields_autoplaced)
+  (hierarchical_label "IN1_ACTIVE" (shape input) (at 119.38 30.48 180) (fields_autoplaced)
     (effects (font (size 1.27 1.27)) (justify right))
   )
@@
     (effects (font (size 1.27 1.27)) (justify left))
   )
-  (hierarchical_label "IN2_ACTIVE" (shape input) (at 33.02 52.07 180) (fields_autoplaced)
+  (hierarchical_label "IN2_ACTIVE" (shape input) (at 116.84 59.69 180) (fields_autoplaced)
     (effects (font (size 1.27 1.27)) (justify right))
   )
@@
     (effects (font (size 1.27 1.27)) (justify left))
   )
-  (hierarchical_label "IN4_ACTIVE" (shape input) (at 33.02 57.15 180) (fields_autoplaced)
+  (hierarchical_label "IN4_ACTIVE" (shape input) (at 116.84 147.32 180) (fields_autoplaced)
     (effects (font (size 1.27 1.27)) (justify right))
   )

Commit message: Progressed ECAD.
Parts:
- U10, U11, U12, U8, U9: footprint (none) -> Package_TO_SOT_SMD:SOT-23-5; MFN (none) -> 74AHC1G08W5-7
- U13: footprint (none) -> Package_TO_SOT_SMD:SOT-23-5; MFN (none) -> 74AHC1G14W5-7
- U5, U6, U7: footprint (none) -> Package_TO_SOT_SMD:SOT-23-5; MFN (none) -> 74AHC1G04W5-7
Changed lines of the file:
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@@
+      (effects (font (size 1.27 1.27)) hide)
+    )
+    (property "MFN" "" (at 211.582 29.972 0)
       (effects (font (size 1.27 1.27)) hide)
     )
@@
       (effects (font (size 1.27 1.27)))
     )
-    (property "Footprint" "" (at 181.102 149.606 0)
-      (effects (font (size 1.27 1.27)) hide)
-    )
-    (property "Datasheet" "http://www.ti.com/lit/sg/scyt129e/scyt129e.pdf" (at 181.102 149.606 0)
+    (property "Footprint" "Package_TO_SOT_SMD:SOT-23-5" (at 181.102 149.606 0)
+      (effects (font (size 1.27 1.27)) hide)
+    )
+    (property "Datasheet" "https://datasheet.lcsc.com/lcsc/1912111437_Diodes-Incorporated-74AHC1G08W5-7_C460487.pdf" (at 181.102 149.606 0)
+      (effects (font (size 1.27 1.27)) hide)
+    )
+    (property "MFN" "74AHC1G08W5-7" (at 181.102 149.606 0)
       (effects (font (size 1.27 1.27)) hide)
     )
@@
       (effects (font (size 1.27 1.27)))
     )
-    (property "Footprint" "" (at 243.078 31.496 0)
-      (effects (font (size 1.27 1.27)) hide)
-    )
-    (property "Datasheet" "https://www.ti.com/lit/ds/symlink/sn74lvc1g14.pdf" (at 243.078 31.496 0)
+    (property "Footprint" "Package_TO_SOT_SMD:SOT-23-5" (at 243.078 31.496 0)
+      (effects (font (size 1.27 1.27)) hide)
+    )
+    (property "Datasheet" "https://datasheet.lcsc.com/lcsc/2304140030_Diodes-Incorporated-74AHC1G14W5-7_C176916.pdf" (at 243.078 31.496 0)
+      (effects (font (size 1.27 1.27)) hide)
+    )
+    (property "MFN" "74AHC1G14W5-7" (at 243.078 31.496 0)
       (effects (font (size 1.27 1.27)) hide)
     )
@@
       (effects (font (size 1.27 1.27)))
     )
-    (property "Footprint" "" (at 144.78 72.136 0)
-      (effects (font (size 1.27 1.27)) hide)
-    )
-    (property "Datasheet" "http://www.ti.com/lit/sg/scyt129e/scyt129e.pdf" (at 144.78 72.136 0)
+    (property "Footprint" "Package_TO_SOT_SMD:SOT-23-5" (at 144.78 72.136 0)
+      (effects (font (size 1.27 1.27)) hide)
+    )
+    (property "Datasheet" "https://datasheet.lcsc.com/lcsc/1912111437_Diodes-Incorporated-74AHC1G04W5-7_C460486.pdf" (at 144.78 72.136 0)
+      (effects (font (size 1.27 1.27)) hide)
+    )
+    (property "MFN" "74AHC1G04W5-7" (at 144.78 72.136 0)
       (effects (font (size 1.27 1.27)) hide)
     )
@@
       (effects (font (size 1.27 1.27)))
     )
-    (property "Footprint" "" (at 181.102 106.172 0)
-      (effects (font (size 1.27 1.27)) hide)
-    )
-    (property "Datasheet" "http://www.ti.com/lit/sg/scyt129e/scyt129e.pdf" (at 181.102 106.172 0)
+    (property "Footprint" "Package_TO_SOT_SMD:SOT-23-5" (at 181.102 106.172 0)
+      (effects (font (size 1.27 1.27)) hide)
+    )
+    (property "Datasheet" "https://datasheet.lcsc.com/lcsc/1912111437_Diodes-Incorporated-74AHC1G08W5-7_C460487.pdf" (at 181.102 106.172 0)
+      (effects (font (size 1.27 1.27)) hide)
+    )
+    (property "MFN" "74AHC1G08W5-7" (at 181.102 106.172 0)
       (effects (font (size 1.27 1.27)) hide)
     )
@@
       (effects (font (size 1.27 1.27)) hide)
     )
-    (property "Sim.Device" "D" (at 211.582 33.02 0)
-      (effects (font (size 1.27 1.27)) hide)
-    )
-    (property "Sim.Pins" "1=K 2=A" (at 211.582 33.02 0)
+    (property "MFN" "" (at 211.582 33.02 0)
       (effects (font (size 1.27 1.27)) hide)
     )
@@
       (effects (font (size 1.27 1.27)))
     )
-    (property "Footprint" "" (at 144.78 115.57 0)
-      (effects (font (size 1.27 1.27)) hide)
-    )
-    (property "Datasheet" "http://www.ti.com/lit/sg/scyt129e/scyt129e.pdf" (at 144.78 115.57 0)
+    (property "Footprint" "Package_TO_SOT_SMD:SOT-23-5" (at 144.78 115.57 0)
+      (effects (font (size 1.27 1.27)) hide)
+    )
+    (property "Datasheet" "https://datasheet.lcsc.com/lcsc/1912111437_Diodes-Incorporated-74AHC1G04W5-7_C460486.pdf" (at 144.78 115.57 0)
+      (effects (font (size 1.27 1.27)) hide)
+    )
+    (property "MFN" "74AHC1G04W5-7" (at 144.78 115.57 0)
       (effects (font (size 1.27 1.27)) hide)
     )
@@
       (effects (font (size 1.27 1.27)))
     )
-    (property "Footprint" "" (at 162.306 88.646 0)
-      (effects (font (size 1.27 1.27)) hide)
-    )
-    (property "Datasheet" "http://www.ti.com/lit/sg/scyt129e/scyt129e.pdf" (at 162.306 88.646 0)
+    (property "Footprint" "Package_TO_SOT_SMD:SOT-23-5" (at 162.306 88.646 0)
+      (effects (font (size 1.27 1.27)) hide)
+    )
+    (property "Datasheet" "https://datasheet.lcsc.com/lcsc/1912111437_Diodes-Incorporated-74AHC1G08W5-7_C460487.pdf" (at 162.306 88.646 0)
+      (effects (font (size 1.27 1.27)) hide)
+    )
+    (property "MFN" "74AHC1G08W5-7" (at 162.306 88.646 0)
       (effects (font (size 1.27 1.27)) hide)
     )
@@
       (effects (font (size 1.27 1.27)))
     )
-    (property "Footprint" "" (at 144.78 43.434 0)
-      (effects (font (size 1.27 1.27)) hide)
-    )
-    (property "Datasheet" "http://www.ti.com/lit/sg/scyt129e/scyt129e.pdf" (at 144.78 43.434 0)
+    (property "Footprint" "Package_TO_SOT_SMD:SOT-23-5" (at 144.78 43.434 0)
+      (effects (font (size 1.27 1.27)) hide)
+    )
+    (property "Datasheet" "https://datasheet.lcsc.com/lcsc/1912111437_Diodes-Incorporated-74AHC1G04W5-7_C460486.pdf" (at 144.78 43.434 0)
+      (effects (font (size 1.27 1.27)) hide)
+    )
+    (property "MFN" "74AHC1G04W5-7" (at 144.78 43.434 0)
       (effects (font (size 1.27 1.27)) hide)
     )
@@
       (effects (font (size 1.27 1.27)))
     )
-    (property "Footprint" "" (at 162.306 132.08 0)
-      (effects (font (size 1.27 1.27)) hide)
-    )
-    (property "Datasheet" "http://www.ti.com/lit/sg/scyt129e/scyt129e.pdf" (at 162.306 132.08 0)
+    (property "Footprint" "Package_TO_SOT_SMD:SOT-23-5" (at 162.306 132.08 0)
+      (effects (font (size 1.27 1.27)) hide)
+    )
+    (property "Datasheet" "https://datasheet.lcsc.com/lcsc/1912111437_Diodes-Incorporated-74AHC1G08W5-7_C460487.pdf" (at 162.306 132.08 0)
+      (effects (font (size 1.27 1.27)) hide)
+    )
+    (property "MFN" "74AHC1G08W5-7" (at 162.306 132.08 0)
       (effects (font (size 1.27 1.27)) hide)
     )
@@
       (effects (font (size 1.27 1.27)))
     )
-    (property "Footprint" "" (at 181.102 62.738 0)
-      (effects (font (size 1.27 1.27)) hide)
-    )
-    (property "Datasheet" "http://www.ti.com/lit/sg/scyt129e/scyt129e.pdf" (at 181.102 62.738 0)
+    (property "Footprint" "Package_TO_SOT_SMD:SOT-23-5" (at 181.102 62.738 0)
+      (effects (font (size 1.27 1.27)) hide)
+    )
+    (property "Datasheet" "https://datasheet.lcsc.com/lcsc/1912111437_Diodes-Incorporated-74AHC1G08W5-7_C460487.pdf" (at 181.102 62.738 0)
+      (effects (font (size 1.27 1.27)) hide)
+    )
+    (property "MFN" "74AHC1G08W5-7" (at 181.102 62.738 0)
       (effects (font (size 1.27 1.27)) hide)
     )
@@
     )
     (property "Datasheet" "~" (at 225.298 40.64 0)
+      (effects (font (size 1.27 1.27)) hide)
+    )
+    (property "MFN" "" (at 225.298 40.64 0)
       (effects (font (size 1.27 1.27)) hide)
     )
@@
       (effects (font (size 1.27 1.27)) hide)
     )
+    (property "MFN" "" (at 221.234 40.64 0)
+      (effects (font (size 1.27 1.27)) hide)
+    )

Commit message: Circuit simplification
Changed lines of the file:
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@@
     (effects (font (size 1.27 1.27)) (justify right bottom))
-  )
-  (hierarchical_label "IN4_VIDEO_4_3" (shape input) (at 20.32 88.9 0) (fields_autoplaced)
-    (effects (font (size 1.27 1.27)) (justify left))
-  )
-  (hierarchical_label "IN3_VIDEO_4_3" (shape input) (at 20.32 85.09 0) (fields_autoplaced)
-    (effects (font (size 1.27 1.27)) (justify left))
   )
   (hierarchical_label "IN3_ACTIVE" (shape input) (at 116.84 102.87 180) (fields_autoplaced)
@@
   (hierarchical_label "IN8_ACTIVE" (shape input) (at 33.0089 67.4096 180) (fields_autoplaced)
     (effects (font (size 1.27 1.27)) (justify right))
-  )
-  (hierarchical_label "IN10_VIDEO_4_3" (shape input) (at 20.32 113.03 0) (fields_autoplaced)
-    (effects (font (size 1.27 1.27)) (justify left))
   )
   (hierarchical_label "IN8_ENABLE" (shape output) (at 257.81 88.9 0) (fields_autoplaced)
@@
     (effects (font (size 1.27 1.27)) (justify right))
   )
-  (hierarchical_label "IN6_VIDEO_4_3" (shape input) (at 20.2777 96.5495 0) (fields_autoplaced)
-    (effects (font (size 1.27 1.27)) (justify left))
-  )
   (hierarchical_label "IN9_ENABLE" (shape output) (at 257.81 91.44 0) (fields_autoplaced)
     (effects (font (size 1.27 1.27)) (justify left))
@@
     (effects (font (size 1.27 1.27)) (justify right))
   )
-  (hierarchical_label "IN2_VIDEO_4_3" (shape input) (at 20.32 81.28 0) (fields_autoplaced)
-    (effects (font (size 1.27 1.27)) (justify left))
-  )
-  (hierarchical_label "IN9_VIDEO_4_3" (shape input) (at 20.32 109.22 0) (fields_autoplaced)
-    (effects (font (size 1.27 1.27)) (justify left))
-  )
   (hierarchical_label "IN6_ACTIVE" (shape input) (at 33.02 62.23 180) (fields_autoplaced)
     (effects (font (size 1.27 1.27)) (justify right))
-  )
-  (hierarchical_label "IN1_VIDEO_4_3" (shape input) (at 20.32 78.74 0) (fields_autoplaced)
-    (effects (font (size 1.27 1.27)) (justify left))
-  )
-  (hierarchical_label "IN8_VIDEO_4_3" (shape input) (at 20.32 105.41 0) (fields_autoplaced)
-    (effects (font (size 1.27 1.27)) (justify left))
   )
   (hierarchical_label "IN2_ACTIVE" (shape input) (at 116.84 59.69 180) (fields_autoplaced)
@@
     (effects (font (size 1.27 1.27)) (justify left))
   )
-  (hierarchical_label "IN7_VIDEO_4_3" (shape input) (at 20.32 100.33 0) (fields_autoplaced)
-    (effects (font (size 1.27 1.27)) (justify left))
-  )
   (hierarchical_label "IN7_ENABLE" (shape output) (at 257.81 86.36 0) (fields_autoplaced)
-    (effects (font (size 1.27 1.27)) (justify left))
-  )
-  (hierarchical_label "IN5_VIDEO_4_3" (shape input) (at 20.32 92.71 0) (fields_autoplaced)
     (effects (font (size 1.27 1.27)) (justify left))
   )
@@
     (effects (font (size 1.27 1.27)) (justify right))
   )
-  (hierarchical_label "VIDEO_4_3" (shape output) (at 261.62 105.41 0) (fields_autoplaced)
-    (effects (font (size 1.27 1.27)) (justify left))
-  )
   (hierarchical_label "IN3_ENABLE" (shape output) (at 210.82 106.68 0) (fields_autoplaced)
