File: ECAD/SCART_switcher/priority_encoder.kicad_sch (KiCad schematic)
At the start: 13 parts, among them U10 74AHC1G08, U11 74AHC1G08, U12 74AHC1G08, U13 74AHC1G14, U5 74AHC1G04, U6 74AHC1G04, U7 74AHC1G04, U8 74AHC1G08, U9 74AHC1G08

Commit message: Progressed ECAD
Parts:
- removed C15: 2n2C, symbol Device:C
- removed D1: BAS316, symbol Device:D
- removed R25: 2k2R, Resistor_SMD:R_0805_2012Metric_Pad1.20x1.40mm_HandSolder, symbol Device:R
- removed R26: 10kR, Resistor_SMD:R_0805_2012Metric_Pad1.20x1.40mm_HandSolder, symbol Device:R
- removed U10, U11, U12, U8, U9: 74AHC1G08, Package_TO_SOT_SMD:SOT-23-5, symbol 74xGxx:74AHC1G08
- removed U13: 74AHC1G14, Package_TO_SOT_SMD:SOT-23-5, symbol 74xGxx:74AHC1G14
- removed U5, U6, U7: 74AHC1G04, Package_TO_SOT_SMD:SOT-23-5, symbol 74xGxx:74AHC1G04
Other:
- added sheet Priority Level 0 (priority_level_start.kicad_sch)
- added sheet Priority Level 1 (priority_level.kicad_sch)
- added sheet Priority Level 2 (priority_level.kicad_sch)
- added sheet Priority Level 3 (priority_level.kicad_sch)
- added sheet Priority Level 4 (priority_level.kicad_sch)
- added sheet Priority Level 5 (priority_level.kicad_sch)
- added sheet Priority Level 6 (priority_level.kicad_sch)
- added sheet Priority Level 7 (priority_level.kicad_sch)
- added sheet Priority Level 8 (priority_level.kicad_sch)
- added sheet Priority Level 9 (priority_level_end.kicad_sch)
- note removed: "Dead time delay to allow for break before make input video selection."
- note removed: "tbd: add delay to the enable case such that "break before make" type of behaviour is built."
