File: ECAD/SCART_switcher/priority_level_end.kicad_sch (KiCad schematic)
At the start: 5 parts, among them U10 74AHC1G08, U6 74AHC1G04, U8 74AHC1G08

Commit message: progressed ECAD
Parts:
- renumbered C6 to C?, U8 to U?, U6 to U?, U10 to U?
Connections:
- net +3.3V renamed +5V
