File: ECAD/SCART_switcher/priority_level_end.kicad_sch (KiCad schematic)
At the start: 5 parts

Commit message: progressed ecad
Parts:
- C?: MPN (none) -> CL21B104KBCNNNC
Changed lines of the file:
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@@
       (effects (font (size 1.27 1.27)) hide)
     )
-    (property "Datasheet" "~" (at 88.9 92.71 0)
+    (property "Datasheet" "https://datasheet.lcsc.com/lcsc/1810191215_Samsung-Electro-Mechanics-CL21B104KBCNNNC_C1711.pdf" (at 88.9 92.71 0)
       (effects (font (size 1.27 1.27)) hide)
     )
@@
       (effects (font (size 1.27 1.27)) hide)
     )
+    (property "MPN" "CL21B104KBCNNNC" (at 88.9 92.71 0)
+      (effects (font (size 1.27 1.27)) hide)
+    )
