File: ECAD/SCART_switcher/priority_level_end.kicad_sch (KiCad schematic)
At the start: 5 parts

Commit message: Progressed ECAD.
Parts:
- C?: footprint Capacitor_SMD:C_0805_2012Metric_Pad1.18x1.45mm_HandSolder -> Capacitor_SMD:C_0805_2012Metric
Changed lines of the file:
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@@
       (effects (font (size 1.27 1.27)) (justify left))
     )
-    (property "Footprint" "Capacitor_SMD:C_0805_2012Metric_Pad1.18x1.45mm_HandSolder" (at 89.8652 96.52 0)
+    (property "Footprint" "Capacitor_SMD:C_0805_2012Metric" (at 89.8652 96.52 0)
       (effects (font (size 1.27 1.27)) hide)
     )

Commit message: Progressed ECAD.
Parts:
- U? (x2): MPN 74AHC1G08W5-7 -> SN74AHC1G08DBVR
- U? (x2): MPN 74AHC1G04W5-7 -> SN74AHC1G04DBVR
Changed lines of the file:
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@@
       (effects (font (size 1.27 1.27)) hide)
     )
-    (property "Datasheet" "https://datasheet.lcsc.com/lcsc/1912111437_Diodes-Incorporated-74AHC1G08W5-7_C460487.pdf" (at 146.05 102.87 0)
-      (effects (font (size 1.27 1.27)) hide)
-    )
-    (property "MPN" "74AHC1G08W5-7" (at 146.05 102.87 0)
+    (property "Datasheet" "https://datasheet.lcsc.com/lcsc/1809151118_Texas-Instruments-SN74AHC1G08DBVR_C7467.pdf" (at 146.05 102.87 0)
+      (effects (font (size 1.27 1.27)) hide)
+    )
+    (property "MPN" "SN74AHC1G08DBVR" (at 146.05 102.87 0)
       (effects (font (size 1.27 1.27)) hide)
     )
@@
       (effects (font (size 1.27 1.27)) hide)
     )
-    (property "Datasheet" "https://datasheet.lcsc.com/lcsc/1912111437_Diodes-Incorporated-74AHC1G04W5-7_C460486.pdf" (at 176.53 119.38 0)
-      (effects (font (size 1.27 1.27)) hide)
-    )
-    (property "MPN" "74AHC1G04W5-7" (at 176.53 119.38 0)
+    (property "Datasheet" "https://datasheet.lcsc.com/lcsc/2001061132_Texas-Instruments-SN74AHC1G04DBVR_C7465.pdf" (at 176.53 119.38 0)
+      (effects (font (size 1.27 1.27)) hide)
+    )
+    (property "MPN" "SN74AHC1G04DBVR" (at 176.53 119.38 0)
       (effects (font (size 1.27 1.27)) hide)
     )
@@
       (effects (font (size 1.27 1.27)) hide)
     )
-    (property "Datasheet" "https://datasheet.lcsc.com/lcsc/1912111437_Diodes-Incorporated-74AHC1G04W5-7_C460486.pdf" (at 129.54 86.36 0)
-      (effects (font (size 1.27 1.27)) hide)
-    )
-    (property "MPN" "74AHC1G04W5-7" (at 129.54 86.36 0)
+    (property "Datasheet" "https://datasheet.lcsc.com/lcsc/2001061132_Texas-Instruments-SN74AHC1G04DBVR_C7465.pdf" (at 129.54 86.36 0)
+      (effects (font (size 1.27 1.27)) hide)
+    )
+    (property "MPN" "SN74AHC1G04DBVR" (at 129.54 86.36 0)
       (effects (font (size 1.27 1.27)) hide)
     )
@@
       (effects (font (size 1.27 1.27)) hide)
     )
-    (property "Datasheet" "https://datasheet.lcsc.com/lcsc/1912111437_Diodes-Incorporated-74AHC1G08W5-7_C460487.pdf" (at 165.1 71.12 0)
-      (effects (font (size 1.27 1.27)) hide)
-    )
-    (property "MPN" "74AHC1G08W5-7" (at 165.1 71.12 0)
-      (effects (font (size 1.27 1.27)) hide)
-    )
+    (property "Datasheet" "https://datasheet.lcsc.com/lcsc/1809151118_Texas-Instruments-SN74AHC1G08DBVR_C7467.pdf" (at 165.1 71.12 0)
+      (effects (font (size 1.27 1.27)) hide)
+    )
+    (property "MPN" "SN74AHC1G08DBVR" (at 165.1 71.12 0)
+      (effects (font (size 1.27 1.27)) hide)
+    )

Commit message: Progressed ECAD.
Parts:
- U? (x2): value 74AHC1G08 -> 74LVC1G08; footprint Package_TO_SOT_SMD:SOT-23-5 -> Package_TO_SOT_SMD:SOT-353_SC-70-5; MPN SN74AHC1G08DBVR -> SN74LVC1G08DCKR; Status (none) -> OK
- U? (x2): value 74AHC1G04 -> 74LVC1G04; footprint Package_TO_SOT_SMD:SOT-23-5 -> Package_TO_SOT_SMD:SOT-353_SC-70-5; MPN SN74AHC1G04DBVR -> SN74LVC1G04DCKR; Status (none) -> OK
Changed lines of the file:
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@@
       (effects (font (size 1.27 1.27)))
     )
-    (property "Value" "74AHC1G08" (at 156.21 106.68 90)
-      (effects (font (size 1.27 1.27)))
-    )
-    (property "Footprint" "Package_TO_SOT_SMD:SOT-23-5" (at 146.05 102.87 0)
-      (effects (font (size 1.27 1.27)) hide)
-    )
-    (property "Datasheet" "https://datasheet.lcsc.com/lcsc/1809151118_Texas-Instruments-SN74AHC1G08DBVR_C7467.pdf" (at 146.05 102.87 0)
-      (effects (font (size 1.27 1.27)) hide)
-    )
-    (property "MPN" "SN74AHC1G08DBVR" (at 146.05 102.87 0)
-      (effects (font (size 1.27 1.27)) hide)
-    )
-    (property "Status" "" (at 146.05 102.87 0)
+    (property "Value" "74LVC1G08" (at 156.21 106.68 90)
+      (effects (font (size 1.27 1.27)))
+    )
+    (property "Footprint" "Package_TO_SOT_SMD:SOT-353_SC-70-5" (at 146.05 102.87 0)
+      (effects (font (size 1.27 1.27)) hide)
+    )
+    (property "Datasheet" "https://datasheet.lcsc.com/lcsc/1809051811_Texas-Instruments-SN74LVC1G08DCKR_C7832.pdf" (at 146.05 102.87 0)
+      (effects (font (size 1.27 1.27)) hide)
+    )
+    (property "MPN" "SN74LVC1G08DCKR" (at 146.05 102.87 0)
+      (effects (font (size 1.27 1.27)) hide)
+    )
+    (property "Status" "OK" (at 146.05 102.87 0)
       (effects (font (size 1.27 1.27)) hide)
     )
@@
       (effects (font (size 1.27 1.27)))
     )
-    (property "Value" "74AHC1G04" (at 181.61 114.3 0)
-      (effects (font (size 1.27 1.27)))
-    )
-    (property "Footprint" "Package_TO_SOT_SMD:SOT-23-5" (at 176.53 119.38 0)
-      (effects (font (size 1.27 1.27)) hide)
-    )
-    (property "Datasheet" "https://datasheet.lcsc.com/lcsc/2001061132_Texas-Instruments-SN74AHC1G04DBVR_C7465.pdf" (at 176.53 119.38 0)
-      (effects (font (size 1.27 1.27)) hide)
-    )
-    (property "MPN" "SN74AHC1G04DBVR" (at 176.53 119.38 0)
-      (effects (font (size 1.27 1.27)) hide)
-    )
-    (property "Status" "" (at 176.53 119.38 0)
+    (property "Value" "74LVC1G04" (at 181.61 114.3 0)
+      (effects (font (size 1.27 1.27)))
+    )
+    (property "Footprint" "Package_TO_SOT_SMD:SOT-353_SC-70-5" (at 176.53 119.38 0)
+      (effects (font (size 1.27 1.27)) hide)
+    )
+    (property "Datasheet" "https://datasheet.lcsc.com/lcsc/1811021113_Texas-Instruments-SN74LVC1G04DCKR_C8207.pdf" (at 176.53 119.38 0)
+      (effects (font (size 1.27 1.27)) hide)
+    )
+    (property "MPN" "SN74LVC1G04DCKR" (at 176.53 119.38 0)
+      (effects (font (size 1.27 1.27)) hide)
+    )
+    (property "Status" "OK" (at 176.53 119.38 0)
       (effects (font (size 1.27 1.27)) hide)
     )
@@
       (effects (font (size 1.27 1.27)))
     )
-    (property "Value" "74AHC1G04" (at 134.62 81.28 0)
-      (effects (font (size 1.27 1.27)))
-    )
-    (property "Footprint" "Package_TO_SOT_SMD:SOT-23-5" (at 129.54 86.36 0)
-      (effects (font (size 1.27 1.27)) hide)
-    )
-    (property "Datasheet" "https://datasheet.lcsc.com/lcsc/2001061132_Texas-Instruments-SN74AHC1G04DBVR_C7465.pdf" (at 129.54 86.36 0)
-      (effects (font (size 1.27 1.27)) hide)
-    )
-    (property "MPN" "SN74AHC1G04DBVR" (at 129.54 86.36 0)
-      (effects (font (size 1.27 1.27)) hide)
-    )
-    (property "Status" "" (at 129.54 86.36 0)
+    (property "Value" "74LVC1G04" (at 134.62 81.28 0)
+      (effects (font (size 1.27 1.27)))
+    )
+    (property "Footprint" "Package_TO_SOT_SMD:SOT-353_SC-70-5" (at 129.54 86.36 0)
+      (effects (font (size 1.27 1.27)) hide)
+    )
+    (property "Datasheet" "https://datasheet.lcsc.com/lcsc/1811021113_Texas-Instruments-SN74LVC1G04DCKR_C8207.pdf" (at 129.54 86.36 0)
+      (effects (font (size 1.27 1.27)) hide)
+    )
+    (property "MPN" "SN74LVC1G04DCKR" (at 129.54 86.36 0)
+      (effects (font (size 1.27 1.27)) hide)
+    )
+    (property "Status" "OK" (at 129.54 86.36 0)
       (effects (font (size 1.27 1.27)) hide)
     )
@@
       (effects (font (size 1.27 1.27)))
     )
-    (property "Value" "74AHC1G08" (at 173.99 66.04 0)
-      (effects (font (size 1.27 1.27)))
-    )
-    (property "Footprint" "Package_TO_SOT_SMD:SOT-23-5" (at 165.1 71.12 0)
-      (effects (font (size 1.27 1.27)) hide)
-    )
-    (property "Datasheet" "https://datasheet.lcsc.com/lcsc/1809151118_Texas-Instruments-SN74AHC1G08DBVR_C7467.pdf" (at 165.1 71.12 0)
-      (effects (font (size 1.27 1.27)) hide)
-    )
-    (property "MPN" "SN74AHC1G08DBVR" (at 165.1 71.12 0)
-      (effects (font (size 1.27 1.27)) hide)
-    )
-    (property "Status" "" (at 165.1 71.12 0)
-      (effects (font (size 1.27 1.27)) hide)
-    )
+    (property "Value" "74LVC1G08" (at 173.99 66.04 0)
+      (effects (font (size 1.27 1.27)))
+    )
+    (property "Footprint" "Package_TO_SOT_SMD:SOT-353_SC-70-5" (at 165.1 71.12 0)
+      (effects (font (size 1.27 1.27)) hide)
+    )
+    (property "Datasheet" "https://datasheet.lcsc.com/lcsc/1809051811_Texas-Instruments-SN74LVC1G08DCKR_C7832.pdf" (at 165.1 71.12 0)
+      (effects (font (size 1.27 1.27)) hide)
+    )
+    (property "MPN" "SN74LVC1G08DCKR" (at 165.1 71.12 0)
+      (effects (font (size 1.27 1.27)) hide)
+    )
+    (property "Status" "OK" (at 165.1 71.12 0)
+      (effects (font (size 1.27 1.27)) hide)
+    )

Commit message: Progressed ECAD.
Parts:
- gave numbers to parts that had none: 5
