File: ECAD/SCART_switcher/audio_in.kicad_sch (KiCad schematic)
At the start: 17 parts, among them Q3 MMBFJ111, Q4 MMBFJ111, Q57 BC847, U4 CD4066BPW

Commit message: progressed ecad
Parts:
- added Q57: BC847, Package_TO_SOT_SMD:SOT-23, symbol Transistor_BJT:BC847
- added R28, R282, R292, R302: R, symbol Device:R
Connections:
- net +9V: now also Q57.3 (C), R282.1
- net ENABLE: now also R28.1, R302.1
- net GND: now also R292.2
- net AUDIO_OUT_ENABLE: now reaches U4.12, U4.13, U4.5, U4.6
- net AUDIO_OUT_ENABLE: now also Q57.2 (E), R292.1
- net MUTE: now reaches Q4.3 (G)
- net MUTE: now also Q3.3 (G), Q57.3 (C), R282.2
- net at Q57.1 (B): now also R28.2
- new net: Q57.1 (B), R302.2
Other:
- note added: "(*1)"
- note added: "(*1) RF input RC filter. Should be placed near the input connector as possible."
- note added: "(*2)"
- note added: "(*2) Drain resistor to discharge the DC blocking capacitor."
- note added: "(*3)"
- note added: "(*3) This JFET is added to improve channel isolation when this channel is off."
- note removed: "Drain resistor to discharge the DC blocking capacitor."
- note removed: "JFETs to improve channel isolation."
- note removed: "RF input filter. Place near connector."
- moved on the sheet: C10, Q57, U4E

Commit message: Progressed ECAD.
Parts:
- renumbered C9 to C?, C10 to C?, C8 to C?, Q4 to Q?, Q3 to Q?, Q57 to Q?, R28 to R82, R282 to R83, R302 to R88, R292 to R91, R13 to R?, R20 to R?, R17 to R?, R16 to R?, R12 to R?, R21 to R?, R18 to R?, R19 to R?, U4 to U?

Commit message: progressed ecad
Parts:
- C?: MPN (none) -> CL21B104KBCNNNC
Other:
- note added: "(*3) This JFET is added to improve channel isolation when this input channel is off."
- note removed: "(*3) This JFET is added to improve channel isolation when this channel is off."
Changed lines of the file:
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@@
     (effects (font (size 1.27 1.27)) (justify left bottom))
   )
-  (text "(*3) This JFET is added to improve channel isolation when this channel is off."
+  (text "(*3) This JFET is added to improve channel isolation when this input channel is off."
     (at 177.8 176.53 0)
     (effects (font (size 1.27 1.27)) (justify left bottom))
@@
       (effects (font (size 1.27 1.27)) hide)
     )
-    (property "Datasheet" "~" (at 163.83 135.89 0)
+    (property "Datasheet" "https://datasheet.lcsc.com/lcsc/1810191215_Samsung-Electro-Mechanics-CL21B104KBCNNNC_C1711.pdf" (at 163.83 135.89 0)
       (effects (font (size 1.27 1.27)) hide)
     )
@@
       (effects (font (size 1.27 1.27)) hide)
     )
+    (property "MPN" "CL21B104KBCNNNC" (at 163.83 135.89 0)
+      (effects (font (size 1.27 1.27)) hide)
+    )

Commit message: progressed ecad
Parts:
- C? (x2): value 100pC -> 1nC
Other:
- note added: "(*1) RF input low pass RC filter. Should be placed near the input connector as possible. Assuming a max source impedance of 1k ohm, the cut-off (-3 db point) frequency will be at 145kHz."
- note added: "(*3) JFET added to improve channel isolation when this input channel is off."
- note added: "(*4)"
- note added: "(*4) Two switches are used in paralel to improve linearity and reduce total series resistence."
- note added: "Input conditioning circuit"
- note removed: "(*1) RF input RC filter. Should be placed near the input connector as possible."
- note removed: "(*3) This JFET is added to improve channel isolation when this input channel is off."
- note removed: "Audio signals buffer"
Changed lines of the file:
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@@
     (stroke (width 0) (type default))
   )
-  (text "Audio signals buffer" (at 128.27 40.64 0)
+  (text "Input conditioning circuit" (at 124.46 33.02 0)
     (effects (font (size 1.27 1.27)) (justify left bottom))
   )
-  (text "(*1) RF input RC filter. Should be placed near the input connector as possible."
-    (at 177.8 168.91 0)
+  (text "(*1) RF input low pass RC filter. Should be placed near the input connector as possible.\nAssuming a max source impedance of 1k ohm, the cut-off (-3 db point) frequency will be at 145kHz."
+    (at 177.8 171.45 0)
     (effects (font (size 1.27 1.27)) (justify left bottom))
   )
@@
     (effects (font (size 1.27 1.27)) (justify left bottom))
   )
-  (text "(*1)" (at 92.71 67.31 0)
+  (text "(*1)" (at 95.25 58.42 0)
     (effects (font (size 1.27 1.27)) (justify left bottom))
   )
   (text "(*2) Drain resistor to discharge the DC blocking capacitor."
-    (at 177.8 172.72 0)
+    (at 177.8 173.99 0)
     (effects (font (size 1.27 1.27)) (justify left bottom))
   )
-  (text "(*3) This JFET is added to improve channel isolation when this input channel is off."
+  (text "(*3) JFET added to improve channel isolation when this input channel is off."
     (at 177.8 176.53 0)
+    (effects (font (size 1.27 1.27)) (justify left bottom))
+  )
+  (text "(*4)" (at 171.45 53.34 0)
+    (effects (font (size 1.27 1.27)) (justify left bottom))
+  )
+  (text "(*4) Two switches are used in paralel to improve linearity and reduce total series resistence."
+    (at 177.8 179.07 0)
     (effects (font (size 1.27 1.27)) (justify left bottom))
   )
@@
       (effects (font (size 1.27 1.27)) (justify left))
     )
-    (property "Value" "100pC" (at 97.028 62.23 0)
+    (property "Value" "1nC" (at 97.028 62.23 0)
       (effects (font (size 1.27 1.27)) (justify left))
     )
@@
       (effects (font (size 1.27 1.27)) (justify left))
     )
-    (property "Value" "100pC" (at 97.028 107.95 0)
+    (property "Value" "1nC" (at 97.028 107.95 0)
       (effects (font (size 1.27 1.27)) (justify left))
     )

Commit message: progressed ecad
Parts:
- added D?: BAS16W, Package_TO_SOT_SMD:SOT-323_SC-70, symbol Diode:BAS16W
- added R83: 680kR, symbol Device:R
- renumbered R82 to R81, R83 to R82
Connections:
- net +4V5: now also R83.2
- net ENABLE: no longer R88.1
- net MUTE: now also D?.1 (A), R83.1; no longer Q?.3 (C), R82.2
- new net: D?.3 (K), Q?.3 (C), R82.2
Other:
- note added: "(*2) Drain resistor to discharge the DC blocking capacitor when no input connected to avoid pop sounds."
- note removed: "(*2) Drain resistor to discharge the DC blocking capacitor."
- moved on the sheet: Q?, R81, R82

Commit message: Update audio_in.kicad_sch
Parts:
- removed Q?: BC847, Package_TO_SOT_SMD:SOT-23, symbol Transistor_BJT:BC847
- removed R88, R91: R, symbol Device:R
- added Q28: BC847, Package_TO_SOT_SMD:SOT-23, symbol Transistor_BJT:BC847
- added R82, R84: R, symbol Device:R
- renumbered R82 to R83, R83 to R85
Connections:
- net +9V: now also R84.1
- net AUDIO_OUT_ENABLE: now also Q28.3 (C), R84.2
- net ENABLE: now also Q28.2 (E)
- new net: Q28.1 (B), R82.2
- new net +5V: R82.1

Commit message: progressed ecad
Parts:
- Q? (x2): value MMBFJ111 -> MMBFJ113
- renumbered Q28 to Q25, R81 to R78, R82 to R79, R83 to R80, R84 to R81, R85 to R82

Commit message: progressed ecad
Parts:
- Q? (x2): value MMBFJ113 -> 2SK209; footprint Package_TO_SOT_SMD:SOT-23 -> Package_TO_SOT_SMD:SC-59_Handsoldering; MFN (none) -> 2SK209-GR(TE85L,F)
Changed lines of the file:
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@@
       (effects (font (size 1.27 1.27)) (justify left))
     )
-    (property "Value" "MMBFJ113" (at 135.89 111.76 0)
+    (property "Value" "2SK209" (at 135.89 111.76 0)
       (effects (font (size 1.27 1.27)) (justify left))
     )
-    (property "Footprint" "Package_TO_SOT_SMD:SOT-23" (at 151.13 108.585 0)
+    (property "Footprint" "Package_TO_SOT_SMD:SC-59_Handsoldering" (at 151.13 108.585 0)
       (effects (font (size 1.27 1.27) italic) (justify left) hide)
     )
-    (property "Datasheet" "https://www.onsemi.com/pub/Collateral/MMBFJ113-D.PDF" (at 146.05 106.68 0)
+    (property "Datasheet" "https://datasheet.lcsc.com/lcsc/1810271708_TOSHIBA-2SK209-GR-TE85L-F_C61792.pdf" (at 146.05 106.68 0)
       (effects (font (size 1.27 1.27)) (justify left) hide)
+    )
+    (property "MFN" "2SK209-GR(TE85L,F)" (at 146.05 106.68 0)
+      (effects (font (size 1.27 1.27)) hide)
     )
     (pin "1")
@@
       (effects (font (size 1.27 1.27)) (justify left))
     )
-    (property "Value" "MMBFJ113" (at 135.89 66.04 0)
+    (property "Value" "2SK209" (at 135.89 66.04 0)
       (effects (font (size 1.27 1.27)) (justify left))
     )
-    (property "Footprint" "Package_TO_SOT_SMD:SOT-23" (at 151.13 62.865 0)
+    (property "Footprint" "Package_TO_SOT_SMD:SC-59_Handsoldering" (at 151.13 62.865 0)
       (effects (font (size 1.27 1.27) italic) (justify left) hide)
     )
-    (property "Datasheet" "https://www.onsemi.com/pub/Collateral/MMBFJ113-D.PDF" (at 146.05 60.96 0)
+    (property "Datasheet" "https://datasheet.lcsc.com/lcsc/1810271708_TOSHIBA-2SK209-GR-TE85L-F_C61792.pdf" (at 146.05 60.96 0)
       (effects (font (size 1.27 1.27)) (justify left) hide)
     )
-    (pin "1")
+    (property "MFN" "2SK209-GR(TE85L,F)" (at 146.05 60.96 0)
+      (effects (font (size 1.27 1.27)) hide)
+    )
+    (pin "1")
