File: ECAD/SCART_switcher/audio_in.kicad_sch (KiCad schematic)
At the start: 28 parts, among them Q25 BC847

Commit message: progressed ecad
Parts:
- R82: value 680kR -> 220kR
- R? (x2): value 22kR -> 20kR
Other:
- note added: "(*5)"
- note added: "(*5) Use thin film resistor with 1% or better tolerance."
Changed lines of the file:
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@@
+    (stroke (width 0) (type default))
+  )
+  (wire (pts (xy 39.37 181.61) (xy 43.18 181.61))
     (stroke (width 0) (type default))
   )
@@
     (stroke (width 0) (type default))
   )
+  (text "(*5) Use thin film resistor with 1% or better tolerance."
+    (at 177.8 180.34 0)
+    (effects (font (size 1.27 1.27)) (justify left bottom))
+  )
   (text "Input conditioning circuit" (at 124.46 33.02 0)
     (effects (font (size 1.27 1.27)) (justify left bottom))
   )
   (text "(*1) RF input low pass RC filter. Should be placed near the input connector as possible.\nAssuming a max source impedance of 1k ohm, the cut-off (-3 db point) frequency will be at 145kHz."
-    (at 177.8 171.45 0)
+    (at 177.8 170.18 0)
+    (effects (font (size 1.27 1.27)) (justify left bottom))
+  )
+  (text "(*5)" (at 130.81 50.8 0)
     (effects (font (size 1.27 1.27)) (justify left bottom))
   )
@@
   )
   (text "(*2) Drain resistor to discharge the DC blocking capacitor when no input connected to avoid pop sounds."
-    (at 177.8 173.99 0)
+    (at 177.8 172.72 0)
     (effects (font (size 1.27 1.27)) (justify left bottom))
   )
   (text "(*3) JFET added to improve channel isolation when this input channel is off."
-    (at 177.8 176.53 0)
+    (at 177.8 175.26 0)
     (effects (font (size 1.27 1.27)) (justify left bottom))
   )
@@
   )
   (text "(*4) Two switches are used in paralel to improve linearity and reduce total series resistence."
-    (at 177.8 179.07 0)
+    (at 177.8 177.8 0)
     (effects (font (size 1.27 1.27)) (justify left bottom))
   )
@@
     (effects (font (size 1.27 1.27)) (justify right))
   )
-  (hierarchical_label "ENABLE" (shape input) (at 43.18 181.61 180) (fields_autoplaced)
+  (hierarchical_label "ENABLE" (shape input) (at 39.37 181.61 180) (fields_autoplaced)
     (effects (font (size 1.27 1.27)) (justify right))
   )
@@
       (effects (font (size 1.27 1.27)))
     )
-    (property "Value" "22kR" (at 137.16 49.53 90)
+    (property "Value" "20kR" (at 137.16 49.53 90)
       (effects (font (size 1.27 1.27)))
     )
@@
       (effects (font (size 1.27 1.27)) (justify left))
     )
-    (property "Value" "680kR" (at 81.28 142.24 0)
+    (property "Value" "220kR" (at 81.28 142.24 0)
       (effects (font (size 1.27 1.27)) (justify left))
     )
@@
       (effects (font (size 1.27 1.27)))
     )
-    (property "Value" "22kR" (at 137.16 95.25 90)
-      (effects (font (size 1.27 1.27)))
-    )
+    (property "Value" "20kR" (at 137.16 95.25 90)
+      (effects (font (size 1.27 1.27)))
+    )

Commit message: progressed ecad
Other:
- note added: "Audio switch control"
- note added: "Mute control"
- moved on the sheet: D?, Q25, Q?, R78, R79, R80, R81, R82

Commit message: progresed ECAD
Parts:
- R78, R79, R80, R81, R82: footprint (none) -> Resistor_SMD:R_0805_2012Metric_Pad1.20x1.40mm_HandSolder
Changed lines of the file:
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@@
       (effects (font (size 1.27 1.27)) (justify left))
     )
-    (property "Footprint" "" (at 68.072 134.62 90)
+    (property "Footprint" "Resistor_SMD:R_0805_2012Metric_Pad1.20x1.40mm_HandSolder" (at 68.072 134.62 90)
       (effects (font (size 1.27 1.27)) hide)
     )
@@
       (effects (font (size 1.27 1.27)) (justify left))
     )
-    (property "Footprint" "" (at 57.912 171.45 90)
+    (property "Footprint" "Resistor_SMD:R_0805_2012Metric_Pad1.20x1.40mm_HandSolder" (at 57.912 171.45 90)
       (effects (font (size 1.27 1.27)) hide)
     )
@@
       (effects (font (size 1.27 1.27)))
     )
-    (property "Footprint" "" (at 38.1 135.128 90)
+    (property "Footprint" "Resistor_SMD:R_0805_2012Metric_Pad1.20x1.40mm_HandSolder" (at 38.1 135.128 90)
       (effects (font (size 1.27 1.27)) hide)
     )
@@
       (effects (font (size 1.27 1.27)) (justify left))
     )
-    (property "Footprint" "" (at 46.482 171.45 90)
+    (property "Footprint" "Resistor_SMD:R_0805_2012Metric_Pad1.20x1.40mm_HandSolder" (at 46.482 171.45 90)
       (effects (font (size 1.27 1.27)) hide)
     )
@@
       (effects (font (size 1.27 1.27)) (justify left))
     )
-    (property "Footprint" "" (at 47.752 124.46 90)
-      (effects (font (size 1.27 1.27)) hide)
-    )
+    (property "Footprint" "Resistor_SMD:R_0805_2012Metric_Pad1.20x1.40mm_HandSolder" (at 47.752 124.46 90)
+      (effects (font (size 1.27 1.27)) hide)
+    )

Commit message: progressed ecad
Parts:
- added R82: 10kR, Resistor_SMD:R_0805_2012Metric_Pad1.20x1.40mm_HandSolder, symbol Device:R
- R78, R79: value R -> 100kR
- R80, R81: value R -> 10kR
- renumbered Q25 to Q26, R82 to R83
Connections:
- net AUDIO_OUT_ENABLE: now also R82.2; no longer R81.2
- new net: R81.2, R82.1
Other:
- moved on the sheet: R81

Commit message: progressed ecad
Parts:
- removed Q26: BC847, Package_TO_SOT_SMD:SOT-23, symbol Transistor_BJT:BC847
- removed R79: 100kR, Resistor_SMD:R_0805_2012Metric_Pad1.20x1.40mm_HandSolder, symbol Device:R
- removed R81: 10kR, Resistor_SMD:R_0805_2012Metric_Pad1.20x1.40mm_HandSolder, symbol Device:R
- added Q26: BC857, Package_TO_SOT_SMD:SOT-23, symbol Transistor_BJT:BC857
- added R80: 100kR, Resistor_SMD:R_0805_2012Metric_Pad1.20x1.40mm_HandSolder, symbol Device:R
- renumbered R80 to R79, R83 to R81
Connections:
- net +9V: now also Q26.2 (E)
- net AUDIO_OUT_ENABLE: now also R82.1, Q26.3 (C); no longer R82.2
- net GND: now also R82.2
- net at D?.3 (K), Q?.3 (C), R79.2: now also R80.1
- new net: Q26.1 (B), R80.2
Other:
- moved on the sheet: C?, D?, Q?, R78, R79, R81, R82, R?, U?A, U?B, U?C, U?D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

Commit message: progressed ecad
Parts:
- R78, R80: value 100kR -> 47kR
Changed lines of the file:
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@@
       (effects (font (size 1.27 1.27)))
     )
-    (property "Value" "100kR" (at 73.66 157.48 90)
+    (property "Value" "47kR" (at 73.66 157.48 90)
       (effects (font (size 1.27 1.27)))
     )
@@
       (effects (font (size 1.27 1.27)))
     )
-    (property "Value" "100kR" (at 44.45 129.54 90)
-      (effects (font (size 1.27 1.27)))
-    )
+    (property "Value" "47kR" (at 44.45 129.54 90)
+      (effects (font (size 1.27 1.27)))
+    )

Commit message: progressed ECAD
Parts:
- renumbered Q26 to Q16, R78 to R108, R79 to R109, R80 to R110, R81 to R111, R82 to R112

Commit message: progressed ecad
Parts:
- renumbered Q16 to Q26, R108 to R88, R109 to R89, R110 to R90, R111 to R91, R112 to R92
