File: ECAD/SCART_switcher/audio_out.kicad_sch (KiCad schematic)
At the start: 28 parts, among them U10 RC4580, U9 RC4580, U97 RC4580

Commit message: progressed ecad
Parts:
- removed C23, C24, C25, C26: 100uC, symbol Device:C_Polarized
- added C165, C24, C25, C26: 10uC, symbol Device:C
- R40, R41, R42, R43: value 22kR -> 220kR
Connections:
- net at R43.1, R47.1: now also C26.2
- net at R?.2, U10.1: now also C165.1
- net at R42.1, R46.1: now also C25.2
- net at R?.2, U97.7: now also C26.1
- net at R?.2, U10.7: now also C24.1
- net at R?.2, U97.1: now also C25.1
- net at R41.1, R45.1: now also C24.2
- net at R40.1, R44.1: now also C165.2
Other:
- note added: "10uC DC blocking capacitor chosen assuming a load impedance of 10k ohm. Cut-off frequency at 1.6Hz."
- note added: "Drain resistor to discharge the DC blocking capacitor."
- moved on the sheet: C?, R40, R41, R42, R43, R44, R45, R46, R47, R?, U10A, U10B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

Commit message: progressed ecad
Other:
- note added: "(*1)"
- note added: "(*1) 10uC DC blocking capacitor chosen assuming a load impedance of 10k ohm. Cut-off frequency at 1.6Hz."
- note added: "(*2)"
- note added: "(*2) Drain resistor to discharge the DC blocking capacitor."
- note removed: "10uC DC blocking capacitor chosen assuming a load impedance of 10k ohm. Cut-off frequency at 1.6Hz."
- note removed: "Drain resistor to discharge the DC blocking capacitor."
Changed lines of the file:
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@@
     (stroke (width 0) (type default))
   )
-  (text "Drain resistor\nto discharge\nthe DC blocking\ncapacitor."
-    (at 162.56 165.1 0)
+  (text "(*1)" (at 157.48 144.78 0)
     (effects (font (size 1.27 1.27)) (justify left bottom))
   )
-  (text "10uC DC blocking\ncapacitor chosen\nassuming a load\nimpedance of 10k ohm.\nCut-off frequency at 1.6Hz."
-    (at 156.21 30.48 0)
+  (text "(*2)" (at 161.29 149.86 0)
     (effects (font (size 1.27 1.27)) (justify left bottom))
   )
+  (text "(*2) Drain resistor to discharge the DC blocking capacitor."
+    (at 177.8 175.26 0)
+    (effects (font (size 1.27 1.27)) (justify left bottom))
+  )
+  (text "(*1) 10uC DC blocking capacitor chosen assuming a load impedance of 10k ohm.\nCut-off frequency at 1.6Hz."
+    (at 177.8 171.45 0)
+    (effects (font (size 1.27 1.27)) (justify left bottom))
+  )

Commit message: Progressed ECAD.
Parts:
- added Q? (x2): MMBFJ111, Package_TO_SOT_SMD:SOT-23, symbol Transistor_FET:MMBFJ111
- added Q?: BC847, Package_TO_SOT_SMD:SOT-23, symbol Transistor_BJT:BC847
- added R? (x2): R, symbol Device:R
- renumbered C165 to C55, C24 to C56, C25 to C57, C26 to C58, R43 to R?, R42 to R?, R47 to R?, R44 to R?, R46 to R?, R41 to R?, R45 to R?, R40 to R?, U10 to U?, U97 to U?, U9 to U?
Connections:
- net +4V5: now also Q?.2 (S), Q?.2 (S)
- net +9V: now also R?.1
- net AUDIO_LEFT_IN: now also Q?.1 (D)
- net AUDIO_RIGHT_IN: now also Q?.1 (D)
- net GND: now also Q?.2 (E)
- new net: Q?.1 (B), R?.2
- new net ENABLE: R?.1
- new net MUTE: Q?.3 (C), Q?.3 (G), Q?.3 (G), R?.2
Other:
- note added: "(*3)"
- note added: "(*3) This JFET is added to properly bias the opamp inverting input when no active input source is enabled."
- moved on the sheet: C?, U?C

Commit message: progressed ecad
Parts:
- C? (x3): MPN (none) -> CL21B104KBCNNNC
- R? (x4): value 68R -> 100R; footprint (none) -> Resistor_SMD:R_0805_2012Metric_Pad1.20x1.40mm_HandSolder
Other:
- note added: "(*1) 10uC DC blocking capacitor chosen assuming a load impedance of 10k ohm. Cut-off (-3 db point) frequency at 1.6Hz."
- note added: "(*3) JFET added to properly bias the opamp inverting input when no active input source is enabled."
- note added: "(*4)"
- note added: "(*4) Decoupling resistor to isolate the opamp from the line shunt-capacitance."
- note removed: "(*1) 10uC DC blocking capacitor chosen assuming a load impedance of 10k ohm. Cut-off frequency at 1.6Hz."
- note removed: "(*3) This JFET is added to properly bias the opamp inverting input when no active input source is enabled."
Changed lines of the file:
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@@
     (stroke (width 0) (type default))
   )
-  (text "(*1)" (at 157.48 144.78 0)
+  (text "(*4)" (at 181.61 45.72 0)
     (effects (font (size 1.27 1.27)) (justify left bottom))
   )
-  (text "(*2)" (at 161.29 149.86 0)
+  (text "(*1)" (at 158.75 46.99 0)
+    (effects (font (size 1.27 1.27)) (justify left bottom))
+  )
+  (text "(*4) Decoupling resistor to isolate the opamp from the line shunt-capacitance."
+    (at 177.8 179.07 0)
+    (effects (font (size 1.27 1.27)) (justify left bottom))
+  )
+  (text "(*2)" (at 161.29 52.07 0)
     (effects (font (size 1.27 1.27)) (justify left bottom))
   )
   (text "(*2) Drain resistor to discharge the DC blocking capacitor."
-    (at 177.8 175.26 0)
+    (at 177.8 173.99 0)
     (effects (font (size 1.27 1.27)) (justify left bottom))
   )
-  (text "(*3) This JFET is added to properly bias the opamp inverting input when no active input source is enabled."
-    (at 177.8 179.07 0)
+  (text "(*3) JFET added to properly bias the opamp inverting input when no active input source is enabled."
+    (at 177.8 176.53 0)
     (effects (font (size 1.27 1.27)) (justify left bottom))
   )
-  (text "(*1) 10uC DC blocking capacitor chosen assuming a load impedance of 10k ohm.\nCut-off frequency at 1.6Hz."
+  (text "(*1) 10uC DC blocking capacitor chosen assuming a load impedance of 10k ohm.\nCut-off (-3 db point) frequency at 1.6Hz."
     (at 177.8 171.45 0)
     (effects (font (size 1.27 1.27)) (justify left bottom))
@@
     (effects (font (size 1.27 1.27)) (justify left bottom))
   )
-  (text "(*3)" (at 80.01 72.39 0)
-    (effects (font (size 1.27 1.27)) (justify left bottom))
-  )
   (label "MUTE" (at 74.93 74.93 0) (fields_autoplaced)
     (effects (font (size 1.27 1.27)) (justify left bottom))
@@
       (effects (font (size 1.27 1.27)) hide)
     )
-    (property "Datasheet" "~" (at 72.39 172.72 0)
+    (property "Datasheet" "https://datasheet.lcsc.com/lcsc/1810191215_Samsung-Electro-Mechanics-CL21B104KBCNNNC_C1711.pdf" (at 72.39 172.72 0)
       (effects (font (size 1.27 1.27)) hide)
     )
@@
       (effects (font (size 1.27 1.27)) hide)
     )
+    (property "MPN" "CL21B104KBCNNNC" (at 72.39 172.72 0)
+      (effects (font (size 1.27 1.27)) hide)
+    )
     (pin "1")
     (pin "2")
@@
       (effects (font (size 1.27 1.27)) hide)
     )
-    (property "Datasheet" "~" (at 44.45 172.72 0)
+    (property "Datasheet" "https://datasheet.lcsc.com/lcsc/1810191215_Samsung-Electro-Mechanics-CL21B104KBCNNNC_C1711.pdf" (at 44.45 172.72 0)
       (effects (font (size 1.27 1.27)) hide)
     )
@@
       (effects (font (size 1.27 1.27)) hide)
     )
+    (property "MPN" "CL21B104KBCNNNC" (at 44.45 172.72 0)
+      (effects (font (size 1.27 1.27)) hide)
+    )
     (pin "1")
     (pin "2")
@@
       (effects (font (size 1.27 1.27)))
     )
-    (property "Value" "68R" (at 179.07 137.16 90)
+    (property "Value" "100R" (at 179.07 137.16 90)
       (effects (font (size 1.27 1.27)))
     )
-    (property "Footprint" "" (at 179.07 142.748 90)
+    (property "Footprint" "Resistor_SMD:R_0805_2012Metric_Pad1.20x1.40mm_HandSolder" (at 179.07 142.748 90)
       (effects (font (size 1.27 1.27)) hide)
     )
@@
       (effects (font (size 1.27 1.27)))
     )
-    (property "Value" "68R" (at 179.07 38.1 90)
+    (property "Value" "100R" (at 179.07 38.1 90)
       (effects (font (size 1.27 1.27)))
     )
-    (property "Footprint" "" (at 179.07 43.688 90)
+    (property "Footprint" "Resistor_SMD:R_0805_2012Metric_Pad1.20x1.40mm_HandSolder" (at 179.07 43.688 90)
       (effects (font (size 1.27 1.27)) hide)
     )
@@
       (effects (font (size 1.27 1.27)))
     )
-    (property "Value" "68R" (at 179.07 106.68 90)
+    (property "Value" "100R" (at 179.07 106.68 90)
       (effects (font (size 1.27 1.27)))
     )
-    (property "Footprint" "" (at 179.07 112.268 90)
+    (property "Footprint" "Resistor_SMD:R_0805_2012Metric_Pad1.20x1.40mm_HandSolder" (at 179.07 112.268 90)
       (effects (font (size 1.27 1.27)) hide)
     )
@@
       (effects (font (size 1.27 1.27)))
     )
-    (property "Value" "68R" (at 179.07 68.58 90)
+    (property "Value" "100R" (at 179.07 68.58 90)
       (effects (font (size 1.27 1.27)))
     )
-    (property "Footprint" "" (at 179.07 74.168 90)
+    (property "Footprint" "Resistor_SMD:R_0805_2012Metric_Pad1.20x1.40mm_HandSolder" (at 179.07 74.168 90)
       (effects (font (size 1.27 1.27)) hide)
     )
@@
       (effects (font (size 1.27 1.27)) hide)
     )
-    (property "Datasheet" "~" (at 100.33 172.72 0)
+    (property "Datasheet" "https://datasheet.lcsc.com/lcsc/1810191215_Samsung-Electro-Mechanics-CL21B104KBCNNNC_C1711.pdf" (at 100.33 172.72 0)
       (effects (font (size 1.27 1.27)) hide)
     )
@@
       (effects (font (size 1.27 1.27)) hide)
     )
+    (property "MPN" "CL21B104KBCNNNC" (at 100.33 172.72 0)
+      (effects (font (size 1.27 1.27)) hide)
+    )

Commit message: progressed ecad
Other:
- note added: "(*1) 10uC DC blocking capacitor. Assuming a minimum load impedance of 10k ohm, the cut-off (-3 db point) frequency will be at 1.6Hz."
- note removed: "(*1) 10uC DC blocking capacitor chosen assuming a load impedance of 10k ohm. Cut-off (-3 db point) frequency at 1.6Hz."
Changed lines of the file:
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@@
     (effects (font (size 1.27 1.27)) (justify left bottom))
   )
-  (text "(*1) 10uC DC blocking capacitor chosen assuming a load impedance of 10k ohm.\nCut-off (-3 db point) frequency at 1.6Hz."
+  (text "(*1) 10uC DC blocking capacitor.\nAssuming a minimum load impedance of 10k ohm, the cut-off (-3 db point) frequency will be at 1.6Hz."
     (at 177.8 171.45 0)
     (effects (font (size 1.27 1.27)) (justify left bottom))

Commit message: progressed ecad
Parts:
- added D14: BAS16W, Package_TO_SOT_SMD:SOT-323_SC-70, symbol Diode:BAS16W
- added R?: 680kR, symbol Device:R
- renumbered C55 to C54, C56 to C55, C57 to C56, C58 to C57
Connections:
- net +4V5: now also R?.2
- net MUTE: now also D14.1 (A), R?.1; no longer Q?.3 (C), R?.2
- new net: D14.3 (K), Q?.3 (C), R?.2
Other:
- note added: "(*2) Drain resistor to discharge the DC blocking capacitor when output not connected to avoid pop sounds."
- note removed: "(*2) Drain resistor to discharge the DC blocking capacitor."
- moved on the sheet: Q?, R?

Commit message: progressed ecad
Parts:
- removed D14: BAS16W, Package_TO_SOT_SMD:SOT-323_SC-70, symbol Diode:BAS16W
- removed Q? (x2): MMBFJ111, Package_TO_SOT_SMD:SOT-23, symbol Transistor_FET:MMBFJ111
- removed Q?: BC847, Package_TO_SOT_SMD:SOT-23, symbol Transistor_BJT:BC847
- removed R? (x2): R, symbol Device:R
- removed R?: 680kR, symbol Device:R
Other:
- note added: "(*3) Decoupling resistor to isolate the opamp from the line shunt-capacitance."
- note removed: "(*3) JFET added to properly bias the opamp inverting input when no active input source is enabled."
- note removed: "(*4)"
- note removed: "(*4) Decoupling resistor to isolate the opamp from the line shunt-capacitance."

Commit message: progressed ecad
Parts:
- R? (x3): value 22kR -> 20kR
Other:
- note added: "(*4)"
- note added: "(*4) Use thin film resistor with 1% or better tolerance for lower noise and better gain match."
Changed lines of the file:
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@@
+    (effects (font (size 1.27 1.27)) (justify left bottom))
+  )
+  (text "(*4)" (at 128.27 36.83 0)
+    (effects (font (size 1.27 1.27)) (justify left bottom))
+  )
+  (text "(*4) Use thin film resistor with 1% or better tolerance for lower noise and better gain match."
+    (at 177.8 179.07 0)
+    (effects (font (size 1.27 1.27)) (justify left bottom))
+  )
+  (text "(*4)" (at 152.4 33.02 0)
+    (effects (font (size 1.27 1.27)) (justify left bottom))
+  )
+  (text "(*4)" (at 109.22 29.21 0)
     (effects (font (size 1.27 1.27)) (justify left bottom))
   )
@@
       (effects (font (size 1.27 1.27)))
     )
-    (property "Value" "22kR" (at 134.62 35.56 90)
+    (property "Value" "20kR" (at 134.62 35.56 90)
       (effects (font (size 1.27 1.27)))
     )
@@
       (effects (font (size 1.27 1.27)))
     )
-    (property "Value" "22kR" (at 148.59 30.48 90)
+    (property "Value" "20kR" (at 148.59 30.48 90)
       (effects (font (size 1.27 1.27)))
     )
@@
       (effects (font (size 1.27 1.27)))
     )
-    (property "Value" "22kR" (at 106.68 26.67 90)
-      (effects (font (size 1.27 1.27)))
-    )
+    (property "Value" "20kR" (at 106.68 26.67 90)
+      (effects (font (size 1.27 1.27)))
+    )
