File: ECAD/SCART_switcher/audio_out.kicad_sch (KiCad schematic)
At the start: 34 parts

Commit message: Progressed ECAD.
Parts:
- C? (x3): footprint Capacitor_SMD:C_0805_2012Metric_Pad1.18x1.45mm_HandSolder -> Capacitor_SMD:C_0805_2012Metric
- R? (x18): footprint Resistor_SMD:R_0805_2012Metric_Pad1.20x1.40mm_HandSolder -> Resistor_SMD:R_0805_2012Metric
Changed lines of the file:
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@@
       (effects (font (size 1.27 1.27)) (justify left))
     )
-    (property "Footprint" "Capacitor_SMD:C_0805_2012Metric_Pad1.18x1.45mm_HandSolder" (at 73.3552 176.53 0)
+    (property "Footprint" "Capacitor_SMD:C_0805_2012Metric" (at 73.3552 176.53 0)
       (effects (font (size 1.27 1.27)) hide)
     )
@@
       (effects (font (size 1.27 1.27)) (justify left))
     )
-    (property "Footprint" "Resistor_SMD:R_0805_2012Metric_Pad1.20x1.40mm_HandSolder" (at 165.862 146.05 90)
+    (property "Footprint" "Resistor_SMD:R_0805_2012Metric" (at 165.862 146.05 90)
       (effects (font (size 1.27 1.27)) hide)
     )
@@
       (effects (font (size 1.27 1.27)))
     )
-    (property "Footprint" "Resistor_SMD:R_0805_2012Metric_Pad1.20x1.40mm_HandSolder" (at 134.62 140.208 90)
+    (property "Footprint" "Resistor_SMD:R_0805_2012Metric" (at 134.62 140.208 90)
       (effects (font (size 1.27 1.27)) hide)
     )
@@
       (effects (font (size 1.27 1.27)))
     )
-    (property "Footprint" "Resistor_SMD:R_0805_2012Metric_Pad1.20x1.40mm_HandSolder" (at 134.62 41.148 90)
+    (property "Footprint" "Resistor_SMD:R_0805_2012Metric" (at 134.62 41.148 90)
       (effects (font (size 1.27 1.27)) hide)
     )
@@
       (effects (font (size 1.27 1.27)))
     )
-    (property "Footprint" "Resistor_SMD:R_0805_2012Metric_Pad1.20x1.40mm_HandSolder" (at 148.59 36.068 90)
+    (property "Footprint" "Resistor_SMD:R_0805_2012Metric" (at 148.59 36.068 90)
       (effects (font (size 1.27 1.27)) hide)
     )
@@
       (effects (font (size 1.27 1.27)) (justify left))
     )
-    (property "Footprint" "Resistor_SMD:R_0805_2012Metric_Pad1.20x1.40mm_HandSolder" (at 165.862 115.57 90)
+    (property "Footprint" "Resistor_SMD:R_0805_2012Metric" (at 165.862 115.57 90)
       (effects (font (size 1.27 1.27)) hide)
     )
@@
       (effects (font (size 1.27 1.27)) (justify left))
     )
-    (property "Footprint" "Capacitor_SMD:C_0805_2012Metric_Pad1.18x1.45mm_HandSolder" (at 45.4152 176.53 0)
+    (property "Footprint" "Capacitor_SMD:C_0805_2012Metric" (at 45.4152 176.53 0)
       (effects (font (size 1.27 1.27)) hide)
     )
@@
       (effects (font (size 1.27 1.27)))
     )
-    (property "Footprint" "Resistor_SMD:R_0805_2012Metric_Pad1.20x1.40mm_HandSolder" (at 179.07 142.748 90)
+    (property "Footprint" "Resistor_SMD:R_0805_2012Metric" (at 179.07 142.748 90)
       (effects (font (size 1.27 1.27)) hide)
     )
@@
       (effects (font (size 1.27 1.27)))
     )
-    (property "Footprint" "Resistor_SMD:R_0805_2012Metric_Pad1.20x1.40mm_HandSolder" (at 134.62 71.628 90)
+    (property "Footprint" "Resistor_SMD:R_0805_2012Metric" (at 134.62 71.628 90)
       (effects (font (size 1.27 1.27)) hide)
     )
@@
       (effects (font (size 1.27 1.27)))
     )
-    (property "Footprint" "Resistor_SMD:R_0805_2012Metric_Pad1.20x1.40mm_HandSolder" (at 148.59 104.648 90)
+    (property "Footprint" "Resistor_SMD:R_0805_2012Metric" (at 148.59 104.648 90)
       (effects (font (size 1.27 1.27)) hide)
     )
@@
       (effects (font (size 1.27 1.27)))
     )
-    (property "Footprint" "Resistor_SMD:R_0805_2012Metric_Pad1.20x1.40mm_HandSolder" (at 179.07 43.688 90)
+    (property "Footprint" "Resistor_SMD:R_0805_2012Metric" (at 179.07 43.688 90)
       (effects (font (size 1.27 1.27)) hide)
     )
@@
       (effects (font (size 1.27 1.27)))
     )
-    (property "Footprint" "Resistor_SMD:R_0805_2012Metric_Pad1.20x1.40mm_HandSolder" (at 179.07 112.268 90)
+    (property "Footprint" "Resistor_SMD:R_0805_2012Metric" (at 179.07 112.268 90)
       (effects (font (size 1.27 1.27)) hide)
     )
@@
       (effects (font (size 1.27 1.27)) (justify left))
     )
-    (property "Footprint" "Resistor_SMD:R_0805_2012Metric_Pad1.20x1.40mm_HandSolder" (at 165.862 77.47 90)
+    (property "Footprint" "Resistor_SMD:R_0805_2012Metric" (at 165.862 77.47 90)
       (effects (font (size 1.27 1.27)) hide)
     )
@@
       (effects (font (size 1.27 1.27)))
     )
-    (property "Footprint" "Resistor_SMD:R_0805_2012Metric_Pad1.20x1.40mm_HandSolder" (at 148.59 66.548 90)
+    (property "Footprint" "Resistor_SMD:R_0805_2012Metric" (at 148.59 66.548 90)
       (effects (font (size 1.27 1.27)) hide)
     )
@@
       (effects (font (size 1.27 1.27)))
     )
-    (property "Footprint" "Resistor_SMD:R_0805_2012Metric_Pad1.20x1.40mm_HandSolder" (at 106.68 62.738 90)
+    (property "Footprint" "Resistor_SMD:R_0805_2012Metric" (at 106.68 62.738 90)
       (effects (font (size 1.27 1.27)) hide)
     )
@@
       (effects (font (size 1.27 1.27)))
     )
-    (property "Footprint" "Resistor_SMD:R_0805_2012Metric_Pad1.20x1.40mm_HandSolder" (at 179.07 74.168 90)
+    (property "Footprint" "Resistor_SMD:R_0805_2012Metric" (at 179.07 74.168 90)
       (effects (font (size 1.27 1.27)) hide)
     )
@@
       (effects (font (size 1.27 1.27)))
     )
-    (property "Footprint" "Resistor_SMD:R_0805_2012Metric_Pad1.20x1.40mm_HandSolder" (at 134.62 109.728 90)
+    (property "Footprint" "Resistor_SMD:R_0805_2012Metric" (at 134.62 109.728 90)
       (effects (font (size 1.27 1.27)) hide)
     )
@@
       (effects (font (size 1.27 1.27)) (justify left))
     )
-    (property "Footprint" "Resistor_SMD:R_0805_2012Metric_Pad1.20x1.40mm_HandSolder" (at 165.862 46.99 90)
+    (property "Footprint" "Resistor_SMD:R_0805_2012Metric" (at 165.862 46.99 90)
       (effects (font (size 1.27 1.27)) hide)
     )
@@
       (effects (font (size 1.27 1.27)))
     )
-    (property "Footprint" "Resistor_SMD:R_0805_2012Metric_Pad1.20x1.40mm_HandSolder" (at 106.68 32.258 90)
+    (property "Footprint" "Resistor_SMD:R_0805_2012Metric" (at 106.68 32.258 90)
       (effects (font (size 1.27 1.27)) hide)
     )
@@
       (effects (font (size 1.27 1.27)))
     )
-    (property "Footprint" "Resistor_SMD:R_0805_2012Metric_Pad1.20x1.40mm_HandSolder" (at 148.59 135.128 90)
+    (property "Footprint" "Resistor_SMD:R_0805_2012Metric" (at 148.59 135.128 90)
       (effects (font (size 1.27 1.27)) hide)
     )
@@
       (effects (font (size 1.27 1.27)) (justify left))
     )
-    (property "Footprint" "Capacitor_SMD:C_0805_2012Metric_Pad1.18x1.45mm_HandSolder" (at 101.2952 176.53 0)
-      (effects (font (size 1.27 1.27)) hide)
-    )
+    (property "Footprint" "Capacitor_SMD:C_0805_2012Metric" (at 101.2952 176.53 0)
+      (effects (font (size 1.27 1.27)) hide)
+    )

Commit message: progressed ecad
Parts:
- U? (x9): footprint (none) -> Package_SO:SOIC-8_3.9x4.9mm_P1.27mm; MPN (none) -> RC4580IDR
Changed lines of the file:
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@@
       (effects (font (size 1.27 1.27)) (justify left))
     )
-    (property "Footprint" "" (at 62.23 172.72 0)
-      (effects (font (size 1.27 1.27)) hide)
-    )
-    (property "Datasheet" "https://www.ti.com/lit/ds/symlink/rc4580.pdf" (at 62.23 172.72 0)
+    (property "Footprint" "Package_SO:SOIC-8_3.9x4.9mm_P1.27mm" (at 62.23 172.72 0)
+      (effects (font (size 1.27 1.27)) hide)
+    )
+    (property "Datasheet" "https://datasheet.lcsc.com/lcsc/2304140030_Texas-Instruments-RC4580IDR_C80100.pdf" (at 62.23 172.72 0)
+      (effects (font (size 1.27 1.27)) hide)
+    )
+    (property "MPN" "RC4580IDR" (at 62.23 172.72 0)
       (effects (font (size 1.27 1.27)) hide)
     )
@@
       (effects (font (size 1.27 1.27)) (justify left))
     )
-    (property "Footprint" "" (at 90.17 172.72 0)
-      (effects (font (size 1.27 1.27)) hide)
-    )
-    (property "Datasheet" "https://www.ti.com/lit/ds/symlink/rc4580.pdf" (at 90.17 172.72 0)
+    (property "Footprint" "Package_SO:SOIC-8_3.9x4.9mm_P1.27mm" (at 90.17 172.72 0)
+      (effects (font (size 1.27 1.27)) hide)
+    )
+    (property "Datasheet" "https://datasheet.lcsc.com/lcsc/2304140030_Texas-Instruments-RC4580IDR_C80100.pdf" (at 90.17 172.72 0)
+      (effects (font (size 1.27 1.27)) hide)
+    )
+    (property "MPN" "RC4580IDR" (at 90.17 172.72 0)
       (effects (font (size 1.27 1.27)) hide)
     )
@@
       (effects (font (size 1.27 1.27)))
     )
-    (property "Footprint" "" (at 106.68 39.37 0)
-      (effects (font (size 1.27 1.27)) hide)
-    )
-    (property "Datasheet" "https://www.ti.com/lit/ds/symlink/rc4580.pdf" (at 106.68 39.37 0)
+    (property "Footprint" "Package_SO:SOIC-8_3.9x4.9mm_P1.27mm" (at 106.68 39.37 0)
+      (effects (font (size 1.27 1.27)) hide)
+    )
+    (property "Datasheet" "https://datasheet.lcsc.com/lcsc/2304140030_Texas-Instruments-RC4580IDR_C80100.pdf" (at 106.68 39.37 0)
+      (effects (font (size 1.27 1.27)) hide)
+    )
+    (property "MPN" "RC4580IDR" (at 106.68 39.37 0)
       (effects (font (size 1.27 1.27)) hide)
     )
@@
       (effects (font (size 1.27 1.27)))
     )
-    (property "Footprint" "" (at 148.59 140.97 0)
-      (effects (font (size 1.27 1.27)) hide)
-    )
-    (property "Datasheet" "https://www.ti.com/lit/ds/symlink/rc4580.pdf" (at 148.59 140.97 0)
+    (property "Footprint" "Package_SO:SOIC-8_3.9x4.9mm_P1.27mm" (at 148.59 140.97 0)
+      (effects (font (size 1.27 1.27)) hide)
+    )
+    (property "Datasheet" "https://datasheet.lcsc.com/lcsc/2304140030_Texas-Instruments-RC4580IDR_C80100.pdf" (at 148.59 140.97 0)
+      (effects (font (size 1.27 1.27)) hide)
+    )
+    (property "MPN" "RC4580IDR" (at 148.59 140.97 0)
       (effects (font (size 1.27 1.27)) hide)
     )
@@
       (effects (font (size 1.27 1.27)))
     )
-    (property "Footprint" "" (at 148.59 72.39 0)
-      (effects (font (size 1.27 1.27)) hide)
-    )
-    (property "Datasheet" "https://www.ti.com/lit/ds/symlink/rc4580.pdf" (at 148.59 72.39 0)
+    (property "Footprint" "Package_SO:SOIC-8_3.9x4.9mm_P1.27mm" (at 148.59 72.39 0)
+      (effects (font (size 1.27 1.27)) hide)
+    )
+    (property "Datasheet" "https://datasheet.lcsc.com/lcsc/2304140030_Texas-Instruments-RC4580IDR_C80100.pdf" (at 148.59 72.39 0)
+      (effects (font (size 1.27 1.27)) hide)
+    )
+    (property "MPN" "RC4580IDR" (at 148.59 72.39 0)
       (effects (font (size 1.27 1.27)) hide)
     )
@@
       (effects (font (size 1.27 1.27)))
     )
-    (property "Footprint" "" (at 148.59 110.49 0)
-      (effects (font (size 1.27 1.27)) hide)
-    )
-    (property "Datasheet" "https://www.ti.com/lit/ds/symlink/rc4580.pdf" (at 148.59 110.49 0)
+    (property "Footprint" "Package_SO:SOIC-8_3.9x4.9mm_P1.27mm" (at 148.59 110.49 0)
+      (effects (font (size 1.27 1.27)) hide)
+    )
+    (property "Datasheet" "https://datasheet.lcsc.com/lcsc/2304140030_Texas-Instruments-RC4580IDR_C80100.pdf" (at 148.59 110.49 0)
+      (effects (font (size 1.27 1.27)) hide)
+    )
+    (property "MPN" "RC4580IDR" (at 148.59 110.49 0)
       (effects (font (size 1.27 1.27)) hide)
     )
@@
       (effects (font (size 1.27 1.27)) (justify left))
     )
-    (property "Footprint" "" (at 34.29 172.72 0)
-      (effects (font (size 1.27 1.27)) hide)
-    )
-    (property "Datasheet" "https://www.ti.com/lit/ds/symlink/rc4580.pdf" (at 34.29 172.72 0)
+    (property "Footprint" "Package_SO:SOIC-8_3.9x4.9mm_P1.27mm" (at 34.29 172.72 0)
+      (effects (font (size 1.27 1.27)) hide)
+    )
+    (property "Datasheet" "https://datasheet.lcsc.com/lcsc/2304140030_Texas-Instruments-RC4580IDR_C80100.pdf" (at 34.29 172.72 0)
+      (effects (font (size 1.27 1.27)) hide)
+    )
+    (property "MPN" "RC4580IDR" (at 34.29 172.72 0)
       (effects (font (size 1.27 1.27)) hide)
     )
@@
       (effects (font (size 1.27 1.27)))
     )
-    (property "Footprint" "" (at 106.68 69.85 0)
-      (effects (font (size 1.27 1.27)) hide)
-    )
-    (property "Datasheet" "https://www.ti.com/lit/ds/symlink/rc4580.pdf" (at 106.68 69.85 0)
+    (property "Footprint" "Package_SO:SOIC-8_3.9x4.9mm_P1.27mm" (at 106.68 69.85 0)
+      (effects (font (size 1.27 1.27)) hide)
+    )
+    (property "Datasheet" "https://datasheet.lcsc.com/lcsc/2304140030_Texas-Instruments-RC4580IDR_C80100.pdf" (at 106.68 69.85 0)
+      (effects (font (size 1.27 1.27)) hide)
+    )
+    (property "MPN" "RC4580IDR" (at 106.68 69.85 0)
       (effects (font (size 1.27 1.27)) hide)
     )
@@
       (effects (font (size 1.27 1.27)))
     )
-    (property "Footprint" "" (at 148.59 41.91 0)
-      (effects (font (size 1.27 1.27)) hide)
-    )
-    (property "Datasheet" "https://www.ti.com/lit/ds/symlink/rc4580.pdf" (at 148.59 41.91 0)
-      (effects (font (size 1.27 1.27)) hide)
-    )
+    (property "Footprint" "Package_SO:SOIC-8_3.9x4.9mm_P1.27mm" (at 148.59 41.91 0)
+      (effects (font (size 1.27 1.27)) hide)
+    )
+    (property "Datasheet" "https://datasheet.lcsc.com/lcsc/2304140030_Texas-Instruments-RC4580IDR_C80100.pdf" (at 148.59 41.91 0)
+      (effects (font (size 1.27 1.27)) hide)
+    )
+    (property "MPN" "RC4580IDR" (at 148.59 41.91 0)
+      (effects (font (size 1.27 1.27)) hide)
+    )

Commit message: Progressed ECAD.
Parts:
- U? (x9): Status (none) -> OK
Changed lines of the file:
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@@
       (effects (font (size 1.27 1.27)) hide)
     )
-    (property "Status" "" (at 62.23 172.72 0)
+    (property "Status" "OK" (at 62.23 172.72 0)
       (effects (font (size 1.27 1.27)) hide)
     )
@@
       (effects (font (size 1.27 1.27)) hide)
     )
-    (property "Status" "" (at 90.17 172.72 0)
+    (property "Status" "OK" (at 90.17 172.72 0)
       (effects (font (size 1.27 1.27)) hide)
     )
@@
       (effects (font (size 1.27 1.27)) hide)
     )
-    (property "Status" "" (at 106.68 39.37 0)
+    (property "Status" "OK" (at 106.68 39.37 0)
       (effects (font (size 1.27 1.27)) hide)
     )
@@
       (effects (font (size 1.27 1.27)) hide)
     )
-    (property "Status" "" (at 148.59 140.97 0)
+    (property "Status" "OK" (at 148.59 140.97 0)
       (effects (font (size 1.27 1.27)) hide)
     )
@@
       (effects (font (size 1.27 1.27)) hide)
     )
-    (property "Status" "" (at 148.59 72.39 0)
+    (property "Status" "OK" (at 148.59 72.39 0)
       (effects (font (size 1.27 1.27)) hide)
     )
@@
       (effects (font (size 1.27 1.27)) hide)
     )
-    (property "Status" "" (at 148.59 110.49 0)
+    (property "Status" "OK" (at 148.59 110.49 0)
       (effects (font (size 1.27 1.27)) hide)
     )
@@
       (effects (font (size 1.27 1.27)) hide)
     )
-    (property "Status" "" (at 34.29 172.72 0)
+    (property "Status" "OK" (at 34.29 172.72 0)
       (effects (font (size 1.27 1.27)) hide)
     )
@@
       (effects (font (size 1.27 1.27)) hide)
     )
-    (property "Status" "" (at 106.68 69.85 0)
+    (property "Status" "OK" (at 106.68 69.85 0)
       (effects (font (size 1.27 1.27)) hide)
     )
@@
       (effects (font (size 1.27 1.27)) hide)
     )
-    (property "Status" "" (at 148.59 41.91 0)
-      (effects (font (size 1.27 1.27)) hide)
-    )
+    (property "Status" "OK" (at 148.59 41.91 0)
+      (effects (font (size 1.27 1.27)) hide)
+    )
