File: ECAD/SCART_switcher/audio_out.kicad_sch (KiCad schematic)
At the start: 34 parts

Commit message: Progressed ECAD.
Parts:
- removed C39, C40, C41, C42: 10uC, symbol Device:C
- added C39, C40, C41, C42: 10uC, Capacitor_SMD:CP_Elec_6.3x5.4, symbol Device:C_Polarized
Connections:
- net at R?.1, R?.1: now also C42.2
- net at R?.2, U?.1: now also C39.1
- net at R?.1, R?.1: now also C41.2
- net at R?.2, U?.7: now also C40.1
- net at R?.1, R?.1: now also C40.2
- net at R?.2, U?.7: now also C42.1
- net at R?.2, U?.1: now also C41.1
- net at R?.1, R?.1: now also C39.2
Changed lines of the file:
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@@
-    )
-  )
-  (symbol (lib_id "Device:C") (at 162.56 72.39 90) (unit 1)
-    (in_bom yes) (on_board yes) (dnp no) (fields_autoplaced)
-    (property "Reference" "C40" (at 162.56 64.77 90)
-      (effects (font (size 1.27 1.27)))
-    )
-    (property "Value" "10uC" (at 162.56 67.31 90)
-      (effects (font (size 1.27 1.27)))
-    )
-    (property "Footprint" "" (at 166.37 71.4248 0)
-      (effects (font (size 1.27 1.27)) hide)
-    )
-    (property "Datasheet" "~" (at 162.56 72.39 0)
-      (effects (font (size 1.27 1.27)) hide)
-    )
-    (property "Status" "" (at 162.56 72.39 0)
-      (effects (font (size 1.27 1.27)) hide)
-    )
-    (pin "1")
-    (pin "2")
-    (instances
-      (project "SCART_switcher"
-        (path "/8cd08eb5-4755-4ef5-8eeb-77fd9974b180/6562ea38-5963-42b2-a0ef-a4a12a4c652f/9f74dfb2-70cd-470e-9dfb-02936b5bb451"
-          (reference "C40") (unit 1)
-        )
-      )
     )
   )
@@
     )
   )
+  (symbol (lib_id "Device:C_Polarized") (at 162.56 110.49 90) (unit 1)
+    (in_bom yes) (on_board yes) (dnp no) (fields_autoplaced)
+    (property "Reference" "C41" (at 161.671 102.87 90)
+      (effects (font (size 1.27 1.27)))
+    )
+    (property "Value" "10uC" (at 161.671 105.41 90)
+      (effects (font (size 1.27 1.27)))
+    )
+    (property "Footprint" "Capacitor_SMD:CP_Elec_6.3x5.4" (at 166.37 109.5248 0)
+      (effects (font (size 1.27 1.27)) hide)
+    )
+    (property "Datasheet" "https://datasheet.lcsc.com/lcsc/2304140030_Nichicon-UWX1H100MCL1GB_C134237.pdf" (at 162.56 110.49 0)
+      (effects (font (size 1.27 1.27)) hide)
+    )
+    (property "MPN" "UWX1H100MCL1GB" (at 162.56 110.49 0)
+      (effects (font (size 1.27 1.27)) hide)
+    )
+    (property "Status" "OK" (at 162.56 110.49 0)
+      (effects (font (size 1.27 1.27)) hide)
+    )
+    (pin "2")
+    (pin "1")
+    (instances
+      (project "SCART_switcher"
+        (path "/8cd08eb5-4755-4ef5-8eeb-77fd9974b180/6562ea38-5963-42b2-a0ef-a4a12a4c652f/9f74dfb2-70cd-470e-9dfb-02936b5bb451"
+          (reference "C41") (unit 1)
+        )
+      )
+    )
+  )
   (symbol (lib_id "Device:R") (at 179.07 41.91 90) (unit 1)
     (in_bom yes) (on_board yes) (dnp no) (fields_autoplaced)
@@
         (path "/8cd08eb5-4755-4ef5-8eeb-77fd9974b180/6562ea38-5963-42b2-a0ef-a4a12a4c652f/9f74dfb2-70cd-470e-9dfb-02936b5bb451"
           (reference "R82") (unit 1)
-        )
-      )
-    )
-  )
-  (symbol (lib_id "Device:C") (at 162.56 41.91 90) (unit 1)
-    (in_bom yes) (on_board yes) (dnp no) (fields_autoplaced)
-    (property "Reference" "C39" (at 162.56 34.29 90)
-      (effects (font (size 1.27 1.27)))
-    )
-    (property "Value" "10uC" (at 162.56 36.83 90)
-      (effects (font (size 1.27 1.27)))
-    )
-    (property "Footprint" "" (at 166.37 40.9448 0)
-      (effects (font (size 1.27 1.27)) hide)
-    )
-    (property "Datasheet" "~" (at 162.56 41.91 0)
-      (effects (font (size 1.27 1.27)) hide)
-    )
-    (property "Status" "" (at 162.56 41.91 0)
-      (effects (font (size 1.27 1.27)) hide)
-    )
-    (pin "1")
-    (pin "2")
-    (instances
-      (project "SCART_switcher"
-        (path "/8cd08eb5-4755-4ef5-8eeb-77fd9974b180/6562ea38-5963-42b2-a0ef-a4a12a4c652f/9f74dfb2-70cd-470e-9dfb-02936b5bb451"
-          (reference "C39") (unit 1)
         )
       )
@@
     )
   )
+  (symbol (lib_id "Device:C_Polarized") (at 162.56 72.39 90) (unit 1)
+    (in_bom yes) (on_board yes) (dnp no) (fields_autoplaced)
+    (property "Reference" "C40" (at 161.671 64.77 90)
+      (effects (font (size 1.27 1.27)))
+    )
+    (property "Value" "10uC" (at 161.671 67.31 90)
+      (effects (font (size 1.27 1.27)))
+    )
+    (property "Footprint" "Capacitor_SMD:CP_Elec_6.3x5.4" (at 166.37 71.4248 0)
+      (effects (font (size 1.27 1.27)) hide)
+    )
+    (property "Datasheet" "https://datasheet.lcsc.com/lcsc/2304140030_Nichicon-UWX1H100MCL1GB_C134237.pdf" (at 162.56 72.39 0)
+      (effects (font (size 1.27 1.27)) hide)
+    )
+    (property "MPN" "UWX1H100MCL1GB" (at 162.56 72.39 0)
+      (effects (font (size 1.27 1.27)) hide)
+    )
+    (property "Status" "OK" (at 162.56 72.39 0)
+      (effects (font (size 1.27 1.27)) hide)
+    )
+    (pin "2")
+    (pin "1")
+    (instances
+      (project "SCART_switcher"
+        (path "/8cd08eb5-4755-4ef5-8eeb-77fd9974b180/6562ea38-5963-42b2-a0ef-a4a12a4c652f/9f74dfb2-70cd-470e-9dfb-02936b5bb451"
+          (reference "C40") (unit 1)
+        )
+      )
+    )
+  )
   (symbol (lib_id "power_custom:+4V5") (at 139.7 144.78 0) (mirror x) (unit 1)
     (in_bom yes) (on_board yes) (dnp no)
@@
         (path "/8cd08eb5-4755-4ef5-8eeb-77fd9974b180/6562ea38-5963-42b2-a0ef-a4a12a4c652f/9f74dfb2-70cd-470e-9dfb-02936b5bb451"
           (reference "#PWR0310") (unit 1)
+        )
+      )
+    )
+  )
+  (symbol (lib_id "Device:C_Polarized") (at 162.56 140.97 90) (unit 1)
+    (in_bom yes) (on_board yes) (dnp no) (fields_autoplaced)
+    (property "Reference" "C42" (at 161.671 133.35 90)
+      (effects (font (size 1.27 1.27)))
+    )
+    (property "Value" "10uC" (at 161.671 135.89 90)
+      (effects (font (size 1.27 1.27)))
+    )
+    (property "Footprint" "Capacitor_SMD:CP_Elec_6.3x5.4" (at 166.37 140.0048 0)
+      (effects (font (size 1.27 1.27)) hide)
+    )
+    (property "Datasheet" "https://datasheet.lcsc.com/lcsc/2304140030_Nichicon-UWX1H100MCL1GB_C134237.pdf" (at 162.56 140.97 0)
+      (effects (font (size 1.27 1.27)) hide)
+    )
+    (property "MPN" "UWX1H100MCL1GB" (at 162.56 140.97 0)
+      (effects (font (size 1.27 1.27)) hide)
+    )
+    (property "Status" "OK" (at 162.56 140.97 0)
+      (effects (font (size 1.27 1.27)) hide)
+    )
+    (pin "2")
+    (pin "1")
+    (instances
+      (project "SCART_switcher"
+        (path "/8cd08eb5-4755-4ef5-8eeb-77fd9974b180/6562ea38-5963-42b2-a0ef-a4a12a4c652f/9f74dfb2-70cd-470e-9dfb-02936b5bb451"
+          (reference "C42") (unit 1)
         )
       )
@@
     )
   )
-  (symbol (lib_id "Device:C") (at 162.56 140.97 90) (unit 1)
-    (in_bom yes) (on_board yes) (dnp no) (fields_autoplaced)
-    (property "Reference" "C42" (at 162.56 133.35 90)
-      (effects (font (size 1.27 1.27)))
-    )
-    (property "Value" "10uC" (at 162.56 135.89 90)
-      (effects (font (size 1.27 1.27)))
-    )
-    (property "Footprint" "" (at 166.37 140.0048 0)
-      (effects (font (size 1.27 1.27)) hide)
-    )
-    (property "Datasheet" "~" (at 162.56 140.97 0)
-      (effects (font (size 1.27 1.27)) hide)
-    )
-    (property "Status" "" (at 162.56 140.97 0)
-      (effects (font (size 1.27 1.27)) hide)
-    )
-    (pin "1")
-    (pin "2")
-    (instances
-      (project "SCART_switcher"
-        (path "/8cd08eb5-4755-4ef5-8eeb-77fd9974b180/6562ea38-5963-42b2-a0ef-a4a12a4c652f/9f74dfb2-70cd-470e-9dfb-02936b5bb451"
-          (reference "C42") (unit 1)
-        )
-      )
-    )
-  )
   (symbol (lib_id "power:GND") (at 44.45 176.53 0) (unit 1)
     (in_bom yes) (on_board yes) (dnp no) (fields_autoplaced)
@@
     )
   )
-  (symbol (lib_id "Device:C") (at 162.56 110.49 90) (unit 1)
-    (in_bom yes) (on_board yes) (dnp no) (fields_autoplaced)
-    (property "Reference" "C41" (at 162.56 102.87 90)
-      (effects (font (size 1.27 1.27)))
-    )
-    (property "Value" "10uC" (at 162.56 105.41 90)
-      (effects (font (size 1.27 1.27)))
-    )
-    (property "Footprint" "" (at 166.37 109.5248 0)
-      (effects (font (size 1.27 1.27)) hide)
-    )
-    (property "Datasheet" "~" (at 162.56 110.49 0)
-      (effects (font (size 1.27 1.27)) hide)
-    )
-    (property "Status" "" (at 162.56 110.49 0)
-      (effects (font (size 1.27 1.27)) hide)
-    )
-    (pin "1")
-    (pin "2")
-    (instances
-      (project "SCART_switcher"
-        (path "/8cd08eb5-4755-4ef5-8eeb-77fd9974b180/6562ea38-5963-42b2-a0ef-a4a12a4c652f/9f74dfb2-70cd-470e-9dfb-02936b5bb451"
-          (reference "C41") (unit 1)
-        )
-      )
-    )
-  )
   (symbol (lib_id "Device:R") (at 106.68 30.48 90) (unit 1)
     (in_bom yes) (on_board yes) (dnp no) (fields_autoplaced)
@@
         )
       )
+    )
+  )
+  (symbol (lib_id "Device:C_Polarized") (at 162.56 41.91 90) (unit 1)
+    (in_bom yes) (on_board yes) (dnp no) (fields_autoplaced)
+    (property "Reference" "C39" (at 161.671 34.29 90)
+      (effects (font (size 1.27 1.27)))
+    )
+    (property "Value" "10uC" (at 161.671 36.83 90)
+      (effects (font (size 1.27 1.27)))
+    )
+    (property "Footprint" "Capacitor_SMD:CP_Elec_6.3x5.4" (at 166.37 40.9448 0)
+      (effects (font (size 1.27 1.27)) hide)
+    )
+    (property "Datasheet" "https://datasheet.lcsc.com/lcsc/2304140030_Nichicon-UWX1H100MCL1GB_C134237.pdf" (at 162.56 41.91 0)
+      (effects (font (size 1.27 1.27)) hide)
+    )
+    (property "MPN" "UWX1H100MCL1GB" (at 162.56 41.91 0)
+      (effects (font (size 1.27 1.27)) hide)
+    )
+    (property "Status" "OK" (at 162.56 41.91 0)
+      (effects (font (size 1.27 1.27)) hide)
+    )
+    (pin "2")
+    (pin "1")
+    (instances
+      (project "SCART_switcher"
+        (path "/8cd08eb5-4755-4ef5-8eeb-77fd9974b180/6562ea38-5963-42b2-a0ef-a4a12a4c652f/9f74dfb2-70cd-470e-9dfb-02936b5bb451"
+          (reference "C39") (unit 1)
+        )
+      )

Commit message: Progressed ECAD.
Parts:
- added C34, C36, C38: 10uC, Capacitor_SMD:CP_Elec_6.3x5.4, symbol Device:C_Polarized
Connections:
- net +9V: now also C34.1, C36.1, C38.1
- net GND: now also C34.2, C36.2, C38.2
Other:
- moved on the sheet: C?, U?C

Commit message: Progressed ECAD.
Parts:
- gave numbers to parts that had none: 24
- renumbered C34 to C24, C36 to C26, C38 to C28, C39 to C29, C40 to C30, C41 to C31, C42 to C32

Commit message: Progressed ECAD
Parts:
- renumbered C23 to C29, C24 to C30, C25 to C31, C26 to C32, C27 to C33, C28 to C34, C29 to C35, C30 to C36, C31 to C37, C32 to C38, R66 to R74, R67 to R75, R68 to R76, R69 to R77, R70 to R78, R71 to R79, R72 to R80, R73 to R81, R74 to R82, R75 to R83, R76 to R84, R77 to R85, R78 to R86, R79 to R87, R80 to R88, R81 to R89, R82 to R90, R83 to R91, U15 to U21, U16 to U22, U17 to U23
