File: ECAD/SCART_switcher/priority_level_start.kicad_sch (KiCad schematic)
At the start: 7 parts

Commit message: progressed ecad
Parts:
- C?: MPN (none) -> CL21B104KBCNNNC
Changed lines of the file:
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@@
       (effects (font (size 1.27 1.27)) hide)
     )
-    (property "Datasheet" "~" (at 184.15 87.63 0)
+    (property "Datasheet" "https://datasheet.lcsc.com/lcsc/1810191215_Samsung-Electro-Mechanics-CL21B104KBCNNNC_C1711.pdf" (at 184.15 87.63 0)
       (effects (font (size 1.27 1.27)) hide)
     )
@@
       (effects (font (size 1.27 1.27)) hide)
     )
+    (property "MPN" "CL21B104KBCNNNC" (at 184.15 87.63 0)
+      (effects (font (size 1.27 1.27)) hide)
+    )

Commit message: progressed ecad
Parts:
- removed C?: 2n2C, symbol Device:C
- removed D?: BAS316, symbol Device:D
- removed R?: 2k2R, Resistor_SMD:R_0805_2012Metric_Pad1.20x1.40mm_HandSolder, symbol Device:R
- removed R?: 10kR, Resistor_SMD:R_0805_2012Metric_Pad1.20x1.40mm_HandSolder, symbol Device:R
- removed U?: 74AHC1G14, Package_TO_SOT_SMD:SOT-23-5, symbol 74xGxx:74AHC1G14
Other:
- note removed: "Dead time delay to allow for break before make input video selection."
- note removed: "tbd: add delay to the enable case such that "break before make" type of behaviour is built."
