File: ECAD/SCART_switcher/priority_level_start.kicad_sch (KiCad schematic)
At the start: 2 parts

Commit message: Progressed ECAD. Error fixing and cleanup.
Parts:
- added NT?: NetTie_2, symbol Device:NetTie_2
Connections:
- net IN_ACTIVE: now also NT?.1
- new net IN_ENABLE: NT?.2
Changed lines of the file:
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@@
+    (stroke (width 0) (type default))
+  )
+  (wire (pts (xy 130.81 73.66) (xy 147.32 73.66))
     (stroke (width 0) (type default))
   )
@@
     (stroke (width 0) (type default))
   )
-  (wire (pts (xy 114.3 73.66) (xy 147.32 73.66))
+  (wire (pts (xy 114.3 73.66) (xy 125.73 73.66))
     (stroke (width 0) (type default))
   )
@@
         )
         (path "/8cd08eb5-4755-4ef5-8eeb-77fd9974b180/767093fd-244d-47aa-bb03-1a1276be8d22/f3189d6a-8c8d-437b-9f5d-14c8f4314717"
-          (reference "C33") (unit 1)
+          (reference "C34") (unit 1)
         )
       )
@@
         (path "/8cd08eb5-4755-4ef5-8eeb-77fd9974b180/767093fd-244d-47aa-bb03-1a1276be8d22/f3189d6a-8c8d-437b-9f5d-14c8f4314717"
           (reference "#PWR0280") (unit 1)
+        )
+      )
+    )
+  )
+  (symbol (lib_id "Device:NetTie_2") (at 128.27 73.66 0) (unit 1)
+    (in_bom no) (on_board yes) (dnp no) (fields_autoplaced)
+    (property "Reference" "NT?" (at 128.27 68.58 0)
+      (effects (font (size 1.27 1.27)))
+    )
+    (property "Value" "NetTie_2" (at 128.27 71.12 0)
+      (effects (font (size 1.27 1.27)))
+    )
+    (property "Footprint" "" (at 128.27 73.66 0)
+      (effects (font (size 1.27 1.27)) hide)
+    )
+    (property "Datasheet" "~" (at 128.27 73.66 0)
+      (effects (font (size 1.27 1.27)) hide)
+    )
+    (pin "2")
+    (pin "1")
+    (instances
+      (project "SCART_switcher"
+        (path "/8cd08eb5-4755-4ef5-8eeb-77fd9974b180/6e53f4c9-ed59-4c5d-ac8d-a66f0d353ca7"
+          (reference "NT?") (unit 1)
+        )
+        (path "/8cd08eb5-4755-4ef5-8eeb-77fd9974b180/8ea6db35-25d0-43bc-9de5-3ca23502dcdc"
+          (reference "NT?") (unit 1)
+        )
+        (path "/8cd08eb5-4755-4ef5-8eeb-77fd9974b180/272a4677-3ef2-418e-abc5-b29f59e726f9"
+          (reference "NT?") (unit 1)
+        )
+        (path "/8cd08eb5-4755-4ef5-8eeb-77fd9974b180/56b7edd2-65bf-4844-b6bd-3868b6562f83"
+          (reference "NT?") (unit 1)
+        )
+        (path "/8cd08eb5-4755-4ef5-8eeb-77fd9974b180/a066fdde-5f40-4269-95c1-258d611fd7cb"
+          (reference "NT?") (unit 1)
+        )
+        (path "/8cd08eb5-4755-4ef5-8eeb-77fd9974b180/ec158eb5-f3e0-409c-b64c-a90e3358941f"
+          (reference "NT?") (unit 1)
+        )
+        (path "/8cd08eb5-4755-4ef5-8eeb-77fd9974b180/6c53b757-b2e6-4d60-b760-4a4a0f832c07"
+          (reference "NT?") (unit 1)
+        )
+        (path "/8cd08eb5-4755-4ef5-8eeb-77fd9974b180/0223a704-ac47-44ed-9ba1-f418acceedb3"
+          (reference "NT?") (unit 1)
+        )
+        (path "/8cd08eb5-4755-4ef5-8eeb-77fd9974b180/2ffa7ecd-d29d-4261-a577-43650ca26099"
+          (reference "NT?") (unit 1)
+        )
+        (path "/8cd08eb5-4755-4ef5-8eeb-77fd9974b180/f71a1287-269d-4354-9179-cb80a7e1dbca"
+          (reference "NT?") (unit 1)
+        )
+        (path "/8cd08eb5-4755-4ef5-8eeb-77fd9974b180/767093fd-244d-47aa-bb03-1a1276be8d22/f3189d6a-8c8d-437b-9f5d-14c8f4314717"
+          (reference "NT1") (unit 1)
         )
       )
@@
         )
         (path "/8cd08eb5-4755-4ef5-8eeb-77fd9974b180/767093fd-244d-47aa-bb03-1a1276be8d22/f3189d6a-8c8d-437b-9f5d-14c8f4314717"
-          (reference "U40") (unit 1)
-        )
-      )
+          (reference "U39") (unit 1)
+        )
+      )

Commit message: Progressed ECAD.
Parts:
- U?: MFN 74AHC1G04W5-7 -> (none); MPN (none) -> 74AHC1G04W5-7
Changed lines of the file:
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@@
-      (effects (font (size 1.27 1.27)) hide)
-    )
-    (property "MFN" "" (at 184.15 87.63 0)
       (effects (font (size 1.27 1.27)) hide)
     )
@@
       (effects (font (size 1.27 1.27)) hide)
     )
-    (property "MFN" "74AHC1G04W5-7" (at 130.81 91.44 0)
-      (effects (font (size 1.27 1.27)) hide)
-    )
+    (property "MPN" "74AHC1G04W5-7" (at 130.81 91.44 0)
+      (effects (font (size 1.27 1.27)) hide)
+    )
