File: ECAD/SCART_switcher/priority_level_start.kicad_sch (KiCad schematic)
At the start: 3 parts

Commit message: Progressed ECAD.
Parts:
- C?: footprint Capacitor_SMD:C_0805_2012Metric_Pad1.18x1.45mm_HandSolder -> Capacitor_SMD:C_0805_2012Metric
Changed lines of the file:
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@@
       (effects (font (size 1.27 1.27)) (justify left))
     )
-    (property "Footprint" "Capacitor_SMD:C_0805_2012Metric_Pad1.18x1.45mm_HandSolder" (at 185.1152 91.44 0)
+    (property "Footprint" "Capacitor_SMD:C_0805_2012Metric" (at 185.1152 91.44 0)
       (effects (font (size 1.27 1.27)) hide)
     )

Commit message: Progressed ECAD.
Parts:
- NT?: MPN (none) -> N/A; Status (none) -> OK
Changed lines of the file:
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@@
+      (effects (font (size 1.27 1.27)) hide)
+    )
+    (property "Status" "" (at 184.15 87.63 0)
       (effects (font (size 1.27 1.27)) hide)
     )
@@
       (effects (font (size 1.27 1.27)) hide)
     )
+    (property "Status" "OK" (at 128.27 73.66 0)
+      (effects (font (size 1.27 1.27)) hide)
+    )
+    (property "MPN" "N/A" (at 128.27 73.66 0)
+      (effects (font (size 1.27 1.27)) hide)
+    )
     (pin "2")
     (pin "1")
@@
       (effects (font (size 1.27 1.27)) hide)
     )
+    (property "Status" "" (at 130.81 91.44 0)
+      (effects (font (size 1.27 1.27)) hide)
+    )

Commit message: Progressed ECAD.
Parts:
- U?: MPN 74AHC1G04W5-7 -> SN74AHC1G04DBVR
Changed lines of the file:
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@@
       (effects (font (size 1.27 1.27)) hide)
     )
-    (property "Datasheet" "https://datasheet.lcsc.com/lcsc/1912111437_Diodes-Incorporated-74AHC1G04W5-7_C460486.pdf" (at 130.81 91.44 0)
+    (property "Datasheet" "https://datasheet.lcsc.com/lcsc/2001061132_Texas-Instruments-SN74AHC1G04DBVR_C7465.pdf" (at 130.81 91.44 0)
       (effects (font (size 1.27 1.27)) hide)
     )
-    (property "MPN" "74AHC1G04W5-7" (at 130.81 91.44 0)
+    (property "MPN" "SN74AHC1G04DBVR" (at 130.81 91.44 0)
       (effects (font (size 1.27 1.27)) hide)
     )

Commit message: Progressed ECAD.
Parts:
- U?: value 74AHC1G04 -> 74LVC1G04; footprint Package_TO_SOT_SMD:SOT-23-5 -> Package_TO_SOT_SMD:SOT-353_SC-70-5; MPN SN74AHC1G04DBVR -> SN74LVC1G04DCKR; Status (none) -> OK
Changed lines of the file:
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@@
       (effects (font (size 1.27 1.27)))
     )
-    (property "Value" "74AHC1G04" (at 135.89 86.36 0)
+    (property "Value" "74LVC1G04" (at 135.89 86.36 0)
       (effects (font (size 1.27 1.27)))
     )
-    (property "Footprint" "Package_TO_SOT_SMD:SOT-23-5" (at 130.81 91.44 0)
+    (property "Footprint" "Package_TO_SOT_SMD:SOT-353_SC-70-5" (at 130.81 91.44 0)
       (effects (font (size 1.27 1.27)) hide)
     )
-    (property "Datasheet" "https://datasheet.lcsc.com/lcsc/2001061132_Texas-Instruments-SN74AHC1G04DBVR_C7465.pdf" (at 130.81 91.44 0)
+    (property "Datasheet" "https://datasheet.lcsc.com/lcsc/1811021113_Texas-Instruments-SN74LVC1G04DCKR_C8207.pdf" (at 130.81 91.44 0)
       (effects (font (size 1.27 1.27)) hide)
     )
-    (property "MPN" "SN74AHC1G04DBVR" (at 130.81 91.44 0)
+    (property "MPN" "SN74LVC1G04DCKR" (at 130.81 91.44 0)
       (effects (font (size 1.27 1.27)) hide)
     )
-    (property "Status" "" (at 130.81 91.44 0)
+    (property "Status" "OK" (at 130.81 91.44 0)
       (effects (font (size 1.27 1.27)) hide)
     )

Commit message: Progressed ECAD.
Parts:
- removed NT?: NetTie_2, symbol Device:NetTie_2
Changed lines of the file:
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@@
     (stroke (width 0) (type default))
   )
-  (wire (pts (xy 130.81 73.66) (xy 147.32 73.66))
+  (wire (pts (xy 114.3 73.66) (xy 147.32 73.66))
     (stroke (width 0) (type default))
   )
   (wire (pts (xy 109.22 73.66) (xy 114.3 73.66))
-    (stroke (width 0) (type default))
-  )
-  (wire (pts (xy 114.3 73.66) (xy 125.73 73.66))
     (stroke (width 0) (type default))
   )
@@
         )
         (path "/8cd08eb5-4755-4ef5-8eeb-77fd9974b180/767093fd-244d-47aa-bb03-1a1276be8d22/f3189d6a-8c8d-437b-9f5d-14c8f4314717"
-          (reference "#PWR0278") (unit 1)
+          (reference "#PWR0275") (unit 1)
         )
       )
@@
         )
         (path "/8cd08eb5-4755-4ef5-8eeb-77fd9974b180/767093fd-244d-47aa-bb03-1a1276be8d22/f3189d6a-8c8d-437b-9f5d-14c8f4314717"
-          (reference "C34") (unit 1)
+          (reference "C31") (unit 1)
         )
       )
@@
         )
         (path "/8cd08eb5-4755-4ef5-8eeb-77fd9974b180/767093fd-244d-47aa-bb03-1a1276be8d22/f3189d6a-8c8d-437b-9f5d-14c8f4314717"
-          (reference "#PWR0280") (unit 1)
-        )
-      )
-    )
-  )
-  (symbol (lib_id "Device:NetTie_2") (at 128.27 73.66 0) (unit 1)
-    (in_bom no) (on_board yes) (dnp no) (fields_autoplaced)
-    (property "Reference" "NT?" (at 128.27 68.58 0)
-      (effects (font (size 1.27 1.27)))
-    )
-    (property "Value" "NetTie_2" (at 128.27 71.12 0)
-      (effects (font (size 1.27 1.27)))
-    )
-    (property "Footprint" "" (at 128.27 73.66 0)
-      (effects (font (size 1.27 1.27)) hide)
-    )
-    (property "Datasheet" "~" (at 128.27 73.66 0)
-      (effects (font (size 1.27 1.27)) hide)
-    )
-    (property "Status" "OK" (at 128.27 73.66 0)
-      (effects (font (size 1.27 1.27)) hide)
-    )
-    (property "MPN" "N/A" (at 128.27 73.66 0)
-      (effects (font (size 1.27 1.27)) hide)
-    )
-    (pin "2")
-    (pin "1")
-    (instances
-      (project "SCART_switcher"
-        (path "/8cd08eb5-4755-4ef5-8eeb-77fd9974b180/6e53f4c9-ed59-4c5d-ac8d-a66f0d353ca7"
-          (reference "NT?") (unit 1)
-        )
-        (path "/8cd08eb5-4755-4ef5-8eeb-77fd9974b180/8ea6db35-25d0-43bc-9de5-3ca23502dcdc"
-          (reference "NT?") (unit 1)
-        )
-        (path "/8cd08eb5-4755-4ef5-8eeb-77fd9974b180/272a4677-3ef2-418e-abc5-b29f59e726f9"
-          (reference "NT?") (unit 1)
-        )
-        (path "/8cd08eb5-4755-4ef5-8eeb-77fd9974b180/56b7edd2-65bf-4844-b6bd-3868b6562f83"
-          (reference "NT?") (unit 1)
-        )
-        (path "/8cd08eb5-4755-4ef5-8eeb-77fd9974b180/a066fdde-5f40-4269-95c1-258d611fd7cb"
-          (reference "NT?") (unit 1)
-        )
-        (path "/8cd08eb5-4755-4ef5-8eeb-77fd9974b180/ec158eb5-f3e0-409c-b64c-a90e3358941f"
-          (reference "NT?") (unit 1)
-        )
-        (path "/8cd08eb5-4755-4ef5-8eeb-77fd9974b180/6c53b757-b2e6-4d60-b760-4a4a0f832c07"
-          (reference "NT?") (unit 1)
-        )
-        (path "/8cd08eb5-4755-4ef5-8eeb-77fd9974b180/0223a704-ac47-44ed-9ba1-f418acceedb3"
-          (reference "NT?") (unit 1)
-        )
-        (path "/8cd08eb5-4755-4ef5-8eeb-77fd9974b180/2ffa7ecd-d29d-4261-a577-43650ca26099"
-          (reference "NT?") (unit 1)
-        )
-        (path "/8cd08eb5-4755-4ef5-8eeb-77fd9974b180/f71a1287-269d-4354-9179-cb80a7e1dbca"
-          (reference "NT?") (unit 1)
-        )
-        (path "/8cd08eb5-4755-4ef5-8eeb-77fd9974b180/767093fd-244d-47aa-bb03-1a1276be8d22/f3189d6a-8c8d-437b-9f5d-14c8f4314717"
-          (reference "NT1") (unit 1)
+          (reference "#PWR0277") (unit 1)
         )
       )
@@
         )
         (path "/8cd08eb5-4755-4ef5-8eeb-77fd9974b180/767093fd-244d-47aa-bb03-1a1276be8d22/f3189d6a-8c8d-437b-9f5d-14c8f4314717"
-          (reference "#PWR0279") (unit 1)
+          (reference "#PWR0276") (unit 1)
         )
       )
@@
         )
         (path "/8cd08eb5-4755-4ef5-8eeb-77fd9974b180/767093fd-244d-47aa-bb03-1a1276be8d22/f3189d6a-8c8d-437b-9f5d-14c8f4314717"
-          (reference "#PWR0281") (unit 1)
-        )
-      )
+          (reference "#PWR0278") (unit 1)
+        )
+      )

Commit message: Progressed ECAD.
Parts:
- gave numbers to parts that had none: 2
