File: ECAD/SCART_switcher/SCART_output.kicad_sch (KiCad schematic)
At the start: 10 parts, among them J2 RCA Left, J3 RCA Right, Q3 BC847

Commit message: Progressed ECAD.
Parts:
- Q3: MFN BC847B,215 -> (none); MPN (none) -> BC847B,215
- R7, R?: MPN (none) -> RC0805FR-0710KL
Changed lines of the file:
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@@
       (effects (font (size 1.27 1.27)) hide)
     )
-    (property "Datasheet" "~" (at 105.41 77.47 0)
+    (property "Datasheet" "https://datasheet.lcsc.com/lcsc/1810201611_YAGEO-RC0805FR-0710KL_C84376.pdf" (at 105.41 77.47 0)
+      (effects (font (size 1.27 1.27)) hide)
+    )
+    (property "MPN" "RC0805FR-0710KL" (at 105.41 77.47 0)
       (effects (font (size 1.27 1.27)) hide)
     )
@@
     )
     (property "Datasheet" " ~" (at 220.98 123.19 0)
-      (effects (font (size 1.27 1.27)) hide)
-    )
-    (property "MFN" "" (at 220.98 124.46 0)
       (effects (font (size 1.27 1.27)) hide)
     )
@@
       (effects (font (size 1.27 1.27)) hide)
     )
-    (property "Datasheet" "~" (at 81.28 64.77 0)
-      (effects (font (size 1.27 1.27)) hide)
-    )
-    (property "MFN" "" (at 81.28 64.77 0)
+    (property "Datasheet" "https://datasheet.lcsc.com/lcsc/1810201611_YAGEO-RC0805FR-0710KL_C84376.pdf" (at 81.28 64.77 0)
+      (effects (font (size 1.27 1.27)) hide)
+    )
+    (property "MPN" "RC0805FR-0710KL" (at 81.28 64.77 0)
       (effects (font (size 1.27 1.27)) hide)
     )
@@
       (effects (font (size 1.27 1.27)) (justify left) hide)
     )
-    (property "MFN" "BC847B,215" (at 78.74 73.66 0)
-      (effects (font (size 1.27 1.27)) hide)
-    )
+    (property "MPN" "BC847B,215" (at 78.74 73.66 0)
+      (effects (font (size 1.27 1.27)) hide)
+    )

Commit message: Progressed ECAD.
Other:
- added sheet Silent output (dummy_input.kicad_sch)
- moved on the sheet: J2, J3, Q3, Q?, R10, R7, R?

Commit message: Progressed ECAD.
Parts:
- R10, R7, R? (x3): footprint Resistor_SMD:R_0805_2012Metric_Pad1.20x1.40mm_HandSolder -> Resistor_SMD:R_0805_2012Metric

Commit message: Progressed ECAD.
Parts:
- J2, J3, J?: MPN (none) -> N/A; Status (none) -> OK
- Q3: MPN BC847B,215 -> BC847C,215; Status (none) -> OK
- Q?: MPN (none) -> BC857C,215; Status (none) -> OK
Changed lines of the file:
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@@
+      (effects (font (size 1.27 1.27)) hide)
+    )
+    (property "Status" "OK" (at 220.98 54.61 0)
+      (effects (font (size 1.27 1.27)) hide)
+    )
+    (property "MPN" "N/A" (at 220.98 54.61 0)
       (effects (font (size 1.27 1.27)) hide)
     )
@@
       (effects (font (size 1.27 1.27)) hide)
     )
+    (property "Status" "" (at 95.25 146.05 0)
+      (effects (font (size 1.27 1.27)) hide)
+    )
     (pin "1")
     (pin "2")
@@
     )
     (property "Datasheet" "~" (at 71.12 151.13 0)
+      (effects (font (size 1.27 1.27)) hide)
+    )
+    (property "Status" "" (at 71.12 151.13 0)
       (effects (font (size 1.27 1.27)) hide)
     )
@@
       (effects (font (size 1.27 1.27)) hide)
     )
+    (property "Status" "" (at 106.68 154.94 0)
+      (effects (font (size 1.27 1.27)) hide)
+    )
     (pin "1")
     (pin "2")
@@
     )
     (property "Datasheet" " ~" (at 220.98 123.19 0)
+      (effects (font (size 1.27 1.27)) hide)
+    )
+    (property "Status" "OK" (at 220.98 124.46 0)
+      (effects (font (size 1.27 1.27)) hide)
+    )
+    (property "MPN" "N/A" (at 220.98 124.46 0)
       (effects (font (size 1.27 1.27)) hide)
     )
@@
       (effects (font (size 1.27 1.27)) hide)
     )
+    (property "Status" "OK" (at 220.98 36.83 0)
+      (effects (font (size 1.27 1.27)) hide)
+    )
+    (property "MPN" "N/A" (at 220.98 36.83 0)
+      (effects (font (size 1.27 1.27)) hide)
+    )
     (pin "1")
     (pin "2")
@@
     )
     (property "MPN" "RC0805FR-0710KL" (at 82.55 142.24 0)
+      (effects (font (size 1.27 1.27)) hide)
+    )
+    (property "Status" "" (at 82.55 142.24 0)
       (effects (font (size 1.27 1.27)) hide)
     )
@@
       (effects (font (size 1.27 1.27) italic) (justify left) hide)
     )
-    (property "Datasheet" "https://www.onsemi.com/pub/Collateral/BC860-D.pdf" (at 104.14 146.05 0)
+    (property "Datasheet" "https://datasheet.lcsc.com/lcsc/2304140030_Nexperia-BC857C-215_C8666.pdf" (at 104.14 146.05 0)
       (effects (font (size 1.27 1.27)) (justify left) hide)
+    )
+    (property "Status" "OK" (at 104.14 146.05 0)
+      (effects (font (size 1.27 1.27)) hide)
+    )
+    (property "MPN" "BC857C,215" (at 104.14 146.05 0)
+      (effects (font (size 1.27 1.27)) hide)
     )
     (pin "1")
@@
       (effects (font (size 1.27 1.27)) hide)
     )
+    (property "Status" "" (at 120.65 151.13 0)
+      (effects (font (size 1.27 1.27)) hide)
+    )
     (pin "1")
     (pin "2")
@@
       (effects (font (size 1.27 1.27) italic) (justify left) hide)
     )
-    (property "Datasheet" "https://datasheet.lcsc.com/lcsc/2304140030_Nexperia-BC847B-215_C57668.pdf" (at 80.01 151.13 0)
+    (property "Datasheet" "https://datasheet.lcsc.com/lcsc/1811141238_Nexperia-BC847C-215_C8664.pdf" (at 80.01 151.13 0)
       (effects (font (size 1.27 1.27)) (justify left) hide)
     )
-    (property "MPN" "BC847B,215" (at 80.01 151.13 0)
-      (effects (font (size 1.27 1.27)) hide)
-    )
+    (property "MPN" "BC847C,215" (at 80.01 151.13 0)
+      (effects (font (size 1.27 1.27)) hide)
+    )
+    (property "Status" "OK" (at 80.01 151.13 0)
+      (effects (font (size 1.27 1.27)) hide)
+    )

Commit message: Progressed ECAD.
Parts:
- gave numbers to parts that had none: 5
Other:
- note added: "check polarity add not !!!!!!!!!!!!!!!!"

Commit message: Progressed ECAD.
Parts:
- removed Q4: BC857, Package_TO_SOT_SMD:SOT-23, symbol Transistor_BJT:BC857
- removed R8: 47kR, Resistor_SMD:R_0805_2012Metric, symbol Device:R
- removed R9: 10kR, Resistor_SMD:R_0805_2012Metric, symbol Device:R
Connections:
- net at Q3.3 (C), R7.2: now also R10.1
- net OUT_ACTIVE renamed ~{OUT_ACTIVE}
Other:
- note removed: "check polarity add not !!!!!!!!!!!!!!!!"
- moved on the sheet: R10
Changed lines of the file:
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@@
   (junction (at 77.47 27.94) (diameter 0) (color 0 0 0 0)
-  )
-  (junction (at 106.68 151.13) (diameter 0) (color 0 0 0 0)
   )
   (no_connect (at 205.74 149.86))
@@
     (stroke (width 0) (type default))
   )
-  (wire (pts (xy 124.46 151.13) (xy 134.62 151.13))
+  (wire (pts (xy 100.33 146.05) (xy 110.49 146.05))
     (stroke (width 0) (type default))
   )
@@
     (stroke (width 0) (type default))
   )
-  (wire (pts (xy 82.55 146.05) (xy 91.44 146.05))
+  (wire (pts (xy 82.55 146.05) (xy 92.71 146.05))
     (stroke (width 0) (type default))
   )
@@
   )
   (wire (pts (xy 80.01 68.58) (xy 80.01 30.48))
-    (stroke (width 0) (type default))
-  )
-  (wire (pts (xy 106.68 151.13) (xy 116.84 151.13))
     (stroke (width 0) (type default))
   )
@@
     (effects (font (size 1.27 1.27)) (justify left bottom))
   )
-  (text "(*1)" (at 127 153.67 0)
+  (text "(*1)" (at 102.87 148.59 0)
     (effects (font (size 1.27 1.27)) (justify left bottom))
   )
@@
     (effects (font (size 1.27 1.27)) (justify left bottom))
   )
-  (text "check polarity\nadd not !!!!!!!!!!!!!!!!" (at 38.1 153.67 0)
-    (effects (font (size 1.27 1.27)) (justify left bottom))
-  )
   (label "RED" (at 194.31 114.3 0) (fields_autoplaced)
     (effects (font (size 1.27 1.27)) (justify left bottom))
@@
     (effects (font (size 1.27 1.27)) (justify right bottom))
   )
-  (label "FUNCTION" (at 134.62 151.13 180) (fields_autoplaced)
+  (label "FUNCTION" (at 110.49 146.05 180) (fields_autoplaced)
     (effects (font (size 1.27 1.27)) (justify right bottom))
   )
@@
     (effects (font (size 1.27 1.27)) (justify right))
   )
-  (hierarchical_label "OUT_ACTIVE" (shape input) (at 67.31 151.13 180) (fields_autoplaced)
+  (hierarchical_label "~{OUT_ACTIVE}" (shape input) (at 67.31 151.13 180) (fields_autoplaced)
     (effects (font (size 1.27 1.27)) (justify right))
   )
@@
     (effects (font (size 1.27 1.27)) (justify right))
   )
-  (hierarchical_label "OUT_ACTIVE" (shape input) (at 41.91 86.36 180) (fields_autoplaced)
+  (hierarchical_label "~{OUT_ACTIVE}" (shape input) (at 41.91 86.36 180) (fields_autoplaced)
     (effects (font (size 1.27 1.27)) (justify right))
   )
@@
     )
   )
-  (symbol (lib_id "Device:R") (at 95.25 146.05 90) (unit 1)
-    (in_bom yes) (on_board yes) (dnp no) (fields_autoplaced)
-    (property "Reference" "R8" (at 95.25 139.7 90)
-      (effects (font (size 1.27 1.27)))
-    )
-    (property "Value" "47kR" (at 95.25 142.24 90)
-      (effects (font (size 1.27 1.27)))
-    )
-    (property "Footprint" "Resistor_SMD:R_0805_2012Metric" (at 95.25 147.828 90)
-      (effects (font (size 1.27 1.27)) hide)
-    )
-    (property "Datasheet" "~" (at 95.25 146.05 0)
-      (effects (font (size 1.27 1.27)) hide)
-    )
-    (property "Status" "" (at 95.25 146.05 0)
+  (symbol (lib_id "Device:R") (at 71.12 151.13 90) (unit 1)
+    (in_bom yes) (on_board yes) (dnp no) (fields_autoplaced)
+    (property "Reference" "R6" (at 71.12 144.78 90)
+      (effects (font (size 1.27 1.27)))
+    )
+    (property "Value" "47kR" (at 71.12 147.32 90)
+      (effects (font (size 1.27 1.27)))
+    )
+    (property "Footprint" "Resistor_SMD:R_0805_2012Metric" (at 71.12 152.908 90)
+      (effects (font (size 1.27 1.27)) hide)
+    )
+    (property "Datasheet" "~" (at 71.12 151.13 0)
+      (effects (font (size 1.27 1.27)) hide)
+    )
+    (property "Status" "" (at 71.12 151.13 0)
       (effects (font (size 1.27 1.27)) hide)
     )
@@
       (project "SCART_switcher"
         (path "/8cd08eb5-4755-4ef5-8eeb-77fd9974b180/6562ea38-5963-42b2-a0ef-a4a12a4c652f"
-          (reference "R8") (unit 1)
-        )
-      )
-    )
-  )
-  (symbol (lib_id "Device:R") (at 71.12 151.13 90) (unit 1)
-    (in_bom yes) (on_board yes) (dnp no) (fields_autoplaced)
-    (property "Reference" "R6" (at 71.12 144.78 90)
-      (effects (font (size 1.27 1.27)))
-    )
-    (property "Value" "47kR" (at 71.12 147.32 90)
-      (effects (font (size 1.27 1.27)))
-    )
-    (property "Footprint" "Resistor_SMD:R_0805_2012Metric" (at 71.12 152.908 90)
-      (effects (font (size 1.27 1.27)) hide)
-    )
-    (property "Datasheet" "~" (at 71.12 151.13 0)
-      (effects (font (size 1.27 1.27)) hide)
-    )
-    (property "Status" "" (at 71.12 151.13 0)
-      (effects (font (size 1.27 1.27)) hide)
-    )
-    (pin "1")
-    (pin "2")
-    (instances
-      (project "SCART_switcher"
-        (path "/8cd08eb5-4755-4ef5-8eeb-77fd9974b180/6562ea38-5963-42b2-a0ef-a4a12a4c652f"
           (reference "R6") (unit 1)
-        )
-      )
-    )
-  )
-  (symbol (lib_id "Device:R") (at 106.68 154.94 0) (unit 1)
-    (in_bom yes) (on_board yes) (dnp no) (fields_autoplaced)
-    (property "Reference" "R9" (at 109.22 153.67 0)
-      (effects (font (size 1.27 1.27)) (justify left))
-    )
-    (property "Value" "10kR" (at 109.22 156.21 0)
-      (effects (font (size 1.27 1.27)) (justify left))
-    )
-    (property "Footprint" "Resistor_SMD:R_0805_2012Metric" (at 104.902 154.94 90)
-      (effects (font (size 1.27 1.27)) hide)
-    )
-    (property "Datasheet" "https://datasheet.lcsc.com/lcsc/1810201611_YAGEO-RC0805FR-0710KL_C84376.pdf" (at 106.68 154.94 0)
-      (effects (font (size 1.27 1.27)) hide)
-    )
-    (property "MPN" "RC0805FR-0710KL" (at 106.68 154.94 0)
-      (effects (font (size 1.27 1.27)) hide)
-    )
-    (property "Status" "" (at 106.68 154.94 0)
-      (effects (font (size 1.27 1.27)) hide)
-    )
-    (pin "1")
-    (pin "2")
-    (instances
-      (project "SCART_switcher"
-        (path "/8cd08eb5-4755-4ef5-8eeb-77fd9974b180/6562ea38-5963-42b2-a0ef-a4a12a4c652f"
-          (reference "R9") (unit 1)
         )
       )
@@
     )
   )
-  (symbol (lib_id "power:+12V") (at 106.68 140.97 0) (unit 1)
-    (in_bom yes) (on_board yes) (dnp no) (fields_autoplaced)
-    (property "Reference" "#PWR020" (at 106.68 144.78 0)
-      (effects (font (size 1.27 1.27)) hide)
-    )
-    (property "Value" "+12V" (at 106.68 136.144 0)
-      (effects (font (size 1.27 1.27)))
-    )
-    (property "Footprint" "" (at 106.68 140.97 0)
-      (effects (font (size 1.27 1.27)) hide)
-    )
-    (property "Datasheet" "" (at 106.68 140.97 0)
-      (effects (font (size 1.27 1.27)) hide)
-    )
-    (pin "1")
-    (instances
-      (project "SCART_switcher"
-        (path "/8cd08eb5-4755-4ef5-8eeb-77fd9974b180/6562ea38-5963-42b2-a0ef-a4a12a4c652f"
-          (reference "#PWR020") (unit 1)
-        )
-      )
-    )
-  )
   (symbol (lib_id "power:GND") (at 205.74 99.06 270) (unit 1)
     (in_bom yes) (on_board yes) (dnp no) (fields_autoplaced)
@@
     )
   )
-  (symbol (lib_id "Transistor_BJT:BC857") (at 104.14 146.05 0) (mirror x) (unit 1)
-    (in_bom yes) (on_board yes) (dnp no)
-    (property "Reference" "Q4" (at 109.22 147.32 0)
-      (effects (font (size 1.27 1.27)) (justify left))
-    )
-    (property "Value" "BC857" (at 109.22 144.78 0)
-      (effects (font (size 1.27 1.27)) (justify left))
-    )
-    (property "Footprint" "Package_TO_SOT_SMD:SOT-23" (at 109.22 144.145 0)
-      (effects (font (size 1.27 1.27) italic) (justify left) hide)
-    )
-    (property "Datasheet" "https://datasheet.lcsc.com/lcsc/2304140030_Nexperia-BC857C-215_C8666.pdf" (at 104.14 146.05 0)
-      (effects (font (size 1.27 1.27)) (justify left) hide)
-    )
-    (property "Status" "OK" (at 104.14 146.05 0)
-      (effects (font (size 1.27 1.27)) hide)
-    )
-    (property "MPN" "BC857C,215" (at 104.14 146.05 0)
-      (effects (font (size 1.27 1.27)) hide)
-    )
-    (pin "1")
-    (pin "2")
-    (pin "3")
-    (instances
-      (project "SCART_switcher"
-        (path "/8cd08eb5-4755-4ef5-8eeb-77fd9974b180/6562ea38-5963-42b2-a0ef-a4a12a4c652f"
-          (reference "Q4") (unit 1)
-        )
-      )
-    )
-  )
   (symbol (lib_id "power:GND") (at 236.22 116.84 90) (unit 1)
     (in_bom yes) (on_board yes) (dnp no) (fields_autoplaced)
@@
     )
   )
-  (symbol (lib_id "power:GND") (at 106.68 158.75 0) (unit 1)
-    (in_bom yes) (on_board yes) (dnp no) (fields_autoplaced)
-    (property "Reference" "#PWR021" (at 106.68 165.1 0)
-      (effects (font (size 1.27 1.27)) hide)
-    )
-    (property "Value" "GND" (at 106.68 163.83 0)
-      (effects (font (size 1.27 1.27)))
-    )
-    (property "Footprint" "" (at 106.68 158.75 0)
-      (effects (font (size 1.27 1.27)) hide)
-    )
-    (property "Datasheet" "" (at 106.68 158.75 0)
-      (effects (font (size 1.27 1.27)) hide)
-    )
-    (pin "1")
-    (instances
-      (project "SCART_switcher"
-        (path "/8cd08eb5-4755-4ef5-8eeb-77fd9974b180/6562ea38-5963-42b2-a0ef-a4a12a4c652f"
-          (reference "#PWR021") (unit 1)
-        )
-      )
-    )
-  )
-  (symbol (lib_id "Device:R") (at 120.65 151.13 90) (unit 1)
-    (in_bom yes) (on_board yes) (dnp no) (fields_autoplaced)
-    (property "Reference" "R10" (at 120.65 144.78 90)
-      (effects (font (size 1.27 1.27)))
-    )
-    (property "Value" "100R" (at 120.65 147.32 90)
-      (effects (font (size 1.27 1.27)))
-    )
-    (property "Footprint" "Resistor_SMD:R_0805_2012Metric" (at 120.65 152.908 90)
-      (effects (font (size 1.27 1.27)) hide)
-    )
-    (property "Datasheet" "~" (at 120.65 151.13 0)
-      (effects (font (size 1.27 1.27)) hide)
-    )
-    (property "Status" "" (at 120.65 151.13 0)
-      (effects (font (size 1.27 1.27)) hide)
-    )
+  (symbol (lib_id "Device:R") (at 96.52 146.05 90) (unit 1)
+    (in_bom yes) (on_board yes) (dnp no) (fields_autoplaced)
+    (property "Reference" "R10" (at 96.52 139.7 90)
+      (effects (font (size 1.27 1.27)))
+    )
+    (property "Value" "100R" (at 96.52 142.24 90)
+      (effects (font (size 1.27 1.27)))
+    )
+    (property "Footprint" "Resistor_SMD:R_0805_2012Metric" (at 96.52 147.828 90)
+      (effects (font (size 1.27 1.27)) hide)
+    )
+    (property "Datasheet" "~" (at 96.52 146.05 0)
+      (effects (font (size 1.27 1.27)) hide)
+    )
+    (property "Status" "" (at 96.52 146.05 0)
+      (effects (font (size 1.27 1.27)) hide)
+    )

Commit message: Progressed ECAD
Parts:
- renumbered R10 to R8
Other:
- removed sheet Silent output
- moved on the sheet: Q3, R6, R7, R8

Commit message: Progressed ECAD.
Parts:
- added C2: 100nC, Capacitor_SMD:C_0805_2012Metric, symbol Device:C
- added Q4: BC857, Package_TO_SOT_SMD:SOT-23, symbol Transistor_BJT:BC857
- added R10: 100R, Resistor_SMD:R_0805_2012Metric, symbol Device:R
- added R9: 100kR, Resistor_SMD:R_0805_2012Metric, symbol Device:R
- added U2: 74LVC1G04, Package_TO_SOT_SMD:SOT-353_SC-70-5, symbol 74xGxx:74AHC1G04
- R6: value 47kR -> 10kR; MPN (none) -> RC0805FR-0710KL
- R8: value 100R -> 10kR; MPN (none) -> RC0805FR-0710KL
Connections:
- net +12V: now also Q4.2 (E)
- net FUNCTION: now also R10.2; no longer R8.2
- net GND: now also C2.2, R9.2, U2.3 (GND)
- net ~{OUT_ACTIVE}: now also U2.2; no longer R6.1
- new net: Q4.1 (B), R8.2
- new net: Q4.3 (C), R10.1, R9.1
- new net: R6.1, U2.4
- new net +5V: C2.1, U2.5 (VCC)
Other:
- moved on the sheet: Q3, R7
