File: ECAD/SCART_switcher/SCART_output.kicad_sch (KiCad schematic)
At the start: 12 parts, among them J2 RCA Left, J3 RCA Right, J4 SCART-F, Q3 BC847, Q4 BC857, U2 74LVC1G04

Commit message: Progressed ECAD.
Parts:
- renumbered C2 to C3, U2 to U3
Changed lines of the file:
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@@
   (symbol (lib_id "power:+12V") (at 104.14 144.78 0) (unit 1)
     (in_bom yes) (on_board yes) (dnp no) (fields_autoplaced)
-    (property "Reference" "#PWR022" (at 104.14 148.59 0)
+    (property "Reference" "#PWR026" (at 104.14 148.59 0)
       (effects (font (size 1.27 1.27)) hide)
     )
@@
       (project "SCART_switcher"
         (path "/8cd08eb5-4755-4ef5-8eeb-77fd9974b180/6562ea38-5963-42b2-a0ef-a4a12a4c652f"
-          (reference "#PWR022") (unit 1)
+          (reference "#PWR026") (unit 1)
         )
       )
@@
   (symbol (lib_id "power:GND") (at 236.22 142.24 90) (unit 1)
     (in_bom yes) (on_board yes) (dnp no) (fields_autoplaced)
-    (property "Reference" "#PWR034" (at 242.57 142.24 0)
+    (property "Reference" "#PWR038" (at 242.57 142.24 0)
       (effects (font (size 1.27 1.27)) hide)
     )
@@
       (project "SCART_switcher"
         (path "/8cd08eb5-4755-4ef5-8eeb-77fd9974b180/6562ea38-5963-42b2-a0ef-a4a12a4c652f"
-          (reference "#PWR034") (unit 1)
+          (reference "#PWR038") (unit 1)
         )
       )
@@
   (symbol (lib_id "power:+5V") (at 36.83 153.67 0) (unit 1)
     (in_bom yes) (on_board yes) (dnp no) (fields_autoplaced)
-    (property "Reference" "#PWR018" (at 36.83 157.48 0)
+    (property "Reference" "#PWR022" (at 36.83 157.48 0)
       (effects (font (size 1.27 1.27)) hide)
     )
@@
       (project "SCART_switcher"
         (path "/8cd08eb5-4755-4ef5-8eeb-77fd9974b180/6562ea38-5963-42b2-a0ef-a4a12a4c652f"
-          (reference "#PWR018") (unit 1)
+          (reference "#PWR022") (unit 1)
         )
       )
@@
   (symbol (lib_id "74xGxx:74AHC1G04") (at 76.2 157.48 0) (unit 1)
     (in_bom yes) (on_board yes) (dnp no)
-    (property "Reference" "U2" (at 81.28 149.86 0)
+    (property "Reference" "U3" (at 81.28 149.86 0)
       (effects (font (size 1.27 1.27)))
     )
@@
       (project "SCART_switcher"
         (path "/8cd08eb5-4755-4ef5-8eeb-77fd9974b180/6562ea38-5963-42b2-a0ef-a4a12a4c652f"
-          (reference "U2") (unit 1)
+          (reference "U3") (unit 1)
         )
       )
@@
   (symbol (lib_id "power:GND") (at 205.74 139.7 270) (unit 1)
     (in_bom yes) (on_board yes) (dnp no) (fields_autoplaced)
-    (property "Reference" "#PWR029" (at 199.39 139.7 0)
+    (property "Reference" "#PWR033" (at 199.39 139.7 0)
       (effects (font (size 1.27 1.27)) hide)
     )
@@
       (project "SCART_switcher"
         (path "/8cd08eb5-4755-4ef5-8eeb-77fd9974b180/6562ea38-5963-42b2-a0ef-a4a12a4c652f"
-          (reference "#PWR029") (unit 1)
+          (reference "#PWR033") (unit 1)
         )
       )
@@
   (symbol (lib_id "Device:C") (at 36.83 157.48 0) (unit 1)
     (in_bom yes) (on_board yes) (dnp no) (fields_autoplaced)
-    (property "Reference" "C2" (at 40.132 156.21 0)
+    (property "Reference" "C3" (at 40.132 156.21 0)
       (effects (font (size 1.27 1.27)) (justify left))
     )
@@
       (project "SCART_switcher"
         (path "/8cd08eb5-4755-4ef5-8eeb-77fd9974b180/6562ea38-5963-42b2-a0ef-a4a12a4c652f"
-          (reference "C2") (unit 1)
+          (reference "C3") (unit 1)
         )
       )
@@
   (symbol (lib_id "power:+12V") (at 128.27 147.32 0) (unit 1)
     (in_bom yes) (on_board yes) (dnp no) (fields_autoplaced)
-    (property "Reference" "#PWR024" (at 128.27 151.13 0)
+    (property "Reference" "#PWR028" (at 128.27 151.13 0)
       (effects (font (size 1.27 1.27)) hide)
     )
@@
       (project "SCART_switcher"
         (path "/8cd08eb5-4755-4ef5-8eeb-77fd9974b180/6562ea38-5963-42b2-a0ef-a4a12a4c652f"
-          (reference "#PWR024") (unit 1)
+          (reference "#PWR028") (unit 1)
         )
       )
@@
   (symbol (lib_id "power:GND") (at 104.14 162.56 0) (unit 1)
     (in_bom yes) (on_board yes) (dnp no) (fields_autoplaced)
-    (property "Reference" "#PWR023" (at 104.14 168.91 0)
+    (property "Reference" "#PWR027" (at 104.14 168.91 0)
       (effects (font (size 1.27 1.27)) hide)
     )
@@
       (project "SCART_switcher"
         (path "/8cd08eb5-4755-4ef5-8eeb-77fd9974b180/6562ea38-5963-42b2-a0ef-a4a12a4c652f"
-          (reference "#PWR023") (unit 1)
+          (reference "#PWR027") (unit 1)
         )
       )
@@
   (symbol (lib_id "power:GND") (at 205.74 99.06 270) (unit 1)
     (in_bom yes) (on_board yes) (dnp no) (fields_autoplaced)
-    (property "Reference" "#PWR026" (at 199.39 99.06 0)
+    (property "Reference" "#PWR030" (at 199.39 99.06 0)
       (effects (font (size 1.27 1.27)) hide)
     )
@@
       (project "SCART_switcher"
         (path "/8cd08eb5-4755-4ef5-8eeb-77fd9974b180/6562ea38-5963-42b2-a0ef-a4a12a4c652f"
-          (reference "#PWR026") (unit 1)
+          (reference "#PWR030") (unit 1)
         )
       )
@@
   (symbol (lib_id "power:GND") (at 36.83 161.29 0) (unit 1)
     (in_bom yes) (on_board yes) (dnp no) (fields_autoplaced)
-    (property "Reference" "#PWR019" (at 36.83 167.64 0)
+    (property "Reference" "#PWR023" (at 36.83 167.64 0)
       (effects (font (size 1.27 1.27)) hide)
     )
@@
       (project "SCART_switcher"
         (path "/8cd08eb5-4755-4ef5-8eeb-77fd9974b180/6562ea38-5963-42b2-a0ef-a4a12a4c652f"
-          (reference "#PWR019") (unit 1)
+          (reference "#PWR023") (unit 1)
         )
       )
@@
   (symbol (lib_id "power:+5V") (at 71.12 147.32 0) (unit 1)
     (in_bom yes) (on_board yes) (dnp no) (fields_autoplaced)
-    (property "Reference" "#PWR020" (at 71.12 151.13 0)
+    (property "Reference" "#PWR024" (at 71.12 151.13 0)
       (effects (font (size 1.27 1.27)) hide)
     )
@@
       (project "SCART_switcher"
         (path "/8cd08eb5-4755-4ef5-8eeb-77fd9974b180/6562ea38-5963-42b2-a0ef-a4a12a4c652f"
-          (reference "#PWR020") (unit 1)
+          (reference "#PWR024") (unit 1)
         )
       )
@@
   (symbol (lib_id "power:GND") (at 220.98 59.69 0) (unit 1)
     (in_bom yes) (on_board yes) (dnp no) (fields_autoplaced)
-    (property "Reference" "#PWR031" (at 220.98 66.04 0)
+    (property "Reference" "#PWR035" (at 220.98 66.04 0)
       (effects (font (size 1.27 1.27)) hide)
     )
@@
       (project "SCART_switcher"
         (path "/8cd08eb5-4755-4ef5-8eeb-77fd9974b180/6562ea38-5963-42b2-a0ef-a4a12a4c652f"
-          (reference "#PWR031") (unit 1)
+          (reference "#PWR035") (unit 1)
         )
       )
@@
   (symbol (lib_id "power:GND") (at 236.22 106.68 90) (unit 1)
     (in_bom yes) (on_board yes) (dnp no) (fields_autoplaced)
-    (property "Reference" "#PWR032" (at 242.57 106.68 0)
+    (property "Reference" "#PWR036" (at 242.57 106.68 0)
       (effects (font (size 1.27 1.27)) hide)
     )
@@
       (project "SCART_switcher"
         (path "/8cd08eb5-4755-4ef5-8eeb-77fd9974b180/6562ea38-5963-42b2-a0ef-a4a12a4c652f"
-          (reference "#PWR032") (unit 1)
+          (reference "#PWR036") (unit 1)
         )
       )
@@
   (symbol (lib_id "power:GND") (at 128.27 165.1 0) (unit 1)
     (in_bom yes) (on_board yes) (dnp no) (fields_autoplaced)
-    (property "Reference" "#PWR025" (at 128.27 171.45 0)
+    (property "Reference" "#PWR029" (at 128.27 171.45 0)
       (effects (font (size 1.27 1.27)) hide)
     )
@@
       (project "SCART_switcher"
         (path "/8cd08eb5-4755-4ef5-8eeb-77fd9974b180/6562ea38-5963-42b2-a0ef-a4a12a4c652f"
-          (reference "#PWR025") (unit 1)
+          (reference "#PWR029") (unit 1)
         )
       )
@@
   (symbol (lib_id "power:GND") (at 220.98 41.91 0) (unit 1)
     (in_bom yes) (on_board yes) (dnp no) (fields_autoplaced)
-    (property "Reference" "#PWR030" (at 220.98 48.26 0)
+    (property "Reference" "#PWR034" (at 220.98 48.26 0)
       (effects (font (size 1.27 1.27)) hide)
     )
@@
       (project "SCART_switcher"
         (path "/8cd08eb5-4755-4ef5-8eeb-77fd9974b180/6562ea38-5963-42b2-a0ef-a4a12a4c652f"
-          (reference "#PWR030") (unit 1)
+          (reference "#PWR034") (unit 1)
         )
       )
@@
   (symbol (lib_id "power:GND") (at 236.22 116.84 90) (unit 1)
     (in_bom yes) (on_board yes) (dnp no) (fields_autoplaced)
-    (property "Reference" "#PWR033" (at 242.57 116.84 0)
+    (property "Reference" "#PWR037" (at 242.57 116.84 0)
       (effects (font (size 1.27 1.27)) hide)
     )
@@
       (project "SCART_switcher"
         (path "/8cd08eb5-4755-4ef5-8eeb-77fd9974b180/6562ea38-5963-42b2-a0ef-a4a12a4c652f"
-          (reference "#PWR033") (unit 1)
+          (reference "#PWR037") (unit 1)
         )
       )
@@
   (symbol (lib_id "power:GND") (at 71.12 167.64 0) (unit 1)
     (in_bom yes) (on_board yes) (dnp no) (fields_autoplaced)
-    (property "Reference" "#PWR021" (at 71.12 173.99 0)
+    (property "Reference" "#PWR025" (at 71.12 173.99 0)
       (effects (font (size 1.27 1.27)) hide)
     )
@@
       (project "SCART_switcher"
         (path "/8cd08eb5-4755-4ef5-8eeb-77fd9974b180/6562ea38-5963-42b2-a0ef-a4a12a4c652f"
-          (reference "#PWR021") (unit 1)
+          (reference "#PWR025") (unit 1)
         )
       )
@@
   (symbol (lib_id "power:GND") (at 205.74 119.38 270) (unit 1)
     (in_bom yes) (on_board yes) (dnp no) (fields_autoplaced)
-    (property "Reference" "#PWR027" (at 199.39 119.38 0)
+    (property "Reference" "#PWR031" (at 199.39 119.38 0)
       (effects (font (size 1.27 1.27)) hide)
     )
@@
       (project "SCART_switcher"
         (path "/8cd08eb5-4755-4ef5-8eeb-77fd9974b180/6562ea38-5963-42b2-a0ef-a4a12a4c652f"
-          (reference "#PWR027") (unit 1)
+          (reference "#PWR031") (unit 1)
         )
       )
@@
   (symbol (lib_id "power:GND") (at 205.74 129.54 270) (unit 1)
     (in_bom yes) (on_board yes) (dnp no) (fields_autoplaced)
-    (property "Reference" "#PWR028" (at 199.39 129.54 0)
+    (property "Reference" "#PWR032" (at 199.39 129.54 0)
       (effects (font (size 1.27 1.27)) hide)
     )
@@
       (project "SCART_switcher"
         (path "/8cd08eb5-4755-4ef5-8eeb-77fd9974b180/6562ea38-5963-42b2-a0ef-a4a12a4c652f"
-          (reference "#PWR028") (unit 1)
-        )
-      )
+          (reference "#PWR032") (unit 1)
+        )
+      )

Commit message: Progressed ECAD.
Parts:
- C3: footprint Capacitor_SMD:C_0805_2012Metric -> Capacitor_SMD:C_0603_1608Metric
Changed lines of the file:
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@@
       (effects (font (size 1.27 1.27)) (justify left))
     )
-    (property "Footprint" "Capacitor_SMD:C_0805_2012Metric" (at 37.7952 161.29 0)
+    (property "Footprint" "Capacitor_SMD:C_0603_1608Metric" (at 37.7952 161.29 0)
       (effects (font (size 1.27 1.27)) hide)
     )

Commit message: Progressed ECAD.
Other:
- note added: "I_{12V}=4mA"
- note added: "I_{5V}=200mA"
- note added: "I_{9V}=30mA"
Changed lines of the file:
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@@
     (stroke (width 0) (type default))
+  )
+  (text "I_{5V}=200mA" (at 81.28 85.09 0)
+    (effects (font (size 1.27 1.27)) (justify left bottom))
   )
   (text "SCART output" (at 214.63 83.82 0)
@@
     (effects (font (size 1.27 1.27)) (justify left bottom))
   )
+  (text "I_{12V}=4mA" (at 106.68 175.26 0)
+    (effects (font (size 1.27 1.27)) (justify left bottom))
+  )
   (text "(*1) FUNCTION pin has the following signaling:\n	Level 0: 0 V to +2 V (SCART off)\n	Level 1A: +4.5 V to +7 V (SCART on, 16:9)\n	Level 1B: +9.5 V to +12 V (SCART on)\nThe circuit doesn't distinguish between levels 1A and 1B as these are frequently not respected in consumer\nproducts. This way it is simpler to default to 4:3 format (12V) when the video output is active and\nif needed manualy adjust the TV to 16:9."
     (at 177.8 180.34 0)
@@
     (effects (font (size 1.27 1.27)) (justify left bottom))
   )
+  (text "I_{9V}=30mA" (at 82.55 63.5 0)
+    (effects (font (size 1.27 1.27)) (justify left bottom))
+  )

Commit message: Progressed ECAD.
Parts:
- R6, R7, R8: MPN RC0805FR-0710KL -> AC0805FR-0710KL; Status (none) -> OK
- R9: MPN (none) -> RC0805FR-07100KL; Status (none) -> OK
Changed lines of the file:
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@@
       (effects (font (size 1.27 1.27)) hide)
     )
-    (property "Datasheet" "https://datasheet.lcsc.com/lcsc/1810201611_YAGEO-RC0805FR-0710KL_C84376.pdf" (at 92.71 157.48 0)
-      (effects (font (size 1.27 1.27)) hide)
-    )
-    (property "MPN" "RC0805FR-0710KL" (at 92.71 157.48 0)
-      (effects (font (size 1.27 1.27)) hide)
-    )
-    (property "Status" "" (at 92.71 157.48 0)
+    (property "Datasheet" "https://datasheet.lcsc.com/lcsc/2304140030_YAGEO-AC0805FR-0710KL_C140868.pdf" (at 92.71 157.48 0)
+      (effects (font (size 1.27 1.27)) hide)
+    )
+    (property "MPN" "AC0805FR-0710KL" (at 92.71 157.48 0)
+      (effects (font (size 1.27 1.27)) hide)
+    )
+    (property "Status" "OK" (at 92.71 157.48 0)
       (effects (font (size 1.27 1.27)) hide)
     )
@@
       (effects (font (size 1.27 1.27)) hide)
     )
-    (property "Datasheet" "https://datasheet.lcsc.com/lcsc/1810201611_YAGEO-RC0805FR-0710KL_C84376.pdf" (at 116.84 152.4 0)
-      (effects (font (size 1.27 1.27)) hide)
-    )
-    (property "MPN" "RC0805FR-0710KL" (at 116.84 152.4 0)
-      (effects (font (size 1.27 1.27)) hide)
-    )
-    (property "Status" "" (at 116.84 152.4 0)
+    (property "Datasheet" "https://datasheet.lcsc.com/lcsc/2304140030_YAGEO-AC0805FR-0710KL_C140868.pdf" (at 116.84 152.4 0)
+      (effects (font (size 1.27 1.27)) hide)
+    )
+    (property "MPN" "AC0805FR-0710KL" (at 116.84 152.4 0)
+      (effects (font (size 1.27 1.27)) hide)
+    )
+    (property "Status" "OK" (at 116.84 152.4 0)
       (effects (font (size 1.27 1.27)) hide)
     )
@@
       (effects (font (size 1.27 1.27)) hide)
     )
-    (property "Datasheet" "https://datasheet.lcsc.com/lcsc/1810201611_YAGEO-RC0805FR-0710KL_C84376.pdf" (at 104.14 148.59 0)
-      (effects (font (size 1.27 1.27)) hide)
-    )
-    (property "MPN" "RC0805FR-0710KL" (at 104.14 148.59 0)
-      (effects (font (size 1.27 1.27)) hide)
-    )
-    (property "Status" "" (at 104.14 148.59 0)
+    (property "Datasheet" "https://datasheet.lcsc.com/lcsc/2304140030_YAGEO-AC0805FR-0710KL_C140868.pdf" (at 104.14 148.59 0)
+      (effects (font (size 1.27 1.27)) hide)
+    )
+    (property "MPN" "AC0805FR-0710KL" (at 104.14 148.59 0)
+      (effects (font (size 1.27 1.27)) hide)
+    )
+    (property "Status" "OK" (at 104.14 148.59 0)
       (effects (font (size 1.27 1.27)) hide)
     )
@@
       (effects (font (size 1.27 1.27)) hide)
     )
-    (property "Datasheet" "" (at 128.27 161.29 0)
-      (effects (font (size 1.27 1.27)) hide)
-    )
-    (property "MPN" "" (at 128.27 161.29 0)
-      (effects (font (size 1.27 1.27)) hide)
-    )
-    (property "Status" "" (at 128.27 161.29 0)
-      (effects (font (size 1.27 1.27)) hide)
-    )
+    (property "Datasheet" "https://datasheet.lcsc.com/lcsc/2304140030_YAGEO-RC0805FR-07100KL_C96346.pdf" (at 128.27 161.29 0)
+      (effects (font (size 1.27 1.27)) hide)
+    )
+    (property "MPN" "RC0805FR-07100KL" (at 128.27 161.29 0)
+      (effects (font (size 1.27 1.27)) hide)
+    )
+    (property "Status" "OK" (at 128.27 161.29 0)
+      (effects (font (size 1.27 1.27)) hide)
+    )

Commit message: Progressed ECAD.
Parts:
- C3: MPN CL21B104KBCNNNC -> CL10B104KO8NNNC; Status (none) -> OK
- R10: MPN (none) -> RT0805BRD07100RL; Status (none) -> OK
Changed lines of the file:
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@@
       (effects (font (size 1.27 1.27)) hide)
     )
-    (property "Datasheet" "~" (at 142.24 157.48 0)
+    (property "Datasheet" "https://datasheet.lcsc.com/lcsc/2304140030_YAGEO-RT0805BRD07100RL_C110773.pdf" (at 142.24 157.48 0)
       (effects (font (size 1.27 1.27)) hide)
     )
-    (property "Status" "" (at 142.24 157.48 0)
+    (property "Status" "OK" (at 142.24 157.48 0)
+      (effects (font (size 1.27 1.27)) hide)
+    )
+    (property "MPN" "RT0805BRD07100RL" (at 142.24 157.48 0)
       (effects (font (size 1.27 1.27)) hide)
     )
@@
       (effects (font (size 1.27 1.27)) hide)
     )
-    (property "Datasheet" "https://datasheet.lcsc.com/lcsc/1810191215_Samsung-Electro-Mechanics-CL21B104KBCNNNC_C1711.pdf" (at 36.83 157.48 0)
+    (property "Datasheet" "https://datasheet.lcsc.com/lcsc/1810271710_Samsung-Electro-Mechanics-CL10B104KO8NNNC_C66501.pdf" (at 36.83 157.48 0)
       (effects (font (size 1.27 1.27)) hide)
     )
-    (property "MPN" "CL21B104KBCNNNC" (at 36.83 157.48 0)
+    (property "MPN" "CL10B104KO8NNNC" (at 36.83 157.48 0)
       (effects (font (size 1.27 1.27)) hide)
     )
-    (property "Status" "" (at 36.83 157.48 0)
+    (property "Status" "OK" (at 36.83 157.48 0)
       (effects (font (size 1.27 1.27)) hide)
     )

Commit message: Progressed ECAD.
Parts:
- Q3: MPN_MOUSER (none) -> BC847C,215
- Q4: MPN_MOUSER (none) -> BC857C,215
- U3: MPN_MOUSER (none) -> SN74LVC1G04DCKR

Commit message: Progressed ECAD.
Parts:
- J2, J3, J4: MPN_MOUSER (none) -> N/A
Changed lines of the file:
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@@
       (effects (font (size 1.27 1.27)) hide)
     )
-    (property "Datasheet" " ~" (at 220.98 36.83 0)
+    (property "Datasheet" "N/A" (at 220.98 36.83 0)
       (effects (font (size 1.27 1.27)) hide)
     )
@@
       (effects (font (size 1.27 1.27)) hide)
     )
-    (property "MPN_MOUSER" "" (at 220.98 36.83 0)
+    (property "MPN_MOUSER" "N/A" (at 220.98 36.83 0)
       (effects (font (size 1.27 1.27)) hide)
     )
@@
       (effects (font (size 1.27 1.27)) hide)
     )
-    (property "Datasheet" " ~" (at 220.98 123.19 0)
+    (property "Datasheet" "N/A" (at 220.98 123.19 0)
       (effects (font (size 1.27 1.27)) hide)
     )
@@
       (effects (font (size 1.27 1.27)) hide)
     )
-    (property "MPN_MOUSER" "" (at 220.98 124.46 0)
+    (property "MPN_MOUSER" "N/A" (at 220.98 124.46 0)
       (effects (font (size 1.27 1.27)) hide)
     )
@@
       (effects (font (size 1.27 1.27)) hide)
     )
-    (property "Datasheet" " ~" (at 220.98 54.61 0)
+    (property "Datasheet" "N/A" (at 220.98 54.61 0)
       (effects (font (size 1.27 1.27)) hide)
     )
@@
       (effects (font (size 1.27 1.27)) hide)
     )
-    (property "MPN_MOUSER" "" (at 220.98 54.61 0)
-      (effects (font (size 1.27 1.27)) hide)
-    )
+    (property "MPN_MOUSER" "N/A" (at 220.98 54.61 0)
+      (effects (font (size 1.27 1.27)) hide)
+    )
