File: ECAD/SCART_switcher/SCART_output.kicad_sch (KiCad schematic)
At the start: 12 parts, among them J2 RCA Left, J3 RCA Right, J4 SCART-F, Q3 BC847, Q4 BC857, U3 74LVC1G04

Commit message: Progressed ECAD.
Parts:
- R10: MPN RT0805BRD07100RL -> RT0805FRD07100RL; R % tol (none) -> 1%; R pwr (none) -> 125mW
- R6, R7, R8: MPN AC0805FR-0710KL -> RC0805JR-0710KL; R % tol (none) -> 5%; R pwr (none) -> 125mW
- R9: MPN RC0805FR-07100KL -> RC0805JR-07100KL; R % tol (none) -> 5%; R pwr (none) -> 125mW
Changed lines of the file:
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@@
+      (effects (font (size 1.27 1.27)) hide)
+    )
+    (property "R % tol" "" (at 220.98 36.83 0)
+      (effects (font (size 1.27 1.27)) hide)
+    )
+    (property "R pwr" "" (at 220.98 36.83 0)
       (effects (font (size 1.27 1.27)) hide)
     )
@@
       (effects (font (size 1.27 1.27)) hide)
     )
+    (property "R % tol" "" (at 125.73 152.4 0)
+      (effects (font (size 1.27 1.27)) hide)
+    )
+    (property "R pwr" "" (at 125.73 152.4 0)
+      (effects (font (size 1.27 1.27)) hide)
+    )
     (pin "1")
     (pin "2")
@@
       (effects (font (size 1.27 1.27)) hide)
     )
-    (property "Datasheet" "https://datasheet.lcsc.com/lcsc/2304140030_YAGEO-AC0805FR-0710KL_C140868.pdf" (at 92.71 157.48 0)
-      (effects (font (size 1.27 1.27)) hide)
-    )
-    (property "MPN" "AC0805FR-0710KL" (at 92.71 157.48 0)
+    (property "Datasheet" "https://datasheet.lcsc.com/lcsc/1810171610_YAGEO-RC0805JR-0710KL_C100047.pdf" (at 92.71 157.48 0)
+      (effects (font (size 1.27 1.27)) hide)
+    )
+    (property "MPN" "RC0805JR-0710KL" (at 92.71 157.48 0)
       (effects (font (size 1.27 1.27)) hide)
     )
@@
       (effects (font (size 1.27 1.27)) hide)
     )
+    (property "R % tol" "5%" (at 92.71 157.48 0)
+      (effects (font (size 1.27 1.27)) hide)
+    )
+    (property "R pwr" "125mW" (at 92.71 157.48 0)
+      (effects (font (size 1.27 1.27)) hide)
+    )
     (pin "1")
     (pin "2")
@@
       (effects (font (size 1.27 1.27)) hide)
     )
-    (property "Datasheet" "https://datasheet.lcsc.com/lcsc/2304140030_YAGEO-RT0805BRD07100RL_C110773.pdf" (at 142.24 157.48 0)
+    (property "Datasheet" "https://datasheet.lcsc.com/lcsc/2304140030_YAGEO-RT0805FRD07100RL_C143843.pdf" (at 142.24 157.48 0)
       (effects (font (size 1.27 1.27)) hide)
     )
@@
       (effects (font (size 1.27 1.27)) hide)
     )
-    (property "MPN" "RT0805BRD07100RL" (at 142.24 157.48 0)
+    (property "MPN" "RT0805FRD07100RL" (at 142.24 157.48 0)
       (effects (font (size 1.27 1.27)) hide)
     )
     (property "MPN_MOUSER" "" (at 142.24 157.48 0)
+      (effects (font (size 1.27 1.27)) hide)
+    )
+    (property "R % tol" "1%" (at 142.24 157.48 0)
+      (effects (font (size 1.27 1.27)) hide)
+    )
+    (property "R pwr" "125mW" (at 142.24 157.48 0)
       (effects (font (size 1.27 1.27)) hide)
     )
@@
       (effects (font (size 1.27 1.27)) hide)
     )
+    (property "R % tol" "" (at 76.2 157.48 0)
+      (effects (font (size 1.27 1.27)) hide)
+    )
+    (property "R pwr" "" (at 76.2 157.48 0)
+      (effects (font (size 1.27 1.27)) hide)
+    )
     (pin "2")
     (pin "3")
@@
       (effects (font (size 1.27 1.27)) hide)
     )
+    (property "R % tol" "" (at 36.83 157.48 0)
+      (effects (font (size 1.27 1.27)) hide)
+    )
+    (property "R pwr" "" (at 36.83 157.48 0)
+      (effects (font (size 1.27 1.27)) hide)
+    )
     (pin "1")
     (pin "2")
@@
     )
     (property "MPN_MOUSER" "N/A" (at 220.98 124.46 0)
+      (effects (font (size 1.27 1.27)) hide)
+    )
+    (property "R % tol" "" (at 220.98 124.46 0)
+      (effects (font (size 1.27 1.27)) hide)
+    )
+    (property "R pwr" "" (at 220.98 124.46 0)
       (effects (font (size 1.27 1.27)) hide)
     )
@@
       (effects (font (size 1.27 1.27)) hide)
     )
-    (property "Datasheet" "https://datasheet.lcsc.com/lcsc/2304140030_YAGEO-AC0805FR-0710KL_C140868.pdf" (at 116.84 152.4 0)
-      (effects (font (size 1.27 1.27)) hide)
-    )
-    (property "MPN" "AC0805FR-0710KL" (at 116.84 152.4 0)
+    (property "Datasheet" "https://datasheet.lcsc.com/lcsc/1810171610_YAGEO-RC0805JR-0710KL_C100047.pdf" (at 116.84 152.4 0)
+      (effects (font (size 1.27 1.27)) hide)
+    )
+    (property "MPN" "RC0805JR-0710KL" (at 116.84 152.4 0)
       (effects (font (size 1.27 1.27)) hide)
     )
@@
     )
     (property "MPN_MOUSER" "" (at 116.84 152.4 0)
+      (effects (font (size 1.27 1.27)) hide)
+    )
+    (property "R % tol" "5%" (at 116.84 152.4 0)
+      (effects (font (size 1.27 1.27)) hide)
+    )
+    (property "R pwr" "125mW" (at 116.84 152.4 0)
       (effects (font (size 1.27 1.27)) hide)
     )
@@
       (effects (font (size 1.27 1.27)) hide)
     )
-    (property "Datasheet" "https://datasheet.lcsc.com/lcsc/2304140030_YAGEO-AC0805FR-0710KL_C140868.pdf" (at 104.14 148.59 0)
-      (effects (font (size 1.27 1.27)) hide)
-    )
-    (property "MPN" "AC0805FR-0710KL" (at 104.14 148.59 0)
+    (property "Datasheet" "https://datasheet.lcsc.com/lcsc/1810171610_YAGEO-RC0805JR-0710KL_C100047.pdf" (at 104.14 148.59 0)
+      (effects (font (size 1.27 1.27)) hide)
+    )
+    (property "MPN" "RC0805JR-0710KL" (at 104.14 148.59 0)
       (effects (font (size 1.27 1.27)) hide)
     )
@@
       (effects (font (size 1.27 1.27)) hide)
     )
+    (property "R % tol" "5%" (at 104.14 148.59 0)
+      (effects (font (size 1.27 1.27)) hide)
+    )
+    (property "R pwr" "125mW" (at 104.14 148.59 0)
+      (effects (font (size 1.27 1.27)) hide)
+    )
     (pin "1")
     (pin "2")
@@
       (effects (font (size 1.27 1.27)) hide)
     )
-    (property "Datasheet" "https://datasheet.lcsc.com/lcsc/2304140030_YAGEO-RC0805FR-07100KL_C96346.pdf" (at 128.27 161.29 0)
-      (effects (font (size 1.27 1.27)) hide)
-    )
-    (property "MPN" "RC0805FR-07100KL" (at 128.27 161.29 0)
+    (property "Datasheet" "https://datasheet.lcsc.com/lcsc/2304140030_YAGEO-RC0805JR-07100KL_C100049.pdf" (at 128.27 161.29 0)
+      (effects (font (size 1.27 1.27)) hide)
+    )
+    (property "MPN" "RC0805JR-07100KL" (at 128.27 161.29 0)
       (effects (font (size 1.27 1.27)) hide)
     )
@@
       (effects (font (size 1.27 1.27)) hide)
     )
+    (property "R % tol" "5%" (at 128.27 161.29 0)
+      (effects (font (size 1.27 1.27)) hide)
+    )
+    (property "R pwr" "125mW" (at 128.27 161.29 0)
+      (effects (font (size 1.27 1.27)) hide)
+    )
     (pin "1")
     (pin "2")
@@
     )
     (property "MPN_MOUSER" "N/A" (at 220.98 54.61 0)
+      (effects (font (size 1.27 1.27)) hide)
+    )
+    (property "R % tol" "" (at 220.98 54.61 0)
+      (effects (font (size 1.27 1.27)) hide)
+    )
+    (property "R pwr" "" (at 220.98 54.61 0)
       (effects (font (size 1.27 1.27)) hide)
     )
@@
       (effects (font (size 1.27 1.27)) hide)
     )
+    (property "R % tol" "" (at 101.6 157.48 0)
+      (effects (font (size 1.27 1.27)) hide)
+    )
+    (property "R pwr" "" (at 101.6 157.48 0)
+      (effects (font (size 1.27 1.27)) hide)
+    )
