File: ECAD/SCART_switcher/priority_level.kicad_sch (KiCad schematic)
At the start: 4 parts

Commit message: Progressed ECAD.
Parts:
- U?: MFN 74AHC1G04W5-7 -> (none); MPN (none) -> 74AHC1G04W5-7
- U? (x2): MFN 74AHC1G08W5-7 -> (none); MPN (none) -> 74AHC1G08W5-7
Changed lines of the file:
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@@
       (effects (font (size 1.27 1.27)) hide)
     )
-    (property "MFN" "74AHC1G04W5-7" (at 132.08 93.98 0)
+    (property "MPN" "74AHC1G04W5-7" (at 132.08 93.98 0)
       (effects (font (size 1.27 1.27)) hide)
     )
@@
       (effects (font (size 1.27 1.27)) hide)
     )
-    (property "MFN" "" (at 91.44 100.33 0)
-      (effects (font (size 1.27 1.27)) hide)
-    )
     (property "MPN" "CL21B104KBCNNNC" (at 91.44 100.33 0)
       (effects (font (size 1.27 1.27)) hide)
@@
       (effects (font (size 1.27 1.27)) hide)
     )
-    (property "MFN" "74AHC1G08W5-7" (at 148.59 110.49 0)
+    (property "MPN" "74AHC1G08W5-7" (at 148.59 110.49 0)
       (effects (font (size 1.27 1.27)) hide)
     )
@@
       (effects (font (size 1.27 1.27)) hide)
     )
-    (property "MFN" "74AHC1G08W5-7" (at 167.64 78.74 0)
-      (effects (font (size 1.27 1.27)) hide)
-    )
+    (property "MPN" "74AHC1G08W5-7" (at 167.64 78.74 0)
+      (effects (font (size 1.27 1.27)) hide)
+    )

Commit message: Progressed ECAD.
Parts:
- C?: footprint Capacitor_SMD:C_0805_2012Metric_Pad1.18x1.45mm_HandSolder -> Capacitor_SMD:C_0805_2012Metric
Changed lines of the file:
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@@
       (effects (font (size 1.27 1.27)) (justify left))
     )
-    (property "Footprint" "Capacitor_SMD:C_0805_2012Metric_Pad1.18x1.45mm_HandSolder" (at 92.4052 104.14 0)
+    (property "Footprint" "Capacitor_SMD:C_0805_2012Metric" (at 92.4052 104.14 0)
       (effects (font (size 1.27 1.27)) hide)
     )
