File: ECAD/SCART_switcher/priority_level.kicad_sch (KiCad schematic)
At the start: 4 parts

Commit message: Progressed ECAD.
Parts:
- U?: MPN 74AHC1G04W5-7 -> SN74AHC1G04DBVR
- U? (x2): MPN 74AHC1G08W5-7 -> SN74AHC1G08DBVR
Changed lines of the file:
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@@
       (effects (font (size 1.27 1.27)) hide)
     )
-    (property "Datasheet" "https://datasheet.lcsc.com/lcsc/1912111437_Diodes-Incorporated-74AHC1G04W5-7_C460486.pdf" (at 132.08 93.98 0)
-      (effects (font (size 1.27 1.27)) hide)
-    )
-    (property "MPN" "74AHC1G04W5-7" (at 132.08 93.98 0)
+    (property "Datasheet" "https://datasheet.lcsc.com/lcsc/2001061132_Texas-Instruments-SN74AHC1G04DBVR_C7465.pdf" (at 132.08 93.98 0)
+      (effects (font (size 1.27 1.27)) hide)
+    )
+    (property "MPN" "SN74AHC1G04DBVR" (at 132.08 93.98 0)
       (effects (font (size 1.27 1.27)) hide)
     )
@@
       (effects (font (size 1.27 1.27)) hide)
     )
-    (property "Datasheet" "https://datasheet.lcsc.com/lcsc/1912111437_Diodes-Incorporated-74AHC1G08W5-7_C460487.pdf" (at 148.59 110.49 0)
-      (effects (font (size 1.27 1.27)) hide)
-    )
-    (property "MPN" "74AHC1G08W5-7" (at 148.59 110.49 0)
+    (property "Datasheet" "https://datasheet.lcsc.com/lcsc/1809151118_Texas-Instruments-SN74AHC1G08DBVR_C7467.pdf" (at 148.59 110.49 0)
+      (effects (font (size 1.27 1.27)) hide)
+    )
+    (property "MPN" "SN74AHC1G08DBVR" (at 148.59 110.49 0)
       (effects (font (size 1.27 1.27)) hide)
     )
@@
       (effects (font (size 1.27 1.27)) hide)
     )
-    (property "Datasheet" "https://datasheet.lcsc.com/lcsc/1912111437_Diodes-Incorporated-74AHC1G08W5-7_C460487.pdf" (at 167.64 78.74 0)
-      (effects (font (size 1.27 1.27)) hide)
-    )
-    (property "MPN" "74AHC1G08W5-7" (at 167.64 78.74 0)
-      (effects (font (size 1.27 1.27)) hide)
-    )
+    (property "Datasheet" "https://datasheet.lcsc.com/lcsc/1809151118_Texas-Instruments-SN74AHC1G08DBVR_C7467.pdf" (at 167.64 78.74 0)
+      (effects (font (size 1.27 1.27)) hide)
+    )
+    (property "MPN" "SN74AHC1G08DBVR" (at 167.64 78.74 0)
+      (effects (font (size 1.27 1.27)) hide)
+    )

Commit message: Progressed ECAD.
Parts:
- U?: value 74AHC1G04 -> 74LVC1G04; footprint Package_TO_SOT_SMD:SOT-23-5 -> Package_TO_SOT_SMD:SOT-353_SC-70-5; MPN SN74AHC1G04DBVR -> SN74LVC1G04DCKR; Status (none) -> OK
- U? (x2): value 74AHC1G08 -> 74LVC1G08; footprint Package_TO_SOT_SMD:SOT-23-5 -> Package_TO_SOT_SMD:SOT-353_SC-70-5; MPN SN74AHC1G08DBVR -> SN74LVC1G08DCKR; Status (none) -> OK
Changed lines of the file:
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@@
       (effects (font (size 1.27 1.27)))
     )
-    (property "Value" "74AHC1G04" (at 137.16 88.9 0)
-      (effects (font (size 1.27 1.27)))
-    )
-    (property "Footprint" "Package_TO_SOT_SMD:SOT-23-5" (at 132.08 93.98 0)
-      (effects (font (size 1.27 1.27)) hide)
-    )
-    (property "Datasheet" "https://datasheet.lcsc.com/lcsc/2001061132_Texas-Instruments-SN74AHC1G04DBVR_C7465.pdf" (at 132.08 93.98 0)
-      (effects (font (size 1.27 1.27)) hide)
-    )
-    (property "MPN" "SN74AHC1G04DBVR" (at 132.08 93.98 0)
-      (effects (font (size 1.27 1.27)) hide)
-    )
-    (property "Status" "" (at 132.08 93.98 0)
+    (property "Value" "74LVC1G04" (at 137.16 88.9 0)
+      (effects (font (size 1.27 1.27)))
+    )
+    (property "Footprint" "Package_TO_SOT_SMD:SOT-353_SC-70-5" (at 132.08 93.98 0)
+      (effects (font (size 1.27 1.27)) hide)
+    )
+    (property "Datasheet" "https://datasheet.lcsc.com/lcsc/1811021113_Texas-Instruments-SN74LVC1G04DCKR_C8207.pdf" (at 132.08 93.98 0)
+      (effects (font (size 1.27 1.27)) hide)
+    )
+    (property "MPN" "SN74LVC1G04DCKR" (at 132.08 93.98 0)
+      (effects (font (size 1.27 1.27)) hide)
+    )
+    (property "Status" "OK" (at 132.08 93.98 0)
       (effects (font (size 1.27 1.27)) hide)
     )
@@
       (effects (font (size 1.27 1.27)))
     )
-    (property "Value" "74AHC1G08" (at 158.75 114.3 90)
-      (effects (font (size 1.27 1.27)))
-    )
-    (property "Footprint" "Package_TO_SOT_SMD:SOT-23-5" (at 148.59 110.49 0)
-      (effects (font (size 1.27 1.27)) hide)
-    )
-    (property "Datasheet" "https://datasheet.lcsc.com/lcsc/1809151118_Texas-Instruments-SN74AHC1G08DBVR_C7467.pdf" (at 148.59 110.49 0)
-      (effects (font (size 1.27 1.27)) hide)
-    )
-    (property "MPN" "SN74AHC1G08DBVR" (at 148.59 110.49 0)
-      (effects (font (size 1.27 1.27)) hide)
-    )
-    (property "Status" "" (at 148.59 110.49 0)
+    (property "Value" "74LVC1G08" (at 158.75 114.3 90)
+      (effects (font (size 1.27 1.27)))
+    )
+    (property "Footprint" "Package_TO_SOT_SMD:SOT-353_SC-70-5" (at 148.59 110.49 0)
+      (effects (font (size 1.27 1.27)) hide)
+    )
+    (property "Datasheet" "https://datasheet.lcsc.com/lcsc/1809051811_Texas-Instruments-SN74LVC1G08DCKR_C7832.pdf" (at 148.59 110.49 0)
+      (effects (font (size 1.27 1.27)) hide)
+    )
+    (property "MPN" "SN74LVC1G08DCKR" (at 148.59 110.49 0)
+      (effects (font (size 1.27 1.27)) hide)
+    )
+    (property "Status" "OK" (at 148.59 110.49 0)
       (effects (font (size 1.27 1.27)) hide)
     )
@@
       (effects (font (size 1.27 1.27)))
     )
-    (property "Value" "74AHC1G08" (at 176.53 73.66 0)
-      (effects (font (size 1.27 1.27)))
-    )
-    (property "Footprint" "Package_TO_SOT_SMD:SOT-23-5" (at 167.64 78.74 0)
-      (effects (font (size 1.27 1.27)) hide)
-    )
-    (property "Datasheet" "https://datasheet.lcsc.com/lcsc/1809151118_Texas-Instruments-SN74AHC1G08DBVR_C7467.pdf" (at 167.64 78.74 0)
-      (effects (font (size 1.27 1.27)) hide)
-    )
-    (property "MPN" "SN74AHC1G08DBVR" (at 167.64 78.74 0)
-      (effects (font (size 1.27 1.27)) hide)
-    )
-    (property "Status" "" (at 167.64 78.74 0)
-      (effects (font (size 1.27 1.27)) hide)
-    )
+    (property "Value" "74LVC1G08" (at 176.53 73.66 0)
+      (effects (font (size 1.27 1.27)))
+    )
+    (property "Footprint" "Package_TO_SOT_SMD:SOT-353_SC-70-5" (at 167.64 78.74 0)
+      (effects (font (size 1.27 1.27)) hide)
+    )
+    (property "Datasheet" "https://datasheet.lcsc.com/lcsc/1809051811_Texas-Instruments-SN74LVC1G08DCKR_C7832.pdf" (at 167.64 78.74 0)
+      (effects (font (size 1.27 1.27)) hide)
+    )
+    (property "MPN" "SN74LVC1G08DCKR" (at 167.64 78.74 0)
+      (effects (font (size 1.27 1.27)) hide)
+    )
+    (property "Status" "OK" (at 167.64 78.74 0)
+      (effects (font (size 1.27 1.27)) hide)
+    )

Commit message: Progressed ECAD.
Parts:
- gave numbers to parts that had none: 4

Commit message: Progressed ECAD
Parts:
- renumbered C45 to C44, U26 to U25, U27 to U26, U28 to U27

Commit message: Progressed ECAD.
Parts:
- renumbered C44 to C45, U25 to U26, U26 to U27, U27 to U28

Commit message: Progressed ECAD.
Parts:
- renumbered C45 to C46, U26 to U27, U27 to U28, U28 to U29
