File: ECAD/SCART_switcher/priority_level.kicad_sch (KiCad schematic)
At the start: 4 parts, among them U27 74LVC1G04, U28 74LVC1G08, U29 74LVC1G08

Commit message: Progressed ECAD.
Parts:
- added C58, C59: 100nC, Capacitor_SMD:C_0805_2012Metric, symbol Device:C
- renumbered C46 to C57, U27 to U38, U28 to U39, U29 to U40
Connections:
- net +5V: now also C58.1, C59.1
- net GND: now also C58.2, C59.2
Other:
- moved on the sheet: C57

Commit message: Progressed ECAD.
Parts:
- removed U39: 74LVC1G08, Package_TO_SOT_SMD:SOT-353_SC-70-5, symbol 74xGxx:74AHC1G08
- added U40: 74LVC1G08, Package_TO_SOT_SMD:SOT-353_SC-70-5, symbol 74xGxx:74AHC1G08
- renumbered U40 to U39
Connections:
- net +5V: now also U40.5 (VCC)
- net CARRY_IN: now also U39.1, U40.1; no longer U39.2
- net CARRY_OUT: now also U40.4
- net GND: now also U40.3 (GND)
- net IN_ACTIVE: now also U39.2; no longer U39.1
- net at U38.4: now also U40.2
Other:
- note added: "CARRY_IN | IN_ACTIVE || CARRY_OUT ----------------------- 0V 0V 0V 0V 5V 0V 5V 0V 5V 5V 5V 0V"
- note added: "CARRY_IN | IN_ACTIVE || IN_ENABLE ----------------------- 0V 0V 0V 0V 5V 0V 5V 0V 0V 5V 5V 5V"
- note added: "CARRY_OUT = CARRY_IN AND ~{IN_ACTIVE}"
- note added: "IN_ENABLE = CARRY_IN AND IN_ACTIVE"
- moved on the sheet: C57, C58, C59, U38, U39

Commit message: Progressed ECAD.
Parts:
- C57, C58, C59: footprint Capacitor_SMD:C_0805_2012Metric -> Capacitor_SMD:C_0603_1608Metric
Changed lines of the file:
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@@
       (effects (font (size 1.27 1.27)) (justify left))
     )
-    (property "Footprint" "Capacitor_SMD:C_0805_2012Metric" (at 174.9552 113.03 0)
+    (property "Footprint" "Capacitor_SMD:C_0603_1608Metric" (at 174.9552 113.03 0)
       (effects (font (size 1.27 1.27)) hide)
     )
@@
       (effects (font (size 1.27 1.27)) (justify left))
     )
-    (property "Footprint" "Capacitor_SMD:C_0805_2012Metric" (at 174.9552 77.47 0)
+    (property "Footprint" "Capacitor_SMD:C_0603_1608Metric" (at 174.9552 77.47 0)
       (effects (font (size 1.27 1.27)) hide)
     )
@@
       (effects (font (size 1.27 1.27)) (justify left))
     )
-    (property "Footprint" "Capacitor_SMD:C_0805_2012Metric" (at 101.2952 143.51 0)
-      (effects (font (size 1.27 1.27)) hide)
-    )
+    (property "Footprint" "Capacitor_SMD:C_0603_1608Metric" (at 101.2952 143.51 0)
+      (effects (font (size 1.27 1.27)) hide)
+    )

Commit message: Progressed ECAD.
Parts:
- renumbered C57 to C61, C58 to C62, C59 to C63, U38 to U39, U39 to U40, U40 to U41

Commit message: Progressed ECAD.
Parts:
- renumbered C61 to C59, C62 to C60, C63 to C61

Commit message: Cleanup and new power supply pcb
Parts:
- renumbered C59 to C53, C60 to C54, C61 to C55, U39 to U36, U40 to U37, U41 to U38

Commit message: Progressed ECAD.
Parts:
- renumbered C53 to C51, C54 to C52, C55 to C53
