File: ECAD/SCART_switcher/power.kicad_sch (KiCad schematic)
At the start: 40 parts, among them SW1 SW_Push_DPDT, U11 L7805, U12 L7809

Commit message: progressed ecad
Parts:
- U? (x6): footprint (none) -> Package_SO:SOIC-8_3.9x4.9mm_P1.27mm; MPN (none) -> RC4580IDR
Changed lines of the file:
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@@
       (effects (font (size 1.27 1.27)))
     )
-    (property "Footprint" "" (at 147.32 153.67 0)
+    (property "Footprint" "Package_SO:SOIC-8_3.9x4.9mm_P1.27mm" (at 147.32 153.67 0)
       (effects (font (size 1.27 1.27)) hide)
     )
-    (property "Datasheet" "https://www.ti.com/lit/ds/symlink/rc4580.pdf" (at 147.32 153.67 0)
+    (property "Datasheet" "https://datasheet.lcsc.com/lcsc/2304140030_Texas-Instruments-RC4580IDR_C80100.pdf" (at 147.32 153.67 0)
+      (effects (font (size 1.27 1.27)) hide)
+    )
+    (property "MPN" "RC4580IDR" (at 147.32 153.67 0)
       (effects (font (size 1.27 1.27)) hide)
     )
@@
       (effects (font (size 1.27 1.27)))
     )
-    (property "Footprint" "" (at 147.32 78.74 0)
+    (property "Footprint" "Package_SO:SOIC-8_3.9x4.9mm_P1.27mm" (at 147.32 78.74 0)
+      (effects (font (size 1.27 1.27)) hide)
+    )
+    (property "Datasheet" "https://datasheet.lcsc.com/lcsc/2304140030_Texas-Instruments-RC4580IDR_C80100.pdf" (at 147.32 78.74 0)
       (effects (font (size 1.27 1.27)) hide)
     )
-    (property "Datasheet" "https://www.ti.com/lit/ds/symlink/rc4580.pdf" (at 147.32 78.74 0)
+    (property "MPN" "RC4580IDR" (at 147.32 78.74 0)
       (effects (font (size 1.27 1.27)) hide)
     )
@@
       (effects (font (size 1.27 1.27)) (justify left))
     )
-    (property "Footprint" "" (at 213.36 88.9 0)
+    (property "Footprint" "Package_SO:SOIC-8_3.9x4.9mm_P1.27mm" (at 213.36 88.9 0)
+      (effects (font (size 1.27 1.27)) hide)
+    )
+    (property "Datasheet" "https://datasheet.lcsc.com/lcsc/2304140030_Texas-Instruments-RC4580IDR_C80100.pdf" (at 213.36 88.9 0)
       (effects (font (size 1.27 1.27)) hide)
     )
-    (property "Datasheet" "https://www.ti.com/lit/ds/symlink/rc4580.pdf" (at 213.36 88.9 0)
+    (property "MPN" "RC4580IDR" (at 213.36 88.9 0)
       (effects (font (size 1.27 1.27)) hide)
     )
@@
       (effects (font (size 1.27 1.27)))
     )
-    (property "Footprint" "" (at 147.32 133.35 0)
+    (property "Footprint" "Package_SO:SOIC-8_3.9x4.9mm_P1.27mm" (at 147.32 133.35 0)
       (effects (font (size 1.27 1.27)) hide)
     )
-    (property "Datasheet" "https://www.ti.com/lit/ds/symlink/rc4580.pdf" (at 147.32 133.35 0)
+    (property "Datasheet" "https://datasheet.lcsc.com/lcsc/2304140030_Texas-Instruments-RC4580IDR_C80100.pdf" (at 147.32 133.35 0)
+      (effects (font (size 1.27 1.27)) hide)
+    )
+    (property "MPN" "RC4580IDR" (at 147.32 133.35 0)
       (effects (font (size 1.27 1.27)) hide)
     )
@@
       (effects (font (size 1.27 1.27)))
     )
-    (property "Footprint" "" (at 147.32 99.06 0)
+    (property "Footprint" "Package_SO:SOIC-8_3.9x4.9mm_P1.27mm" (at 147.32 99.06 0)
+      (effects (font (size 1.27 1.27)) hide)
+    )
+    (property "Datasheet" "https://datasheet.lcsc.com/lcsc/2304140030_Texas-Instruments-RC4580IDR_C80100.pdf" (at 147.32 99.06 0)
       (effects (font (size 1.27 1.27)) hide)
     )
-    (property "Datasheet" "https://www.ti.com/lit/ds/symlink/rc4580.pdf" (at 147.32 99.06 0)
+    (property "MPN" "RC4580IDR" (at 147.32 99.06 0)
       (effects (font (size 1.27 1.27)) hide)
     )
@@
       (effects (font (size 1.27 1.27)) (justify left))
     )
-    (property "Footprint" "" (at 213.36 143.51 0)
+    (property "Footprint" "Package_SO:SOIC-8_3.9x4.9mm_P1.27mm" (at 213.36 143.51 0)
+      (effects (font (size 1.27 1.27)) hide)
+    )
+    (property "Datasheet" "https://datasheet.lcsc.com/lcsc/2304140030_Texas-Instruments-RC4580IDR_C80100.pdf" (at 213.36 143.51 0)
       (effects (font (size 1.27 1.27)) hide)
     )
-    (property "Datasheet" "https://www.ti.com/lit/ds/symlink/rc4580.pdf" (at 213.36 143.51 0)
+    (property "MPN" "RC4580IDR" (at 213.36 143.51 0)
       (effects (font (size 1.27 1.27)) hide)
     )
