File: ECAD/SCART_switcher/power.kicad_sch (KiCad schematic)
At the start: 40 parts, among them SW1 SW_Push_DPDT, U11 L7805, U12 L7809

Commit message: Progressed ECAD.
Parts:
- D22: MPN (none) -> BZX84C10-7-F; Status (none) -> OK
- J?, Q?: Status (none) -> OK
Changed lines of the file:
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@@
       (effects (font (size 1.27 1.27)) hide)
     )
+    (property "Status" "" (at 187.96 149.86 0)
+      (effects (font (size 1.27 1.27)) hide)
+    )
     (pin "1")
     (pin "2")
@@
       (effects (font (size 1.27 1.27)) hide)
     )
+    (property "Status" "" (at 147.32 153.67 0)
+      (effects (font (size 1.27 1.27)) hide)
+    )
     (pin "1")
     (pin "2")
@@
       (effects (font (size 1.27 1.27)) hide)
     )
-    (property "Datasheet" "" (at 76.2 35.306 0)
+    (property "Datasheet" "https://datasheet.lcsc.com/lcsc/2108131730_Korean-Hroparts-Elec-DC-005-20A_C136744.pdf" (at 76.2 35.306 0)
       (effects (font (size 1.27 1.27)) hide)
     )
@@
       (effects (font (size 1.27 1.27)) hide)
     )
+    (property "Status" "OK" (at 74.93 34.29 0)
+      (effects (font (size 1.27 1.27)) hide)
+    )
     (pin "1")
     (pin "2")
@@
       (effects (font (size 1.27 1.27)) hide)
     )
+    (property "Status" "" (at 167.64 36.83 0)
+      (effects (font (size 1.27 1.27)) hide)
+    )
     (pin "1")
     (pin "2")
@@
       (effects (font (size 1.27 1.27)) hide)
     )
+    (property "Status" "" (at 87.63 148.59 0)
+      (effects (font (size 1.27 1.27)) hide)
+    )
     (pin "1")
     (pin "2")
@@
       (effects (font (size 1.27 1.27)) hide)
     )
+    (property "Status" "" (at 147.32 78.74 0)
+      (effects (font (size 1.27 1.27)) hide)
+    )
     (pin "1")
     (pin "2")
@@
       (effects (font (size 1.27 1.27)) hide)
     )
+    (property "Status" "" (at 109.22 148.59 0)
+      (effects (font (size 1.27 1.27)) hide)
+    )
     (pin "2")
     (pin "1")
@@
       (effects (font (size 1.27 1.27)) hide)
     )
+    (property "Status" "" (at 124.46 36.83 0)
+      (effects (font (size 1.27 1.27)) hide)
+    )
     (pin "1")
     (pin "2")
@@
       (effects (font (size 1.27 1.27)) hide)
     )
+    (property "Status" "" (at 162.56 153.67 0)
+      (effects (font (size 1.27 1.27)) hide)
+    )
     (pin "1")
     (pin "2")
@@
       (effects (font (size 1.27 1.27)) hide)
     )
+    (property "Status" "" (at 205.74 36.83 0)
+      (effects (font (size 1.27 1.27)) hide)
+    )
     (pin "1")
     (pin "2")
@@
       (effects (font (size 1.27 1.27)) hide)
     )
+    (property "Status" "" (at 87.63 93.98 0)
+      (effects (font (size 1.27 1.27)) hide)
+    )
     (pin "1")
     (pin "2")
@@
       (effects (font (size 1.27 1.27)) hide)
     )
+    (property "Status" "" (at 109.22 83.82 0)
+      (effects (font (size 1.27 1.27)) hide)
+    )
     (pin "2")
     (pin "1")
@@
       (effects (font (size 1.27 1.27)) hide)
     )
+    (property "Status" "" (at 213.36 88.9 0)
+      (effects (font (size 1.27 1.27)) hide)
+    )
     (pin "1")
     (pin "2")
@@
       (effects (font (size 1.27 1.27)) hide)
     )
+    (property "Status" "" (at 101.6 31.75 0)
+      (effects (font (size 1.27 1.27)) hide)
+    )
     (pin "3")
     (pin "2")
@@
       (effects (font (size 1.27 1.27)) hide)
     )
+    (property "Status" "" (at 54.61 93.98 0)
+      (effects (font (size 1.27 1.27)) hide)
+    )
     (pin "1")
     (pin "2")
@@
       (effects (font (size 1.27 1.27)) hide)
     )
+    (property "Status" "" (at 224.79 143.51 0)
+      (effects (font (size 1.27 1.27)) hide)
+    )
     (pin "1")
     (pin "2")
@@
       (effects (font (size 1.27 1.27)) hide)
     )
+    (property "Status" "" (at 147.32 133.35 0)
+      (effects (font (size 1.27 1.27)) hide)
+    )
     (pin "1")
     (pin "2")
@@
       (effects (font (size 1.27 1.27)) hide)
     )
+    (property "Status" "" (at 162.56 133.35 0)
+      (effects (font (size 1.27 1.27)) hide)
+    )
     (pin "1")
     (pin "2")
@@
       (effects (font (size 1.27 1.27)) hide)
     )
+    (property "Status" "" (at 179.07 31.75 0)
+      (effects (font (size 1.27 1.27)) hide)
+    )
     (pin "1")
     (pin "2")
@@
       (effects (font (size 1.27 1.27)) hide)
     )
+    (property "Status" "" (at 109.22 93.98 0)
+      (effects (font (size 1.27 1.27)) hide)
+    )
     (pin "2")
     (pin "1")
@@
       (effects (font (size 1.27 1.27)) hide)
     )
+    (property "Status" "" (at 250.19 33.02 0)
+      (effects (font (size 1.27 1.27)) hide)
+    )
     (pin "1")
     (pin "2")
@@
       (effects (font (size 1.27 1.27)) hide)
     )
+    (property "Status" "" (at 173.99 149.86 0)
+      (effects (font (size 1.27 1.27)) hide)
+    )
     (pin "1")
     (pin "2")
@@
       (effects (font (size 1.27 1.27)) hide)
     )
+    (property "Status" "" (at 147.32 99.06 0)
+      (effects (font (size 1.27 1.27)) hide)
+    )
     (pin "1")
     (pin "2")
@@
       (effects (font (size 1.27 1.27)) hide)
     )
-    (property "Datasheet" "https://diotec.com/tl_files/diotec/files/pdf/datasheets/bzx84c2v4.pdf" (at 146.05 35.56 0)
+    (property "Datasheet" "https://datasheet.lcsc.com/lcsc/2304140030_Diodes-Incorporated-BZX84C10-7-F_C500793.pdf" (at 146.05 35.56 0)
+      (effects (font (size 1.27 1.27)) hide)
+    )
+    (property "Status" "OK" (at 146.05 35.56 0)
+      (effects (font (size 1.27 1.27)) hide)
+    )
+    (property "MPN" "BZX84C10-7-F" (at 146.05 35.56 0)
       (effects (font (size 1.27 1.27)) hide)
     )
@@
       (effects (font (size 1.27 1.27)) hide)
     )
+    (property "Status" "" (at 162.56 78.74 0)
+      (effects (font (size 1.27 1.27)) hide)
+    )
     (pin "1")
     (pin "2")
@@
       (effects (font (size 1.27 1.27)) hide)
     )
+    (property "Status" "" (at 162.56 99.06 0)
+      (effects (font (size 1.27 1.27)) hide)
+    )
     (pin "1")
     (pin "2")
@@
       (effects (font (size 1.27 1.27)) hide)
     )
+    (property "Status" "" (at 120.65 93.98 0)
+      (effects (font (size 1.27 1.27)) hide)
+    )
     (pin "1")
     (pin "2")
@@
       (effects (font (size 1.27 1.27)) hide)
     )
+    (property "Status" "" (at 71.12 88.9 0)
+      (effects (font (size 1.27 1.27)) hide)
+    )
     (pin "1")
     (pin "2")
@@
       (effects (font (size 1.27 1.27)) hide)
     )
+    (property "Status" "" (at 120.65 148.59 0)
+      (effects (font (size 1.27 1.27)) hide)
+    )
     (pin "1")
     (pin "2")
@@
       (effects (font (size 1.27 1.27)) hide)
     )
+    (property "Status" "" (at 109.22 138.43 0)
+      (effects (font (size 1.27 1.27)) hide)
+    )
     (pin "2")
     (pin "1")
@@
       (effects (font (size 1.27 1.27)) hide)
     )
+    (property "Status" "" (at 224.79 88.9 0)
+      (effects (font (size 1.27 1.27)) hide)
+    )
     (pin "1")
     (pin "2")
@@
       (effects (font (size 1.27 1.27)) hide)
     )
+    (property "Status" "" (at 250.19 40.64 0)
+      (effects (font (size 1.27 1.27)) hide)
+    )
     (pin "1")
     (pin "2")
@@
       (effects (font (size 1.27 1.27)) hide)
     )
+    (property "Status" "OK" (at 140.97 34.29 0)
+      (effects (font (size 1.27 1.27)) hide)
+    )
     (pin "1")
     (pin "2")
@@
       (effects (font (size 1.27 1.27)) hide)
     )
+    (property "Status" "" (at 54.61 148.59 0)
+      (effects (font (size 1.27 1.27)) hide)
+    )
     (pin "1")
     (pin "2")
@@
       (effects (font (size 1.27 1.27)) hide)
     )
+    (property "Status" "" (at 189.23 36.83 0)
+      (effects (font (size 1.27 1.27)) hide)
+    )
     (pin "1")
     (pin "2")
@@
       (effects (font (size 1.27 1.27)) hide)
     )
+    (property "Status" "" (at 213.36 143.51 0)
+      (effects (font (size 1.27 1.27)) hide)
+    )
     (pin "1")
     (pin "2")
@@
       (effects (font (size 1.27 1.27)) hide)
     )
+    (property "Status" "" (at 187.96 95.25 0)
+      (effects (font (size 1.27 1.27)) hide)
+    )
     (pin "1")
     (pin "2")
@@
       (effects (font (size 1.27 1.27)) hide)
     )
+    (property "Status" "" (at 173.99 95.25 0)
+      (effects (font (size 1.27 1.27)) hide)
+    )
     (pin "1")
     (pin "2")
@@
       (effects (font (size 1.27 1.27)) hide)
     )
+    (property "Status" "" (at 71.12 143.51 0)
+      (effects (font (size 1.27 1.27)) hide)
+    )
     (pin "1")
     (pin "2")
@@
       (effects (font (size 1.27 1.27)) hide)
     )
+    (property "Status" "" (at 140.97 43.18 0)
+      (effects (font (size 1.27 1.27)) hide)
+    )

Commit message: Progressed ECAD.
Parts:
- D? (x2), U? (x6): Status (none) -> OK
Changed lines of the file:
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@@
       (effects (font (size 1.27 1.27)) hide)
     )
-    (property "Status" "" (at 147.32 153.67 0)
+    (property "Status" "OK" (at 147.32 153.67 0)
       (effects (font (size 1.27 1.27)) hide)
     )
@@
       (effects (font (size 1.27 1.27)) hide)
     )
-    (property "Status" "" (at 147.32 78.74 0)
+    (property "Status" "OK" (at 147.32 78.74 0)
       (effects (font (size 1.27 1.27)) hide)
     )
@@
       (effects (font (size 1.27 1.27)) hide)
     )
-    (property "Status" "" (at 124.46 36.83 0)
+    (property "Status" "OK" (at 124.46 36.83 0)
       (effects (font (size 1.27 1.27)) hide)
     )
@@
       (effects (font (size 1.27 1.27)) hide)
     )
-    (property "Status" "" (at 213.36 88.9 0)
+    (property "Status" "OK" (at 213.36 88.9 0)
       (effects (font (size 1.27 1.27)) hide)
     )
@@
       (effects (font (size 1.27 1.27)) hide)
     )
-    (property "Status" "" (at 147.32 133.35 0)
+    (property "Status" "OK" (at 147.32 133.35 0)
       (effects (font (size 1.27 1.27)) hide)
     )
@@
       (effects (font (size 1.27 1.27)) hide)
     )
-    (property "Status" "" (at 147.32 99.06 0)
+    (property "Status" "OK" (at 147.32 99.06 0)
       (effects (font (size 1.27 1.27)) hide)
     )
@@
       (effects (font (size 1.27 1.27)) hide)
     )
-    (property "Status" "" (at 250.19 40.64 0)
+    (property "Status" "OK" (at 250.19 40.64 0)
       (effects (font (size 1.27 1.27)) hide)
     )
@@
       (effects (font (size 1.27 1.27)) hide)
     )
-    (property "Status" "" (at 213.36 143.51 0)
+    (property "Status" "OK" (at 213.36 143.51 0)
       (effects (font (size 1.27 1.27)) hide)
     )

Commit message: Progressed ECAD.
Parts:
- SW1: footprint (none) -> Button_Switch_THT_custom:PN22SJNA03QE; MPN (none) -> PS-22E05; Status (none) -> OK
Connections:
- net at D?.2 (A2), Q?.5 (D), Q?.6 (D)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: now also SW1.1 (A), SW1.4 (A); no longer SW1.3 (C), SW1.6 (C)
Changed lines of the file:
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@@
   (junction (at 189.23 31.75) (diameter 0) (color 0 0 0 0)
   )
+  (junction (at 107.95 31.75) (diameter 0) (color 0 0 0 0)
+  )
   (junction (at 156.21 133.35) (diameter 0) (color 0 0 0 0)
   )
@@
   (junction (at 156.21 153.67) (diameter 0) (color 0 0 0 0)
   )
-  (junction (at 107.95 31.75) (diameter 0) (color 0 0 0 0)
-  )
   (junction (at 120.65 88.9) (diameter 0) (color 0 0 0 0)
   )
@@
   (junction (at 146.05 31.75) (diameter 0) (color 0 0 0 0)
   )
-  (no_connect (at 106.68 24.13))
-  (no_connect (at 106.68 34.29))
+  (no_connect (at 106.68 29.21))
+  (no_connect (at 106.68 39.37))
   (wire (pts (xy 82.55 36.83) (xy 83.82 36.83))
     (stroke (width 0) (type default))
@@
     (stroke (width 0) (type default))
   )
+  (wire (pts (xy 106.68 24.13) (xy 107.95 24.13))
+    (stroke (width 0) (type default))
+  )
   (wire (pts (xy 173.99 146.05) (xy 173.99 143.51))
     (stroke (width 0) (type default))
@@
     (stroke (width 0) (type default))
   )
+  (wire (pts (xy 106.68 34.29) (xy 107.95 34.29))
+    (stroke (width 0) (type default))
+  )
   (wire (pts (xy 133.35 88.9) (xy 133.35 81.28))
     (stroke (width 0) (type default))
@@
     (stroke (width 0) (type default))
   )
-  (wire (pts (xy 107.95 39.37) (xy 106.68 39.37))
-    (stroke (width 0) (type default))
-  )
   (wire (pts (xy 154.94 99.06) (xy 156.21 99.06))
     (stroke (width 0) (type default))
@@
     (stroke (width 0) (type default))
   )
-  (wire (pts (xy 107.95 31.75) (xy 107.95 39.37))
-    (stroke (width 0) (type default))
-  )
   (wire (pts (xy 140.97 39.37) (xy 146.05 39.37))
     (stroke (width 0) (type default))
@@
     (stroke (width 0) (type default))
   )
-  (wire (pts (xy 107.95 29.21) (xy 107.95 31.75))
+  (wire (pts (xy 107.95 24.13) (xy 107.95 31.75))
     (stroke (width 0) (type default))
   )
@@
     (stroke (width 0) (type default))
   )
-  (wire (pts (xy 106.68 29.21) (xy 107.95 29.21))
+  (wire (pts (xy 107.95 34.29) (xy 107.95 31.75))
     (stroke (width 0) (type default))
   )
@@
       (effects (font (size 1.27 1.27)))
     )
-    (property "Footprint" "" (at 101.6 26.67 0)
-      (effects (font (size 1.27 1.27)) hide)
-    )
-    (property "Datasheet" "~" (at 101.6 26.67 0)
-      (effects (font (size 1.27 1.27)) hide)
-    )
-    (property "Status" "" (at 101.6 31.75 0)
-      (effects (font (size 1.27 1.27)) hide)
-    )
+    (property "Footprint" "Button_Switch_THT_custom:PN22SJNA03QE" (at 101.6 26.67 0)
+      (effects (font (size 1.27 1.27)) hide)
+    )
+    (property "Datasheet" "https://datasheet.lcsc.com/lcsc/2108301530_G-Switch-PS-22E05_C2848949.pdf" (at 101.6 26.67 0)
+      (effects (font (size 1.27 1.27)) hide)
+    )
+    (property "Status" "OK" (at 101.6 31.75 0)
+      (effects (font (size 1.27 1.27)) hide)
+    )
+    (property "MPN" "PS-22E05" (at 101.6 31.75 0)
+      (effects (font (size 1.27 1.27)) hide)
+    )

Commit message: Progressed ECAD.
Parts:
- C? (x2): footprint (none) -> Capacitor_SMD:CP_Elec_6.3x5.4; MPN (none) -> UWX1H100MCL1GB; Status (none) -> OK
Changed lines of the file:
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@@
       (effects (font (size 1.27 1.27)) (justify right))
     )
-    (property "Footprint" "" (at 186.9948 146.05 0)
+    (property "Footprint" "Capacitor_SMD:CP_Elec_6.3x5.4" (at 186.9948 146.05 0)
       (effects (font (size 1.27 1.27)) hide)
     )
-    (property "Datasheet" "~" (at 187.96 149.86 0)
+    (property "Datasheet" "https://datasheet.lcsc.com/lcsc/2304140030_Nichicon-UWX1H100MCL1GB_C134237.pdf" (at 187.96 149.86 0)
       (effects (font (size 1.27 1.27)) hide)
     )
-    (property "Status" "" (at 187.96 149.86 0)
+    (property "Status" "OK" (at 187.96 149.86 0)
+      (effects (font (size 1.27 1.27)) hide)
+    )
+    (property "MPN" "UWX1H100MCL1GB" (at 187.96 149.86 0)
       (effects (font (size 1.27 1.27)) hide)
     )
@@
       (effects (font (size 1.27 1.27)) (justify right))
     )
-    (property "Footprint" "" (at 186.9948 91.44 0)
+    (property "Footprint" "Capacitor_SMD:CP_Elec_6.3x5.4" (at 186.9948 91.44 0)
+      (effects (font (size 1.27 1.27)) hide)
+    )
+    (property "Datasheet" "https://datasheet.lcsc.com/lcsc/2304140030_Nichicon-UWX1H100MCL1GB_C134237.pdf" (at 187.96 95.25 0)
       (effects (font (size 1.27 1.27)) hide)
     )
-    (property "Datasheet" "~" (at 187.96 95.25 0)
+    (property "Status" "OK" (at 187.96 95.25 0)
       (effects (font (size 1.27 1.27)) hide)
     )
-    (property "Status" "" (at 187.96 95.25 0)
+    (property "MPN" "UWX1H100MCL1GB" (at 187.96 95.25 0)
       (effects (font (size 1.27 1.27)) hide)
     )

Commit message: Error fix.
Parts:
- removed C? (x2): 10uC, Capacitor_SMD:CP_Elec_6.3x5.4, symbol Device:C
- added C? (x2): 10uC, Capacitor_SMD:CP_Elec_6.3x5.4, symbol Device:C_Polarized
Connections:
- net +2V5: now also C?.1
- net +4V5: now also C?.1
- net GND: now also C?.2, C?.2
Changed lines of the file:
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@@
     (effects (font (size 1.27 1.27)) (justify left bottom))
   )
-  (symbol (lib_id "Device:C") (at 187.96 149.86 180) (unit 1)
-    (in_bom yes) (on_board yes) (dnp no) (fields_autoplaced)
-    (property "Reference" "C?" (at 191.77 148.59 0)
-      (effects (font (size 1.27 1.27)) (justify right))
-    )
-    (property "Value" "10uC" (at 191.77 151.13 0)
-      (effects (font (size 1.27 1.27)) (justify right))
-    )
-    (property "Footprint" "Capacitor_SMD:CP_Elec_6.3x5.4" (at 186.9948 146.05 0)
-      (effects (font (size 1.27 1.27)) hide)
-    )
-    (property "Datasheet" "https://datasheet.lcsc.com/lcsc/2304140030_Nichicon-UWX1H100MCL1GB_C134237.pdf" (at 187.96 149.86 0)
-      (effects (font (size 1.27 1.27)) hide)
-    )
-    (property "Status" "OK" (at 187.96 149.86 0)
-      (effects (font (size 1.27 1.27)) hide)
-    )
-    (property "MPN" "UWX1H100MCL1GB" (at 187.96 149.86 0)
-      (effects (font (size 1.27 1.27)) hide)
-    )
-    (pin "1")
-    (pin "2")
-    (instances
-      (project "SCART_switcher"
-        (path "/8cd08eb5-4755-4ef5-8eeb-77fd9974b180/6562ea38-5963-42b2-a0ef-a4a12a4c652f/9f74dfb2-70cd-470e-9dfb-02936b5bb451"
-          (reference "C?") (unit 1)
-        )
-        (path "/8cd08eb5-4755-4ef5-8eeb-77fd9974b180/19b1c794-1d68-480b-a4cd-c99f5e9ef1e6"
-          (reference "C21") (unit 1)
-        )
-      )
-    )
-  )
   (symbol (lib_id "power:GND") (at 205.74 40.64 0) (unit 1)
     (in_bom yes) (on_board yes) (dnp no) (fields_autoplaced)
@@
     )
   )
+  (symbol (lib_id "Device:C_Polarized") (at 187.96 149.86 0) (unit 1)
+    (in_bom yes) (on_board yes) (dnp no) (fields_autoplaced)
+    (property "Reference" "C?" (at 191.77 147.701 0)
+      (effects (font (size 1.27 1.27)) (justify left))
+    )
+    (property "Value" "10uC" (at 191.77 150.241 0)
+      (effects (font (size 1.27 1.27)) (justify left))
+    )
+    (property "Footprint" "Capacitor_SMD:CP_Elec_6.3x5.4" (at 188.9252 153.67 0)
+      (effects (font (size 1.27 1.27)) hide)
+    )
+    (property "Datasheet" "https://datasheet.lcsc.com/lcsc/2304140030_Nichicon-UWX1H100MCL1GB_C134237.pdf" (at 187.96 149.86 0)
+      (effects (font (size 1.27 1.27)) hide)
+    )
+    (property "MPN" "UWX1H100MCL1GB" (at 187.96 149.86 0)
+      (effects (font (size 1.27 1.27)) hide)
+    )
+    (property "Status" "OK" (at 187.96 149.86 0)
+      (effects (font (size 1.27 1.27)) hide)
+    )
+    (pin "2")
+    (pin "1")
+    (instances
+      (project "SCART_switcher"
+        (path "/8cd08eb5-4755-4ef5-8eeb-77fd9974b180/6562ea38-5963-42b2-a0ef-a4a12a4c652f/9f74dfb2-70cd-470e-9dfb-02936b5bb451"
+          (reference "C?") (unit 1)
+        )
+        (path "/8cd08eb5-4755-4ef5-8eeb-77fd9974b180/19b1c794-1d68-480b-a4cd-c99f5e9ef1e6"
+          (reference "C21") (unit 1)
+        )
+      )
+    )
+  )
   (symbol (lib_id "power:GND") (at 173.99 99.06 0) (unit 1)
     (in_bom yes) (on_board yes) (dnp no) (fields_autoplaced)
@@
     )
   )
+  (symbol (lib_id "Device:C_Polarized") (at 187.96 95.25 0) (unit 1)
+    (in_bom yes) (on_board yes) (dnp no) (fields_autoplaced)
+    (property "Reference" "C?" (at 191.77 93.091 0)
+      (effects (font (size 1.27 1.27)) (justify left))
+    )
+    (property "Value" "10uC" (at 191.77 95.631 0)
+      (effects (font (size 1.27 1.27)) (justify left))
+    )
+    (property "Footprint" "Capacitor_SMD:CP_Elec_6.3x5.4" (at 188.9252 99.06 0)
+      (effects (font (size 1.27 1.27)) hide)
+    )
+    (property "Datasheet" "https://datasheet.lcsc.com/lcsc/2304140030_Nichicon-UWX1H100MCL1GB_C134237.pdf" (at 187.96 95.25 0)
+      (effects (font (size 1.27 1.27)) hide)
+    )
+    (property "MPN" "UWX1H100MCL1GB" (at 187.96 95.25 0)
+      (effects (font (size 1.27 1.27)) hide)
+    )
+    (property "Status" "OK" (at 187.96 95.25 0)
+      (effects (font (size 1.27 1.27)) hide)
+    )
+    (pin "2")
+    (pin "1")
+    (instances
+      (project "SCART_switcher"
+        (path "/8cd08eb5-4755-4ef5-8eeb-77fd9974b180/6562ea38-5963-42b2-a0ef-a4a12a4c652f/9f74dfb2-70cd-470e-9dfb-02936b5bb451"
+          (reference "C?") (unit 1)
+        )
+        (path "/8cd08eb5-4755-4ef5-8eeb-77fd9974b180/19b1c794-1d68-480b-a4cd-c99f5e9ef1e6"
+          (reference "C20") (unit 1)
+        )
+      )
+    )
+  )
   (symbol (lib_id "Diode:BZX84Cxx") (at 146.05 35.56 270) (unit 1)
     (in_bom yes) (on_board yes) (dnp no) (fields_autoplaced)
@@
         )
       )
-    )
-  )
-  (symbol (lib_id "Device:C") (at 187.96 95.25 180) (unit 1)
-    (in_bom yes) (on_board yes) (dnp no) (fields_autoplaced)
-    (property "Reference" "C?" (at 191.77 93.98 0)
-      (effects (font (size 1.27 1.27)) (justify right))
-    )
-    (property "Value" "10uC" (at 191.77 96.52 0)
-      (effects (font (size 1.27 1.27)) (justify right))
-    )
-    (property "Footprint" "Capacitor_SMD:CP_Elec_6.3x5.4" (at 186.9948 91.44 0)
-      (effects (font (size 1.27 1.27)) hide)
-    )
-    (property "Datasheet" "https://datasheet.lcsc.com/lcsc/2304140030_Nichicon-UWX1H100MCL1GB_C134237.pdf" (at 187.96 95.25 0)
-      (effects (font (size 1.27 1.27)) hide)
-    )
-    (property "Status" "OK" (at 187.96 95.25 0)
-      (effects (font (size 1.27 1.27)) hide)
-    )
-    (property "MPN" "UWX1H100MCL1GB" (at 187.96 95.25 0)
-      (effects (font (size 1.27 1.27)) hide)
-    )
-    (pin "1")
-    (pin "2")
-    (instances
-      (project "SCART_switcher"
-        (path "/8cd08eb5-4755-4ef5-8eeb-77fd9974b180/6562ea38-5963-42b2-a0ef-a4a12a4c652f/9f74dfb2-70cd-470e-9dfb-02936b5bb451"
-          (reference "C?") (unit 1)
-        )
-        (path "/8cd08eb5-4755-4ef5-8eeb-77fd9974b180/19b1c794-1d68-480b-a4cd-c99f5e9ef1e6"
-          (reference "C20") (unit 1)
-        )
-      )

Commit message: Progressed ECAD.
Parts:
- removed C? (x2): 100nC, Capacitor_SMD:C_0805_2012Metric, symbol Device:C
- removed C?: 220uC, Capacitor_THT:CP_Radial_D8.0mm_P3.50mm, symbol Device:C_Polarized
- removed FB?: FerriteBead, Inductor_SMD:L_1806_4516Metric, symbol Device:FerriteBead
Connections:
- net +12V: now also D22.3 (K), Q?.1 (S), Q?.2 (S), Q?.3 (S)
Other:
- note removed: "Power supply line filter (PI filter)"

Commit message: Progressed ECAD.
Parts:
- gave numbers to parts that had none: 18

Commit message: Progressed ECAD
Parts:
- removed Q?: DMP3037LSS-13, Package_SO:SOIC-8_3.9x4.9mm_P1.27mm, symbol Transistor_FET:IRF7404
- added Q24: DMP3037LSS-13, Package_SO:SOIC-8_3.9x4.9mm_P1.27mm, symbol Transistor_FET:IRF7404
- renumbered C13 to C19, C14 to C20, C17 to C23, C18 to C24, C19 to C25, C20 to C26, C21 to C27, C22 to C28, R56 to R64, R57 to R65, R58 to R66, R59 to R67, R61 to R69, R62 to R70, R63 to R71, R64 to R72, U11 to U17, U12 to U18, U13 to U19, U14 to U20
Connections:
- net +12V: now also Q24.1 (S), Q24.2 (S), Q24.3 (S)
- net at D?.2 (A2), SW1.1 (A), SW1.4 (A): now also Q24.5 (D), Q24.6 (D), Q24.7 (D), Q24.8 (D)
- net at D22.1 (A), R?.1: now also Q24.4 (G)
