File: ECAD/SCART_switcher/power.kicad_sch (KiCad schematic)
At the start: 17 parts, among them J14 Conn_01x06, U29 LM4041LP-ADJ, U30 LM4041LP-ADJ

Commit message: Progressed ECAD.
Parts:
- removed R70: 10kR, Resistor_SMD:R_0805_2012Metric, symbol Device:R
- added R68, R73: 1kR, Resistor_SMD:R_0805_2012Metric, symbol Device:R
- added R72: 379R, Resistor_SMD:R_0805_2012Metric, symbol Device:R
- R64, R67: value 10kR -> 976R; MPN RC0805FR-0710KL -> (none)
- R65: value 10kR -> 1kR; MPN RC0805FR-0710KL -> (none)
- R66: value 10kR -> 379R; MPN RC0805FR-0710KL -> (none)
- R69: renamed from R68; value 10kR -> 379R; MPN RC0805FR-0710KL -> (none)
- R70: renamed from R69; value 10kR -> 1kR; MPN RC0805FR-0710KL -> (none)
- R71: value 10kR -> 100R; MPN RC0805FR-0710KL -> (none)
Connections:
- net +2V5: now also R68.1
- net +4V5: now also R72.2, R73.1; no longer R71.2
- net +9V: now also R71.1
- net GND: now also R68.2, R73.2
- net at C32.1: now also R71.2, R72.1; no longer R71.1
Other:
- moved on the sheet: C29, C32

Commit message: Update power.kicad_sch
Parts:
- J14: footprint (none) -> Connector_PinSocket_2.54mm:PinSocket_1x06_P2.54mm_Horizontal
Changed lines of the file:
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@@
       (effects (font (size 1.27 1.27)) (justify left))
     )
-    (property "Footprint" "" (at 77.47 161.29 0)
+    (property "Footprint" "Connector_PinSocket_2.54mm:PinSocket_1x06_P2.54mm_Horizontal" (at 77.47 161.29 0)
       (effects (font (size 1.27 1.27)) hide)
     )

Commit message: Progressed ECAD.
Parts:
- J14: MPN (none) -> PM254-1-06-W-8.5; Status (none) -> OK
Changed lines of the file:
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@@
       (effects (font (size 1.27 1.27)) hide)
     )
-    (property "Datasheet" "~" (at 77.47 161.29 0)
+    (property "Datasheet" "https://datasheet.lcsc.com/lcsc/2306091006_HCTL-PM254-1-06-W-8-5_C2897388.pdf" (at 77.47 161.29 0)
       (effects (font (size 1.27 1.27)) hide)
     )
+    (property "MPN" "PM254-1-06-W-8.5" (at 77.47 161.29 0)
+      (effects (font (size 1.27 1.27)) hide)
+    )
+    (property "Status" "OK" (at 77.47 161.29 0)
+      (effects (font (size 1.27 1.27)) hide)
+    )

Commit message: Progressed ECAD.
Parts:
- C30, C33: MPN CL21B104KBCNNNC -> CL10B104KO8NNNC; Status (none) -> OK
- R64, R67: MPN (none) -> RT0805BRD07976RL; Status (none) -> OK
- R65, R68, R70, R73: MPN (none) -> RT0805BRD071KL; Status (none) -> OK
- R66, R69, R72: MPN (none) -> PTFR0805B374RP9; Status (none) -> OK
- R71: MPN (none) -> RT0805BRD07100RL; Status (none) -> OK
Changed lines of the file:
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@@
       (effects (font (size 1.27 1.27)) hide)
     )
-    (property "Datasheet" "" (at 74.93 93.98 0)
-      (effects (font (size 1.27 1.27)) hide)
-    )
-    (property "MPN" "" (at 74.93 93.98 0)
-      (effects (font (size 1.27 1.27)) hide)
-    )
-    (property "Status" "" (at 74.93 93.98 0)
+    (property "Datasheet" "https://datasheet.lcsc.com/lcsc/2304140030_YAGEO-RT0805BRD071KL_C110774.pdf" (at 74.93 93.98 0)
+      (effects (font (size 1.27 1.27)) hide)
+    )
+    (property "MPN" "RT0805BRD071KL" (at 74.93 93.98 0)
+      (effects (font (size 1.27 1.27)) hide)
+    )
+    (property "Status" "OK" (at 74.93 93.98 0)
       (effects (font (size 1.27 1.27)) hide)
     )
@@
       (effects (font (size 1.27 1.27)) hide)
     )
-    (property "Datasheet" "" (at 81.28 63.5 0)
-      (effects (font (size 1.27 1.27)) hide)
-    )
-    (property "MPN" "" (at 81.28 63.5 0)
-      (effects (font (size 1.27 1.27)) hide)
-    )
-    (property "Status" "" (at 81.28 63.5 0)
+    (property "Datasheet" "https://datasheet.lcsc.com/lcsc/2310201549_RESI-PTFR0805B374RP9_C2849198.pdf" (at 81.28 63.5 0)
+      (effects (font (size 1.27 1.27)) hide)
+    )
+    (property "MPN" "PTFR0805B374RP9" (at 81.28 63.5 0)
+      (effects (font (size 1.27 1.27)) hide)
+    )
+    (property "Status" "OK" (at 81.28 63.5 0)
       (effects (font (size 1.27 1.27)) hide)
     )
@@
       (effects (font (size 1.27 1.27)) hide)
     )
-    (property "Datasheet" "https://datasheet.lcsc.com/lcsc/1810191215_Samsung-Electro-Mechanics-CL21B104KBCNNNC_C1711.pdf" (at 102.87 88.9 0)
-      (effects (font (size 1.27 1.27)) hide)
-    )
-    (property "MPN" "CL21B104KBCNNNC" (at 102.87 88.9 0)
-      (effects (font (size 1.27 1.27)) hide)
-    )
-    (property "Status" "" (at 102.87 88.9 0)
+    (property "Datasheet" "https://datasheet.lcsc.com/lcsc/1810271710_Samsung-Electro-Mechanics-CL10B104KO8NNNC_C66501.pdf" (at 102.87 88.9 0)
+      (effects (font (size 1.27 1.27)) hide)
+    )
+    (property "MPN" "CL10B104KO8NNNC" (at 102.87 88.9 0)
+      (effects (font (size 1.27 1.27)) hide)
+    )
+    (property "Status" "OK" (at 102.87 88.9 0)
       (effects (font (size 1.27 1.27)) hide)
     )
@@
       (effects (font (size 1.27 1.27)) hide)
     )
-    (property "Datasheet" "https://datasheet.lcsc.com/lcsc/1810191215_Samsung-Electro-Mechanics-CL21B104KBCNNNC_C1711.pdf" (at 217.17 88.9 0)
-      (effects (font (size 1.27 1.27)) hide)
-    )
-    (property "MPN" "CL21B104KBCNNNC" (at 217.17 88.9 0)
-      (effects (font (size 1.27 1.27)) hide)
-    )
-    (property "Status" "" (at 217.17 88.9 0)
+    (property "Datasheet" "https://datasheet.lcsc.com/lcsc/1810271710_Samsung-Electro-Mechanics-CL10B104KO8NNNC_C66501.pdf" (at 217.17 88.9 0)
+      (effects (font (size 1.27 1.27)) hide)
+    )
+    (property "MPN" "CL10B104KO8NNNC" (at 217.17 88.9 0)
+      (effects (font (size 1.27 1.27)) hide)
+    )
+    (property "Status" "OK" (at 217.17 88.9 0)
       (effects (font (size 1.27 1.27)) hide)
     )
@@
       (effects (font (size 1.27 1.27)) hide)
     )
-    (property "Datasheet" "" (at 195.58 73.66 0)
-      (effects (font (size 1.27 1.27)) hide)
-    )
-    (property "MPN" "" (at 195.58 73.66 0)
-      (effects (font (size 1.27 1.27)) hide)
-    )
-    (property "Status" "" (at 195.58 73.66 0)
+    (property "Datasheet" "https://datasheet.lcsc.com/lcsc/2310201549_RESI-PTFR0805B374RP9_C2849198.pdf" (at 195.58 73.66 0)
+      (effects (font (size 1.27 1.27)) hide)
+    )
+    (property "MPN" "PTFR0805B374RP9" (at 195.58 73.66 0)
+      (effects (font (size 1.27 1.27)) hide)
+    )
+    (property "Status" "OK" (at 195.58 73.66 0)
       (effects (font (size 1.27 1.27)) hide)
     )
@@
       (effects (font (size 1.27 1.27)) hide)
     )
-    (property "Datasheet" "" (at 195.58 63.5 0)
-      (effects (font (size 1.27 1.27)) hide)
-    )
-    (property "MPN" "" (at 195.58 63.5 0)
-      (effects (font (size 1.27 1.27)) hide)
-    )
-    (property "Status" "" (at 195.58 63.5 0)
+    (property "Datasheet" "https://datasheet.lcsc.com/lcsc/2304140030_YAGEO-RT0805BRD07100RL_C110773.pdf" (at 195.58 63.5 0)
+      (effects (font (size 1.27 1.27)) hide)
+    )
+    (property "MPN" "RT0805BRD07100RL" (at 195.58 63.5 0)
+      (effects (font (size 1.27 1.27)) hide)
+    )
+    (property "Status" "OK" (at 195.58 63.5 0)
       (effects (font (size 1.27 1.27)) hide)
     )
@@
       (effects (font (size 1.27 1.27)) hide)
     )
-    (property "Datasheet" "" (at 189.23 93.98 0)
-      (effects (font (size 1.27 1.27)) hide)
-    )
-    (property "MPN" "" (at 189.23 93.98 0)
-      (effects (font (size 1.27 1.27)) hide)
-    )
-    (property "Status" "" (at 189.23 93.98 0)
+    (property "Datasheet" "https://datasheet.lcsc.com/lcsc/2304140030_YAGEO-RT0805BRD071KL_C110774.pdf" (at 189.23 93.98 0)
+      (effects (font (size 1.27 1.27)) hide)
+    )
+    (property "MPN" "RT0805BRD071KL" (at 189.23 93.98 0)
+      (effects (font (size 1.27 1.27)) hide)
+    )
+    (property "Status" "OK" (at 189.23 93.98 0)
       (effects (font (size 1.27 1.27)) hide)
     )
@@
       (effects (font (size 1.27 1.27)) hide)
     )
-    (property "Datasheet" "" (at 74.93 83.82 0)
-      (effects (font (size 1.27 1.27)) hide)
-    )
-    (property "MPN" "" (at 74.93 83.82 0)
-      (effects (font (size 1.27 1.27)) hide)
-    )
-    (property "Status" "" (at 74.93 83.82 0)
+    (property "Datasheet" "https://datasheet.lcsc.com/lcsc/2311211102_YAGEO-RT0805BRD07976RL_C865714.pdf" (at 74.93 83.82 0)
+      (effects (font (size 1.27 1.27)) hide)
+    )
+    (property "MPN" "RT0805BRD07976RL" (at 74.93 83.82 0)
+      (effects (font (size 1.27 1.27)) hide)
+    )
+    (property "Status" "OK" (at 74.93 83.82 0)
       (effects (font (size 1.27 1.27)) hide)
     )
@@
       (effects (font (size 1.27 1.27)) hide)
     )
-    (property "Datasheet" "" (at 138.43 86.36 0)
-      (effects (font (size 1.27 1.27)) hide)
-    )
-    (property "MPN" "" (at 138.43 86.36 0)
-      (effects (font (size 1.27 1.27)) hide)
-    )
-    (property "Status" "" (at 138.43 86.36 0)
+    (property "Datasheet" "https://datasheet.lcsc.com/lcsc/2304140030_YAGEO-RT0805BRD071KL_C110774.pdf" (at 138.43 86.36 0)
+      (effects (font (size 1.27 1.27)) hide)
+    )
+    (property "MPN" "RT0805BRD071KL" (at 138.43 86.36 0)
+      (effects (font (size 1.27 1.27)) hide)
+    )
+    (property "Status" "OK" (at 138.43 86.36 0)
       (effects (font (size 1.27 1.27)) hide)
     )
@@
       (effects (font (size 1.27 1.27)) hide)
     )
-    (property "Datasheet" "" (at 81.28 73.66 0)
-      (effects (font (size 1.27 1.27)) hide)
-    )
-    (property "MPN" "" (at 81.28 73.66 0)
-      (effects (font (size 1.27 1.27)) hide)
-    )
-    (property "Status" "" (at 81.28 73.66 0)
+    (property "Datasheet" "https://datasheet.lcsc.com/lcsc/2311211102_YAGEO-RT0805BRD07976RL_C865714.pdf" (at 81.28 73.66 0)
+      (effects (font (size 1.27 1.27)) hide)
+    )
+    (property "MPN" "RT0805BRD07976RL" (at 81.28 73.66 0)
+      (effects (font (size 1.27 1.27)) hide)
+    )
+    (property "Status" "OK" (at 81.28 73.66 0)
       (effects (font (size 1.27 1.27)) hide)
     )
@@
       (effects (font (size 1.27 1.27)) hide)
     )
-    (property "Datasheet" "" (at 189.23 83.82 0)
-      (effects (font (size 1.27 1.27)) hide)
-    )
-    (property "MPN" "" (at 189.23 83.82 0)
-      (effects (font (size 1.27 1.27)) hide)
-    )
-    (property "Status" "" (at 189.23 83.82 0)
+    (property "Datasheet" "https://datasheet.lcsc.com/lcsc/2310201549_RESI-PTFR0805B374RP9_C2849198.pdf" (at 189.23 83.82 0)
+      (effects (font (size 1.27 1.27)) hide)
+    )
+    (property "MPN" "PTFR0805B374RP9" (at 189.23 83.82 0)
+      (effects (font (size 1.27 1.27)) hide)
+    )
+    (property "Status" "OK" (at 189.23 83.82 0)
       (effects (font (size 1.27 1.27)) hide)
     )
@@
       (effects (font (size 1.27 1.27)) hide)
     )
-    (property "Datasheet" "" (at 251.46 86.36 0)
-      (effects (font (size 1.27 1.27)) hide)
-    )
-    (property "MPN" "" (at 251.46 86.36 0)
-      (effects (font (size 1.27 1.27)) hide)
-    )
-    (property "Status" "" (at 251.46 86.36 0)
-      (effects (font (size 1.27 1.27)) hide)
-    )
+    (property "Datasheet" "https://datasheet.lcsc.com/lcsc/2304140030_YAGEO-RT0805BRD071KL_C110774.pdf" (at 251.46 86.36 0)
+      (effects (font (size 1.27 1.27)) hide)
+    )
+    (property "MPN" "RT0805BRD071KL" (at 251.46 86.36 0)
+      (effects (font (size 1.27 1.27)) hide)
+    )
+    (property "Status" "OK" (at 251.46 86.36 0)
+      (effects (font (size 1.27 1.27)) hide)
+    )

Commit message: Progressed ECAD.
Parts:
- U29, U30: MPN_MOUSER (none) -> LM4041DIDBZT

Commit message: Progressed ECAD.
Parts:
- R64, R65, R67, R68, R70, R73: R % tol (none) -> 0.1%; R pwr (none) -> 125mW
- R66, R69, R72: value 379R -> 374R; R % tol (none) -> 0.1%; R pwr (none) -> 130mW
- R71: MPN RT0805BRD07100RL -> RT0805FRD07100RL; R % tol (none) -> 1%; R pwr (none) -> 125mW
Changed lines of the file:
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@@
+      (effects (font (size 1.27 1.27)) hide)
+    )
+    (property "R % tol" "" (at 195.58 88.9 0)
+      (effects (font (size 1.27 1.27)) hide)
+    )
+    (property "R pwr" "" (at 195.58 88.9 0)
       (effects (font (size 1.27 1.27)) hide)
     )
@@
       (effects (font (size 1.27 1.27)) hide)
     )
+    (property "R % tol" "0.1%" (at 74.93 93.98 0)
+      (effects (font (size 1.27 1.27)) hide)
+    )
+    (property "R pwr" "125mW" (at 74.93 93.98 0)
+      (effects (font (size 1.27 1.27)) hide)
+    )
     (pin "2")
     (pin "1")
@@
       (effects (font (size 1.27 1.27)) (justify left))
     )
-    (property "Value" "379R" (at 83.82 64.77 0)
+    (property "Value" "374R" (at 83.82 64.77 0)
       (effects (font (size 1.27 1.27)) (justify left))
     )
@@
       (effects (font (size 1.27 1.27)) hide)
     )
+    (property "R % tol" "0.1%" (at 81.28 63.5 0)
+      (effects (font (size 1.27 1.27)) hide)
+    )
+    (property "R pwr" "130mW " (at 81.28 63.5 0)
+      (effects (font (size 1.27 1.27)) hide)
+    )
     (pin "2")
     (pin "1")
@@
     )
     (property "MPN_MOUSER" "" (at 102.87 88.9 0)
+      (effects (font (size 1.27 1.27)) hide)
+    )
+    (property "R % tol" "" (at 102.87 88.9 0)
+      (effects (font (size 1.27 1.27)) hide)
+    )
+    (property "R pwr" "" (at 102.87 88.9 0)
       (effects (font (size 1.27 1.27)) hide)
     )
@@
       (effects (font (size 1.27 1.27)) hide)
     )
+    (property "R % tol" "" (at 175.26 73.66 0)
+      (effects (font (size 1.27 1.27)) hide)
+    )
+    (property "R pwr" "" (at 175.26 73.66 0)
+      (effects (font (size 1.27 1.27)) hide)
+    )
     (pin "2")
     (pin "1")
@@
       (effects (font (size 1.27 1.27)) hide)
     )
+    (property "R % tol" "" (at 217.17 88.9 0)
+      (effects (font (size 1.27 1.27)) hide)
+    )
+    (property "R pwr" "" (at 217.17 88.9 0)
+      (effects (font (size 1.27 1.27)) hide)
+    )
     (pin "1")
     (pin "2")
@@
       (effects (font (size 1.27 1.27)) (justify left))
     )
-    (property "Value" "379R" (at 198.12 74.93 0)
+    (property "Value" "374R" (at 198.12 74.93 0)
       (effects (font (size 1.27 1.27)) (justify left))
     )
@@
       (effects (font (size 1.27 1.27)) hide)
     )
+    (property "R % tol" "0.1%" (at 195.58 73.66 0)
+      (effects (font (size 1.27 1.27)) hide)
+    )
+    (property "R pwr" "130mW " (at 195.58 73.66 0)
+      (effects (font (size 1.27 1.27)) hide)
+    )
     (pin "2")
     (pin "1")
@@
       (effects (font (size 1.27 1.27)) hide)
     )
+    (property "R % tol" "" (at 231.14 88.9 0)
+      (effects (font (size 1.27 1.27)) hide)
+    )
+    (property "R pwr" "" (at 231.14 88.9 0)
+      (effects (font (size 1.27 1.27)) hide)
+    )
     (pin "2")
     (pin "1")
@@
       (effects (font (size 1.27 1.27)) hide)
     )
-    (property "Datasheet" "https://datasheet.lcsc.com/lcsc/2304140030_YAGEO-RT0805BRD07100RL_C110773.pdf" (at 195.58 63.5 0)
-      (effects (font (size 1.27 1.27)) hide)
-    )
-    (property "MPN" "RT0805BRD07100RL" (at 195.58 63.5 0)
+    (property "Datasheet" "https://datasheet.lcsc.com/lcsc/2304140030_YAGEO-RT0805FRD07100RL_C143843.pdf" (at 195.58 63.5 0)
+      (effects (font (size 1.27 1.27)) hide)
+    )
+    (property "MPN" "RT0805FRD07100RL" (at 195.58 63.5 0)
       (effects (font (size 1.27 1.27)) hide)
     )
@@
     )
     (property "MPN_MOUSER" "" (at 195.58 63.5 0)
+      (effects (font (size 1.27 1.27)) hide)
+    )
+    (property "R % tol" "1%" (at 195.58 63.5 0)
+      (effects (font (size 1.27 1.27)) hide)
+    )
+    (property "R pwr" "125mW" (at 195.58 63.5 0)
       (effects (font (size 1.27 1.27)) hide)
     )
@@
     )
     (property "MPN_MOUSER" "LM4041DIDBZT" (at 81.28 88.9 0)
+      (effects (font (size 1.27 1.27)) hide)
+    )
+    (property "R % tol" "" (at 81.28 88.9 0)
+      (effects (font (size 1.27 1.27)) hide)
+    )
+    (property "R pwr" "" (at 81.28 88.9 0)
       (effects (font (size 1.27 1.27)) hide)
     )
@@
       (effects (font (size 1.27 1.27)) hide)
     )
+    (property "R % tol" "0.1%" (at 189.23 93.98 0)
+      (effects (font (size 1.27 1.27)) hide)
+    )
+    (property "R pwr" "125mW" (at 189.23 93.98 0)
+      (effects (font (size 1.27 1.27)) hide)
+    )
     (pin "2")
     (pin "1")
@@
       (effects (font (size 1.27 1.27)) hide)
     )
+    (property "R % tol" "" (at 60.96 73.66 0)
+      (effects (font (size 1.27 1.27)) hide)
+    )
+    (property "R pwr" "" (at 60.96 73.66 0)
+      (effects (font (size 1.27 1.27)) hide)
+    )
     (pin "2")
     (pin "1")
@@
       (effects (font (size 1.27 1.27)) hide)
     )
+    (property "R % tol" "" (at 77.47 161.29 0)
+      (effects (font (size 1.27 1.27)) hide)
+    )
+    (property "R pwr" "" (at 77.47 161.29 0)
+      (effects (font (size 1.27 1.27)) hide)
+    )
     (pin "4")
     (pin "5")
@@
       (effects (font (size 1.27 1.27)) hide)
     )
+    (property "R % tol" "0.1%" (at 74.93 83.82 0)
+      (effects (font (size 1.27 1.27)) hide)
+    )
+    (property "R pwr" "125mW" (at 74.93 83.82 0)
+      (effects (font (size 1.27 1.27)) hide)
+    )
     (pin "2")
     (pin "1")
@@
       (effects (font (size 1.27 1.27)) hide)
     )
+    (property "R % tol" "0.1%" (at 138.43 86.36 0)
+      (effects (font (size 1.27 1.27)) hide)
+    )
+    (property "R pwr" "125mW" (at 138.43 86.36 0)
+      (effects (font (size 1.27 1.27)) hide)
+    )
     (pin "2")
     (pin "1")
@@
       (effects (font (size 1.27 1.27)) hide)
     )
+    (property "R % tol" "0.1%" (at 81.28 73.66 0)
+      (effects (font (size 1.27 1.27)) hide)
+    )
+    (property "R pwr" "125mW" (at 81.28 73.66 0)
+      (effects (font (size 1.27 1.27)) hide)
+    )
     (pin "2")
     (pin "1")
@@
     )
     (property "MPN_MOUSER" "" (at 116.84 88.9 0)
+      (effects (font (size 1.27 1.27)) hide)
+    )
+    (property "R % tol" "" (at 116.84 88.9 0)
+      (effects (font (size 1.27 1.27)) hide)
+    )
+    (property "R pwr" "" (at 116.84 88.9 0)
       (effects (font (size 1.27 1.27)) hide)
     )
@@
       (effects (font (size 1.27 1.27)) (justify left))
     )
-    (property "Value" "379R" (at 186.69 85.09 0)
+    (property "Value" "374R" (at 186.69 85.09 0)
       (effects (font (size 1.27 1.27)) (justify left))
     )
@@
       (effects (font (size 1.27 1.27)) hide)
     )
+    (property "R % tol" "0.1%" (at 189.23 83.82 0)
+      (effects (font (size 1.27 1.27)) hide)
+    )
+    (property "R pwr" "130mW " (at 189.23 83.82 0)
+      (effects (font (size 1.27 1.27)) hide)
+    )
     (pin "2")
     (pin "1")
@@
       (effects (font (size 1.27 1.27)) hide)
     )
+    (property "R % tol" "0.1%" (at 251.46 86.36 0)
+      (effects (font (size 1.27 1.27)) hide)
+    )
+    (property "R pwr" "125mW" (at 251.46 86.36 0)
+      (effects (font (size 1.27 1.27)) hide)
+    )

Commit message: Progressed ECAD
Parts:
- C29, C31, C32, C34: footprint Capacitor_SMD:CP_Elec_6.3x5.4 -> Capacitor_SMD:CP_Elec_4x5.4; MPN UWX1H100MCL1GB -> UWX1C100MCL1GB
Changed lines of the file:
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@@
       (effects (font (size 1.27 1.27)) (justify left))
     )
-    (property "Footprint" "Capacitor_SMD:CP_Elec_6.3x5.4" (at 174.2948 77.47 0)
-      (effects (font (size 1.27 1.27)) hide)
-    )
-    (property "Datasheet" "https://datasheet.lcsc.com/lcsc/2304140030_Nichicon-UWX1H100MCL1GB_C134237.pdf" (at 175.26 73.66 0)
-      (effects (font (size 1.27 1.27)) hide)
-    )
-    (property "MPN" "UWX1H100MCL1GB" (at 175.26 73.66 0)
+    (property "Footprint" "Capacitor_SMD:CP_Elec_4x5.4" (at 174.2948 77.47 0)
+      (effects (font (size 1.27 1.27)) hide)
+    )
+    (property "Datasheet" "https://datasheet.lcsc.com/lcsc/2304140030_Nichicon-UWX1C100MCL1GB_C445047.pdf" (at 175.26 73.66 0)
+      (effects (font (size 1.27 1.27)) hide)
+    )
+    (property "MPN" "UWX1C100MCL1GB" (at 175.26 73.66 0)
       (effects (font (size 1.27 1.27)) hide)
     )
@@
       (effects (font (size 1.27 1.27)) (justify left))
     )
-    (property "Footprint" "Capacitor_SMD:CP_Elec_6.3x5.4" (at 232.1052 92.71 0)
-      (effects (font (size 1.27 1.27)) hide)
-    )
-    (property "Datasheet" "https://datasheet.lcsc.com/lcsc/2304140030_Nichicon-UWX1H100MCL1GB_C134237.pdf" (at 231.14 88.9 0)
-      (effects (font (size 1.27 1.27)) hide)
-    )
-    (property "MPN" "UWX1H100MCL1GB" (at 231.14 88.9 0)
+    (property "Footprint" "Capacitor_SMD:CP_Elec_4x5.4" (at 232.1052 92.71 0)
+      (effects (font (size 1.27 1.27)) hide)
+    )
+    (property "Datasheet" "https://datasheet.lcsc.com/lcsc/2304140030_Nichicon-UWX1C100MCL1GB_C445047.pdf" (at 231.14 88.9 0)
+      (effects (font (size 1.27 1.27)) hide)
+    )
+    (property "MPN" "UWX1C100MCL1GB" (at 231.14 88.9 0)
       (effects (font (size 1.27 1.27)) hide)
     )
@@
       (effects (font (size 1.27 1.27)) (justify left))
     )
-    (property "Footprint" "Capacitor_SMD:CP_Elec_6.3x5.4" (at 59.9948 77.47 0)
-      (effects (font (size 1.27 1.27)) hide)
-    )
-    (property "Datasheet" "https://datasheet.lcsc.com/lcsc/2304140030_Nichicon-UWX1H100MCL1GB_C134237.pdf" (at 60.96 73.66 0)
-      (effects (font (size 1.27 1.27)) hide)
-    )
-    (property "MPN" "UWX1H100MCL1GB" (at 60.96 73.66 0)
+    (property "Footprint" "Capacitor_SMD:CP_Elec_4x5.4" (at 59.9948 77.47 0)
+      (effects (font (size 1.27 1.27)) hide)
+    )
+    (property "Datasheet" "https://datasheet.lcsc.com/lcsc/2304140030_Nichicon-UWX1C100MCL1GB_C445047.pdf" (at 60.96 73.66 0)
+      (effects (font (size 1.27 1.27)) hide)
+    )
+    (property "MPN" "UWX1C100MCL1GB" (at 60.96 73.66 0)
       (effects (font (size 1.27 1.27)) hide)
     )
@@
       (effects (font (size 1.27 1.27)) (justify left))
     )
-    (property "Footprint" "Capacitor_SMD:CP_Elec_6.3x5.4" (at 117.8052 92.71 0)
-      (effects (font (size 1.27 1.27)) hide)
-    )
-    (property "Datasheet" "https://datasheet.lcsc.com/lcsc/2304140030_Nichicon-UWX1H100MCL1GB_C134237.pdf" (at 116.84 88.9 0)
-      (effects (font (size 1.27 1.27)) hide)
-    )
-    (property "MPN" "UWX1H100MCL1GB" (at 116.84 88.9 0)
-      (effects (font (size 1.27 1.27)) hide)
-    )
+    (property "Footprint" "Capacitor_SMD:CP_Elec_4x5.4" (at 117.8052 92.71 0)
+      (effects (font (size 1.27 1.27)) hide)
+    )
+    (property "Datasheet" "https://datasheet.lcsc.com/lcsc/2304140030_Nichicon-UWX1C100MCL1GB_C445047.pdf" (at 116.84 88.9 0)
+      (effects (font (size 1.27 1.27)) hide)
+    )
+    (property "MPN" "UWX1C100MCL1GB" (at 116.84 88.9 0)
+      (effects (font (size 1.27 1.27)) hide)
+    )

Commit message: PRogressed ECAD.
Parts:
- J14: footprint Connector_PinSocket_2.54mm:PinSocket_1x06_P2.54mm_Horizontal -> Connector_PinSocket_2.54mm:PinSocket_1x06_P2.54mm_Vertical; MPN PM254-1-06-W-8.5 -> (none); Status OK -> (none)
Changed lines of the file:
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@@
       (effects (font (size 1.27 1.27)) (justify left))
     )
-    (property "Footprint" "Connector_PinSocket_2.54mm:PinSocket_1x06_P2.54mm_Horizontal" (at 77.47 161.29 0)
+    (property "Footprint" "Connector_PinSocket_2.54mm:PinSocket_1x06_P2.54mm_Vertical" (at 77.47 161.29 0)
       (effects (font (size 1.27 1.27)) hide)
     )
-    (property "Datasheet" "https://datasheet.lcsc.com/lcsc/2306091006_HCTL-PM254-1-06-W-8-5_C2897388.pdf" (at 77.47 161.29 0)
+    (property "Datasheet" "" (at 77.47 161.29 0)
       (effects (font (size 1.27 1.27)) hide)
     )
-    (property "MPN" "PM254-1-06-W-8.5" (at 77.47 161.29 0)
+    (property "MPN" "" (at 77.47 161.29 0)
       (effects (font (size 1.27 1.27)) hide)
     )
-    (property "Status" "OK" (at 77.47 161.29 0)
+    (property "Status" "" (at 77.47 161.29 0)
       (effects (font (size 1.27 1.27)) hide)
     )
