File: ECAD/SCART_switcher/dummy_input.kicad_sch (KiCad schematic)
At the start: 34 parts

Commit message: progressed ecad
Parts:
- U? (x5): value CD4066BPW -> CD4066; footprint Package_SO:TSSOP-14_4.4x5mm_P0.65mm -> Package_SO:SOIC-14_3.9x8.7mm_P1.27mm; MPN (none) -> CD4066BM96
Changed lines of the file:
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@@
       (effects (font (size 1.27 1.27)))
     )
-    (property "Value" "CD4066BPW" (at 210.82 34.29 0)
-      (effects (font (size 1.27 1.27)))
-    )
-    (property "Footprint" "Package_SO:TSSOP-14_4.4x5mm_P0.65mm" (at 203.2 27.94 0)
-      (effects (font (size 1.27 1.27)) hide)
-    )
-    (property "Datasheet" "https://www.ti.com/lit/ds/symlink/cd4066b.pdf" (at 203.2 30.48 0)
+    (property "Value" "CD4066" (at 210.82 34.29 0)
+      (effects (font (size 1.27 1.27)))
+    )
+    (property "Footprint" "Package_SO:SOIC-14_3.9x8.7mm_P1.27mm" (at 203.2 27.94 0)
+      (effects (font (size 1.27 1.27)) hide)
+    )
+    (property "Datasheet" "https://datasheet.lcsc.com/lcsc/1810171510_Texas-Instruments-CD4066BM96_C54755.pdf" (at 203.2 30.48 0)
+      (effects (font (size 1.27 1.27)) hide)
+    )
+    (property "MPN" "CD4066BM96" (at 203.2 30.48 0)
       (effects (font (size 1.27 1.27)) hide)
     )
@@
       (effects (font (size 1.27 1.27)) (justify left))
     )
-    (property "Value" "CD4066BPW" (at 270.51 38.1 0)
+    (property "Value" "CD4066" (at 270.51 38.1 0)
       (effects (font (size 1.27 1.27)) (justify left))
     )
-    (property "Footprint" "Package_SO:TSSOP-14_4.4x5mm_P0.65mm" (at 265.43 39.37 0)
-      (effects (font (size 1.27 1.27)) hide)
-    )
-    (property "Datasheet" "https://www.ti.com/lit/ds/symlink/cd4066b.pdf" (at 265.43 36.83 0)
+    (property "Footprint" "Package_SO:SOIC-14_3.9x8.7mm_P1.27mm" (at 265.43 39.37 0)
+      (effects (font (size 1.27 1.27)) hide)
+    )
+    (property "Datasheet" "https://datasheet.lcsc.com/lcsc/1810171510_Texas-Instruments-CD4066BM96_C54755.pdf" (at 265.43 36.83 0)
+      (effects (font (size 1.27 1.27)) hide)
+    )
+    (property "MPN" "CD4066BM96" (at 265.43 36.83 0)
       (effects (font (size 1.27 1.27)) hide)
     )
@@
       (effects (font (size 1.27 1.27)))
     )
-    (property "Value" "CD4066BPW" (at 119.38 36.83 0)
-      (effects (font (size 1.27 1.27)))
-    )
-    (property "Footprint" "Package_SO:TSSOP-14_4.4x5mm_P0.65mm" (at 127 27.94 0)
-      (effects (font (size 1.27 1.27)) hide)
-    )
-    (property "Datasheet" "https://www.ti.com/lit/ds/symlink/cd4066b.pdf" (at 127 30.48 0)
+    (property "Value" "CD4066" (at 119.38 36.83 0)
+      (effects (font (size 1.27 1.27)))
+    )
+    (property "Footprint" "Package_SO:SOIC-14_3.9x8.7mm_P1.27mm" (at 127 27.94 0)
+      (effects (font (size 1.27 1.27)) hide)
+    )
+    (property "Datasheet" "https://datasheet.lcsc.com/lcsc/1810171510_Texas-Instruments-CD4066BM96_C54755.pdf" (at 127 30.48 0)
+      (effects (font (size 1.27 1.27)) hide)
+    )
+    (property "MPN" "CD4066BM96" (at 127 30.48 0)
       (effects (font (size 1.27 1.27)) hide)
     )
@@
       (effects (font (size 1.27 1.27)))
     )
-    (property "Value" "CD4066BPW" (at 195.58 39.37 0)
-      (effects (font (size 1.27 1.27)))
-    )
-    (property "Footprint" "Package_SO:TSSOP-14_4.4x5mm_P0.65mm" (at 203.2 45.72 0)
-      (effects (font (size 1.27 1.27)) hide)
-    )
-    (property "Datasheet" "https://www.ti.com/lit/ds/symlink/cd4066b.pdf" (at 203.2 43.18 0)
+    (property "Value" "CD4066" (at 195.58 39.37 0)
+      (effects (font (size 1.27 1.27)))
+    )
+    (property "Footprint" "Package_SO:SOIC-14_3.9x8.7mm_P1.27mm" (at 203.2 45.72 0)
+      (effects (font (size 1.27 1.27)) hide)
+    )
+    (property "Datasheet" "https://datasheet.lcsc.com/lcsc/1810171510_Texas-Instruments-CD4066BM96_C54755.pdf" (at 203.2 43.18 0)
+      (effects (font (size 1.27 1.27)) hide)
+    )
+    (property "MPN" "CD4066BM96" (at 203.2 43.18 0)
       (effects (font (size 1.27 1.27)) hide)
     )
@@
       (effects (font (size 1.27 1.27)))
     )
-    (property "Value" "CD4066BPW" (at 134.62 39.37 0)
-      (effects (font (size 1.27 1.27)))
-    )
-    (property "Footprint" "Package_SO:TSSOP-14_4.4x5mm_P0.65mm" (at 127 45.72 0)
-      (effects (font (size 1.27 1.27)) hide)
-    )
-    (property "Datasheet" "https://www.ti.com/lit/ds/symlink/cd4066b.pdf" (at 127 43.18 0)
-      (effects (font (size 1.27 1.27)) hide)
-    )
+    (property "Value" "CD4066" (at 134.62 39.37 0)
+      (effects (font (size 1.27 1.27)))
+    )
+    (property "Footprint" "Package_SO:SOIC-14_3.9x8.7mm_P1.27mm" (at 127 45.72 0)
+      (effects (font (size 1.27 1.27)) hide)
+    )
+    (property "Datasheet" "https://datasheet.lcsc.com/lcsc/1810171510_Texas-Instruments-CD4066BM96_C54755.pdf" (at 127 43.18 0)
+      (effects (font (size 1.27 1.27)) hide)
+    )
+    (property "MPN" "CD4066BM96" (at 127 43.18 0)
+      (effects (font (size 1.27 1.27)) hide)
+    )

Commit message: progressed ecad
Parts:
- U? (x8): value TS5A63157DBV -> 74LVC1G3157; footprint Package_TO_SOT_SMD:SOT-23-6 -> Package_TO_SOT_SMD:SOT-363_SC-70-6; MPN (none) -> SN74LVC1G3157DCKR
Changed lines of the file:
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@@
       (effects (font (size 1.27 1.27)) (justify left))
     )
-    (property "Value" "TS5A63157DBV" (at 240.03 124.46 0)
+    (property "Value" "74LVC1G3157" (at 240.03 124.46 0)
       (effects (font (size 1.27 1.27)) (justify left))
     )
-    (property "Footprint" "Package_TO_SOT_SMD:SOT-23-6" (at 234.95 130.81 0)
+    (property "Footprint" "Package_TO_SOT_SMD:SOT-363_SC-70-6" (at 234.95 130.81 0)
       (effects (font (size 1.27 1.27)) hide)
     )
-    (property "Datasheet" "https://www.ti.com/lit/ds/symlink/ts5a63157.pdf" (at 234.95 123.19 0)
+    (property "Datasheet" "https://datasheet.lcsc.com/lcsc/1811031937_Texas-Instruments-SN74LVC1G3157DCKR_C38663.pdf" (at 234.95 123.19 0)
+      (effects (font (size 1.27 1.27)) hide)
+    )
+    (property "MPN" "SN74LVC1G3157DCKR" (at 234.95 123.19 0)
       (effects (font (size 1.27 1.27)) hide)
     )
@@
       (effects (font (size 1.27 1.27)) (justify left))
     )
-    (property "Value" "TS5A63157DBV" (at 240.03 83.82 0)
+    (property "Value" "74LVC1G3157" (at 240.03 83.82 0)
       (effects (font (size 1.27 1.27)) (justify left))
     )
-    (property "Footprint" "Package_TO_SOT_SMD:SOT-23-6" (at 234.95 90.17 0)
+    (property "Footprint" "Package_TO_SOT_SMD:SOT-363_SC-70-6" (at 234.95 90.17 0)
+      (effects (font (size 1.27 1.27)) hide)
+    )
+    (property "Datasheet" "https://datasheet.lcsc.com/lcsc/1811031937_Texas-Instruments-SN74LVC1G3157DCKR_C38663.pdf" (at 234.95 82.55 0)
       (effects (font (size 1.27 1.27)) hide)
     )
-    (property "Datasheet" "https://www.ti.com/lit/ds/symlink/ts5a63157.pdf" (at 234.95 82.55 0)
+    (property "MPN" "SN74LVC1G3157DCKR" (at 234.95 82.55 0)
       (effects (font (size 1.27 1.27)) hide)
     )
@@
       (effects (font (size 1.27 1.27)))
     )
-    (property "Value" "TS5A63157DBV" (at 182.88 88.9 0)
+    (property "Value" "74LVC1G3157" (at 182.88 88.9 0)
       (effects (font (size 1.27 1.27)))
     )
-    (property "Footprint" "Package_TO_SOT_SMD:SOT-23-6" (at 182.88 77.47 0)
+    (property "Footprint" "Package_TO_SOT_SMD:SOT-363_SC-70-6" (at 182.88 77.47 0)
       (effects (font (size 1.27 1.27)) hide)
     )
-    (property "Datasheet" "https://www.ti.com/lit/ds/symlink/ts5a63157.pdf" (at 182.88 85.09 0)
+    (property "Datasheet" "https://datasheet.lcsc.com/lcsc/1811031937_Texas-Instruments-SN74LVC1G3157DCKR_C38663.pdf" (at 182.88 85.09 0)
+      (effects (font (size 1.27 1.27)) hide)
+    )
+    (property "MPN" "SN74LVC1G3157DCKR" (at 182.88 85.09 0)
       (effects (font (size 1.27 1.27)) hide)
     )
@@
       (effects (font (size 1.27 1.27)) (justify left))
     )
-    (property "Value" "TS5A63157DBV" (at 115.57 125.73 0)
+    (property "Value" "74LVC1G3157" (at 115.57 125.73 0)
       (effects (font (size 1.27 1.27)) (justify left))
     )
-    (property "Footprint" "Package_TO_SOT_SMD:SOT-23-6" (at 110.49 132.08 0)
+    (property "Footprint" "Package_TO_SOT_SMD:SOT-363_SC-70-6" (at 110.49 132.08 0)
+      (effects (font (size 1.27 1.27)) hide)
+    )
+    (property "Datasheet" "https://datasheet.lcsc.com/lcsc/1811031937_Texas-Instruments-SN74LVC1G3157DCKR_C38663.pdf" (at 110.49 124.46 0)
       (effects (font (size 1.27 1.27)) hide)
     )
-    (property "Datasheet" "https://www.ti.com/lit/ds/symlink/ts5a63157.pdf" (at 110.49 124.46 0)
+    (property "MPN" "SN74LVC1G3157DCKR" (at 110.49 124.46 0)
       (effects (font (size 1.27 1.27)) hide)
     )
@@
       (effects (font (size 1.27 1.27)))
     )
-    (property "Value" "TS5A63157DBV" (at 58.42 88.9 0)
+    (property "Value" "74LVC1G3157" (at 58.42 88.9 0)
       (effects (font (size 1.27 1.27)))
     )
-    (property "Footprint" "Package_TO_SOT_SMD:SOT-23-6" (at 58.42 77.47 0)
+    (property "Footprint" "Package_TO_SOT_SMD:SOT-363_SC-70-6" (at 58.42 77.47 0)
       (effects (font (size 1.27 1.27)) hide)
     )
-    (property "Datasheet" "https://www.ti.com/lit/ds/symlink/ts5a63157.pdf" (at 58.42 85.09 0)
+    (property "Datasheet" "https://datasheet.lcsc.com/lcsc/1811031937_Texas-Instruments-SN74LVC1G3157DCKR_C38663.pdf" (at 58.42 85.09 0)
+      (effects (font (size 1.27 1.27)) hide)
+    )
+    (property "MPN" "SN74LVC1G3157DCKR" (at 58.42 85.09 0)
       (effects (font (size 1.27 1.27)) hide)
     )
@@
       (effects (font (size 1.27 1.27)) (justify left))
     )
-    (property "Value" "TS5A63157DBV" (at 116.84 83.82 0)
+    (property "Value" "74LVC1G3157" (at 116.84 83.82 0)
       (effects (font (size 1.27 1.27)) (justify left))
     )
-    (property "Footprint" "Package_TO_SOT_SMD:SOT-23-6" (at 110.49 90.17 0)
+    (property "Footprint" "Package_TO_SOT_SMD:SOT-363_SC-70-6" (at 110.49 90.17 0)
+      (effects (font (size 1.27 1.27)) hide)
+    )
+    (property "Datasheet" "https://datasheet.lcsc.com/lcsc/1811031937_Texas-Instruments-SN74LVC1G3157DCKR_C38663.pdf" (at 110.49 82.55 0)
       (effects (font (size 1.27 1.27)) hide)
     )
-    (property "Datasheet" "https://www.ti.com/lit/ds/symlink/ts5a63157.pdf" (at 110.49 82.55 0)
+    (property "MPN" "SN74LVC1G3157DCKR" (at 110.49 82.55 0)
       (effects (font (size 1.27 1.27)) hide)
     )
@@
       (effects (font (size 1.27 1.27)))
     )
-    (property "Value" "TS5A63157DBV" (at 58.42 130.81 0)
+    (property "Value" "74LVC1G3157" (at 58.42 130.81 0)
       (effects (font (size 1.27 1.27)))
     )
-    (property "Footprint" "Package_TO_SOT_SMD:SOT-23-6" (at 58.42 119.38 0)
+    (property "Footprint" "Package_TO_SOT_SMD:SOT-363_SC-70-6" (at 58.42 119.38 0)
       (effects (font (size 1.27 1.27)) hide)
     )
-    (property "Datasheet" "https://www.ti.com/lit/ds/symlink/ts5a63157.pdf" (at 58.42 127 0)
+    (property "Datasheet" "https://datasheet.lcsc.com/lcsc/1811031937_Texas-Instruments-SN74LVC1G3157DCKR_C38663.pdf" (at 58.42 127 0)
+      (effects (font (size 1.27 1.27)) hide)
+    )
+    (property "MPN" "SN74LVC1G3157DCKR" (at 58.42 127 0)
       (effects (font (size 1.27 1.27)) hide)
     )
@@
       (effects (font (size 1.27 1.27)))
     )
-    (property "Value" "TS5A63157DBV" (at 182.88 129.54 0)
+    (property "Value" "74LVC1G3157" (at 182.88 129.54 0)
       (effects (font (size 1.27 1.27)))
     )
-    (property "Footprint" "Package_TO_SOT_SMD:SOT-23-6" (at 182.88 118.11 0)
+    (property "Footprint" "Package_TO_SOT_SMD:SOT-363_SC-70-6" (at 182.88 118.11 0)
+      (effects (font (size 1.27 1.27)) hide)
+    )
+    (property "Datasheet" "https://datasheet.lcsc.com/lcsc/1811031937_Texas-Instruments-SN74LVC1G3157DCKR_C38663.pdf" (at 182.88 125.73 0)
       (effects (font (size 1.27 1.27)) hide)
     )
-    (property "Datasheet" "https://www.ti.com/lit/ds/symlink/ts5a63157.pdf" (at 182.88 125.73 0)
+    (property "MPN" "SN74LVC1G3157DCKR" (at 182.88 125.73 0)
       (effects (font (size 1.27 1.27)) hide)
     )
