File: ECAD/SCART_switcher/dummy_input.kicad_sch (KiCad schematic)
At the start: 34 parts

Commit message: Progressed ECAD.
Parts:
- Q?: MPN BC847B,215 -> BC847C,215; Status (none) -> OK
- Q?: MPN (none) -> BC857C,215; Status (none) -> OK
Changed lines of the file:
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@@
       (effects (font (size 1.27 1.27)) hide)
     )
+    (property "Status" "" (at 26.67 41.91 0)
+      (effects (font (size 1.27 1.27)) hide)
+    )
     (pin "1")
     (pin "2")
@@
       (effects (font (size 1.27 1.27)) hide)
     )
+    (property "Status" "" (at 39.37 129.54 0)
+      (effects (font (size 1.27 1.27)) hide)
+    )
     (pin "1")
     (pin "2")
@@
       (effects (font (size 1.27 1.27) italic) (justify left) hide)
     )
-    (property "Datasheet" "https://datasheet.lcsc.com/lcsc/2304140030_Nexperia-BC847B-215_C57668.pdf" (at 35.56 41.91 0)
+    (property "Datasheet" "https://datasheet.lcsc.com/lcsc/1811141238_Nexperia-BC847C-215_C8664.pdf" (at 35.56 41.91 0)
       (effects (font (size 1.27 1.27)) (justify left) hide)
     )
-    (property "MPN" "BC847B,215" (at 35.56 41.91 0)
+    (property "MPN" "BC847C,215" (at 35.56 41.91 0)
+      (effects (font (size 1.27 1.27)) hide)
+    )
+    (property "Status" "OK" (at 35.56 41.91 0)
       (effects (font (size 1.27 1.27)) hide)
     )
@@
       (effects (font (size 1.27 1.27)) hide)
     )
+    (property "Status" "" (at 250.19 36.83 0)
+      (effects (font (size 1.27 1.27)) hide)
+    )
     (pin "1")
     (pin "2")
@@
       (effects (font (size 1.27 1.27)) hide)
     )
+    (property "Status" "" (at 234.95 123.19 0)
+      (effects (font (size 1.27 1.27)) hide)
+    )
     (pin "1")
     (pin "2")
@@
       (effects (font (size 1.27 1.27)) hide)
     )
+    (property "Status" "" (at 163.83 128.27 0)
+      (effects (font (size 1.27 1.27)) hide)
+    )
     (pin "1")
     (pin "2")
@@
       (effects (font (size 1.27 1.27)) hide)
     )
+    (property "Status" "" (at 234.95 82.55 0)
+      (effects (font (size 1.27 1.27)) hide)
+    )
     (pin "1")
     (pin "2")
@@
       (effects (font (size 1.27 1.27)) hide)
     )
+    (property "Status" "" (at 219.71 82.55 0)
+      (effects (font (size 1.27 1.27)) hide)
+    )
     (pin "1")
     (pin "2")
@@
       (effects (font (size 1.27 1.27)) hide)
     )
+    (property "Status" "" (at 38.1 33.02 0)
+      (effects (font (size 1.27 1.27)) hide)
+    )
     (pin "1")
     (pin "2")
@@
       (effects (font (size 1.27 1.27)) hide)
     )
+    (property "Status" "" (at 173.99 44.45 0)
+      (effects (font (size 1.27 1.27)) hide)
+    )
     (pin "1")
     (pin "2")
@@
       (effects (font (size 1.27 1.27)) hide)
     )
+    (property "Status" "" (at 127 173.99 0)
+      (effects (font (size 1.27 1.27)) hide)
+    )
     (pin "1")
     (pin "2")
@@
       (effects (font (size 1.27 1.27)) hide)
     )
+    (property "Status" "" (at 64.77 45.72 0)
+      (effects (font (size 1.27 1.27)) hide)
+    )
     (pin "1")
     (pin "2")
@@
       (effects (font (size 1.27 1.27)) hide)
     )
+    (property "Status" "" (at 39.37 87.63 0)
+      (effects (font (size 1.27 1.27)) hide)
+    )
     (pin "1")
     (pin "2")
@@
       (effects (font (size 1.27 1.27)) hide)
     )
+    (property "Status" "" (at 53.34 36.83 0)
+      (effects (font (size 1.27 1.27)) hide)
+    )
     (pin "1")
     (pin "2")
@@
       (effects (font (size 1.27 1.27)) hide)
     )
+    (property "Status" "" (at 182.88 85.09 0)
+      (effects (font (size 1.27 1.27)) hide)
+    )
     (pin "1")
     (pin "2")
@@
       (effects (font (size 1.27 1.27)) hide)
     )
+    (property "Status" "" (at 110.49 124.46 0)
+      (effects (font (size 1.27 1.27)) hide)
+    )
     (pin "1")
     (pin "2")
@@
       (effects (font (size 1.27 1.27)) hide)
     )
+    (property "Status" "" (at 57.15 173.99 0)
+      (effects (font (size 1.27 1.27)) hide)
+    )
     (pin "2")
     (pin "3")
@@
       (effects (font (size 1.27 1.27) italic) (justify left) hide)
     )
-    (property "Datasheet" "https://www.onsemi.com/pub/Collateral/BC860-D.pdf" (at 62.23 36.83 0)
+    (property "Datasheet" "https://datasheet.lcsc.com/lcsc/2304140030_Nexperia-BC857C-215_C8666.pdf" (at 62.23 36.83 0)
       (effects (font (size 1.27 1.27)) (justify left) hide)
     )
+    (property "Status" "OK" (at 62.23 36.83 0)
+      (effects (font (size 1.27 1.27)) hide)
+    )
+    (property "MPN" "BC857C,215" (at 62.23 36.83 0)
+      (effects (font (size 1.27 1.27)) hide)
+    )
     (pin "1")
     (pin "2")
@@
       (effects (font (size 1.27 1.27)) hide)
     )
+    (property "Status" "" (at 95.25 82.55 0)
+      (effects (font (size 1.27 1.27)) hide)
+    )
     (pin "1")
     (pin "2")
@@
       (effects (font (size 1.27 1.27)) hide)
     )
+    (property "Status" "" (at 58.42 85.09 0)
+      (effects (font (size 1.27 1.27)) hide)
+    )
     (pin "4")
     (pin "5")
@@
       (effects (font (size 1.27 1.27)) hide)
     )
+    (property "Status" "" (at 163.83 87.63 0)
+      (effects (font (size 1.27 1.27)) hide)
+    )
     (pin "1")
     (pin "2")
@@
       (effects (font (size 1.27 1.27)) hide)
     )
+    (property "Status" "" (at 83.82 173.99 0)
+      (effects (font (size 1.27 1.27)) hide)
+    )
     (pin "1")
     (pin "2")
@@
       (effects (font (size 1.27 1.27)) hide)
     )
+    (property "Status" "" (at 95.25 124.46 0)
+      (effects (font (size 1.27 1.27)) hide)
+    )
     (pin "1")
     (pin "2")
@@
       (effects (font (size 1.27 1.27)) hide)
     )
+    (property "Status" "" (at 97.79 44.45 0)
+      (effects (font (size 1.27 1.27)) hide)
+    )
     (pin "1")
     (pin "2")
@@
       (effects (font (size 1.27 1.27)) hide)
     )
+    (property "Status" "" (at 203.2 30.48 0)
+      (effects (font (size 1.27 1.27)) hide)
+    )
     (pin "1")
     (pin "13")
@@
       (effects (font (size 1.27 1.27)) hide)
     )
+    (property "Status" "" (at 219.71 123.19 0)
+      (effects (font (size 1.27 1.27)) hide)
+    )
     (pin "1")
     (pin "2")
@@
       (effects (font (size 1.27 1.27)) hide)
     )
+    (property "Status" "" (at 265.43 36.83 0)
+      (effects (font (size 1.27 1.27)) hide)
+    )
     (pin "1")
     (pin "13")
@@
       (effects (font (size 1.27 1.27)) hide)
     )
+    (property "Status" "" (at 156.21 173.99 0)
+      (effects (font (size 1.27 1.27)) hide)
+    )
     (pin "1")
     (pin "2")
@@
       (effects (font (size 1.27 1.27)) hide)
     )
+    (property "Status" "" (at 127 30.48 0)
+      (effects (font (size 1.27 1.27)) hide)
+    )
     (pin "1")
     (pin "13")
@@
       (effects (font (size 1.27 1.27)) hide)
     )
+    (property "Status" "" (at 110.49 82.55 0)
+      (effects (font (size 1.27 1.27)) hide)
+    )
     (pin "4")
     (pin "5")
@@
       (effects (font (size 1.27 1.27)) hide)
     )
+    (property "Status" "" (at 58.42 127 0)
+      (effects (font (size 1.27 1.27)) hide)
+    )
     (pin "1")
     (pin "2")
@@
       (effects (font (size 1.27 1.27)) hide)
     )
+    (property "Status" "" (at 203.2 43.18 0)
+      (effects (font (size 1.27 1.27)) hide)
+    )
     (pin "1")
     (pin "13")
@@
       (effects (font (size 1.27 1.27)) hide)
     )
+    (property "Status" "" (at 182.88 125.73 0)
+      (effects (font (size 1.27 1.27)) hide)
+    )
     (pin "1")
     (pin "2")
@@
       (effects (font (size 1.27 1.27)) hide)
     )
+    (property "Status" "" (at 127 43.18 0)
+      (effects (font (size 1.27 1.27)) hide)
+    )

Commit message: Progressed ECAD.
Parts:
- U?: footprint (none) -> Package_TO_SOT_SMD:SOT-23-5; MPN 74AHC1G126W5-7 -> SN74AHC1G126DBVR
- U?: MPN 74AHC1G04W5-7 -> SN74AHC1G04DBVR
- U? (x5): Status (none) -> OK
Changed lines of the file:
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@@
       (effects (font (size 1.27 1.27)))
     )
-    (property "Footprint" "" (at 127 173.99 0)
+    (property "Footprint" "Package_TO_SOT_SMD:SOT-23-5" (at 127 173.99 0)
       (effects (font (size 1.27 1.27)) hide)
     )
-    (property "Datasheet" "https://datasheet.lcsc.com/lcsc/2201131130_Diodes-Incorporated-74AHC1G126W5-7_C842263.pdf" (at 127 173.99 0)
+    (property "Datasheet" "https://datasheet.lcsc.com/lcsc/1810010909_Texas-Instruments-SN74AHC1G126DBVR_C145145.pdf" (at 127 173.99 0)
       (effects (font (size 1.27 1.27)) hide)
     )
-    (property "MPN" "74AHC1G126W5-7" (at 127 173.99 0)
+    (property "MPN" "SN74AHC1G126DBVR" (at 127 173.99 0)
       (effects (font (size 1.27 1.27)) hide)
     )
@@
       (effects (font (size 1.27 1.27)) hide)
     )
-    (property "Datasheet" "https://datasheet.lcsc.com/lcsc/1912111437_Diodes-Incorporated-74AHC1G04W5-7_C460486.pdf" (at 57.15 173.99 0)
+    (property "Datasheet" "https://datasheet.lcsc.com/lcsc/2001061132_Texas-Instruments-SN74AHC1G04DBVR_C7465.pdf" (at 57.15 173.99 0)
       (effects (font (size 1.27 1.27)) hide)
     )
-    (property "MPN" "74AHC1G04W5-7" (at 57.15 173.99 0)
+    (property "MPN" "SN74AHC1G04DBVR" (at 57.15 173.99 0)
       (effects (font (size 1.27 1.27)) hide)
     )
@@
       (effects (font (size 1.27 1.27)) hide)
     )
-    (property "Status" "" (at 203.2 30.48 0)
+    (property "Status" "OK" (at 203.2 30.48 0)
       (effects (font (size 1.27 1.27)) hide)
     )
@@
       (effects (font (size 1.27 1.27)) hide)
     )
-    (property "Status" "" (at 265.43 36.83 0)
+    (property "Status" "OK" (at 265.43 36.83 0)
       (effects (font (size 1.27 1.27)) hide)
     )
@@
       (effects (font (size 1.27 1.27)) hide)
     )
-    (property "Status" "" (at 127 30.48 0)
+    (property "Status" "OK" (at 127 30.48 0)
       (effects (font (size 1.27 1.27)) hide)
     )
@@
       (effects (font (size 1.27 1.27)) hide)
     )
-    (property "Status" "" (at 203.2 43.18 0)
+    (property "Status" "OK" (at 203.2 43.18 0)
       (effects (font (size 1.27 1.27)) hide)
     )
@@
       (effects (font (size 1.27 1.27)) hide)
     )
-    (property "Status" "" (at 127 43.18 0)
+    (property "Status" "OK" (at 127 43.18 0)
       (effects (font (size 1.27 1.27)) hide)
     )

Commit message: Progressed ECAD.
Parts:
- U? (x8): Status (none) -> OK
- U?: value 74AHC1G126 -> 74LVC1G126; footprint Package_TO_SOT_SMD:SOT-23-5 -> Package_TO_SOT_SMD:SOT-353_SC-70-5; MPN SN74AHC1G126DBVR -> SN74LVC1G126DCKR; Status (none) -> OK
- U?: value 74AHC1G04 -> 74LVC1G04; footprint Package_TO_SOT_SMD:SOT-23-5 -> Package_TO_SOT_SMD:SOT-353_SC-70-5; MPN SN74AHC1G04DBVR -> SN74LVC1G04DCKR; Status (none) -> OK
Changed lines of the file:
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@@
       (effects (font (size 1.27 1.27)) hide)
     )
-    (property "Status" "" (at 234.95 123.19 0)
+    (property "Status" "OK" (at 234.95 123.19 0)
       (effects (font (size 1.27 1.27)) hide)
     )
@@
       (effects (font (size 1.27 1.27)) hide)
     )
-    (property "Status" "" (at 234.95 82.55 0)
+    (property "Status" "OK" (at 234.95 82.55 0)
       (effects (font (size 1.27 1.27)) hide)
     )
@@
       (effects (font (size 1.27 1.27)))
     )
-    (property "Value" "74AHC1G126" (at 133.35 177.8 0)
+    (property "Value" "74LVC1G126" (at 133.35 177.8 0)
       (effects (font (size 1.27 1.27)))
     )
-    (property "Footprint" "Package_TO_SOT_SMD:SOT-23-5" (at 127 173.99 0)
+    (property "Footprint" "Package_TO_SOT_SMD:SOT-353_SC-70-5" (at 127 173.99 0)
       (effects (font (size 1.27 1.27)) hide)
     )
-    (property "Datasheet" "https://datasheet.lcsc.com/lcsc/1810010909_Texas-Instruments-SN74AHC1G126DBVR_C145145.pdf" (at 127 173.99 0)
+    (property "Datasheet" "https://datasheet.lcsc.com/lcsc/1811082050_Texas-Instruments-SN74LVC1G126DCKR_C88039.pdf" (at 127 173.99 0)
       (effects (font (size 1.27 1.27)) hide)
     )
-    (property "MPN" "SN74AHC1G126DBVR" (at 127 173.99 0)
+    (property "MPN" "SN74LVC1G126DCKR" (at 127 173.99 0)
       (effects (font (size 1.27 1.27)) hide)
     )
-    (property "Status" "" (at 127 173.99 0)
+    (property "Status" "OK" (at 127 173.99 0)
       (effects (font (size 1.27 1.27)) hide)
     )
@@
       (effects (font (size 1.27 1.27)) hide)
     )
-    (property "Status" "" (at 182.88 85.09 0)
+    (property "Status" "OK" (at 182.88 85.09 0)
       (effects (font (size 1.27 1.27)) hide)
     )
@@
       (effects (font (size 1.27 1.27)) hide)
     )
-    (property "Status" "" (at 110.49 124.46 0)
+    (property "Status" "OK" (at 110.49 124.46 0)
       (effects (font (size 1.27 1.27)) hide)
     )
@@
       (effects (font (size 1.27 1.27)))
     )
-    (property "Value" "74AHC1G04" (at 62.23 168.91 0)
+    (property "Value" "74LVC1G04" (at 62.23 168.91 0)
       (effects (font (size 1.27 1.27)))
     )
-    (property "Footprint" "Package_TO_SOT_SMD:SOT-23-5" (at 57.15 173.99 0)
+    (property "Footprint" "Package_TO_SOT_SMD:SOT-353_SC-70-5" (at 57.15 173.99 0)
       (effects (font (size 1.27 1.27)) hide)
     )
-    (property "Datasheet" "https://datasheet.lcsc.com/lcsc/2001061132_Texas-Instruments-SN74AHC1G04DBVR_C7465.pdf" (at 57.15 173.99 0)
+    (property "Datasheet" "https://datasheet.lcsc.com/lcsc/1811021113_Texas-Instruments-SN74LVC1G04DCKR_C8207.pdf" (at 57.15 173.99 0)
       (effects (font (size 1.27 1.27)) hide)
     )
-    (property "MPN" "SN74AHC1G04DBVR" (at 57.15 173.99 0)
+    (property "MPN" "SN74LVC1G04DCKR" (at 57.15 173.99 0)
       (effects (font (size 1.27 1.27)) hide)
     )
-    (property "Status" "" (at 57.15 173.99 0)
+    (property "Status" "OK" (at 57.15 173.99 0)
       (effects (font (size 1.27 1.27)) hide)
     )
@@
       (effects (font (size 1.27 1.27)) hide)
     )
-    (property "Status" "" (at 58.42 85.09 0)
+    (property "Status" "OK" (at 58.42 85.09 0)
       (effects (font (size 1.27 1.27)) hide)
     )
@@
       (effects (font (size 1.27 1.27)) hide)
     )
-    (property "Status" "" (at 110.49 82.55 0)
+    (property "Status" "OK" (at 110.49 82.55 0)
       (effects (font (size 1.27 1.27)) hide)
     )
@@
       (effects (font (size 1.27 1.27)) hide)
     )
-    (property "Status" "" (at 58.42 127 0)
+    (property "Status" "OK" (at 58.42 127 0)
       (effects (font (size 1.27 1.27)) hide)
     )
@@
       (effects (font (size 1.27 1.27)) hide)
     )
-    (property "Status" "" (at 182.88 125.73 0)
+    (property "Status" "OK" (at 182.88 125.73 0)
       (effects (font (size 1.27 1.27)) hide)
     )

Commit message: Progressed ECAD.
Parts:
- removed U? (x8): 74LVC1G3157, Package_TO_SOT_SMD:SOT-363_SC-70-6, symbol Analog_Switch:TS5A63157DBV
- added U20, U21, U24, U25: 74LVC1G3157, Package_TO_SOT_SMD:SOT-363_SC-70-6, symbol Analog_Switch:TS5A63157DBV
- gave numbers to parts that had none: 22
Connections:
- net +2V5: now also U20.3, U21.3, U24.3, U25.3
- net +5V: now also U20.5 (V+), U21.5 (V+), U24.5 (V+), U25.5 (V+)
- net BLUE: now also U24.1
- net ENABLE: now also U20.6, U21.6, U24.6, U25.6
- net GND: now also U20.2 (GND), U21.2 (GND), U24.2 (GND), U25.2 (GND)
- net GREEN: now also U20.1
- net RED: now also U21.1
- net VIDEO_RGB_SYNC: now also U25.1
- net at R100.1: now also U21.4
- net at R105.1: now also U25.4
- net at R99.1: now also U20.4
- net at R104.1: now also U24.4

Commit message: Progressed ECAD.
Parts:
- removed C38: 100nC, Capacitor_SMD:C_0805_2012Metric, symbol Device:C
- removed U19: 74LVC1G04, Package_TO_SOT_SMD:SOT-353_SC-70-5, symbol 74xGxx:74AHC1G04
Changed lines of the file:
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@@
-    )
-  )
-  (symbol (lib_id "power:+5V") (at 52.07 163.83 0) (unit 1)
-    (in_bom yes) (on_board yes) (dnp no) (fields_autoplaced)
-    (property "Reference" "#PWR0261" (at 52.07 167.64 0)
-      (effects (font (size 1.27 1.27)) hide)
-    )
-    (property "Value" "+5V" (at 52.07 158.75 0)
-      (effects (font (size 1.27 1.27)))
-    )
-    (property "Footprint" "" (at 52.07 163.83 0)
-      (effects (font (size 1.27 1.27)) hide)
-    )
-    (property "Datasheet" "" (at 52.07 163.83 0)
-      (effects (font (size 1.27 1.27)) hide)
-    )
-    (pin "1")
-    (instances
-      (project "SCART_switcher"
-        (path "/8cd08eb5-4755-4ef5-8eeb-77fd9974b180/6562ea38-5963-42b2-a0ef-a4a12a4c652f/32c156af-ff54-4356-ac90-a2b1f82b1e02"
-          (reference "#PWR0261") (unit 1)
-        )
-      )
     )
   )
@@
     )
   )
-  (symbol (lib_id "power:+5V") (at 83.82 170.18 0) (unit 1)
-    (in_bom yes) (on_board yes) (dnp no) (fields_autoplaced)
-    (property "Reference" "#PWR0267" (at 83.82 173.99 0)
-      (effects (font (size 1.27 1.27)) hide)
-    )
-    (property "Value" "+5V" (at 83.82 165.1 0)
-      (effects (font (size 1.27 1.27)))
-    )
-    (property "Footprint" "" (at 83.82 170.18 0)
-      (effects (font (size 1.27 1.27)) hide)
-    )
-    (property "Datasheet" "" (at 83.82 170.18 0)
-      (effects (font (size 1.27 1.27)) hide)
-    )
-    (pin "1")
-    (instances
-      (project "SCART_switcher"
-        (path "/8cd08eb5-4755-4ef5-8eeb-77fd9974b180/6562ea38-5963-42b2-a0ef-a4a12a4c652f/32c156af-ff54-4356-ac90-a2b1f82b1e02"
-          (reference "#PWR0267") (unit 1)
-        )
-      )
-    )
-  )
   (symbol (lib_name "TS5A63157DBV_1") (lib_id "Analog_Switch:TS5A63157DBV") (at 58.42 124.46 0) (mirror x) (unit 1)
     (in_bom yes) (on_board yes) (dnp no)
@@
     )
   )
-  (symbol (lib_id "74xGxx:74AHC1G04") (at 57.15 173.99 0) (unit 1)
-    (in_bom yes) (on_board yes) (dnp no)
-    (property "Reference" "U19" (at 62.23 166.37 0)
-      (effects (font (size 1.27 1.27)))
-    )
-    (property "Value" "74LVC1G04" (at 62.23 168.91 0)
-      (effects (font (size 1.27 1.27)))
-    )
-    (property "Footprint" "Package_TO_SOT_SMD:SOT-353_SC-70-5" (at 57.15 173.99 0)
-      (effects (font (size 1.27 1.27)) hide)
-    )
-    (property "Datasheet" "https://datasheet.lcsc.com/lcsc/1811021113_Texas-Instruments-SN74LVC1G04DCKR_C8207.pdf" (at 57.15 173.99 0)
-      (effects (font (size 1.27 1.27)) hide)
-    )
-    (property "MPN" "SN74LVC1G04DCKR" (at 57.15 173.99 0)
-      (effects (font (size 1.27 1.27)) hide)
-    )
-    (property "Status" "OK" (at 57.15 173.99 0)
-      (effects (font (size 1.27 1.27)) hide)
-    )
-    (pin "2")
-    (pin "3")
-    (pin "4")
-    (pin "5")
-    (instances
-      (project "SCART_switcher"
-        (path "/8cd08eb5-4755-4ef5-8eeb-77fd9974b180/6562ea38-5963-42b2-a0ef-a4a12a4c652f/32c156af-ff54-4356-ac90-a2b1f82b1e02"
-          (reference "U19") (unit 1)
-        )
-      )
-    )
-  )
   (symbol (lib_id "Transistor_BJT:BC857") (at 62.23 36.83 0) (mirror x) (unit 1)
     (in_bom yes) (on_board yes) (dnp no)
@@
     )
   )
-  (symbol (lib_id "Device:C") (at 83.82 173.99 0) (unit 1)
-    (in_bom yes) (on_board yes) (dnp no) (fields_autoplaced)
-    (property "Reference" "C38" (at 87.122 172.72 0)
-      (effects (font (size 1.27 1.27)) (justify left))
-    )
-    (property "Value" "100nC" (at 87.122 175.26 0)
-      (effects (font (size 1.27 1.27)) (justify left))
-    )
-    (property "Footprint" "Capacitor_SMD:C_0805_2012Metric" (at 84.7852 177.8 0)
-      (effects (font (size 1.27 1.27)) hide)
-    )
-    (property "Datasheet" "https://datasheet.lcsc.com/lcsc/1810191215_Samsung-Electro-Mechanics-CL21B104KBCNNNC_C1711.pdf" (at 83.82 173.99 0)
-      (effects (font (size 1.27 1.27)) hide)
-    )
-    (property "MPN" "CL21B104KBCNNNC" (at 83.82 173.99 0)
-      (effects (font (size 1.27 1.27)) hide)
-    )
-    (property "Status" "" (at 83.82 173.99 0)
-      (effects (font (size 1.27 1.27)) hide)
-    )
-    (pin "1")
-    (pin "2")
-    (instances
-      (project "SCART_switcher"
-        (path "/8cd08eb5-4755-4ef5-8eeb-77fd9974b180/6562ea38-5963-42b2-a0ef-a4a12a4c652f/32c156af-ff54-4356-ac90-a2b1f82b1e02"
-          (reference "C38") (unit 1)
-        )
-      )
-    )
-  )
   (symbol (lib_id "power:+2V5") (at 39.37 133.35 180) (unit 1)
     (in_bom yes) (on_board yes) (dnp no) (fields_autoplaced)
@@
         (path "/8cd08eb5-4755-4ef5-8eeb-77fd9974b180/6562ea38-5963-42b2-a0ef-a4a12a4c652f/32c156af-ff54-4356-ac90-a2b1f82b1e02"
           (reference "U20") (unit 1)
-        )
-      )
-    )
-  )
-  (symbol (lib_id "power:GND") (at 83.82 177.8 0) (unit 1)
-    (in_bom yes) (on_board yes) (dnp no) (fields_autoplaced)
-    (property "Reference" "#PWR0268" (at 83.82 184.15 0)
-      (effects (font (size 1.27 1.27)) hide)
-    )
-    (property "Value" "GND" (at 83.82 182.88 0)
-      (effects (font (size 1.27 1.27)))
-    )
-    (property "Footprint" "" (at 83.82 177.8 0)
-      (effects (font (size 1.27 1.27)) hide)
-    )
-    (property "Datasheet" "" (at 83.82 177.8 0)
-      (effects (font (size 1.27 1.27)) hide)
-    )
-    (pin "1")
-    (instances
-      (project "SCART_switcher"
-        (path "/8cd08eb5-4755-4ef5-8eeb-77fd9974b180/6562ea38-5963-42b2-a0ef-a4a12a4c652f/32c156af-ff54-4356-ac90-a2b1f82b1e02"
-          (reference "#PWR0268") (unit 1)
         )
       )
@@
         )
       )
-    )
-  )
-  (symbol (lib_id "power:GND") (at 52.07 184.15 0) (unit 1)
-    (in_bom yes) (on_board yes) (dnp no) (fields_autoplaced)
-    (property "Reference" "#PWR0262" (at 52.07 190.5 0)
-      (effects (font (size 1.27 1.27)) hide)
-    )
-    (property "Value" "GND" (at 52.07 189.23 0)
-      (effects (font (size 1.27 1.27)))
-    )
-    (property "Footprint" "" (at 52.07 184.15 0)
-      (effects (font (size 1.27 1.27)) hide)
-    )
-    (property "Datasheet" "" (at 52.07 184.15 0)
-      (effects (font (size 1.27 1.27)) hide)
-    )
-    (pin "1")
-    (instances
-      (project "SCART_switcher"
-        (path "/8cd08eb5-4755-4ef5-8eeb-77fd9974b180/6562ea38-5963-42b2-a0ef-a4a12a4c652f/32c156af-ff54-4356-ac90-a2b1f82b1e02"
-          (reference "#PWR0262") (unit 1)
-        )
-      )

Commit message: Progressed ECAD
Parts:
- renumbered C39 to C2, C40 to C3, C41 to C4, C42 to C5, C43 to C6, C44 to C7, Q28 to Q4, Q29 to Q5, R98 to R10, R99 to R11, R100 to R12, R101 to R13, R102 to R14, R103 to R15, R104 to R16, R105 to R17, R106 to R18, R97 to R9, U20 to U2, U21 to U3, U22 to U4, U23 to U5, U24 to U6, U25 to U7

Commit message: Update dummy_input.kicad_sch
Parts:
- removed Q5: BC857, Package_TO_SOT_SMD:SOT-23, symbol Transistor_BJT:BC857
- removed R10: 10kR, Resistor_SMD:R_0805_2012Metric, symbol Device:R
- added Q5: BC847, Package_TO_SOT_SMD:SOT-23, symbol Transistor_BJT:BC847
- added R12: 4k7R, Resistor_SMD:R_0805_2012Metric, symbol Device:R
- R13, R9: value 47kR -> 10kR; MPN (none) -> RC0805FR-0710KL
- R14: value 10kR -> 4k7R; MPN RC0805FR-0710KL -> (none)
- renumbered R11 to R10, R12 to R11, U5 to U4, U4 to U5
Connections:
- net ENABLE is gone; now on net ~{OUT_ACTIVE}: R9.1, U2.6, U3.6, U4.1, U6.6, U7.6
- net +2V5: now also U2.1, U3.1, U6.1, U7.1; no longer U2.3, U3.3, U6.3, U7.3
- net +9V: now also R14.1, R12.1
- net AUDIO_OUT_ENABLE: now also R14.2, Q5.3 (C); no longer R14.1
- net BLUE: now also U6.3; no longer U6.1
- net GND: now also Q5.2 (E); no longer R14.2
- net GREEN: now also U2.3; no longer U2.1
- net RED: now also U3.3; no longer U3.1
- net VIDEO_RGB_SYNC: now also U7.3; no longer U7.1
- net at Q4.3 (C), R13.1: now also R12.2
- net at R13.2: now also Q5.1 (B)
Other:
- note removed: "Dummy input enable is active low"
- moved on the sheet: R15, R18, U2A, U3A, U5A, U5B, U5C, U5D, U6A, U7A
