File: ECAD/SCART_switcher/dummy_input.kicad_sch (KiCad schematic)
At the start: 24 parts, among them Q4 BC847, Q5 BC847, U2 74LVC1G3157, U3 74LVC1G3157, U4 74LVC1G126, U5 CD4066, U6 74LVC1G3157, U7 74LVC1G3157

Commit message: Progressed ECAD.
Parts:
- removed Q4: BC847, Package_TO_SOT_SMD:SOT-23, symbol Transistor_BJT:BC847
- removed R12: 4k7R, Resistor_SMD:R_0805_2012Metric, symbol Device:R
- removed R9: 10kR, Resistor_SMD:R_0805_2012Metric, symbol Device:R
- added C2: 100nC, Capacitor_SMD:C_0805_2012Metric, symbol Device:C
- added U2: 74LVC1G04, Package_TO_SOT_SMD:SOT-353_SC-70-5, symbol 74xGxx:74AHC1G04
- renumbered C2 to C3, C3 to C4, C4 to C5, C5 to C6, C6 to C7, C7 to C8, Q5 to Q4, R11 to R10, R13 to R11, R14 to R12, R15 to R13, R16 to R14, R17 to R15, R18 to R16, R10 to R9, U2 to U3, U3 to U4, U4 to U5, U5 to U6, U6 to U7, U7 to U8
Connections:
- net +5V: now also C2.1, U2.5 (VCC)
- net GND: now also C2.2, U2.3 (GND)
- net ~{OUT_ACTIVE}: now also U2.2
- net at R11.1: now also U2.4
Other:
- moved on the sheet: C8, Q4, R11, R12, R13, R16, U6A, U6B, U6C, U6D, U6E

Commit message: Progressed ECAD.
Parts:
- renumbered C2 to C3, C3 to C4, C4 to C5, C5 to C6, C6 to C7, C7 to C8, C8 to C9, Q4 to Q5, R9 to R11, R10 to R12, R11 to R13, R12 to R14, R13 to R15, R14 to R16, R15 to R17, R16 to R18, U2 to U3, U3 to U4, U4 to U5, U5 to U6, U6 to U7, U7 to U8, U8 to U9

Commit message: Progressed ECAD.
Parts:
- renumbered C9 to C10, C3 to C4, C4 to C5, C5 to C6, C6 to C7, C7 to C8, C8 to C9, U9 to U10, U3 to U4, U4 to U5, U5 to U6, U6 to U7, U7 to U8, U8 to U9

Commit message: Progressed ECAD.
Parts:
- C10, C4, C5, C6, C7, C8, C9: footprint Capacitor_SMD:C_0805_2012Metric -> Capacitor_SMD:C_0603_1608Metric
Changed lines of the file:
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@@
       (effects (font (size 1.27 1.27)) (justify left))
     )
-    (property "Footprint" "Capacitor_SMD:C_0805_2012Metric" (at 253.6952 40.64 0)
+    (property "Footprint" "Capacitor_SMD:C_0603_1608Metric" (at 253.6952 40.64 0)
       (effects (font (size 1.27 1.27)) hide)
     )
@@
       (effects (font (size 1.27 1.27)) (justify left))
     )
-    (property "Footprint" "Capacitor_SMD:C_0805_2012Metric" (at 220.6752 86.36 0)
+    (property "Footprint" "Capacitor_SMD:C_0603_1608Metric" (at 220.6752 86.36 0)
       (effects (font (size 1.27 1.27)) hide)
     )
@@
       (effects (font (size 1.27 1.27)) (justify left))
     )
-    (property "Footprint" "Capacitor_SMD:C_0805_2012Metric" (at 16.2052 44.45 0)
+    (property "Footprint" "Capacitor_SMD:C_0603_1608Metric" (at 16.2052 44.45 0)
       (effects (font (size 1.27 1.27)) hide)
     )
@@
       (effects (font (size 1.27 1.27)) (justify left))
     )
-    (property "Footprint" "Capacitor_SMD:C_0805_2012Metric" (at 96.2152 86.36 0)
+    (property "Footprint" "Capacitor_SMD:C_0603_1608Metric" (at 96.2152 86.36 0)
       (effects (font (size 1.27 1.27)) hide)
     )
@@
       (effects (font (size 1.27 1.27)) (justify left))
     )
-    (property "Footprint" "Capacitor_SMD:C_0805_2012Metric" (at 96.2152 128.27 0)
+    (property "Footprint" "Capacitor_SMD:C_0603_1608Metric" (at 96.2152 128.27 0)
       (effects (font (size 1.27 1.27)) hide)
     )
@@
       (effects (font (size 1.27 1.27)) (justify left))
     )
-    (property "Footprint" "Capacitor_SMD:C_0805_2012Metric" (at 220.6752 127 0)
+    (property "Footprint" "Capacitor_SMD:C_0603_1608Metric" (at 220.6752 127 0)
       (effects (font (size 1.27 1.27)) hide)
     )
@@
       (effects (font (size 1.27 1.27)) (justify left))
     )
-    (property "Footprint" "Capacitor_SMD:C_0805_2012Metric" (at 157.1752 177.8 0)
-      (effects (font (size 1.27 1.27)) hide)
-    )
+    (property "Footprint" "Capacitor_SMD:C_0603_1608Metric" (at 157.1752 177.8 0)
+      (effects (font (size 1.27 1.27)) hide)
+    )

Commit message: Progressed ECAD.
Parts:
- removed U7: 74LVC1G126, Package_TO_SOT_SMD:SOT-353_SC-70-5, symbol 74xGxx:74AHC1G126
- added U7: 74LVC1G3157, Package_TO_SOT_SMD:SOT-363_SC-70-6, symbol Analog_Switch:TS5A63157DBV
Connections:
- net +5V: now also U7.5 (V+)
- net BLANKING: now also U7.3
- net GND: now also U7.1, U7.2 (GND), U7.4
- net ~{OUT_ACTIVE}: now also U7.6
Other:
- note removed: "Dummy BLANKING input"

Commit message: Progressed ECAD.
Other:
- note added: "I_{on}=1mA"
- note added: "I_{on}=2mA"
Changed lines of the file:
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@@
     (stroke (width 0) (type default))
+  )
+  (text "I_{on}=1mA" (at 45.72 24.13 0)
+    (effects (font (size 1.27 1.27)) (justify left bottom))
   )
   (text "Dummy video (zero level) input" (at 128.27 63.5 0)
@@
     (effects (font (size 1.27 1.27)) (justify left bottom))
   )
+  (text "I_{on}=2mA" (at 78.74 21.59 0)
+    (effects (font (size 1.27 1.27)) (justify left bottom))
+  )

Commit message: Progressed ECAD.
Parts:
- R11, R12, R15, R16, R17, R18: MPN (none) -> RC0805FR-07100KL; Status (none) -> OK
- R13: MPN RC0805FR-0710KL -> AC0805FR-0710KL; Status (none) -> OK
Changed lines of the file:
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@@
       (effects (font (size 1.27 1.27)) hide)
     )
-    (property "Datasheet" "~" (at 39.37 129.54 0)
-      (effects (font (size 1.27 1.27)) hide)
-    )
-    (property "Status" "" (at 39.37 129.54 0)
+    (property "Datasheet" "https://datasheet.lcsc.com/lcsc/2304140030_YAGEO-RC0805FR-07100KL_C96346.pdf" (at 39.37 129.54 0)
+      (effects (font (size 1.27 1.27)) hide)
+    )
+    (property "Status" "OK" (at 39.37 129.54 0)
+      (effects (font (size 1.27 1.27)) hide)
+    )
+    (property "MPN" "RC0805FR-07100KL" (at 39.37 129.54 0)
       (effects (font (size 1.27 1.27)) hide)
     )
@@
       (effects (font (size 1.27 1.27)) hide)
     )
-    (property "Datasheet" "~" (at 163.83 128.27 0)
-      (effects (font (size 1.27 1.27)) hide)
-    )
-    (property "Status" "" (at 163.83 128.27 0)
+    (property "Datasheet" "https://datasheet.lcsc.com/lcsc/2304140030_YAGEO-RC0805FR-07100KL_C96346.pdf" (at 163.83 128.27 0)
+      (effects (font (size 1.27 1.27)) hide)
+    )
+    (property "Status" "OK" (at 163.83 128.27 0)
+      (effects (font (size 1.27 1.27)) hide)
+    )
+    (property "MPN" "RC0805FR-07100KL" (at 163.83 128.27 0)
       (effects (font (size 1.27 1.27)) hide)
     )
@@
       (effects (font (size 1.27 1.27)) hide)
     )
-    (property "Datasheet" "~" (at 184.15 44.45 0)
-      (effects (font (size 1.27 1.27)) hide)
-    )
-    (property "Status" "" (at 184.15 44.45 0)
+    (property "Datasheet" "https://datasheet.lcsc.com/lcsc/2304140030_YAGEO-RC0805FR-07100KL_C96346.pdf" (at 184.15 44.45 0)
+      (effects (font (size 1.27 1.27)) hide)
+    )
+    (property "Status" "OK" (at 184.15 44.45 0)
+      (effects (font (size 1.27 1.27)) hide)
+    )
+    (property "MPN" "RC0805FR-07100KL" (at 184.15 44.45 0)
       (effects (font (size 1.27 1.27)) hide)
     )
@@
       (effects (font (size 1.27 1.27)) hide)
     )
-    (property "Datasheet" "https://datasheet.lcsc.com/lcsc/1810201611_YAGEO-RC0805FR-0710KL_C84376.pdf" (at 71.12 40.64 0)
-      (effects (font (size 1.27 1.27)) hide)
-    )
-    (property "MPN" "RC0805FR-0710KL" (at 71.12 40.64 0)
-      (effects (font (size 1.27 1.27)) hide)
-    )
-    (property "Status" "" (at 71.12 40.64 0)
+    (property "Datasheet" "https://datasheet.lcsc.com/lcsc/2304140030_YAGEO-AC0805FR-0710KL_C140868.pdf" (at 71.12 40.64 0)
+      (effects (font (size 1.27 1.27)) hide)
+    )
+    (property "MPN" "AC0805FR-0710KL" (at 71.12 40.64 0)
+      (effects (font (size 1.27 1.27)) hide)
+    )
+    (property "Status" "OK" (at 71.12 40.64 0)
       (effects (font (size 1.27 1.27)) hide)
     )
@@
       (effects (font (size 1.27 1.27)) hide)
     )
-    (property "Datasheet" "~" (at 39.37 87.63 0)
-      (effects (font (size 1.27 1.27)) hide)
-    )
-    (property "Status" "" (at 39.37 87.63 0)
+    (property "Datasheet" "https://datasheet.lcsc.com/lcsc/2304140030_YAGEO-RC0805FR-07100KL_C96346.pdf" (at 39.37 87.63 0)
+      (effects (font (size 1.27 1.27)) hide)
+    )
+    (property "Status" "OK" (at 39.37 87.63 0)
+      (effects (font (size 1.27 1.27)) hide)
+    )
+    (property "MPN" "RC0805FR-07100KL" (at 39.37 87.63 0)
       (effects (font (size 1.27 1.27)) hide)
     )
@@
       (effects (font (size 1.27 1.27)) hide)
     )
-    (property "Datasheet" "~" (at 163.83 87.63 0)
-      (effects (font (size 1.27 1.27)) hide)
-    )
-    (property "Status" "" (at 163.83 87.63 0)
+    (property "Datasheet" "https://datasheet.lcsc.com/lcsc/2304140030_YAGEO-RC0805FR-07100KL_C96346.pdf" (at 163.83 87.63 0)
+      (effects (font (size 1.27 1.27)) hide)
+    )
+    (property "Status" "OK" (at 163.83 87.63 0)
+      (effects (font (size 1.27 1.27)) hide)
+    )
+    (property "MPN" "RC0805FR-07100KL" (at 163.83 87.63 0)
       (effects (font (size 1.27 1.27)) hide)
     )
@@
       (effects (font (size 1.27 1.27)) hide)
     )
-    (property "Datasheet" "~" (at 116.84 44.45 0)
-      (effects (font (size 1.27 1.27)) hide)
-    )
-    (property "Status" "" (at 116.84 44.45 0)
-      (effects (font (size 1.27 1.27)) hide)
-    )
+    (property "Datasheet" "https://datasheet.lcsc.com/lcsc/2304140030_YAGEO-RC0805FR-07100KL_C96346.pdf" (at 116.84 44.45 0)
+      (effects (font (size 1.27 1.27)) hide)
+    )
+    (property "Status" "OK" (at 116.84 44.45 0)
+      (effects (font (size 1.27 1.27)) hide)
+    )
+    (property "MPN" "RC0805FR-07100KL" (at 116.84 44.45 0)
+      (effects (font (size 1.27 1.27)) hide)
+    )
