File: ECAD/SCART_switcher/video_out.kicad_sch (KiCad schematic)
At the start: 36 parts, among them U55 AD8054, U57 AD8054

Commit message: ERC fixes.
Connections:
- net VIDEO/RGB_SYNC_IN renamed VIDEO_RGB_SYNC_IN
- net VIDEO/RGB_SYNC_OUT renamed VIDEO_RGB_SYNC_OUT

Commit message: Progressed ECAD. Error fixing and cleanup.
Parts:
- renumbered U55 to U54, U57 to U56

Commit message: Progressed ECAD.
Parts:
- R?: MPN (none) -> RC0805FR-0710KL
- U?: MFN 74AHC1G04W5-7 -> (none); MPN (none) -> 74AHC1G04W5-7
Changed lines of the file:
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@@
-      (effects (font (size 1.27 1.27)) hide)
-    )
-    (property "MFN" "" (at 229.87 40.64 0)
       (effects (font (size 1.27 1.27)) hide)
     )
@@
     )
     (property "Datasheet" "https://datasheet.lcsc.com/lcsc/1810191215_Samsung-Electro-Mechanics-CL21B104KBCNNNC_C1711.pdf" (at 80.01 114.3 0)
-      (effects (font (size 1.27 1.27)) hide)
-    )
-    (property "MFN" "" (at 80.01 114.3 0)
       (effects (font (size 1.27 1.27)) hide)
     )
@@
       (effects (font (size 1.27 1.27)) hide)
     )
-    (property "MFN" "" (at 241.3 81.28 0)
-      (effects (font (size 1.27 1.27)) hide)
-    )
     (pin "1")
     (pin "2")
@@
       (effects (font (size 1.27 1.27)) hide)
     )
-    (property "MFN" "" (at 59.69 34.29 0)
-      (effects (font (size 1.27 1.27)) hide)
-    )
     (pin "1")
     (pin "2")
@@
       (effects (font (size 1.27 1.27)) hide)
     )
-    (property "MFN" "" (at 181.61 71.12 0)
-      (effects (font (size 1.27 1.27)) hide)
-    )
     (pin "1")
     (pin "2")
@@
       (effects (font (size 1.27 1.27)) hide)
     )
-    (property "Datasheet" "~" (at 90.17 165.1 0)
-      (effects (font (size 1.27 1.27)) hide)
-    )
-    (property "MFN" "" (at 90.17 165.1 0)
+    (property "Datasheet" "https://datasheet.lcsc.com/lcsc/1810201611_YAGEO-RC0805FR-0710KL_C84376.pdf" (at 90.17 165.1 0)
+      (effects (font (size 1.27 1.27)) hide)
+    )
+    (property "MPN" "RC0805FR-0710KL" (at 90.17 165.1 0)
       (effects (font (size 1.27 1.27)) hide)
     )
@@
       (effects (font (size 1.27 1.27)) hide)
     )
-    (property "MFN" "" (at 229.87 85.09 0)
-      (effects (font (size 1.27 1.27)) hide)
-    )
     (property "MPN" "CL21B104KBCNNNC" (at 229.87 85.09 0)
       (effects (font (size 1.27 1.27)) hide)
@@
       (effects (font (size 1.27 1.27)) hide)
     )
-    (property "MFN" "" (at 139.7 165.1 0)
-      (effects (font (size 1.27 1.27)) hide)
-    )
     (property "MPN" "CL21B104KBCNNNC" (at 139.7 165.1 0)
       (effects (font (size 1.27 1.27)) hide)
@@
       (effects (font (size 1.27 1.27)) hide)
     )
-    (property "MFN" "" (at 107.95 85.09 0)
-      (effects (font (size 1.27 1.27)) hide)
-    )
     (property "MPN" "CL21B104KBCNNNC" (at 107.95 85.09 0)
       (effects (font (size 1.27 1.27)) hide)
@@
       (effects (font (size 1.27 1.27)) hide)
     )
-    (property "MFN" "" (at 107.95 48.26 0)
-      (effects (font (size 1.27 1.27)) hide)
-    )
     (property "MPN" "CL21B104KBCNNNC" (at 107.95 48.26 0)
       (effects (font (size 1.27 1.27)) hide)
@@
     )
     (property "Datasheet" "~" (at 107.95 40.64 0)
-      (effects (font (size 1.27 1.27)) hide)
-    )
-    (property "MFN" "" (at 107.95 40.64 0)
       (effects (font (size 1.27 1.27)) hide)
     )
@@
       (effects (font (size 1.27 1.27)) hide)
     )
-    (property "MFN" "" (at 196.85 41.91 0)
-      (effects (font (size 1.27 1.27)) hide)
-    )
     (pin "1")
     (pin "2")
@@
       (effects (font (size 1.27 1.27)) hide)
     )
-    (property "MFN" "" (at 229.87 77.47 0)
-      (effects (font (size 1.27 1.27)) hide)
-    )
     (pin "1")
     (pin "2")
@@
     )
     (property "Datasheet" "~" (at 119.38 44.45 0)
-      (effects (font (size 1.27 1.27)) hide)
-    )
-    (property "MFN" "" (at 119.38 44.45 0)
       (effects (font (size 1.27 1.27)) hide)
     )
@@
       (effects (font (size 1.27 1.27)) hide)
     )
-    (property "MFN" "" (at 241.3 44.45 0)
-      (effects (font (size 1.27 1.27)) hide)
-    )
     (pin "1")
     (pin "2")
@@
       (effects (font (size 1.27 1.27)) hide)
     )
-    (property "MFN" "" (at 90.17 36.83 0)
-      (effects (font (size 1.27 1.27)) hide)
-    )
     (pin "1")
     (pin "2")
@@
       (effects (font (size 1.27 1.27)) hide)
     )
-    (property "MFN" "" (at 90.17 73.66 0)
-      (effects (font (size 1.27 1.27)) hide)
-    )
     (pin "1")
     (pin "2")
@@
       (effects (font (size 1.27 1.27)) hide)
     )
-    (property "MFN" "" (at 181.61 34.29 0)
-      (effects (font (size 1.27 1.27)) hide)
-    )
     (pin "1")
     (pin "2")
@@
     )
     (property "Datasheet" "~" (at 196.85 78.74 0)
-      (effects (font (size 1.27 1.27)) hide)
-    )
-    (property "MFN" "" (at 196.85 78.74 0)
       (effects (font (size 1.27 1.27)) hide)
     )
@@
       (effects (font (size 1.27 1.27)) hide)
     )
-    (property "MFN" "" (at 101.6 173.99 0)
-      (effects (font (size 1.27 1.27)) hide)
-    )
     (pin "1")
     (pin "2")
@@
       (effects (font (size 1.27 1.27)) hide)
     )
-    (property "MFN" "" (at 74.93 78.74 0)
-      (effects (font (size 1.27 1.27)) hide)
-    )
     (pin "1")
     (pin "2")
@@
       (effects (font (size 1.27 1.27)) hide)
     )
-    (property "MFN" "" (at 212.09 73.66 0)
-      (effects (font (size 1.27 1.27)) hide)
-    )
     (pin "1")
     (pin "2")
@@
     )
     (property "Datasheet" "~" (at 107.95 77.47 0)
-      (effects (font (size 1.27 1.27)) hide)
-    )
-    (property "MFN" "" (at 107.95 77.47 0)
       (effects (font (size 1.27 1.27)) hide)
     )
@@
       (effects (font (size 1.27 1.27)) hide)
     )
-    (property "MFN" "" (at 119.38 81.28 0)
-      (effects (font (size 1.27 1.27)) hide)
-    )
     (pin "1")
     (pin "2")
@@
       (effects (font (size 1.27 1.27)) hide)
     )
-    (property "MFN" "" (at 201.93 114.3 0)
-      (effects (font (size 1.27 1.27)) hide)
-    )
     (property "MPN" "CL21B104KBCNNNC" (at 201.93 114.3 0)
       (effects (font (size 1.27 1.27)) hide)
@@
     )
     (property "Datasheet" "~" (at 212.09 36.83 0)
-      (effects (font (size 1.27 1.27)) hide)
-    )
-    (property "MFN" "" (at 212.09 36.83 0)
       (effects (font (size 1.27 1.27)) hide)
     )
@@
       (effects (font (size 1.27 1.27)) hide)
     )
-    (property "MFN" "" (at 229.87 48.26 0)
-      (effects (font (size 1.27 1.27)) hide)
-    )
     (property "MPN" "CL21B104KBCNNNC" (at 229.87 48.26 0)
       (effects (font (size 1.27 1.27)) hide)
@@
       (effects (font (size 1.27 1.27)) hide)
     )
-    (property "MFN" "" (at 74.93 41.91 0)
-      (effects (font (size 1.27 1.27)) hide)
-    )
     (pin "1")
     (pin "2")
@@
     )
     (property "Datasheet" "~" (at 59.69 71.12 0)
-      (effects (font (size 1.27 1.27)) hide)
-    )
-    (property "MFN" "" (at 59.69 71.12 0)
       (effects (font (size 1.27 1.27)) hide)
     )
@@
       (effects (font (size 1.27 1.27)) hide)
     )
-    (property "MFN" "74AHC1G04W5-7" (at 73.66 165.1 0)
-      (effects (font (size 1.27 1.27)) hide)
-    )
+    (property "MPN" "74AHC1G04W5-7" (at 73.66 165.1 0)
+      (effects (font (size 1.27 1.27)) hide)
+    )

Commit message: Progressed ECAD.
Parts:
- renumbered U54 to U61, U56 to U63

Commit message: Progressed ECAD.
Parts:
- C? (x7): footprint Capacitor_SMD:C_0805_2012Metric_Pad1.18x1.45mm_HandSolder -> Capacitor_SMD:C_0805_2012Metric
- R? (x4): footprint Resistor_SMD:R_1210_3225Metric_Pad1.30x2.65mm_HandSolder -> Resistor_SMD:R_1210_3225Metric
- R? (x15): footprint Resistor_SMD:R_0805_2012Metric_Pad1.20x1.40mm_HandSolder -> Resistor_SMD:R_0805_2012Metric
Changed lines of the file:
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@@
       (effects (font (size 1.27 1.27)) (justify left))
     )
-    (property "Footprint" "Capacitor_SMD:C_0805_2012Metric_Pad1.18x1.45mm_HandSolder" (at 80.9752 118.11 0)
+    (property "Footprint" "Capacitor_SMD:C_0805_2012Metric" (at 80.9752 118.11 0)
       (effects (font (size 1.27 1.27)) hide)
     )
@@
       (effects (font (size 1.27 1.27)))
     )
-    (property "Footprint" "Resistor_SMD:R_1210_3225Metric_Pad1.30x2.65mm_HandSolder" (at 241.3 83.058 90)
+    (property "Footprint" "Resistor_SMD:R_1210_3225Metric" (at 241.3 83.058 90)
       (effects (font (size 1.27 1.27)) hide)
     )
@@
       (effects (font (size 1.27 1.27)))
     )
-    (property "Footprint" "Resistor_SMD:R_0805_2012Metric_Pad1.20x1.40mm_HandSolder" (at 59.69 36.068 90)
+    (property "Footprint" "Resistor_SMD:R_0805_2012Metric" (at 59.69 36.068 90)
       (effects (font (size 1.27 1.27)) hide)
     )
@@
       (effects (font (size 1.27 1.27)))
     )
-    (property "Footprint" "Resistor_SMD:R_0805_2012Metric_Pad1.20x1.40mm_HandSolder" (at 181.61 72.898 90)
+    (property "Footprint" "Resistor_SMD:R_0805_2012Metric" (at 181.61 72.898 90)
       (effects (font (size 1.27 1.27)) hide)
     )
@@
       (effects (font (size 1.27 1.27)))
     )
-    (property "Footprint" "Resistor_SMD:R_0805_2012Metric_Pad1.20x1.40mm_HandSolder" (at 90.17 163.322 90)
+    (property "Footprint" "Resistor_SMD:R_0805_2012Metric" (at 90.17 163.322 90)
       (effects (font (size 1.27 1.27)) hide)
     )
@@
       (effects (font (size 1.27 1.27)))
     )
-    (property "Footprint" "Capacitor_SMD:C_0805_2012Metric_Pad1.18x1.45mm_HandSolder" (at 226.06 84.1248 0)
+    (property "Footprint" "Capacitor_SMD:C_0805_2012Metric" (at 226.06 84.1248 0)
       (effects (font (size 1.27 1.27)) hide)
     )
@@
       (effects (font (size 1.27 1.27)) (justify left))
     )
-    (property "Footprint" "Capacitor_SMD:C_0805_2012Metric_Pad1.18x1.45mm_HandSolder" (at 140.6652 168.91 0)
+    (property "Footprint" "Capacitor_SMD:C_0805_2012Metric" (at 140.6652 168.91 0)
       (effects (font (size 1.27 1.27)) hide)
     )
@@
       (effects (font (size 1.27 1.27)))
     )
-    (property "Footprint" "Capacitor_SMD:C_0805_2012Metric_Pad1.18x1.45mm_HandSolder" (at 104.14 84.1248 0)
+    (property "Footprint" "Capacitor_SMD:C_0805_2012Metric" (at 104.14 84.1248 0)
       (effects (font (size 1.27 1.27)) hide)
     )
@@
       (effects (font (size 1.27 1.27)))
     )
-    (property "Footprint" "Capacitor_SMD:C_0805_2012Metric_Pad1.18x1.45mm_HandSolder" (at 104.14 47.2948 0)
+    (property "Footprint" "Capacitor_SMD:C_0805_2012Metric" (at 104.14 47.2948 0)
       (effects (font (size 1.27 1.27)) hide)
     )
@@
       (effects (font (size 1.27 1.27)))
     )
-    (property "Footprint" "Resistor_SMD:R_0805_2012Metric_Pad1.20x1.40mm_HandSolder" (at 111.76 171.958 90)
+    (property "Footprint" "Resistor_SMD:R_0805_2012Metric" (at 111.76 171.958 90)
       (effects (font (size 1.27 1.27)) hide)
     )
@@
       (effects (font (size 1.27 1.27)))
     )
-    (property "Footprint" "Resistor_SMD:R_0805_2012Metric_Pad1.20x1.40mm_HandSolder" (at 196.85 43.688 90)
+    (property "Footprint" "Resistor_SMD:R_0805_2012Metric" (at 196.85 43.688 90)
       (effects (font (size 1.27 1.27)) hide)
     )
@@
       (effects (font (size 1.27 1.27)))
     )
-    (property "Footprint" "Resistor_SMD:R_1210_3225Metric_Pad1.30x2.65mm_HandSolder" (at 119.38 46.228 90)
+    (property "Footprint" "Resistor_SMD:R_1210_3225Metric" (at 119.38 46.228 90)
       (effects (font (size 1.27 1.27)) hide)
     )
@@
       (effects (font (size 1.27 1.27)))
     )
-    (property "Footprint" "Resistor_SMD:R_1210_3225Metric_Pad1.30x2.65mm_HandSolder" (at 241.3 46.228 90)
+    (property "Footprint" "Resistor_SMD:R_1210_3225Metric" (at 241.3 46.228 90)
       (effects (font (size 1.27 1.27)) hide)
     )
@@
       (effects (font (size 1.27 1.27)))
     )
-    (property "Footprint" "Resistor_SMD:R_0805_2012Metric_Pad1.20x1.40mm_HandSolder" (at 90.17 38.608 90)
+    (property "Footprint" "Resistor_SMD:R_0805_2012Metric" (at 90.17 38.608 90)
       (effects (font (size 1.27 1.27)) hide)
     )
@@
       (effects (font (size 1.27 1.27)))
     )
-    (property "Footprint" "Resistor_SMD:R_0805_2012Metric_Pad1.20x1.40mm_HandSolder" (at 90.17 75.438 90)
+    (property "Footprint" "Resistor_SMD:R_0805_2012Metric" (at 90.17 75.438 90)
       (effects (font (size 1.27 1.27)) hide)
     )
@@
       (effects (font (size 1.27 1.27)))
     )
-    (property "Footprint" "Resistor_SMD:R_0805_2012Metric_Pad1.20x1.40mm_HandSolder" (at 181.61 36.068 90)
+    (property "Footprint" "Resistor_SMD:R_0805_2012Metric" (at 181.61 36.068 90)
       (effects (font (size 1.27 1.27)) hide)
     )
@@
       (effects (font (size 1.27 1.27)))
     )
-    (property "Footprint" "Resistor_SMD:R_0805_2012Metric_Pad1.20x1.40mm_HandSolder" (at 196.85 80.518 90)
+    (property "Footprint" "Resistor_SMD:R_0805_2012Metric" (at 196.85 80.518 90)
       (effects (font (size 1.27 1.27)) hide)
     )
@@
       (effects (font (size 1.27 1.27)) (justify left))
     )
-    (property "Footprint" "Resistor_SMD:R_0805_2012Metric_Pad1.20x1.40mm_HandSolder" (at 103.378 173.99 90)
+    (property "Footprint" "Resistor_SMD:R_0805_2012Metric" (at 103.378 173.99 90)
       (effects (font (size 1.27 1.27)) hide)
     )
@@
       (effects (font (size 1.27 1.27)))
     )
-    (property "Footprint" "Resistor_SMD:R_0805_2012Metric_Pad1.20x1.40mm_HandSolder" (at 74.93 80.518 90)
+    (property "Footprint" "Resistor_SMD:R_0805_2012Metric" (at 74.93 80.518 90)
       (effects (font (size 1.27 1.27)) hide)
     )
@@
       (effects (font (size 1.27 1.27)))
     )
-    (property "Footprint" "Resistor_SMD:R_0805_2012Metric_Pad1.20x1.40mm_HandSolder" (at 212.09 75.438 90)
+    (property "Footprint" "Resistor_SMD:R_0805_2012Metric" (at 212.09 75.438 90)
       (effects (font (size 1.27 1.27)) hide)
     )
@@
       (effects (font (size 1.27 1.27)))
     )
-    (property "Footprint" "Resistor_SMD:R_1210_3225Metric_Pad1.30x2.65mm_HandSolder" (at 119.38 83.058 90)
+    (property "Footprint" "Resistor_SMD:R_1210_3225Metric" (at 119.38 83.058 90)
       (effects (font (size 1.27 1.27)) hide)
     )
@@
       (effects (font (size 1.27 1.27)) (justify left))
     )
-    (property "Footprint" "Capacitor_SMD:C_0805_2012Metric_Pad1.18x1.45mm_HandSolder" (at 202.8952 118.11 0)
+    (property "Footprint" "Capacitor_SMD:C_0805_2012Metric" (at 202.8952 118.11 0)
       (effects (font (size 1.27 1.27)) hide)
     )
@@
       (effects (font (size 1.27 1.27)))
     )
-    (property "Footprint" "Resistor_SMD:R_0805_2012Metric_Pad1.20x1.40mm_HandSolder" (at 212.09 38.608 90)
+    (property "Footprint" "Resistor_SMD:R_0805_2012Metric" (at 212.09 38.608 90)
       (effects (font (size 1.27 1.27)) hide)
     )
@@
       (effects (font (size 1.27 1.27)))
     )
-    (property "Footprint" "Capacitor_SMD:C_0805_2012Metric_Pad1.18x1.45mm_HandSolder" (at 226.06 47.2948 0)
+    (property "Footprint" "Capacitor_SMD:C_0805_2012Metric" (at 226.06 47.2948 0)
       (effects (font (size 1.27 1.27)) hide)
     )
@@
       (effects (font (size 1.27 1.27)))
     )
-    (property "Footprint" "Resistor_SMD:R_0805_2012Metric_Pad1.20x1.40mm_HandSolder" (at 74.93 43.688 90)
+    (property "Footprint" "Resistor_SMD:R_0805_2012Metric" (at 74.93 43.688 90)
       (effects (font (size 1.27 1.27)) hide)
     )
@@
       (effects (font (size 1.27 1.27)))
     )
-    (property "Footprint" "Resistor_SMD:R_0805_2012Metric_Pad1.20x1.40mm_HandSolder" (at 59.69 72.898 90)
-      (effects (font (size 1.27 1.27)) hide)
-    )
+    (property "Footprint" "Resistor_SMD:R_0805_2012Metric" (at 59.69 72.898 90)
+      (effects (font (size 1.27 1.27)) hide)
+    )

Commit message: progressed ecad
Parts:
- U61, U63: footprint Package_SO:SOIC-14_3.9x8.7mm_P1.27mm -> Package_SO:TSSOP-14_4.4x5mm_P0.65mm; MPN (none) -> GS8054-TR
Changed lines of the file:
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@@
       (effects (font (size 1.27 1.27)) (justify left))
     )
-    (property "Footprint" "Package_SO:SOIC-14_3.9x8.7mm_P1.27mm" (at 190.5 114.3 0)
-      (effects (font (size 1.27 1.27)) hide)
-    )
-    (property "Datasheet" "https://datasheet.lcsc.com/lcsc/2310091131_Analog-Devices-AD8054ARU-REEL7_C4370194.pdf" (at 190.5 114.3 0)
+    (property "Footprint" "Package_SO:TSSOP-14_4.4x5mm_P0.65mm" (at 190.5 114.3 0)
+      (effects (font (size 1.27 1.27)) hide)
+    )
+    (property "Datasheet" "https://datasheet.lcsc.com/lcsc/2310091129_Analog-Devices-AD8054ARU-REEL_C4368882.pdf" (at 190.5 114.3 0)
+      (effects (font (size 1.27 1.27)) hide)
+    )
+    (property "MPN" "GS8054-TR" (at 190.5 114.3 0)
       (effects (font (size 1.27 1.27)) hide)
     )
@@
       (effects (font (size 1.27 1.27)))
     )
-    (property "Footprint" "Package_SO:SOIC-14_3.9x8.7mm_P1.27mm" (at 212.09 44.45 0)
-      (effects (font (size 1.27 1.27)) hide)
-    )
-    (property "Datasheet" "https://datasheet.lcsc.com/lcsc/2310091131_Analog-Devices-AD8054ARU-REEL7_C4370194.pdf" (at 212.09 44.45 0)
+    (property "Footprint" "Package_SO:TSSOP-14_4.4x5mm_P0.65mm" (at 212.09 44.45 0)
+      (effects (font (size 1.27 1.27)) hide)
+    )
+    (property "Datasheet" "https://datasheet.lcsc.com/lcsc/2310091129_Analog-Devices-AD8054ARU-REEL_C4368882.pdf" (at 212.09 44.45 0)
+      (effects (font (size 1.27 1.27)) hide)
+    )
+    (property "MPN" "GS8054-TR" (at 212.09 44.45 0)
       (effects (font (size 1.27 1.27)) hide)
     )
@@
       (effects (font (size 1.27 1.27)))
     )
-    (property "Footprint" "Package_SO:SOIC-14_3.9x8.7mm_P1.27mm" (at 90.17 81.28 0)
-      (effects (font (size 1.27 1.27)) hide)
-    )
-    (property "Datasheet" "https://datasheet.lcsc.com/lcsc/2310091131_Analog-Devices-AD8054ARU-REEL7_C4370194.pdf" (at 90.17 81.28 0)
+    (property "Footprint" "Package_SO:TSSOP-14_4.4x5mm_P0.65mm" (at 90.17 81.28 0)
+      (effects (font (size 1.27 1.27)) hide)
+    )
+    (property "Datasheet" "https://datasheet.lcsc.com/lcsc/2310091129_Analog-Devices-AD8054ARU-REEL_C4368882.pdf" (at 90.17 81.28 0)
+      (effects (font (size 1.27 1.27)) hide)
+    )
+    (property "MPN" "GS8054-TR" (at 90.17 81.28 0)
       (effects (font (size 1.27 1.27)) hide)
     )
@@
       (effects (font (size 1.27 1.27)))
     )
-    (property "Footprint" "Package_SO:SOIC-14_3.9x8.7mm_P1.27mm" (at 181.61 41.91 0)
-      (effects (font (size 1.27 1.27)) hide)
-    )
-    (property "Datasheet" "https://datasheet.lcsc.com/lcsc/2310091131_Analog-Devices-AD8054ARU-REEL7_C4370194.pdf" (at 181.61 41.91 0)
+    (property "Footprint" "Package_SO:TSSOP-14_4.4x5mm_P0.65mm" (at 181.61 41.91 0)
+      (effects (font (size 1.27 1.27)) hide)
+    )
+    (property "Datasheet" "https://datasheet.lcsc.com/lcsc/2310091129_Analog-Devices-AD8054ARU-REEL_C4368882.pdf" (at 181.61 41.91 0)
+      (effects (font (size 1.27 1.27)) hide)
+    )
+    (property "MPN" "GS8054-TR" (at 181.61 41.91 0)
       (effects (font (size 1.27 1.27)) hide)
     )
@@
       (effects (font (size 1.27 1.27)))
     )
-    (property "Footprint" "Package_SO:SOIC-14_3.9x8.7mm_P1.27mm" (at 59.69 78.74 0)
-      (effects (font (size 1.27 1.27)) hide)
-    )
-    (property "Datasheet" "https://datasheet.lcsc.com/lcsc/2310091131_Analog-Devices-AD8054ARU-REEL7_C4370194.pdf" (at 59.69 78.74 0)
+    (property "Footprint" "Package_SO:TSSOP-14_4.4x5mm_P0.65mm" (at 59.69 78.74 0)
+      (effects (font (size 1.27 1.27)) hide)
+    )
+    (property "Datasheet" "https://datasheet.lcsc.com/lcsc/2310091129_Analog-Devices-AD8054ARU-REEL_C4368882.pdf" (at 59.69 78.74 0)
+      (effects (font (size 1.27 1.27)) hide)
+    )
+    (property "MPN" "GS8054-TR" (at 59.69 78.74 0)
       (effects (font (size 1.27 1.27)) hide)
     )
@@
       (effects (font (size 1.27 1.27)) (justify left))
     )
-    (property "Footprint" "Package_SO:SOIC-14_3.9x8.7mm_P1.27mm" (at 68.58 114.3 0)
-      (effects (font (size 1.27 1.27)) hide)
-    )
-    (property "Datasheet" "https://datasheet.lcsc.com/lcsc/2310091131_Analog-Devices-AD8054ARU-REEL7_C4370194.pdf" (at 68.58 114.3 0)
+    (property "Footprint" "Package_SO:TSSOP-14_4.4x5mm_P0.65mm" (at 68.58 114.3 0)
+      (effects (font (size 1.27 1.27)) hide)
+    )
+    (property "Datasheet" "https://datasheet.lcsc.com/lcsc/2310091129_Analog-Devices-AD8054ARU-REEL_C4368882.pdf" (at 68.58 114.3 0)
+      (effects (font (size 1.27 1.27)) hide)
+    )
+    (property "MPN" "GS8054-TR" (at 68.58 114.3 0)
       (effects (font (size 1.27 1.27)) hide)
     )
@@
       (effects (font (size 1.27 1.27)))
     )
-    (property "Footprint" "Package_SO:SOIC-14_3.9x8.7mm_P1.27mm" (at 181.61 78.74 0)
-      (effects (font (size 1.27 1.27)) hide)
-    )
-    (property "Datasheet" "https://datasheet.lcsc.com/lcsc/2310091131_Analog-Devices-AD8054ARU-REEL7_C4370194.pdf" (at 181.61 78.74 0)
+    (property "Footprint" "Package_SO:TSSOP-14_4.4x5mm_P0.65mm" (at 181.61 78.74 0)
+      (effects (font (size 1.27 1.27)) hide)
+    )
+    (property "Datasheet" "https://datasheet.lcsc.com/lcsc/2310091129_Analog-Devices-AD8054ARU-REEL_C4368882.pdf" (at 181.61 78.74 0)
+      (effects (font (size 1.27 1.27)) hide)
+    )
+    (property "MPN" "GS8054-TR" (at 181.61 78.74 0)
       (effects (font (size 1.27 1.27)) hide)
     )
@@
       (effects (font (size 1.27 1.27)))
     )
-    (property "Footprint" "Package_SO:SOIC-14_3.9x8.7mm_P1.27mm" (at 59.69 41.91 0)
-      (effects (font (size 1.27 1.27)) hide)
-    )
-    (property "Datasheet" "https://datasheet.lcsc.com/lcsc/2310091131_Analog-Devices-AD8054ARU-REEL7_C4370194.pdf" (at 59.69 41.91 0)
+    (property "Footprint" "Package_SO:TSSOP-14_4.4x5mm_P0.65mm" (at 59.69 41.91 0)
+      (effects (font (size 1.27 1.27)) hide)
+    )
+    (property "Datasheet" "https://datasheet.lcsc.com/lcsc/2310091129_Analog-Devices-AD8054ARU-REEL_C4368882.pdf" (at 59.69 41.91 0)
+      (effects (font (size 1.27 1.27)) hide)
+    )
+    (property "MPN" "GS8054-TR" (at 59.69 41.91 0)
       (effects (font (size 1.27 1.27)) hide)
     )
@@
       (effects (font (size 1.27 1.27)))
     )
-    (property "Footprint" "Package_SO:SOIC-14_3.9x8.7mm_P1.27mm" (at 212.09 81.28 0)
-      (effects (font (size 1.27 1.27)) hide)
-    )
-    (property "Datasheet" "https://datasheet.lcsc.com/lcsc/2310091131_Analog-Devices-AD8054ARU-REEL7_C4370194.pdf" (at 212.09 81.28 0)
+    (property "Footprint" "Package_SO:TSSOP-14_4.4x5mm_P0.65mm" (at 212.09 81.28 0)
+      (effects (font (size 1.27 1.27)) hide)
+    )
+    (property "Datasheet" "https://datasheet.lcsc.com/lcsc/2310091129_Analog-Devices-AD8054ARU-REEL_C4368882.pdf" (at 212.09 81.28 0)
+      (effects (font (size 1.27 1.27)) hide)
+    )
+    (property "MPN" "GS8054-TR" (at 212.09 81.28 0)
       (effects (font (size 1.27 1.27)) hide)
     )
@@
       (effects (font (size 1.27 1.27)))
     )
-    (property "Footprint" "Package_SO:SOIC-14_3.9x8.7mm_P1.27mm" (at 90.17 44.45 0)
-      (effects (font (size 1.27 1.27)) hide)
-    )
-    (property "Datasheet" "https://datasheet.lcsc.com/lcsc/2310091131_Analog-Devices-AD8054ARU-REEL7_C4370194.pdf" (at 90.17 44.45 0)
-      (effects (font (size 1.27 1.27)) hide)
-    )
+    (property "Footprint" "Package_SO:TSSOP-14_4.4x5mm_P0.65mm" (at 90.17 44.45 0)
+      (effects (font (size 1.27 1.27)) hide)
+    )
+    (property "Datasheet" "https://datasheet.lcsc.com/lcsc/2310091129_Analog-Devices-AD8054ARU-REEL_C4368882.pdf" (at 90.17 44.45 0)
+      (effects (font (size 1.27 1.27)) hide)
+    )
+    (property "MPN" "GS8054-TR" (at 90.17 44.45 0)
+      (effects (font (size 1.27 1.27)) hide)
+    )
