File: ECAD/SCART_switcher/video_out.kicad_sch (KiCad schematic)
At the start: 36 parts, among them U61 AD8054, U63 AD8054

Commit message: Progressed ECAD.
Parts:
- Q?: MPN (none) -> BC857C,215; Status (none) -> OK
Changed lines of the file:
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@@
+      (effects (font (size 1.27 1.27)) hide)
+    )
+    (property "Status" "" (at 229.87 40.64 0)
       (effects (font (size 1.27 1.27)) hide)
     )
@@
       (effects (font (size 1.27 1.27)) hide)
     )
+    (property "Status" "" (at 80.01 114.3 0)
+      (effects (font (size 1.27 1.27)) hide)
+    )
     (pin "1")
     (pin "2")
@@
     )
     (property "MPN" "GS8054-TR" (at 190.5 114.3 0)
+      (effects (font (size 1.27 1.27)) hide)
+    )
+    (property "Status" "" (at 190.5 114.3 0)
       (effects (font (size 1.27 1.27)) hide)
     )
@@
       (effects (font (size 1.27 1.27)) hide)
     )
+    (property "Status" "" (at 241.3 81.28 0)
+      (effects (font (size 1.27 1.27)) hide)
+    )
     (pin "1")
     (pin "2")
@@
     )
     (property "MPN" "GS8054-TR" (at 212.09 44.45 0)
+      (effects (font (size 1.27 1.27)) hide)
+    )
+    (property "Status" "" (at 212.09 44.45 0)
       (effects (font (size 1.27 1.27)) hide)
     )
@@
       (effects (font (size 1.27 1.27)) hide)
     )
+    (property "Status" "" (at 59.69 34.29 0)
+      (effects (font (size 1.27 1.27)) hide)
+    )
     (pin "1")
     (pin "2")
@@
       (effects (font (size 1.27 1.27)) hide)
     )
+    (property "Status" "" (at 181.61 71.12 0)
+      (effects (font (size 1.27 1.27)) hide)
+    )
     (pin "1")
     (pin "2")
@@
       (effects (font (size 1.27 1.27)) hide)
     )
+    (property "Status" "" (at 90.17 165.1 0)
+      (effects (font (size 1.27 1.27)) hide)
+    )
     (pin "1")
     (pin "2")
@@
     )
     (property "MPN" "GS8054-TR" (at 90.17 81.28 0)
+      (effects (font (size 1.27 1.27)) hide)
+    )
+    (property "Status" "" (at 90.17 81.28 0)
       (effects (font (size 1.27 1.27)) hide)
     )
@@
       (effects (font (size 1.27 1.27)) hide)
     )
+    (property "Status" "" (at 229.87 85.09 0)
+      (effects (font (size 1.27 1.27)) hide)
+    )
     (pin "1")
     (pin "2")
@@
       (effects (font (size 1.27 1.27)) hide)
     )
+    (property "Status" "" (at 139.7 165.1 0)
+      (effects (font (size 1.27 1.27)) hide)
+    )
     (pin "1")
     (pin "2")
@@
       (effects (font (size 1.27 1.27)) hide)
     )
+    (property "Status" "" (at 107.95 85.09 0)
+      (effects (font (size 1.27 1.27)) hide)
+    )
     (pin "1")
     (pin "2")
@@
       (effects (font (size 1.27 1.27)) hide)
     )
+    (property "Status" "" (at 107.95 48.26 0)
+      (effects (font (size 1.27 1.27)) hide)
+    )
     (pin "1")
     (pin "2")
@@
       (effects (font (size 1.27 1.27)) hide)
     )
+    (property "Status" "" (at 111.76 170.18 0)
+      (effects (font (size 1.27 1.27)) hide)
+    )
     (pin "1")
     (pin "2")
@@
     )
     (property "Datasheet" "~" (at 107.95 40.64 0)
+      (effects (font (size 1.27 1.27)) hide)
+    )
+    (property "Status" "" (at 107.95 40.64 0)
       (effects (font (size 1.27 1.27)) hide)
     )
@@
       (effects (font (size 1.27 1.27) italic) (justify left) hide)
     )
-    (property "Datasheet" "https://www.onsemi.com/pub/Collateral/BC860-D.pdf" (at 99.06 165.1 0)
+    (property "Datasheet" "https://datasheet.lcsc.com/lcsc/2304140030_Nexperia-BC857C-215_C8666.pdf" (at 99.06 165.1 0)
       (effects (font (size 1.27 1.27)) (justify left) hide)
+    )
+    (property "Status" "OK" (at 99.06 165.1 0)
+      (effects (font (size 1.27 1.27)) hide)
+    )
+    (property "MPN" "BC857C,215" (at 99.06 165.1 0)
+      (effects (font (size 1.27 1.27)) hide)
     )
     (pin "1")
@@
       (effects (font (size 1.27 1.27)) hide)
     )
+    (property "Status" "" (at 196.85 41.91 0)
+      (effects (font (size 1.27 1.27)) hide)
+    )
     (pin "1")
     (pin "2")
@@
       (effects (font (size 1.27 1.27)) hide)
     )
+    (property "Status" "" (at 229.87 77.47 0)
+      (effects (font (size 1.27 1.27)) hide)
+    )
     (pin "1")
     (pin "2")
@@
       (effects (font (size 1.27 1.27)) hide)
     )
+    (property "Status" "" (at 119.38 44.45 0)
+      (effects (font (size 1.27 1.27)) hide)
+    )
     (pin "1")
     (pin "2")
@@
     )
     (property "MPN" "GS8054-TR" (at 181.61 41.91 0)
+      (effects (font (size 1.27 1.27)) hide)
+    )
+    (property "Status" "" (at 181.61 41.91 0)
       (effects (font (size 1.27 1.27)) hide)
     )
@@
       (effects (font (size 1.27 1.27)) hide)
     )
+    (property "Status" "" (at 93.98 114.3 0)
+      (effects (font (size 1.27 1.27)) hide)
+    )
     (pin "1")
     (pin "2")
@@
       (effects (font (size 1.27 1.27)) hide)
     )
+    (property "Status" "" (at 241.3 44.45 0)
+      (effects (font (size 1.27 1.27)) hide)
+    )
     (pin "1")
     (pin "2")
@@
       (effects (font (size 1.27 1.27)) hide)
     )
+    (property "Status" "" (at 90.17 36.83 0)
+      (effects (font (size 1.27 1.27)) hide)
+    )
     (pin "1")
     (pin "2")
@@
       (effects (font (size 1.27 1.27)) hide)
     )
+    (property "Status" "" (at 90.17 73.66 0)
+      (effects (font (size 1.27 1.27)) hide)
+    )
     (pin "1")
     (pin "2")
@@
       (effects (font (size 1.27 1.27)) hide)
     )
+    (property "Status" "" (at 181.61 34.29 0)
+      (effects (font (size 1.27 1.27)) hide)
+    )
     (pin "1")
     (pin "2")
@@
       (effects (font (size 1.27 1.27)) hide)
     )
+    (property "Status" "" (at 196.85 78.74 0)
+      (effects (font (size 1.27 1.27)) hide)
+    )
     (pin "1")
     (pin "2")
@@
     )
     (property "MPN" "GS8054-TR" (at 59.69 78.74 0)
+      (effects (font (size 1.27 1.27)) hide)
+    )
+    (property "Status" "" (at 59.69 78.74 0)
       (effects (font (size 1.27 1.27)) hide)
     )
@@
       (effects (font (size 1.27 1.27)) hide)
     )
+    (property "Status" "" (at 101.6 173.99 0)
+      (effects (font (size 1.27 1.27)) hide)
+    )
     (pin "1")
     (pin "2")
@@
     )
     (property "MPN" "GS8054-TR" (at 68.58 114.3 0)
+      (effects (font (size 1.27 1.27)) hide)
+    )
+    (property "Status" "" (at 68.58 114.3 0)
       (effects (font (size 1.27 1.27)) hide)
     )
@@
       (effects (font (size 1.27 1.27)) hide)
     )
+    (property "Status" "" (at 74.93 78.74 0)
+      (effects (font (size 1.27 1.27)) hide)
+    )
     (pin "1")
     (pin "2")
@@
       (effects (font (size 1.27 1.27)) hide)
     )
+    (property "Status" "" (at 212.09 73.66 0)
+      (effects (font (size 1.27 1.27)) hide)
+    )
     (pin "1")
     (pin "2")
@@
       (effects (font (size 1.27 1.27)) hide)
     )
+    (property "Status" "" (at 107.95 77.47 0)
+      (effects (font (size 1.27 1.27)) hide)
+    )
     (pin "1")
     (pin "2")
@@
     )
     (property "MPN" "GS8054-TR" (at 181.61 78.74 0)
+      (effects (font (size 1.27 1.27)) hide)
+    )
+    (property "Status" "" (at 181.61 78.74 0)
       (effects (font (size 1.27 1.27)) hide)
     )
@@
       (effects (font (size 1.27 1.27)) hide)
     )
+    (property "Status" "" (at 119.38 81.28 0)
+      (effects (font (size 1.27 1.27)) hide)
+    )
     (pin "1")
     (pin "2")
@@
       (effects (font (size 1.27 1.27)) hide)
     )
+    (property "Status" "" (at 201.93 114.3 0)
+      (effects (font (size 1.27 1.27)) hide)
+    )
     (pin "1")
     (pin "2")
@@
       (effects (font (size 1.27 1.27)) hide)
     )
+    (property "Status" "" (at 212.09 36.83 0)
+      (effects (font (size 1.27 1.27)) hide)
+    )
     (pin "1")
     (pin "2")
@@
     )
     (property "MPN" "GS8054-TR" (at 59.69 41.91 0)
+      (effects (font (size 1.27 1.27)) hide)
+    )
+    (property "Status" "" (at 59.69 41.91 0)
       (effects (font (size 1.27 1.27)) hide)
     )
@@
       (effects (font (size 1.27 1.27)) hide)
     )
+    (property "Status" "" (at 229.87 48.26 0)
+      (effects (font (size 1.27 1.27)) hide)
+    )
     (pin "1")
     (pin "2")
@@
       (effects (font (size 1.27 1.27)) hide)
     )
+    (property "Status" "" (at 74.93 41.91 0)
+      (effects (font (size 1.27 1.27)) hide)
+    )
     (pin "1")
     (pin "2")
@@
       (effects (font (size 1.27 1.27)) hide)
     )
+    (property "Status" "" (at 59.69 71.12 0)
+      (effects (font (size 1.27 1.27)) hide)
+    )
     (pin "1")
     (pin "2")
@@
     )
     (property "MPN" "GS8054-TR" (at 212.09 81.28 0)
+      (effects (font (size 1.27 1.27)) hide)
+    )
+    (property "Status" "" (at 212.09 81.28 0)
       (effects (font (size 1.27 1.27)) hide)
     )
@@
       (effects (font (size 1.27 1.27)) hide)
     )
+    (property "Status" "" (at 90.17 44.45 0)
+      (effects (font (size 1.27 1.27)) hide)
+    )
     (pin "4")
     (pin "7")
@@
       (effects (font (size 1.27 1.27)) hide)
     )
+    (property "Status" "" (at 215.9 114.3 0)
+      (effects (font (size 1.27 1.27)) hide)
+    )
     (pin "1")
     (pin "2")
@@
       (effects (font (size 1.27 1.27)) hide)
     )
+    (property "Status" "" (at 73.66 165.1 0)
+      (effects (font (size 1.27 1.27)) hide)
+    )

Commit message: Progressed ECAD.
Parts:
- U?: MPN 74AHC1G04W5-7 -> SN74AHC1G04DBVR
Changed lines of the file:
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@@
       (effects (font (size 1.27 1.27)) hide)
     )
-    (property "Datasheet" "https://datasheet.lcsc.com/lcsc/1912111437_Diodes-Incorporated-74AHC1G04W5-7_C460486.pdf" (at 73.66 165.1 0)
+    (property "Datasheet" "https://datasheet.lcsc.com/lcsc/2001061132_Texas-Instruments-SN74AHC1G04DBVR_C7465.pdf" (at 73.66 165.1 0)
       (effects (font (size 1.27 1.27)) hide)
     )
-    (property "MPN" "74AHC1G04W5-7" (at 73.66 165.1 0)
+    (property "MPN" "SN74AHC1G04DBVR" (at 73.66 165.1 0)
       (effects (font (size 1.27 1.27)) hide)
     )
