File: ECAD/SCART_switcher/video_in.kicad_sch (KiCad schematic)
At the start: 32 parts, among them U55 74LVC1G3157, U56 74LVC1G3157, U59 74LVC1G3157, U60 74LVC1G3157

Commit message: Progressed ECAD.
Parts:
- Q?: MPN BC847B,215 -> BC847C,215; Status (none) -> OK
Changed lines of the file:
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@@
       (effects (font (size 1.27 1.27)) hide)
     )
+    (property "Status" "" (at 194.31 83.82 0)
+      (effects (font (size 1.27 1.27)) hide)
+    )
     (pin "1")
     (pin "2")
@@
       (effects (font (size 1.27 1.27)) hide)
     )
+    (property "Status" "" (at 43.18 90.17 0)
+      (effects (font (size 1.27 1.27)) hide)
+    )
     (pin "1")
     (pin "2")
@@
       (effects (font (size 1.27 1.27)) hide)
     )
+    (property "Status" "" (at 36.83 43.18 0)
+      (effects (font (size 1.27 1.27)) hide)
+    )
     (pin "1")
     (pin "2")
@@
       (effects (font (size 1.27 1.27)) hide)
     )
+    (property "Status" "" (at 110.49 139.7 0)
+      (effects (font (size 1.27 1.27)) hide)
+    )
     (pin "2")
     (pin "1")
@@
       (effects (font (size 1.27 1.27)) hide)
     )
+    (property "Status" "" (at 49.53 85.09 0)
+      (effects (font (size 1.27 1.27)) hide)
+    )
     (pin "1")
     (pin "2")
@@
       (effects (font (size 1.27 1.27)) hide)
     )
+    (property "Status" "" (at 29.21 48.26 0)
+      (effects (font (size 1.27 1.27)) hide)
+    )
     (pin "1")
     (pin "2")
@@
       (effects (font (size 1.27 1.27)) hide)
     )
+    (property "Status" "" (at 114.3 43.18 0)
+      (effects (font (size 1.27 1.27)) hide)
+    )
     (pin "4")
     (pin "5")
@@
       (effects (font (size 1.27 1.27)) hide)
     )
+    (property "Status" "" (at 91.44 154.94 0)
+      (effects (font (size 1.27 1.27)) hide)
+    )
     (pin "1")
     (pin "2")
@@
       (effects (font (size 1.27 1.27)) hide)
     )
+    (property "Status" "" (at 62.23 45.72 0)
+      (effects (font (size 1.27 1.27)) hide)
+    )
     (pin "4")
     (pin "5")
@@
       (effects (font (size 1.27 1.27)) hide)
     )
+    (property "Status" "" (at 259.08 43.18 0)
+      (effects (font (size 1.27 1.27)) hide)
+    )
     (pin "1")
     (pin "2")
@@
       (effects (font (size 1.27 1.27)) hide)
     )
+    (property "Status" "" (at 173.99 48.26 0)
+      (effects (font (size 1.27 1.27)) hide)
+    )
     (pin "1")
     (pin "2")
@@
       (effects (font (size 1.27 1.27)) hide)
     )
+    (property "Status" "" (at 187.96 88.9 0)
+      (effects (font (size 1.27 1.27)) hide)
+    )
     (pin "1")
     (pin "2")
@@
       (effects (font (size 1.27 1.27)) hide)
     )
+    (property "Status" "" (at 49.53 43.18 0)
+      (effects (font (size 1.27 1.27)) hide)
+    )
     (pin "1")
     (pin "2")
@@
       (effects (font (size 1.27 1.27)) hide)
     )
+    (property "Status" "" (at 114.3 85.09 0)
+      (effects (font (size 1.27 1.27)) hide)
+    )
     (pin "1")
     (pin "2")
@@
       (effects (font (size 1.27 1.27)) hide)
     )
+    (property "Status" "" (at 99.06 85.09 0)
+      (effects (font (size 1.27 1.27)) hide)
+    )
     (pin "1")
     (pin "2")
@@
       (effects (font (size 1.27 1.27)) hide)
     )
+    (property "Status" "" (at 196.85 143.51 0)
+      (effects (font (size 1.27 1.27)) hide)
+    )
     (pin "1")
     (pin "2")
@@
       (effects (font (size 1.27 1.27) italic) (justify left) hide)
     )
-    (property "Datasheet" "https://datasheet.lcsc.com/lcsc/2304140030_Nexperia-BC847B-215_C57668.pdf" (at 107.95 148.59 0)
+    (property "Datasheet" "https://datasheet.lcsc.com/lcsc/1811141238_Nexperia-BC847C-215_C8664.pdf" (at 107.95 148.59 0)
       (effects (font (size 1.27 1.27)) (justify left) hide)
     )
-    (property "MPN" "BC847B,215" (at 107.95 148.59 0)
+    (property "MPN" "BC847C,215" (at 107.95 148.59 0)
+      (effects (font (size 1.27 1.27)) hide)
+    )
+    (property "Status" "OK" (at 107.95 148.59 0)
       (effects (font (size 1.27 1.27)) hide)
     )
@@
       (effects (font (size 1.27 1.27)) hide)
     )
+    (property "Status" "" (at 43.18 48.26 0)
+      (effects (font (size 1.27 1.27)) hide)
+    )
     (pin "1")
     (pin "2")
@@
       (effects (font (size 1.27 1.27)) hide)
     )
+    (property "Status" "" (at 173.99 88.9 0)
+      (effects (font (size 1.27 1.27)) hide)
+    )
     (pin "1")
     (pin "2")
@@
       (effects (font (size 1.27 1.27)) hide)
     )
+    (property "Status" "" (at 187.96 48.26 0)
+      (effects (font (size 1.27 1.27)) hide)
+    )
     (pin "1")
     (pin "2")
@@
       (effects (font (size 1.27 1.27)) hide)
     )
+    (property "Status" "" (at 62.23 87.63 0)
+      (effects (font (size 1.27 1.27)) hide)
+    )
     (pin "1")
     (pin "2")
@@
       (effects (font (size 1.27 1.27)) hide)
     )
+    (property "Status" "" (at 181.61 43.18 0)
+      (effects (font (size 1.27 1.27)) hide)
+    )
     (pin "1")
     (pin "2")
@@
       (effects (font (size 1.27 1.27)) hide)
     )
+    (property "Status" "" (at 99.06 148.59 0)
+      (effects (font (size 1.27 1.27)) hide)
+    )
     (pin "1")
     (pin "2")
@@
       (effects (font (size 1.27 1.27)) hide)
     )
+    (property "Status" "" (at 210.82 143.51 0)
+      (effects (font (size 1.27 1.27)) hide)
+    )
     (pin "1")
     (pin "2")
@@
       (effects (font (size 1.27 1.27)) hide)
     )
+    (property "Status" "" (at 243.84 43.18 0)
+      (effects (font (size 1.27 1.27)) hide)
+    )
     (pin "1")
     (pin "2")
@@
       (effects (font (size 1.27 1.27)) hide)
     )
+    (property "Status" "" (at 161.29 143.51 0)
+      (effects (font (size 1.27 1.27)) hide)
+    )
     (pin "1")
     (pin "2")
@@
       (effects (font (size 1.27 1.27)) hide)
     )
+    (property "Status" "" (at 243.84 83.82 0)
+      (effects (font (size 1.27 1.27)) hide)
+    )
     (pin "1")
     (pin "2")
@@
       (effects (font (size 1.27 1.27)) hide)
     )
+    (property "Status" "" (at 194.31 43.18 0)
+      (effects (font (size 1.27 1.27)) hide)
+    )
     (pin "1")
     (pin "2")
@@
       (effects (font (size 1.27 1.27)) hide)
     )
+    (property "Status" "" (at 36.83 85.09 0)
+      (effects (font (size 1.27 1.27)) hide)
+    )
     (pin "1")
     (pin "2")
@@
       (effects (font (size 1.27 1.27)) hide)
     )
+    (property "Status" "" (at 207.01 45.72 0)
+      (effects (font (size 1.27 1.27)) hide)
+    )
     (pin "1")
     (pin "2")
@@
       (effects (font (size 1.27 1.27)) hide)
     )
+    (property "Status" "" (at 207.01 86.36 0)
+      (effects (font (size 1.27 1.27)) hide)
+    )
     (pin "1")
     (pin "2")
@@
       (effects (font (size 1.27 1.27)) hide)
     )
+    (property "Status" "" (at 259.08 83.82 0)
+      (effects (font (size 1.27 1.27)) hide)
+    )
     (pin "1")
     (pin "2")
@@
       (effects (font (size 1.27 1.27)) hide)
     )
+    (property "Status" "" (at 29.21 90.17 0)
+      (effects (font (size 1.27 1.27)) hide)
+    )
     (pin "1")
     (pin "2")
@@
       (effects (font (size 1.27 1.27)) hide)
     )
+    (property "Status" "" (at 99.06 43.18 0)
+      (effects (font (size 1.27 1.27)) hide)
+    )
     (pin "1")
     (pin "2")
@@
       (effects (font (size 1.27 1.27)) hide)
     )
+    (property "Status" "" (at 133.35 143.51 0)
+      (effects (font (size 1.27 1.27)) hide)
+    )
     (pin "3")
     (pin "4")
@@
       (effects (font (size 1.27 1.27)) hide)
     )
+    (property "Status" "" (at 181.61 83.82 0)
+      (effects (font (size 1.27 1.27)) hide)
+    )

Commit message: Progressed ECAD.
Parts:
- U?: footprint (none) -> Package_TO_SOT_SMD:SOT-23-5; MPN 74AHC1G126W5-7 -> SN74AHC1G126DBVR
- U?: footprint Package_TO_SOT_SMD:SOT-353_SC-70-5 -> Package_TO_SOT_SMD:SOT-23-5; MPN 74AHC1G14SE-7 -> SN74AHC1G14DBVR
Changed lines of the file:
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@@
       (effects (font (size 1.27 1.27)))
     )
-    (property "Footprint" "" (at 161.29 143.51 0)
-      (effects (font (size 1.27 1.27)) hide)
-    )
-    (property "Datasheet" "https://datasheet.lcsc.com/lcsc/2201131130_Diodes-Incorporated-74AHC1G126W5-7_C842263.pdf" (at 161.29 143.51 0)
-      (effects (font (size 1.27 1.27)) hide)
-    )
-    (property "MPN" "74AHC1G126W5-7" (at 161.29 143.51 0)
+    (property "Footprint" "Package_TO_SOT_SMD:SOT-23-5" (at 161.29 143.51 0)
+      (effects (font (size 1.27 1.27)) hide)
+    )
+    (property "Datasheet" "https://datasheet.lcsc.com/lcsc/1810010909_Texas-Instruments-SN74AHC1G126DBVR_C145145.pdf" (at 161.29 143.51 0)
+      (effects (font (size 1.27 1.27)) hide)
+    )
+    (property "MPN" "SN74AHC1G126DBVR" (at 161.29 143.51 0)
       (effects (font (size 1.27 1.27)) hide)
     )
@@
       (effects (font (size 1.27 1.27)))
     )
-    (property "Footprint" "Package_TO_SOT_SMD:SOT-353_SC-70-5" (at 133.35 143.51 0)
-      (effects (font (size 1.27 1.27)) hide)
-    )
-    (property "Datasheet" "https://datasheet.lcsc.com/lcsc/1912111437_Diodes-Incorporated-74AHC1G14SE-7_C460491.pdf" (at 133.35 143.51 0)
-      (effects (font (size 1.27 1.27)) hide)
-    )
-    (property "MPN" "74AHC1G14SE-7" (at 133.35 143.51 0)
-      (effects (font (size 1.27 1.27)) hide)
-    )
+    (property "Footprint" "Package_TO_SOT_SMD:SOT-23-5" (at 133.35 143.51 0)
+      (effects (font (size 1.27 1.27)) hide)
+    )
+    (property "Datasheet" "https://datasheet.lcsc.com/lcsc/1809192312_Texas-Instruments-SN74AHC1G14DBVR_C7469.pdf" (at 133.35 143.51 0)
+      (effects (font (size 1.27 1.27)) hide)
+    )
+    (property "MPN" "SN74AHC1G14DBVR" (at 133.35 143.51 0)
+      (effects (font (size 1.27 1.27)) hide)
+    )

Commit message: Progressed ECAD.
Parts:
- U55, U56, U59, U60: Status (none) -> OK
- U?: value 74AHC1G126 -> 74LVC1G126; footprint Package_TO_SOT_SMD:SOT-23-5 -> Package_TO_SOT_SMD:SOT-353_SC-70-5; MPN SN74AHC1G126DBVR -> SN74LVC1G126DCKR; Status (none) -> OK
- U?: value 74AHC1G14 -> 74LVC1G14; footprint Package_TO_SOT_SMD:SOT-23-5 -> Package_TO_SOT_SMD:SOT-353_SC-70-5; MPN SN74AHC1G14DBVR -> SN74LVC1G14DCKR; Status (none) -> OK
Changed lines of the file:
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@@
       (effects (font (size 1.27 1.27)) hide)
     )
-    (property "Status" "" (at 114.3 43.18 0)
+    (property "Status" "OK" (at 114.3 43.18 0)
       (effects (font (size 1.27 1.27)) hide)
     )
@@
       (effects (font (size 1.27 1.27)) hide)
     )
-    (property "Status" "" (at 62.23 45.72 0)
+    (property "Status" "OK" (at 62.23 45.72 0)
       (effects (font (size 1.27 1.27)) hide)
     )
@@
       (effects (font (size 1.27 1.27)) hide)
     )
-    (property "Status" "" (at 259.08 43.18 0)
+    (property "Status" "OK" (at 259.08 43.18 0)
       (effects (font (size 1.27 1.27)) hide)
     )
@@
       (effects (font (size 1.27 1.27)) hide)
     )
-    (property "Status" "" (at 114.3 85.09 0)
+    (property "Status" "OK" (at 114.3 85.09 0)
       (effects (font (size 1.27 1.27)) hide)
     )
@@
       (effects (font (size 1.27 1.27)) hide)
     )
-    (property "Status" "" (at 62.23 87.63 0)
+    (property "Status" "OK" (at 62.23 87.63 0)
       (effects (font (size 1.27 1.27)) hide)
     )
@@
       (effects (font (size 1.27 1.27)))
     )
-    (property "Value" "74AHC1G126" (at 167.64 147.32 0)
+    (property "Value" "74LVC1G126" (at 167.64 147.32 0)
       (effects (font (size 1.27 1.27)))
     )
-    (property "Footprint" "Package_TO_SOT_SMD:SOT-23-5" (at 161.29 143.51 0)
+    (property "Footprint" "Package_TO_SOT_SMD:SOT-353_SC-70-5" (at 161.29 143.51 0)
       (effects (font (size 1.27 1.27)) hide)
     )
-    (property "Datasheet" "https://datasheet.lcsc.com/lcsc/1810010909_Texas-Instruments-SN74AHC1G126DBVR_C145145.pdf" (at 161.29 143.51 0)
+    (property "Datasheet" "https://datasheet.lcsc.com/lcsc/1811082050_Texas-Instruments-SN74LVC1G126DCKR_C88039.pdf" (at 161.29 143.51 0)
       (effects (font (size 1.27 1.27)) hide)
     )
-    (property "MPN" "SN74AHC1G126DBVR" (at 161.29 143.51 0)
+    (property "MPN" "SN74LVC1G126DCKR" (at 161.29 143.51 0)
       (effects (font (size 1.27 1.27)) hide)
     )
-    (property "Status" "" (at 161.29 143.51 0)
+    (property "Status" "OK" (at 161.29 143.51 0)
       (effects (font (size 1.27 1.27)) hide)
     )
@@
       (effects (font (size 1.27 1.27)) hide)
     )
-    (property "Status" "" (at 207.01 45.72 0)
+    (property "Status" "OK" (at 207.01 45.72 0)
       (effects (font (size 1.27 1.27)) hide)
     )
@@
       (effects (font (size 1.27 1.27)) hide)
     )
-    (property "Status" "" (at 207.01 86.36 0)
+    (property "Status" "OK" (at 207.01 86.36 0)
       (effects (font (size 1.27 1.27)) hide)
     )
@@
       (effects (font (size 1.27 1.27)) hide)
     )
-    (property "Status" "" (at 259.08 83.82 0)
+    (property "Status" "OK" (at 259.08 83.82 0)
       (effects (font (size 1.27 1.27)) hide)
     )
@@
       (effects (font (size 1.27 1.27)))
     )
-    (property "Value" "74AHC1G14" (at 139.7 139.7 0)
+    (property "Value" "74LVC1G14" (at 139.7 139.7 0)
       (effects (font (size 1.27 1.27)))
     )
-    (property "Footprint" "Package_TO_SOT_SMD:SOT-23-5" (at 133.35 143.51 0)
+    (property "Footprint" "Package_TO_SOT_SMD:SOT-353_SC-70-5" (at 133.35 143.51 0)
       (effects (font (size 1.27 1.27)) hide)
     )
-    (property "Datasheet" "https://datasheet.lcsc.com/lcsc/1809192312_Texas-Instruments-SN74AHC1G14DBVR_C7469.pdf" (at 133.35 143.51 0)
+    (property "Datasheet" "https://datasheet.lcsc.com/lcsc/1811032110_Texas-Instruments-SN74LVC1G14DCKR_C35740.pdf" (at 133.35 143.51 0)
       (effects (font (size 1.27 1.27)) hide)
     )
-    (property "MPN" "SN74AHC1G14DBVR" (at 133.35 143.51 0)
+    (property "MPN" "SN74LVC1G14DCKR" (at 133.35 143.51 0)
       (effects (font (size 1.27 1.27)) hide)
     )
-    (property "Status" "" (at 133.35 143.51 0)
+    (property "Status" "OK" (at 133.35 143.51 0)
       (effects (font (size 1.27 1.27)) hide)
     )

Commit message: Progressed ECAD.
Parts:
- C? (x4): value 22uC -> 47uC
Other:
- note added: "+"
Changed lines of the file:
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@@
     (effects (font (size 1.27 1.27)) (justify left bottom))
   )
+  (text "+" (at 38.1 41.91 0)
+    (effects (font (size 1.27 1.27)) (justify left bottom))
+  )
   (text "(*2) Use thin film resistor with 1% or better tolerance for lower noise and better gain match."
     (at 177.8 175.26 0)
@@
       (effects (font (size 1.27 1.27)))
     )
-    (property "Value" "22uC" (at 36.83 38.1 90)
+    (property "Value" "47uC" (at 36.83 38.1 90)
       (effects (font (size 1.27 1.27)))
     )
@@
       (effects (font (size 1.27 1.27)))
     )
-    (property "Value" "22uC" (at 181.61 38.1 90)
+    (property "Value" "47uC" (at 181.61 38.1 90)
       (effects (font (size 1.27 1.27)))
     )
@@
       (effects (font (size 1.27 1.27)))
     )
-    (property "Value" "22uC" (at 36.83 80.01 90)
+    (property "Value" "47uC" (at 36.83 80.01 90)
       (effects (font (size 1.27 1.27)))
     )
@@
       (effects (font (size 1.27 1.27)))
     )
-    (property "Value" "22uC" (at 181.61 78.74 90)
+    (property "Value" "47uC" (at 181.61 78.74 90)
       (effects (font (size 1.27 1.27)))
     )

Commit message: Progressed ECAD.
Parts:
- C? (x4): footprint (none) -> Capacitor_SMD:CP_Elec_4x5.8; MPN (none) -> EEEFK1C470SR; Status (none) -> OK
Changed lines of the file:
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@@
       (effects (font (size 1.27 1.27)))
     )
-    (property "Footprint" "" (at 40.64 42.2148 0)
+    (property "Footprint" "Capacitor_SMD:CP_Elec_4x5.8" (at 40.64 42.2148 0)
       (effects (font (size 1.27 1.27)) hide)
     )
-    (property "Datasheet" "~" (at 36.83 43.18 0)
+    (property "Datasheet" "https://datasheet.lcsc.com/lcsc/2304140030_PANASONIC-EEEFK1C470SR_C401706.pdf" (at 36.83 43.18 0)
       (effects (font (size 1.27 1.27)) hide)
     )
-    (property "Status" "" (at 36.83 43.18 0)
+    (property "Status" "OK" (at 36.83 43.18 0)
+      (effects (font (size 1.27 1.27)) hide)
+    )
+    (property "MPN" "EEEFK1C470SR" (at 36.83 43.18 0)
       (effects (font (size 1.27 1.27)) hide)
     )
@@
       (effects (font (size 1.27 1.27)))
     )
-    (property "Footprint" "" (at 185.42 42.2148 0)
+    (property "Footprint" "Capacitor_SMD:CP_Elec_4x5.8" (at 185.42 42.2148 0)
+      (effects (font (size 1.27 1.27)) hide)
+    )
+    (property "Datasheet" "https://datasheet.lcsc.com/lcsc/2304140030_PANASONIC-EEEFK1C470SR_C401706.pdf" (at 181.61 43.18 0)
       (effects (font (size 1.27 1.27)) hide)
     )
-    (property "Datasheet" "~" (at 181.61 43.18 0)
+    (property "Status" "OK" (at 181.61 43.18 0)
       (effects (font (size 1.27 1.27)) hide)
     )
-    (property "Status" "" (at 181.61 43.18 0)
+    (property "MPN" "EEEFK1C470SR" (at 181.61 43.18 0)
       (effects (font (size 1.27 1.27)) hide)
     )
@@
       (effects (font (size 1.27 1.27)))
     )
-    (property "Footprint" "" (at 40.64 84.1248 0)
+    (property "Footprint" "Capacitor_SMD:CP_Elec_4x5.8" (at 40.64 84.1248 0)
       (effects (font (size 1.27 1.27)) hide)
     )
-    (property "Datasheet" "~" (at 36.83 85.09 0)
+    (property "Datasheet" "https://datasheet.lcsc.com/lcsc/2304140030_PANASONIC-EEEFK1C470SR_C401706.pdf" (at 36.83 85.09 0)
       (effects (font (size 1.27 1.27)) hide)
     )
-    (property "Status" "" (at 36.83 85.09 0)
+    (property "Status" "OK" (at 36.83 85.09 0)
+      (effects (font (size 1.27 1.27)) hide)
+    )
+    (property "MPN" "EEEFK1C470SR" (at 36.83 85.09 0)
       (effects (font (size 1.27 1.27)) hide)
     )
@@
       (effects (font (size 1.27 1.27)))
     )
-    (property "Footprint" "" (at 185.42 82.8548 0)
+    (property "Footprint" "Capacitor_SMD:CP_Elec_4x5.8" (at 185.42 82.8548 0)
+      (effects (font (size 1.27 1.27)) hide)
+    )
+    (property "Datasheet" "https://datasheet.lcsc.com/lcsc/2304140030_PANASONIC-EEEFK1C470SR_C401706.pdf" (at 181.61 83.82 0)
       (effects (font (size 1.27 1.27)) hide)
     )
-    (property "Datasheet" "~" (at 181.61 83.82 0)
+    (property "Status" "OK" (at 181.61 83.82 0)
       (effects (font (size 1.27 1.27)) hide)
     )
-    (property "Status" "" (at 181.61 83.82 0)
+    (property "MPN" "EEEFK1C470SR" (at 181.61 83.82 0)
       (effects (font (size 1.27 1.27)) hide)
     )

Commit message: Error fix.
Parts:
- removed C? (x4): 47uC, Capacitor_SMD:CP_Elec_4x5.8, symbol Device:C
- added C? (x4): 47uC, Capacitor_SMD:CP_Elec_4x5.8, symbol Device:C_Polarized
Connections:
- net BLUE_IN: now also C?.2
- net GREEN_IN: now also C?.2
- net RED_IN: now also C?.2
- net VIDEO_RGB_SYNC_IN: now also C?.2
- net at R?.1, R?.1: now also C?.1 (x4)
Other:
- note removed: "+"

Commit message: Progressed ECAD.
Parts:
- removed U56, U59, U60: 74LVC1G3157, Package_TO_SOT_SMD:SOT-363_SC-70-6, symbol Analog_Switch:TS5A63157DBV
- added U50, U51, U54: 74LVC1G3157, Package_TO_SOT_SMD:SOT-363_SC-70-6, symbol Analog_Switch:TS5A63157DBV
- gave numbers to parts that had none: 28
Connections:
- net +2V5: now also U50.3, U51.3, U54.3
- net +5V: now also U50.5 (V+), U51.5 (V+), U54.5 (V+)
- net BLUE_OUT: now also U54.1
- net ENABLE: now also U50.6, U51.6, U54.6
- net GND: now also U50.2 (GND), U51.2 (GND), U54.2 (GND)
- net GREEN_OUT: now also U50.1; no longer U55.1
- net RED_OUT: now also U51.1
- net VIDEO_RGB_SYNC_OUT: now also U55.1
- net at R121.2: now also U55.4
- net at R112.2: now also U51.4
- net at R111.2: now also U50.4; no longer U55.4
- net at R120.2: now also U54.4
