File: ECAD/SCART_switcher/video_in.kicad_sch (KiCad schematic)
At the start: 28 parts, among them U62 74LVC1G3157, U63 74LVC1G3157, U64 74LVC1G3157, U65 74LVC1G3157, U66 74LVC1G3157

Commit message: Progressed ECAD.
Parts:
- renumbered C81 to C85, C82 to C86, C83 to C87, C84 to C88, C85 to C89, C86 to C90, C87 to C91, C88 to C92, C89 to C93, R105 to R107, R106 to R108, R107 to R109, R108 to R110, R109 to R111, R110 to R112, R111 to R113, R112 to R114, R113 to R115, R114 to R116, R115 to R117, R116 to R118, R117 to R119, R118 to R120, U62 to U63, U63 to U64, U64 to U65, U65 to U66, U66 to U67

Commit message: Progressed ECAD.
Parts:
- renumbered C85 to C83, C86 to C84, C87 to C85, C88 to C86, C89 to C87, C90 to C88, C91 to C89, C92 to C90, C93 to C91, R107 to R105, R108 to R106, R109 to R107, R110 to R108, R111 to R109, R112 to R110, R113 to R111, R114 to R112, R115 to R113, R116 to R114, R117 to R115, R118 to R116, R119 to R117, R120 to R118

Commit message: Cleanup and new power supply pcb
Parts:
- renumbered C83 to C77, C84 to C78, C85 to C79, C86 to C80, C87 to C81, C88 to C82, C89 to C83, C90 to C84, C91 to C85, R105 to R103, R106 to R104, R107 to R105, R108 to R106, R109 to R107, R110 to R108, R111 to R109, R112 to R110, R113 to R111, R114 to R112, R115 to R113, R116 to R114, R117 to R115, R118 to R116, U63 to U60, U64 to U61, U65 to U62, U66 to U63, U67 to U64

Commit message: Progressed ECAD.
Parts:
- renumbered C77 to C75, C78 to C76, C79 to C77, C80 to C78, C81 to C79, C82 to C80, C83 to C81, C84 to C82, C85 to C83

Commit message: Progressed ECAD.
Parts:
- renumbered R103 to R105, R104 to R106, R105 to R107, R106 to R108, R107 to R109, R108 to R110, R109 to R111, R110 to R112, R111 to R113, R112 to R114, R113 to R115, R114 to R116, R115 to R117, R116 to R118

Commit message: Progressed ECAD.
Parts:
- R107, R108, R115, R116: MPN (none) -> RC0805FR-07100KL; Status (none) -> OK
- R112: MPN RC0805FR-0710KL -> AC0805FR-0710KL; Status (none) -> OK
Changed lines of the file:
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@@
       (effects (font (size 1.27 1.27)) hide)
     )
-    (property "Datasheet" "~" (at 43.18 105.41 0)
-      (effects (font (size 1.27 1.27)) hide)
-    )
-    (property "Status" "" (at 43.18 105.41 0)
+    (property "Datasheet" "https://datasheet.lcsc.com/lcsc/2304140030_YAGEO-RC0805FR-07100KL_C96346.pdf" (at 43.18 105.41 0)
+      (effects (font (size 1.27 1.27)) hide)
+    )
+    (property "Status" "OK" (at 43.18 105.41 0)
+      (effects (font (size 1.27 1.27)) hide)
+    )
+    (property "MPN" "RC0805FR-07100KL" (at 43.18 105.41 0)
       (effects (font (size 1.27 1.27)) hide)
     )
@@
       (effects (font (size 1.27 1.27)) hide)
     )
-    (property "Datasheet" "https://datasheet.lcsc.com/lcsc/1810201611_YAGEO-RC0805FR-0710KL_C84376.pdf" (at 71.12 165.1 0)
-      (effects (font (size 1.27 1.27)) hide)
-    )
-    (property "MPN" "RC0805FR-0710KL" (at 71.12 165.1 0)
-      (effects (font (size 1.27 1.27)) hide)
-    )
-    (property "Status" "" (at 71.12 165.1 0)
+    (property "Datasheet" "https://datasheet.lcsc.com/lcsc/2304140030_YAGEO-AC0805FR-0710KL_C140868.pdf" (at 71.12 165.1 0)
+      (effects (font (size 1.27 1.27)) hide)
+    )
+    (property "MPN" "AC0805FR-0710KL" (at 71.12 165.1 0)
+      (effects (font (size 1.27 1.27)) hide)
+    )
+    (property "Status" "OK" (at 71.12 165.1 0)
       (effects (font (size 1.27 1.27)) hide)
     )
@@
       (effects (font (size 1.27 1.27)) hide)
     )
-    (property "Datasheet" "~" (at 187.96 104.14 0)
-      (effects (font (size 1.27 1.27)) hide)
-    )
-    (property "Status" "" (at 187.96 104.14 0)
+    (property "Datasheet" "https://datasheet.lcsc.com/lcsc/2304140030_YAGEO-RC0805FR-07100KL_C96346.pdf" (at 187.96 104.14 0)
+      (effects (font (size 1.27 1.27)) hide)
+    )
+    (property "Status" "OK" (at 187.96 104.14 0)
+      (effects (font (size 1.27 1.27)) hide)
+    )
+    (property "MPN" "RC0805FR-07100KL" (at 187.96 104.14 0)
       (effects (font (size 1.27 1.27)) hide)
     )
@@
       (effects (font (size 1.27 1.27)) hide)
     )
-    (property "Datasheet" "~" (at 43.18 48.26 0)
-      (effects (font (size 1.27 1.27)) hide)
-    )
-    (property "Status" "" (at 43.18 48.26 0)
+    (property "Datasheet" "https://datasheet.lcsc.com/lcsc/2304140030_YAGEO-RC0805FR-07100KL_C96346.pdf" (at 43.18 48.26 0)
+      (effects (font (size 1.27 1.27)) hide)
+    )
+    (property "Status" "OK" (at 43.18 48.26 0)
+      (effects (font (size 1.27 1.27)) hide)
+    )
+    (property "MPN" "RC0805FR-07100KL" (at 43.18 48.26 0)
       (effects (font (size 1.27 1.27)) hide)
     )
@@
       (effects (font (size 1.27 1.27)) hide)
     )
-    (property "Datasheet" "~" (at 187.96 48.26 0)
-      (effects (font (size 1.27 1.27)) hide)
-    )
-    (property "Status" "" (at 187.96 48.26 0)
-      (effects (font (size 1.27 1.27)) hide)
-    )
+    (property "Datasheet" "https://datasheet.lcsc.com/lcsc/2304140030_YAGEO-RC0805FR-07100KL_C96346.pdf" (at 187.96 48.26 0)
+      (effects (font (size 1.27 1.27)) hide)
+    )
+    (property "Status" "OK" (at 187.96 48.26 0)
+      (effects (font (size 1.27 1.27)) hide)
+    )
+    (property "MPN" "RC0805FR-07100KL" (at 187.96 48.26 0)
+      (effects (font (size 1.27 1.27)) hide)
+    )

Commit message: Progressed ECAD.
Parts:
- C77, C78, C79, C82, C83: MPN CL21B104KBCNNNC -> CL10B104KO8NNNC; Status (none) -> OK
- R105, R106, R109, R113, R114: MPN (none) -> AC1210FR-0775RL; Status (none) -> OK
- R110, R111, R117, R118: MPN (none) -> RT0805BRD071KL; Status (none) -> OK
Changed lines of the file:
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@@
       (effects (font (size 1.27 1.27)) hide)
     )
-    (property "Datasheet" "~" (at 194.31 99.06 0)
+    (property "Datasheet" "https://datasheet.lcsc.com/lcsc/2304140030_YAGEO-RT0805BRD071KL_C110774.pdf" (at 194.31 99.06 0)
       (effects (font (size 1.27 1.27)) hide)
     )
-    (property "Status" "" (at 194.31 99.06 0)
+    (property "Status" "OK" (at 194.31 99.06 0)
+      (effects (font (size 1.27 1.27)) hide)
+    )
+    (property "MPN" "RT0805BRD071KL" (at 194.31 99.06 0)
       (effects (font (size 1.27 1.27)) hide)
     )
@@
       (effects (font (size 1.27 1.27)) hide)
     )
-    (property "Datasheet" "https://datasheet.lcsc.com/lcsc/1810191215_Samsung-Electro-Mechanics-CL21B104KBCNNNC_C1711.pdf" (at 99.06 157.48 0)
+    (property "Datasheet" "https://datasheet.lcsc.com/lcsc/1810271710_Samsung-Electro-Mechanics-CL10B104KO8NNNC_C66501.pdf" (at 99.06 157.48 0)
       (effects (font (size 1.27 1.27)) hide)
     )
-    (property "MPN" "CL21B104KBCNNNC" (at 99.06 157.48 0)
+    (property "MPN" "CL10B104KO8NNNC" (at 99.06 157.48 0)
       (effects (font (size 1.27 1.27)) hide)
     )
-    (property "Status" "" (at 99.06 157.48 0)
+    (property "Status" "OK" (at 99.06 157.48 0)
       (effects (font (size 1.27 1.27)) hide)
     )
@@
       (effects (font (size 1.27 1.27)) hide)
     )
-    (property "Datasheet" "~" (at 49.53 100.33 0)
+    (property "Datasheet" "https://datasheet.lcsc.com/lcsc/2304140030_YAGEO-RT0805BRD071KL_C110774.pdf" (at 49.53 100.33 0)
       (effects (font (size 1.27 1.27)) hide)
     )
-    (property "Status" "" (at 49.53 100.33 0)
+    (property "Status" "OK" (at 49.53 100.33 0)
+      (effects (font (size 1.27 1.27)) hide)
+    )
+    (property "MPN" "RT0805BRD071KL" (at 49.53 100.33 0)
       (effects (font (size 1.27 1.27)) hide)
     )
@@
       (effects (font (size 1.27 1.27)) hide)
     )
-    (property "Datasheet" "~" (at 29.21 48.26 0)
+    (property "Datasheet" "https://datasheet.lcsc.com/lcsc/2304140030_YAGEO-AC1210FR-0775RL_C230341.pdf" (at 29.21 48.26 0)
       (effects (font (size 1.27 1.27)) hide)
     )
-    (property "Status" "" (at 29.21 48.26 0)
+    (property "Status" "OK" (at 29.21 48.26 0)
+      (effects (font (size 1.27 1.27)) hide)
+    )
+    (property "MPN" "AC1210FR-0775RL" (at 29.21 48.26 0)
       (effects (font (size 1.27 1.27)) hide)
     )
@@
       (effects (font (size 1.27 1.27)) hide)
     )
-    (property "Datasheet" "~" (at 173.99 48.26 0)
+    (property "Datasheet" "https://datasheet.lcsc.com/lcsc/2304140030_YAGEO-AC1210FR-0775RL_C230341.pdf" (at 173.99 48.26 0)
+      (effects (font (size 1.27 1.27)) hide)
+    )
+    (property "Status" "OK" (at 173.99 48.26 0)
       (effects (font (size 1.27 1.27)) hide)
     )
-    (property "Status" "" (at 173.99 48.26 0)
+    (property "MPN" "AC1210FR-0775RL" (at 173.99 48.26 0)
       (effects (font (size 1.27 1.27)) hide)
     )
@@
       (effects (font (size 1.27 1.27)) hide)
     )
-    (property "Datasheet" "~" (at 49.53 43.18 0)
+    (property "Datasheet" "https://datasheet.lcsc.com/lcsc/2304140030_YAGEO-RT0805BRD071KL_C110774.pdf" (at 49.53 43.18 0)
+      (effects (font (size 1.27 1.27)) hide)
+    )
+    (property "Status" "OK" (at 49.53 43.18 0)
       (effects (font (size 1.27 1.27)) hide)
     )
-    (property "Status" "" (at 49.53 43.18 0)
+    (property "MPN" "RT0805BRD071KL" (at 49.53 43.18 0)
       (effects (font (size 1.27 1.27)) hide)
     )
@@
       (effects (font (size 1.27 1.27)) hide)
     )
-    (property "Datasheet" "https://datasheet.lcsc.com/lcsc/1810191215_Samsung-Electro-Mechanics-CL21B104KBCNNNC_C1711.pdf" (at 99.06 100.33 0)
+    (property "Datasheet" "https://datasheet.lcsc.com/lcsc/1810271710_Samsung-Electro-Mechanics-CL10B104KO8NNNC_C66501.pdf" (at 99.06 100.33 0)
       (effects (font (size 1.27 1.27)) hide)
     )
-    (property "MPN" "CL21B104KBCNNNC" (at 99.06 100.33 0)
+    (property "MPN" "CL10B104KO8NNNC" (at 99.06 100.33 0)
       (effects (font (size 1.27 1.27)) hide)
     )
-    (property "Status" "" (at 99.06 100.33 0)
+    (property "Status" "OK" (at 99.06 100.33 0)
       (effects (font (size 1.27 1.27)) hide)
     )
@@
       (effects (font (size 1.27 1.27)) hide)
     )
-    (property "Datasheet" "~" (at 46.99 163.83 0)
+    (property "Datasheet" "https://datasheet.lcsc.com/lcsc/2304140030_YAGEO-AC1210FR-0775RL_C230341.pdf" (at 46.99 163.83 0)
+      (effects (font (size 1.27 1.27)) hide)
+    )
+    (property "Status" "OK" (at 46.99 163.83 0)
       (effects (font (size 1.27 1.27)) hide)
     )
-    (property "Status" "" (at 46.99 163.83 0)
+    (property "MPN" "AC1210FR-0775RL" (at 46.99 163.83 0)
       (effects (font (size 1.27 1.27)) hide)
     )
@@
       (effects (font (size 1.27 1.27)) hide)
     )
-    (property "Datasheet" "~" (at 173.99 104.14 0)
+    (property "Datasheet" "https://datasheet.lcsc.com/lcsc/2304140030_YAGEO-AC1210FR-0775RL_C230341.pdf" (at 173.99 104.14 0)
+      (effects (font (size 1.27 1.27)) hide)
+    )
+    (property "Status" "OK" (at 173.99 104.14 0)
       (effects (font (size 1.27 1.27)) hide)
     )
-    (property "Status" "" (at 173.99 104.14 0)
+    (property "MPN" "AC1210FR-0775RL" (at 173.99 104.14 0)
       (effects (font (size 1.27 1.27)) hide)
     )
@@
       (effects (font (size 1.27 1.27)) hide)
     )
-    (property "Datasheet" "https://datasheet.lcsc.com/lcsc/1810191215_Samsung-Electro-Mechanics-CL21B104KBCNNNC_C1711.pdf" (at 243.84 43.18 0)
+    (property "Datasheet" "https://datasheet.lcsc.com/lcsc/1810271710_Samsung-Electro-Mechanics-CL10B104KO8NNNC_C66501.pdf" (at 243.84 43.18 0)
       (effects (font (size 1.27 1.27)) hide)
     )
-    (property "MPN" "CL21B104KBCNNNC" (at 243.84 43.18 0)
+    (property "MPN" "CL10B104KO8NNNC" (at 243.84 43.18 0)
       (effects (font (size 1.27 1.27)) hide)
     )
-    (property "Status" "" (at 243.84 43.18 0)
+    (property "Status" "OK" (at 243.84 43.18 0)
       (effects (font (size 1.27 1.27)) hide)
     )
@@
       (effects (font (size 1.27 1.27)) hide)
     )
-    (property "Datasheet" "https://datasheet.lcsc.com/lcsc/1810191215_Samsung-Electro-Mechanics-CL21B104KBCNNNC_C1711.pdf" (at 243.84 99.06 0)
+    (property "Datasheet" "https://datasheet.lcsc.com/lcsc/1810271710_Samsung-Electro-Mechanics-CL10B104KO8NNNC_C66501.pdf" (at 243.84 99.06 0)
       (effects (font (size 1.27 1.27)) hide)
     )
-    (property "MPN" "CL21B104KBCNNNC" (at 243.84 99.06 0)
+    (property "MPN" "CL10B104KO8NNNC" (at 243.84 99.06 0)
       (effects (font (size 1.27 1.27)) hide)
     )
-    (property "Status" "" (at 243.84 99.06 0)
+    (property "Status" "OK" (at 243.84 99.06 0)
       (effects (font (size 1.27 1.27)) hide)
     )
@@
       (effects (font (size 1.27 1.27)) hide)
     )
-    (property "Datasheet" "~" (at 194.31 43.18 0)
+    (property "Datasheet" "https://datasheet.lcsc.com/lcsc/2304140030_YAGEO-RT0805BRD071KL_C110774.pdf" (at 194.31 43.18 0)
       (effects (font (size 1.27 1.27)) hide)
     )
-    (property "Status" "" (at 194.31 43.18 0)
+    (property "Status" "OK" (at 194.31 43.18 0)
+      (effects (font (size 1.27 1.27)) hide)
+    )
+    (property "MPN" "RT0805BRD071KL" (at 194.31 43.18 0)
       (effects (font (size 1.27 1.27)) hide)
     )
@@
       (effects (font (size 1.27 1.27)) hide)
     )
-    (property "Datasheet" "~" (at 29.21 105.41 0)
+    (property "Datasheet" "https://datasheet.lcsc.com/lcsc/2304140030_YAGEO-AC1210FR-0775RL_C230341.pdf" (at 29.21 105.41 0)
+      (effects (font (size 1.27 1.27)) hide)
+    )
+    (property "Status" "OK" (at 29.21 105.41 0)
       (effects (font (size 1.27 1.27)) hide)
     )
-    (property "Status" "" (at 29.21 105.41 0)
+    (property "MPN" "AC1210FR-0775RL" (at 29.21 105.41 0)
       (effects (font (size 1.27 1.27)) hide)
     )
@@
       (effects (font (size 1.27 1.27)) hide)
     )
-    (property "Datasheet" "https://datasheet.lcsc.com/lcsc/1810191215_Samsung-Electro-Mechanics-CL21B104KBCNNNC_C1711.pdf" (at 99.06 43.18 0)
+    (property "Datasheet" "https://datasheet.lcsc.com/lcsc/1810271710_Samsung-Electro-Mechanics-CL10B104KO8NNNC_C66501.pdf" (at 99.06 43.18 0)
       (effects (font (size 1.27 1.27)) hide)
     )
-    (property "MPN" "CL21B104KBCNNNC" (at 99.06 43.18 0)
+    (property "MPN" "CL10B104KO8NNNC" (at 99.06 43.18 0)
       (effects (font (size 1.27 1.27)) hide)
     )
-    (property "Status" "" (at 99.06 43.18 0)
+    (property "Status" "OK" (at 99.06 43.18 0)
       (effects (font (size 1.27 1.27)) hide)
     )

Commit message: Progressed ECAD.
Parts:
- U60, U61, U62, U63, U64: MPN_MOUSER (none) -> SN74LVC1G3157DCKR
