File: ECAD/SCART_switcher/SCART_switcher.kicad_sch (KiCad schematic)
At the start: 8 parts

Commit message: Progressed ECAD.
Other:
- removed sheet Dummy input

Commit message: Progressed ECAD.
Other:
- note removed: "(*1)"
- note removed: "(*2)"
- note removed: "(*3)"
- note removed: "(*4)"
- note removed: "(*5)"

Commit message: Progressed ECAD.
Parts:
- H1, H2, H3, H4, H5, H6, H7, H8: MPN (none) -> N/A; Status (none) -> OK
Changed lines of the file:
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@@
+      (effects (font (size 1.27 1.27)) hide)
+    )
+    (property "Status" "OK" (at 195.58 158.75 0)
+      (effects (font (size 1.27 1.27)) hide)
+    )
+    (property "MPN" "N/A" (at 195.58 158.75 0)
       (effects (font (size 1.27 1.27)) hide)
     )
@@
       (effects (font (size 1.27 1.27)) hide)
     )
+    (property "Status" "OK" (at 195.58 152.4 0)
+      (effects (font (size 1.27 1.27)) hide)
+    )
+    (property "MPN" "N/A" (at 195.58 152.4 0)
+      (effects (font (size 1.27 1.27)) hide)
+    )
     (instances
       (project "SCART_switcher"
@@
       (effects (font (size 1.27 1.27)) hide)
     )
+    (property "Status" "OK" (at 236.22 152.4 0)
+      (effects (font (size 1.27 1.27)) hide)
+    )
+    (property "MPN" "N/A" (at 236.22 152.4 0)
+      (effects (font (size 1.27 1.27)) hide)
+    )
     (instances
       (project "SCART_switcher"
@@
       (effects (font (size 1.27 1.27)) hide)
     )
+    (property "Status" "OK" (at 236.22 158.75 0)
+      (effects (font (size 1.27 1.27)) hide)
+    )
+    (property "MPN" "N/A" (at 236.22 158.75 0)
+      (effects (font (size 1.27 1.27)) hide)
+    )
     (instances
       (project "SCART_switcher"
@@
       (effects (font (size 1.27 1.27)) hide)
     )
+    (property "Status" "OK" (at 215.9 158.75 0)
+      (effects (font (size 1.27 1.27)) hide)
+    )
+    (property "MPN" "N/A" (at 215.9 158.75 0)
+      (effects (font (size 1.27 1.27)) hide)
+    )
     (instances
       (project "SCART_switcher"
@@
       (effects (font (size 1.27 1.27)) hide)
     )
+    (property "Status" "OK" (at 256.54 152.4 0)
+      (effects (font (size 1.27 1.27)) hide)
+    )
+    (property "MPN" "N/A" (at 256.54 152.4 0)
+      (effects (font (size 1.27 1.27)) hide)
+    )
     (instances
       (project "SCART_switcher"
@@
       (effects (font (size 1.27 1.27)) hide)
     )
+    (property "Status" "OK" (at 256.54 158.75 0)
+      (effects (font (size 1.27 1.27)) hide)
+    )
+    (property "MPN" "N/A" (at 256.54 158.75 0)
+      (effects (font (size 1.27 1.27)) hide)
+    )
     (instances
       (project "SCART_switcher"
@@
       (effects (font (size 1.27 1.27)) hide)
     )
+    (property "Status" "OK" (at 215.9 152.4 0)
+      (effects (font (size 1.27 1.27)) hide)
+    )
+    (property "MPN" "N/A" (at 215.9 152.4 0)
+      (effects (font (size 1.27 1.27)) hide)
+    )

Commit message: Progressed ECAD.
Other:
- removed sheet Priority Encoder
- sheet SCART input 1 ports: added CARRY_IN, CARRY_OUT; removed IN_ACTIVE, IN_ENABLE
- sheet SCART input 10 ports: added CARRY_IN, CARRY_OUT; removed IN_ACTIVE, IN_ENABLE
- sheet SCART input 2 ports: added CARRY_IN, CARRY_OUT; removed IN_ACTIVE, IN_ENABLE
- sheet SCART input 3 ports: added CARRY_IN, CARRY_OUT; removed IN_ACTIVE, IN_ENABLE
- sheet SCART input 4 ports: added CARRY_IN, CARRY_OUT; removed IN_ACTIVE, IN_ENABLE
- sheet SCART input 5 ports: added CARRY_IN, CARRY_OUT; removed IN_ACTIVE, IN_ENABLE
- sheet SCART input 6 ports: added CARRY_IN, CARRY_OUT; removed IN_ACTIVE, IN_ENABLE
- sheet SCART input 7 ports: added CARRY_IN, CARRY_OUT; removed IN_ACTIVE, IN_ENABLE
- sheet SCART input 8 ports: added CARRY_IN, CARRY_OUT; removed IN_ACTIVE, IN_ENABLE
- sheet SCART input 9 ports: added CARRY_IN, CARRY_OUT; removed IN_ACTIVE, IN_ENABLE
- moved on the sheet: H1, H2, H3, H4, H5, H6, H7, H8

Commit message: Progressed ECAD.
Other:
- sheet SCART output ports: added ~{OUT_ACTIVE}; removed OUT_ACTIVE
Changed lines of the file:
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@@
     (stroke (width 0) (type default))
   )
-  (wire (pts (xy 25.4 35.56) (xy 25.4 33.02))
+  (wire (pts (xy 25.4 35.56) (xy 25.4 21.59))
     (stroke (width 0) (type default))
   )
@@
     )
   )
-  (symbol (lib_id "power:+5V") (at 25.4 33.02 0) (unit 1)
+  (symbol (lib_id "power:+5V") (at 25.4 21.59 0) (unit 1)
     (in_bom yes) (on_board yes) (dnp no) (fields_autoplaced)
-    (property "Reference" "#PWR01" (at 25.4 36.83 0)
-      (effects (font (size 1.27 1.27)) hide)
-    )
-    (property "Value" "+5V" (at 25.4 27.94 0)
+    (property "Reference" "#PWR01" (at 25.4 25.4 0)
+      (effects (font (size 1.27 1.27)) hide)
+    )
+    (property "Value" "+5V" (at 25.4 16.51 0)
       (effects (font (size 1.27 1.27)))
     )
-    (property "Footprint" "" (at 25.4 33.02 0)
-      (effects (font (size 1.27 1.27)) hide)
-    )
-    (property "Datasheet" "" (at 25.4 33.02 0)
+    (property "Footprint" "" (at 25.4 21.59 0)
+      (effects (font (size 1.27 1.27)) hide)
+    )
+    (property "Datasheet" "" (at 25.4 21.59 0)
       (effects (font (size 1.27 1.27)) hide)
     )
@@
       (effects (font (size 1.27 1.27)) (justify left))
     )
-    (pin "OUT_ACTIVE" input (at 205.74 48.26 180)
-      (effects (font (size 1.27 1.27)) (justify left))
-    )
     (pin "VIDEO_RGB_SYNC" input (at 205.74 33.02 180)
       (effects (font (size 1.27 1.27)) (justify left))
     )
+    (pin "~{OUT_ACTIVE}" input (at 205.74 48.26 180)
+      (effects (font (size 1.27 1.27)) (justify left))
+    )

Commit message: Progressed ECAD
Other:
- added sheet Silent input (dummy_input.kicad_sch)
Changed lines of the file:
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@@
   (paper "A4")
   (bus_alias "VIDEO_SIGNALS" (members "RED" "BLUE" "GREEN" "VIDEO_RGB_SYNC" "BLANKING" "AUDIO_LEFT" "AUDIO_RIGHT"))
+  (junction (at 165.1 81.28) (diameter 0) (color 0 0 0 0)
+  )
   (bus_entry (at 157.48 63.5) (size -2.54 -2.54)
     (stroke (width 0) (type default))
@@
     (stroke (width 0) (type default))
   )
+  (bus_entry (at 185.42 63.5) (size 2.54 -2.54)
+    (stroke (width 0) (type default))
+  )
   (bus_entry (at 157.48 43.18) (size -2.54 -2.54)
     (stroke (width 0) (type default))
@@
     (stroke (width 0) (type default))
   )
+  (bus_entry (at 185.42 68.58) (size 2.54 -2.54)
+    (stroke (width 0) (type default))
+  )
   (bus_entry (at 78.74 76.2) (size -2.54 -2.54)
     (stroke (width 0) (type default))
@@
     (stroke (width 0) (type default))
   )
+  (bus_entry (at 185.42 66.04) (size 2.54 -2.54)
+    (stroke (width 0) (type default))
+  )
   (bus_entry (at 185.42 38.1) (size 2.54 -2.54)
     (stroke (width 0) (type default))
@@
     (stroke (width 0) (type default))
   )
+  (bus_entry (at 185.42 71.12) (size 2.54 -2.54)
+    (stroke (width 0) (type default))
+  )
+  (bus_entry (at 185.42 73.66) (size 2.54 -2.54)
+    (stroke (width 0) (type default))
+  )
   (bus_entry (at 157.48 68.58) (size -2.54 -2.54)
     (stroke (width 0) (type default))
@@
     (stroke (width 0) (type default))
   )
+  (bus_entry (at 185.42 60.96) (size 2.54 -2.54)
+    (stroke (width 0) (type default))
+  )
   (bus_entry (at 78.74 160.02) (size -2.54 -2.54)
     (stroke (width 0) (type default))
@@
     (stroke (width 0) (type default))
   )
+  (bus_entry (at 185.42 76.2) (size 2.54 -2.54)
+    (stroke (width 0) (type default))
+  )
   (wire (pts (xy 139.7 147.32) (xy 139.7 152.4))
     (stroke (width 0) (type default))
@@
     (stroke (width 0) (type default))
   )
-  (wire (pts (xy 165.1 180.34) (xy 165.1 48.26))
+  (wire (pts (xy 165.1 180.34) (xy 165.1 81.28))
     (stroke (width 0) (type default))
   )
@@
     (stroke (width 0) (type default))
   )
-  (bus (pts (xy 185.42 25.4) (xy 157.48 25.4))
+  (bus (pts (xy 185.42 22.86) (xy 157.48 22.86))
     (stroke (width 0) (type default))
   )
@@
     (stroke (width 0) (type default))
   )
+  (wire (pts (xy 205.74 60.96) (xy 187.96 60.96))
+    (stroke (width 0) (type default))
+  )
   (wire (pts (xy 76.2 101.6) (xy 58.42 101.6))
     (stroke (width 0) (type default))
@@
     (stroke (width 0) (type default))
   )
-  (bus (pts (xy 185.42 27.94) (xy 185.42 25.4))
+  (bus (pts (xy 185.42 27.94) (xy 185.42 22.86))
     (stroke (width 0) (type default))
   )
@@
     (stroke (width 0) (type default))
   )
+  (bus (pts (xy 185.42 73.66) (xy 185.42 76.2))
+    (stroke (width 0) (type default))
+  )
   (bus (pts (xy 78.74 142.24) (xy 78.74 160.02))
     (stroke (width 0) (type default))
@@
     (stroke (width 0) (type default))
   )
+  (wire (pts (xy 165.1 48.26) (xy 165.1 81.28))
+    (stroke (width 0) (type default))
+  )
   (wire (pts (xy 137.16 81.28) (xy 139.7 81.28))
     (stroke (width 0) (type default))
@@
     (stroke (width 0) (type default))
   )
+  (bus (pts (xy 185.42 68.58) (xy 185.42 71.12))
+    (stroke (width 0) (type default))
+  )
+  (bus (pts (xy 185.42 71.12) (xy 185.42 73.66))
+    (stroke (width 0) (type default))
+  )
   (bus (pts (xy 78.74 93.98) (xy 78.74 96.52))
     (stroke (width 0) (type default))
@@
     (stroke (width 0) (type default))
   )
+  (bus (pts (xy 185.42 60.96) (xy 185.42 63.5))
+    (stroke (width 0) (type default))
+  )
+  (bus (pts (xy 185.42 66.04) (xy 185.42 68.58))
+    (stroke (width 0) (type default))
+  )
   (wire (pts (xy 137.16 25.4) (xy 154.94 25.4))
     (stroke (width 0) (type default))
@@
     (stroke (width 0) (type default))
   )
+  (wire (pts (xy 205.74 63.5) (xy 187.96 63.5))
+    (stroke (width 0) (type default))
+  )
   (wire (pts (xy 137.16 30.48) (xy 154.94 30.48))
     (stroke (width 0) (type default))
   )
+  (wire (pts (xy 187.96 73.66) (xy 205.74 73.66))
+    (stroke (width 0) (type default))
+  )
   (bus (pts (xy 185.42 40.64) (xy 185.42 43.18))
     (stroke (width 0) (type default))
@@
     (stroke (width 0) (type default))
   )
+  (wire (pts (xy 187.96 66.04) (xy 205.74 66.04))
+    (stroke (width 0) (type default))
+  )
   (wire (pts (xy 137.16 124.46) (xy 154.94 124.46))
     (stroke (width 0) (type default))
@@
     (stroke (width 0) (type default))
   )
+  (wire (pts (xy 165.1 81.28) (xy 205.74 81.28))
+    (stroke (width 0) (type default))
+  )
   (wire (pts (xy 104.14 134.62) (xy 106.68 134.62))
     (stroke (width 0) (type default))
@@
     (stroke (width 0) (type default))
   )
+  (wire (pts (xy 205.74 58.42) (xy 187.96 58.42))
+    (stroke (width 0) (type default))
+  )
   (bus (pts (xy 157.48 172.72) (xy 157.48 175.26))
     (stroke (width 0) (type default))
@@
     (stroke (width 0) (type default))
   )
-  (bus (pts (xy 157.48 25.4) (xy 157.48 27.94))
+  (bus (pts (xy 157.48 22.86) (xy 157.48 27.94))
     (stroke (width 0) (type default))
   )
@@
     (stroke (width 0) (type default))
   )
+  (bus (pts (xy 185.42 43.18) (xy 185.42 60.96))
+    (stroke (width 0) (type default))
+  )
   (wire (pts (xy 104.14 119.38) (xy 104.14 134.62))
     (stroke (width 0) (type default))
   )
+  (wire (pts (xy 187.96 71.12) (xy 205.74 71.12))
+    (stroke (width 0) (type default))
+  )
   (wire (pts (xy 154.94 68.58) (xy 137.16 68.58))
     (stroke (width 0) (type default))
@@
     (stroke (width 0) (type default))
   )
+  (wire (pts (xy 187.96 68.58) (xy 205.74 68.58))
+    (stroke (width 0) (type default))
+  )
   (bus (pts (xy 157.48 127) (xy 157.48 129.54))
     (stroke (width 0) (type default))
@@
   )
   (wire (pts (xy 137.16 162.56) (xy 154.94 162.56))
+    (stroke (width 0) (type default))
+  )
+  (bus (pts (xy 185.42 63.5) (xy 185.42 66.04))
     (stroke (width 0) (type default))
   )
@@
     (effects (font (size 1.27 1.27)) (justify left bottom))
   )
+  (label "GREEN" (at 187.96 63.5 0) (fields_autoplaced)
+    (effects (font (size 1.27 1.27)) (justify left bottom))
+  )
   (label "BLANKING" (at 187.96 35.56 0) (fields_autoplaced)
     (effects (font (size 1.27 1.27)) (justify left bottom))
@@
     (effects (font (size 1.27 1.27)) (justify right bottom))
   )
+  (label "BLUE" (at 187.96 60.96 0) (fields_autoplaced)
+    (effects (font (size 1.27 1.27)) (justify left bottom))
+  )
   (label "BLUE" (at 154.94 27.94 180) (fields_autoplaced)
     (effects (font (size 1.27 1.27)) (justify right bottom))
@@
     (effects (font (size 1.27 1.27)) (justify right bottom))
   )
+  (label "AUDIO_RIGHT" (at 187.96 73.66 0) (fields_autoplaced)
+    (effects (font (size 1.27 1.27)) (justify left bottom))
+  )
   (label "{VIDEO_SIGNALS}" (at 101.6 187.96 0) (fields_autoplaced)
     (effects (font (size 1.27 1.27)) (justify left bottom))
@@
     (effects (font (size 1.27 1.27)) (justify right bottom))
   )
+  (label "AUDIO_LEFT" (at 187.96 71.12 0) (fields_autoplaced)
+    (effects (font (size 1.27 1.27)) (justify left bottom))
+  )
   (label "GREEN" (at 76.2 162.56 180) (fields_autoplaced)
     (effects (font (size 1.27 1.27)) (justify right bottom))
@@
     (effects (font (size 1.27 1.27)) (justify right bottom))
   )
+  (label "RED" (at 187.96 58.42 0) (fields_autoplaced)
+    (effects (font (size 1.27 1.27)) (justify left bottom))
+  )
   (label "AUDIO_RIGHT" (at 154.94 172.72 180) (fields_autoplaced)
     (effects (font (size 1.27 1.27)) (justify right bottom))
@@
   (label "RED" (at 154.94 58.42 180) (fields_autoplaced)
     (effects (font (size 1.27 1.27)) (justify right bottom))
+  )
+  (label "VIDEO_RGB_SYNC" (at 187.96 66.04 0) (fields_autoplaced)
+    (effects (font (size 1.27 1.27)) (justify left bottom))
   )
   (label "VIDEO_RGB_SYNC" (at 76.2 99.06 180) (fields_autoplaced)
@@
   )
   (label "VIDEO_RGB_SYNC" (at 187.96 33.02 0) (fields_autoplaced)
+    (effects (font (size 1.27 1.27)) (justify left bottom))
+  )
+  (label "BLANKING" (at 187.96 68.58 0) (fields_autoplaced)
     (effects (font (size 1.27 1.27)) (justify left bottom))
   )
@@
       )
     )
+  )
+  (sheet (at 205.74 57.15) (size 30.48 25.4) (fields_autoplaced)
+    (stroke (width 0.1524) (type solid))
+    (fill (color 0 0 0 0.0000))
+    (property "Sheetname" "Silent input" (at 205.74 56.4384 0)
+      (effects (font (size 1.27 1.27)) (justify left bottom))
+    )
+    (property "Sheetfile" "dummy_input.kicad_sch" (at 205.74 83.1346 0)
+      (effects (font (size 1.27 1.27)) (justify left top))
+    )
+    (pin "VIDEO_RGB_SYNC" output (at 205.74 66.04 180)
+      (effects (font (size 1.27 1.27)) (justify left))
+    )
+    (pin "BLANKING" output (at 205.74 68.58 180)
+      (effects (font (size 1.27 1.27)) (justify left))
+    )
+    (pin "~{OUT_ACTIVE}" input (at 205.74 81.28 180)
+      (effects (font (size 1.27 1.27)) (justify left))
+    )
+    (pin "RED" output (at 205.74 58.42 180)
+      (effects (font (size 1.27 1.27)) (justify left))
+    )
+    (pin "BLUE" output (at 205.74 60.96 180)
+      (effects (font (size 1.27 1.27)) (justify left))
+    )
+    (pin "AUDIO_LEFT" output (at 205.74 71.12 180)
+      (effects (font (size 1.27 1.27)) (justify left))
+    )
+    (pin "GREEN" output (at 205.74 63.5 180)
+      (effects (font (size 1.27 1.27)) (justify left))
+    )
+    (pin "AUDIO_RIGHT" output (at 205.74 73.66 180)
+      (effects (font (size 1.27 1.27)) (justify left))
+    )
+    (instances
+      (project "SCART_switcher"
+        (path "/8cd08eb5-4755-4ef5-8eeb-77fd9974b180" (page "4"))
+        (path "/8cd08eb5-4755-4ef5-8eeb-77fd9974b180/6562ea38-5963-42b2-a0ef-a4a12a4c652f" (page "27"))
+      )
+    )

Commit message: Progressed ECAD.
Other:
- note added: "I_{12V}=0mA"
- note added: "I_{12V}=10mA"
- note added: "I_{12V}=10mA + 4mA + 10mA = 24mA"
- note added: "I_{12V}=4mA"
- note added: "I_{5V}=10mA"
- note added: "I_{5V}=1mA"
- note added: "I_{5V}=200mA"
- note added: "I_{5V}=3mA + 1mA*9 + 200mA + 1mA + 10mA = 223mA"
- note added: "I_{9V}=10mA"
- note added: "I_{9V}=2mA"
- note added: "I_{9V}=2mA + 2mA*9 + 30mA + 2mA + 10mA = 62mA"
- note added: "I_{9V}=30mA"
- note added: "I_{OFF_12V}=0mA"
- note added: "I_{OFF_5V}=1mA"
- note added: "I_{OFF_9V}=2mA"
- note added: "I_{ON_12V}=10mA"
- note added: "I_{ON_5V}=3mA"
- note added: "I_{ON_9V}=2mA"
- note added: "Total:"
- note added: "x9"
Changed lines of the file:
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@@
     (stroke (width 0) (type default))
+  )
+  (text "I_{9V}=2mA" (at 237.49 69.85 0)
+    (effects (font (size 1.27 1.27)) (justify left bottom))
+  )
+  (text "Total:" (at 175.26 96.52 0)
+    (effects (font (size 1.27 1.27)) (justify left bottom))
+  )
+  (text "I_{5V}=200mA" (at 237.49 34.29 0)
+    (effects (font (size 1.27 1.27)) (justify left bottom))
+  )
+  (text "I_{ON_9V}=2mA" (at 12.7 45.72 0)
+    (effects (font (size 1.27 1.27)) (justify left bottom))
+  )
+  (text "I_{12V}=0mA" (at 237.49 72.39 0)
+    (effects (font (size 1.27 1.27)) (justify left bottom))
+  )
+  (text "I_{OFF_12V}=0mA" (at 12.7 81.28 0)
+    (effects (font (size 1.27 1.27)) (justify left bottom))
+  )
+  (text "x9" (at 17.78 83.82 0)
+    (effects (font (size 1.27 1.27)) (justify left bottom))
+  )
+  (text "I_{5V}=1mA" (at 237.49 67.31 0)
+    (effects (font (size 1.27 1.27)) (justify left bottom))
+  )
+  (text "I_{ON_12V}=10mA" (at 12.7 48.26 0)
+    (effects (font (size 1.27 1.27)) (justify left bottom))
+  )
+  (text "I_{OFF_9V}=2mA" (at 12.7 78.74 0)
+    (effects (font (size 1.27 1.27)) (justify left bottom))
+  )
+  (text "I_{OFF_5V}=1mA" (at 12.7 76.2 0)
+    (effects (font (size 1.27 1.27)) (justify left bottom))
+  )
+  (text "I_{ON_5V}=3mA" (at 12.7 43.18 0)
+    (effects (font (size 1.27 1.27)) (justify left bottom))
+  )
+  (text "I_{9V}=2mA + 2mA*9 + 30mA + 2mA + 10mA = 62mA" (at 175.26 101.6 0)
+    (effects (font (size 1.27 1.27)) (justify left bottom))
+  )
+  (text "I_{12V}=10mA + 4mA + 10mA = 24mA" (at 175.26 104.14 0)
+    (effects (font (size 1.27 1.27)) (justify left bottom))
+  )
+  (text "I_{12V}=4mA" (at 237.49 39.37 0)
+    (effects (font (size 1.27 1.27)) (justify left bottom))
+  )
+  (text "I_{5V}=3mA + 1mA*9 + 200mA + 1mA + 10mA = 223mA" (at 175.26 99.06 0)
+    (effects (font (size 1.27 1.27)) (justify left bottom))
+  )
+  (text "I_{9V}=30mA" (at 237.49 36.83 0)
+    (effects (font (size 1.27 1.27)) (justify left bottom))
+  )
+  (text "I_{12V}=10mA" (at 237.49 130.81 0)
+    (effects (font (size 1.27 1.27)) (justify left bottom))
+  )
+  (text "I_{5V}=10mA" (at 237.49 125.73 0)
+    (effects (font (size 1.27 1.27)) (justify left bottom))
+  )
+  (text "I_{9V}=10mA" (at 237.49 128.27 0)
+    (effects (font (size 1.27 1.27)) (justify left bottom))
   )
   (label "GREEN" (at 76.2 63.5 180) (fields_autoplaced)
