File: ECAD/SCART_switcher/SCART_switcher.kicad_pcb (KiCad board)
At the start: 2 copper layers, 250 x 140 mm, 0 parts

Commit message: Progressed ECAD.
Parts:
- added C1: 100nC, Capacitor_SMD:C_0603_1608Metric, F.Cu at (-289.3, -89.3)
- added C10: 100nC, Capacitor_SMD:C_0603_1608Metric, F.Cu at (589.6, -180.9)
- added C100: 100nC, Capacitor_SMD:C_1206_3216Metric, F.Cu at (714.8, -177.3)
- added C101: 1000uC, Capacitor_SMD:CP_Elec_10x10.5, F.Cu at (704.8, -161.2)
- added C102: 100nC, Capacitor_SMD:C_1206_3216Metric, F.Cu at (714.8, -173.9)
- added C103: 47uC, Capacitor_SMD:CP_Elec_4x5.8, F.Cu at (-198.6, -209.6)
- added C104: 47uC, Capacitor_SMD:CP_Elec_4x5.8, F.Cu at (-198.6, -203.7)
- added C105: 100nC, Capacitor_SMD:C_0603_1608Metric, F.Cu at (-182.9, -202.4)
- added C106: 100nC, Capacitor_SMD:C_0603_1608Metric, F.Cu at (-182.9, -199.9)
- added C107: 100nC, Capacitor_SMD:C_0603_1608Metric, F.Cu at (-182.9, -197.3)
- added C108: 47uC, Capacitor_SMD:CP_Elec_4x5.8, F.Cu at (-198.6, -197.8)
- added C109: 47uC, Capacitor_SMD:CP_Elec_4x5.8, F.Cu at (-198.6, -192.0)
- added C11: 100nC, Capacitor_SMD:C_0603_1608Metric, F.Cu at (-204.3, -86.3)
- added C110: 100nC, Capacitor_SMD:C_0603_1608Metric, F.Cu at (-182.9, -194.8)
- added C111: 100nC, Capacitor_SMD:C_0603_1608Metric, F.Cu at (-182.9, -192.3)
- added C112: 100nC, Capacitor_SMD:C_0603_1608Metric, F.Cu at (-183.2, -167.5)
- added C113: 1nC, Capacitor_SMD:C_0805_2012Metric, F.Cu at (-205.2, -153.0)
- added C114: 1nC, Capacitor_SMD:C_0805_2012Metric, F.Cu at (-205.2, -150.0)
- added C115: 22uC, Capacitor_SMD:CP_Elec_5x5.4, F.Cu at (-189.7, -169.2)
- added C116: 22uC, Capacitor_SMD:CP_Elec_5x5.4, F.Cu at (-189.7, -162.3)
- added C117: 100nC, Capacitor_SMD:C_0603_1608Metric, F.Cu at (-183.2, -165.0)
- added C118: 47uC, Capacitor_SMD:CP_Elec_4x5.8, F.Cu at (-110.2, -206.5)
- added C119: 47uC, Capacitor_SMD:CP_Elec_4x5.8, F.Cu at (-110.2, -200.7)
- added C12: 100nC, Capacitor_SMD:C_0603_1608Metric, F.Cu at (-204.3, -83.7)
- added C120: 100nC, Capacitor_SMD:C_0603_1608Metric, F.Cu at (-94.4, -199.3)
- added C121: 100nC, Capacitor_SMD:C_0603_1608Metric, F.Cu at (-94.4, -196.8)
- added C122: 100nC, Capacitor_SMD:C_0603_1608Metric, F.Cu at (-94.4, -194.3)
- added C123: 47uC, Capacitor_SMD:CP_Elec_4x5.8, F.Cu at (-110.2, -194.8)
- added C124: 47uC, Capacitor_SMD:CP_Elec_4x5.8, F.Cu at (-110.2, -188.9)
- added C125: 100nC, Capacitor_SMD:C_0603_1608Metric, F.Cu at (-94.4, -191.8)
- added C126: 100nC, Capacitor_SMD:C_0603_1608Metric, F.Cu at (-94.4, -189.3)
- added C127: 100nC, Capacitor_SMD:C_0603_1608Metric, F.Cu at (-88.5, -163.2)
- added C128: 1nC, Capacitor_SMD:C_0805_2012Metric, F.Cu at (-110.5, -148.7)
- added C129: 1nC, Capacitor_SMD:C_0805_2012Metric, F.Cu at (-110.5, -145.7)
- added C13: 100nC, Capacitor_SMD:C_0603_1608Metric, F.Cu at (-118.3, -86.3)
- added C130: 22uC, Capacitor_SMD:CP_Elec_5x5.4, F.Cu at (-95.0, -164.8)
- added C131: 22uC, Capacitor_SMD:CP_Elec_5x5.4, F.Cu at (-95.0, -158.0)
- added C132: 100nC, Capacitor_SMD:C_0603_1608Metric, F.Cu at (-88.5, -160.7)
- added C133: 47uC, Capacitor_SMD:CP_Elec_4x5.8, F.Cu at (-31.0, -202.4)
- added C134: 47uC, Capacitor_SMD:CP_Elec_4x5.8, F.Cu at (-31.0, -196.6)
- added C135: 100nC, Capacitor_SMD:C_0603_1608Metric, F.Cu at (-15.3, -195.3)
- added C136: 100nC, Capacitor_SMD:C_0603_1608Metric, F.Cu at (-15.3, -192.8)
- added C137: 100nC, Capacitor_SMD:C_0603_1608Metric, F.Cu at (-15.3, -190.2)
- added C138: 47uC, Capacitor_SMD:CP_Elec_4x5.8, F.Cu at (-31.0, -190.8)
- added C139: 47uC, Capacitor_SMD:CP_Elec_4x5.8, F.Cu at (-31.0, -184.9)
- added C14: 100nC, Capacitor_SMD:C_0603_1608Metric, F.Cu at (-118.3, -83.7)
- added C140: 100nC, Capacitor_SMD:C_0603_1608Metric, F.Cu at (-15.3, -187.7)
- added C141: 100nC, Capacitor_SMD:C_0603_1608Metric, F.Cu at (-15.3, -185.2)
- added C142: 100nC, Capacitor_SMD:C_0603_1608Metric, F.Cu at (-10.7, -151.2)
- added C143: 1nC, Capacitor_SMD:C_0805_2012Metric, F.Cu at (-32.7, -136.7)
- added C144: 1nC, Capacitor_SMD:C_0805_2012Metric, F.Cu at (-32.7, -133.7)
- added C145: 22uC, Capacitor_SMD:CP_Elec_5x5.4, F.Cu at (-17.2, -152.8)
- added C146: 22uC, Capacitor_SMD:CP_Elec_5x5.4, F.Cu at (-17.2, -146.0)
- added C147: 100nC, Capacitor_SMD:C_0603_1608Metric, F.Cu at (-10.7, -148.7)
- added C148: 47uC, Capacitor_SMD:CP_Elec_4x5.8, F.Cu at (47.4, -200.4)
- added C149: 47uC, Capacitor_SMD:CP_Elec_4x5.8, F.Cu at (47.4, -194.6)
- added C15: 100nC, Capacitor_SMD:C_0603_1608Metric, F.Cu at (-38.3, -85.3)
- added C150: 100nC, Capacitor_SMD:C_0603_1608Metric, F.Cu at (63.1, -193.3)
- added C151: 100nC, Capacitor_SMD:C_0603_1608Metric, F.Cu at (63.1, -190.8)
- added C152: 100nC, Capacitor_SMD:C_0603_1608Metric, F.Cu at (63.1, -188.2)
- added C153: 47uC, Capacitor_SMD:CP_Elec_4x5.8, F.Cu at (47.4, -188.8)
- added C154: 47uC, Capacitor_SMD:CP_Elec_4x5.8, F.Cu at (47.4, -182.9)
- added C155: 100nC, Capacitor_SMD:C_0603_1608Metric, F.Cu at (63.1, -185.7)
- added C156: 100nC, Capacitor_SMD:C_0603_1608Metric, F.Cu at (63.1, -183.2)
- added C157: 100nC, Capacitor_SMD:C_0603_1608Metric, F.Cu at (63.2, -157.0)
- added C158: 1nC, Capacitor_SMD:C_0805_2012Metric, F.Cu at (41.3, -142.5)
- added C159: 1nC, Capacitor_SMD:C_0805_2012Metric, F.Cu at (41.3, -139.5)
- added C16: 100nC, Capacitor_SMD:C_0603_1608Metric, F.Cu at (-38.3, -82.7)
- added C160: 22uC, Capacitor_SMD:CP_Elec_5x5.4, F.Cu at (56.7, -158.7)
- added C161: 22uC, Capacitor_SMD:CP_Elec_5x5.4, F.Cu at (56.7, -151.8)
- added C162: 100nC, Capacitor_SMD:C_0603_1608Metric, F.Cu at (63.2, -154.5)
- added C163: 47uC, Capacitor_SMD:CP_Elec_4x5.8, F.Cu at (140.6, -198.5)
- added C164: 47uC, Capacitor_SMD:CP_Elec_4x5.8, F.Cu at (140.6, -192.7)
- added C165: 100nC, Capacitor_SMD:C_0603_1608Metric, F.Cu at (156.3, -191.3)
- added C166: 100nC, Capacitor_SMD:C_0603_1608Metric, F.Cu at (156.3, -188.8)
- added C167: 100nC, Capacitor_SMD:C_0603_1608Metric, F.Cu at (156.3, -186.3)
- added C168: 47uC, Capacitor_SMD:CP_Elec_4x5.8, F.Cu at (140.6, -186.8)
- added C169: 47uC, Capacitor_SMD:CP_Elec_4x5.8, F.Cu at (140.6, -180.9)
- added C17: 100nC, Capacitor_SMD:C_0603_1608Metric, F.Cu at (44.7, -83.3)
- added C170: 100nC, Capacitor_SMD:C_0603_1608Metric, F.Cu at (156.3, -183.8)
- added C171: 100nC, Capacitor_SMD:C_0603_1608Metric, F.Cu at (156.3, -181.3)
- added C172: 100nC, Capacitor_SMD:C_0603_1608Metric, F.Cu at (158.3, -151.6)
- added C173: 1nC, Capacitor_SMD:C_0805_2012Metric, F.Cu at (136.3, -137.1)
- added C174: 1nC, Capacitor_SMD:C_0805_2012Metric, F.Cu at (136.3, -134.1)
- added C175: 22uC, Capacitor_SMD:CP_Elec_5x5.4, F.Cu at (151.8, -153.3)
- added C176: 22uC, Capacitor_SMD:CP_Elec_5x5.4, F.Cu at (151.8, -146.4)
- added C177: 100nC, Capacitor_SMD:C_0603_1608Metric, F.Cu at (158.3, -149.1)
- added C178: 47uC, Capacitor_SMD:CP_Elec_4x5.8, F.Cu at (218.3, -196.2)
- added C179: 47uC, Capacitor_SMD:CP_Elec_4x5.8, F.Cu at (218.3, -190.3)
- added C18: 100nC, Capacitor_SMD:C_0603_1608Metric, F.Cu at (44.7, -80.7)
- added C180: 100nC, Capacitor_SMD:C_0603_1608Metric, F.Cu at (234.0, -189.0)
- added C181: 100nC, Capacitor_SMD:C_0603_1608Metric, F.Cu at (234.0, -186.5)
- added C182: 100nC, Capacitor_SMD:C_0603_1608Metric, F.Cu at (234.0, -184.0)
- added C183: 47uC, Capacitor_SMD:CP_Elec_4x5.8, F.Cu at (218.3, -184.5)
- added C184: 47uC, Capacitor_SMD:CP_Elec_4x5.8, F.Cu at (218.3, -178.6)
- added C185: 100nC, Capacitor_SMD:C_0603_1608Metric, F.Cu at (234.0, -181.5)
- added C186: 100nC, Capacitor_SMD:C_0603_1608Metric, F.Cu at (234.0, -179.0)
- added C187: 100nC, Capacitor_SMD:C_0603_1608Metric, F.Cu at (237.8, -155.5)
- added C188: 1nC, Capacitor_SMD:C_0805_2012Metric, F.Cu at (215.8, -141.0)
- added C189: 1nC, Capacitor_SMD:C_0805_2012Metric, F.Cu at (215.8, -138.0)
- added C19: 100nC, Capacitor_SMD:C_0603_1608Metric, F.Cu at (132.7, -82.3)
- added C190: 22uC, Capacitor_SMD:CP_Elec_5x5.4, F.Cu at (231.3, -157.2)
- added C191: 22uC, Capacitor_SMD:CP_Elec_5x5.4, F.Cu at (231.3, -150.3)
- added C192: 100nC, Capacitor_SMD:C_0603_1608Metric, F.Cu at (237.8, -153.0)
- added C193: 47uC, Capacitor_SMD:CP_Elec_4x5.8, F.Cu at (309.5, -196.2)
- added C194: 47uC, Capacitor_SMD:CP_Elec_4x5.8, F.Cu at (309.5, -190.3)
- added C195: 100nC, Capacitor_SMD:C_0603_1608Metric, F.Cu at (325.2, -189.0)
- added C196: 100nC, Capacitor_SMD:C_0603_1608Metric, F.Cu at (325.2, -186.5)
- added C197: 100nC, Capacitor_SMD:C_0603_1608Metric, F.Cu at (325.2, -184.0)
- added C198: 47uC, Capacitor_SMD:CP_Elec_4x5.8, F.Cu at (309.5, -184.5)
- added C199: 47uC, Capacitor_SMD:CP_Elec_4x5.8, F.Cu at (309.5, -178.6)
- added C2: 100nC, Capacitor_SMD:C_0603_1608Metric, F.Cu at (-289.3, -86.7)
- added C20: 100nC, Capacitor_SMD:C_0603_1608Metric, F.Cu at (132.7, -79.7)
- added C200: 100nC, Capacitor_SMD:C_0603_1608Metric, F.Cu at (325.2, -181.5)
- added C201: 100nC, Capacitor_SMD:C_0603_1608Metric, F.Cu at (325.2, -179.0)
- added C202: 100nC, Capacitor_SMD:C_0603_1608Metric, F.Cu at (329.5, -156.3)
- added C203: 1nC, Capacitor_SMD:C_0805_2012Metric, F.Cu at (307.5, -141.8)
- added C204: 1nC, Capacitor_SMD:C_0805_2012Metric, F.Cu at (307.5, -138.8)
- added C205: 22uC, Capacitor_SMD:CP_Elec_5x5.4, F.Cu at (323.0, -158.0)
- added C206: 22uC, Capacitor_SMD:CP_Elec_5x5.4, F.Cu at (323.0, -151.2)
- added C207: 100nC, Capacitor_SMD:C_0603_1608Metric, F.Cu at (329.5, -153.8)
- added C208: 47uC, Capacitor_SMD:CP_Elec_4x5.8, F.Cu at (389.0, -193.7)
- added C209: 47uC, Capacitor_SMD:CP_Elec_4x5.8, F.Cu at (389.0, -187.8)
- added C21: 100nC, Capacitor_SMD:C_0603_1608Metric, F.Cu at (214.7, -80.3)
- added C210: 100nC, Capacitor_SMD:C_0603_1608Metric, F.Cu at (404.8, -186.5)
- added C211: 100nC, Capacitor_SMD:C_0603_1608Metric, F.Cu at (404.8, -184.0)
- added C212: 100nC, Capacitor_SMD:C_0603_1608Metric, F.Cu at (404.8, -181.5)
- added C213: 47uC, Capacitor_SMD:CP_Elec_4x5.8, F.Cu at (389.0, -182.0)
- added C214: 47uC, Capacitor_SMD:CP_Elec_4x5.8, F.Cu at (389.0, -176.1)
- added C215: 100nC, Capacitor_SMD:C_0603_1608Metric, F.Cu at (404.8, -179.0)
- added C216: 100nC, Capacitor_SMD:C_0603_1608Metric, F.Cu at (404.8, -176.5)
- added C217: 100nC, Capacitor_SMD:C_0603_1608Metric, F.Cu at (406.1, -153.3)
- added C218: 1nC, Capacitor_SMD:C_0805_2012Metric, F.Cu at (384.1, -138.8)
- added C219: 1nC, Capacitor_SMD:C_0805_2012Metric, F.Cu at (384.1, -135.8)
- added C22: 100nC, Capacitor_SMD:C_0603_1608Metric, F.Cu at (214.7, -77.7)
- added C220: 22uC, Capacitor_SMD:CP_Elec_5x5.4, F.Cu at (399.6, -154.9)
- added C221: 22uC, Capacitor_SMD:CP_Elec_5x5.4, F.Cu at (399.6, -148.1)
- added C222: 100nC, Capacitor_SMD:C_0603_1608Metric, F.Cu at (406.1, -150.8)
- added C223: 47uC, Capacitor_SMD:CP_Elec_4x5.8, F.Cu at (466.5, -203.5)
- added C224: 47uC, Capacitor_SMD:CP_Elec_4x5.8, F.Cu at (466.5, -197.7)
- added C225: 100nC, Capacitor_SMD:C_0603_1608Metric, F.Cu at (482.2, -196.3)
- added C226: 100nC, Capacitor_SMD:C_0603_1608Metric, F.Cu at (482.2, -193.8)
- added C227: 100nC, Capacitor_SMD:C_0603_1608Metric, F.Cu at (482.2, -191.3)
- added C228: 47uC, Capacitor_SMD:CP_Elec_4x5.8, F.Cu at (466.5, -191.8)
- added C229: 47uC, Capacitor_SMD:CP_Elec_4x5.8, F.Cu at (466.5, -185.9)
- added C23: 100nC, Capacitor_SMD:C_0603_1608Metric, F.Cu at (303.7, -78.3)
- added C230: 100nC, Capacitor_SMD:C_0603_1608Metric, F.Cu at (482.2, -188.8)
- added C231: 100nC, Capacitor_SMD:C_0603_1608Metric, F.Cu at (482.2, -186.3)
- added C232: 100nC, Capacitor_SMD:C_0603_1608Metric, F.Cu at (491.1, -146.3)
- added C233: 1nC, Capacitor_SMD:C_0805_2012Metric, F.Cu at (469.1, -131.8)
- added C234: 1nC, Capacitor_SMD:C_0805_2012Metric, F.Cu at (469.1, -128.8)
- added C235: 22uC, Capacitor_SMD:CP_Elec_5x5.4, F.Cu at (484.6, -147.9)
- added C236: 22uC, Capacitor_SMD:CP_Elec_5x5.4, F.Cu at (484.6, -141.1)
- added C237: 100nC, Capacitor_SMD:C_0603_1608Metric, F.Cu at (491.1, -143.8)
- added C24: 100nC, Capacitor_SMD:C_0603_1608Metric, F.Cu at (303.7, -75.7)
- added C25: 100nC, Capacitor_SMD:C_0603_1608Metric, F.Cu at (384.7, -77.3)
- added C26: 100nC, Capacitor_SMD:C_0603_1608Metric, F.Cu at (384.7, -74.7)
- added C27: 100nC, Capacitor_SMD:C_0603_1608Metric, F.Cu at (473.7, -73.3)
- added C28: 100nC, Capacitor_SMD:C_0603_1608Metric, F.Cu at (473.7, -70.7)
- added C29: 10uC, Capacitor_SMD:CP_Elec_4x5.4, F.Cu at (868.6, -154.4)
- added C3: 100nC, Capacitor_SMD:C_0603_1608Metric, F.Cu at (695.6, -84.1)
- added C30: 100nC, Capacitor_SMD:C_0603_1608Metric, F.Cu at (853.4, -138.8)
- added C31: 10uC, Capacitor_SMD:CP_Elec_4x5.4, F.Cu at (868.6, -148.6)
- added C32: 10uC, Capacitor_SMD:CP_Elec_4x5.4, F.Cu at (868.6, -142.8)
- added C33: 100nC, Capacitor_SMD:C_0603_1608Metric, F.Cu at (853.4, -136.3)
- added C34: 10uC, Capacitor_SMD:CP_Elec_4x5.4, F.Cu at (868.6, -136.9)
- added C35: 100nC, Capacitor_SMD:C_0603_1608Metric, F.Cu at (680.8, -181.5)
- added C36: 100nC, Capacitor_SMD:C_0603_1608Metric, F.Cu at (680.8, -179.0)
- added C37: 100nC, Capacitor_SMD:C_0603_1608Metric, F.Cu at (680.8, -176.5)
- added C38: 10uC, Capacitor_SMD:CP_Elec_4x5.4, F.Cu at (666.5, -200.5)
- added C39: 10uC, Capacitor_SMD:CP_Elec_4x5.4, F.Cu at (666.5, -194.7)
- added C4: 100nC, Capacitor_SMD:C_0603_1608Metric, F.Cu at (589.6, -196.0)
- added C40: 10uC, Capacitor_SMD:CP_Elec_4x5.4, F.Cu at (666.5, -188.8)
- added C41: 10uC, Capacitor_SMD:CP_Elec_4x5.4, F.Cu at (666.5, -182.9)
- added C42: 10uC, Capacitor_SMD:CP_Elec_4x5.4, F.Cu at (666.5, -177.1)
- added C43: 10uC, Capacitor_SMD:CP_Elec_4x5.4, F.Cu at (666.5, -171.2)
- added C44: 10uC, Capacitor_SMD:CP_Elec_4x5.4, F.Cu at (666.5, -165.4)
- added C45: 100nC, Capacitor_SMD:C_0603_1608Metric, F.Cu at (-259.8, -167.9)
- added C46: 1nC, Capacitor_SMD:C_0805_2012Metric, F.Cu at (-281.8, -153.4)
- added C47: 1nC, Capacitor_SMD:C_0805_2012Metric, F.Cu at (-281.8, -150.4)
- added C48: 22uC, Capacitor_SMD:CP_Elec_5x5.4, F.Cu at (-266.3, -169.6)
- added C49: 22uC, Capacitor_SMD:CP_Elec_5x5.4, F.Cu at (-266.3, -162.8)
- added C5: 100nC, Capacitor_SMD:C_0603_1608Metric, F.Cu at (589.6, -193.5)
- added C50: 100nC, Capacitor_SMD:C_0603_1608Metric, F.Cu at (-259.8, -165.4)
- added C51: 100nC, Capacitor_SMD:C_0603_1608Metric, F.Cu at (-273.0, -241.0)
- added C52: 100nC, Capacitor_SMD:C_0603_1608Metric, F.Cu at (-273.0, -238.5)
- added C53: 100nC, Capacitor_SMD:C_0603_1608Metric, F.Cu at (-273.0, -236.0)
- added C54: 100nC, Capacitor_SMD:C_0603_1608Metric, F.Cu at (-191.8, -237.0)
- added C55: 100nC, Capacitor_SMD:C_0603_1608Metric, F.Cu at (-191.8, -234.5)
- added C56: 100nC, Capacitor_SMD:C_0603_1608Metric, F.Cu at (-191.8, -232.0)
- added C57: 100nC, Capacitor_SMD:C_0603_1608Metric, F.Cu at (-102.9, -233.9)
- added C58: 100nC, Capacitor_SMD:C_0603_1608Metric, F.Cu at (-102.9, -231.4)
- added C59: 100nC, Capacitor_SMD:C_0603_1608Metric, F.Cu at (-102.9, -228.8)
- added C6: 100nC, Capacitor_SMD:C_0603_1608Metric, F.Cu at (589.6, -190.9)
- added C60: 100nC, Capacitor_SMD:C_0603_1608Metric, F.Cu at (-20.8, -229.0)
- added C61: 100nC, Capacitor_SMD:C_0603_1608Metric, F.Cu at (-20.8, -226.5)
- added C62: 100nC, Capacitor_SMD:C_0603_1608Metric, F.Cu at (-20.8, -224.0)
- added C63: 100nC, Capacitor_SMD:C_0603_1608Metric, F.Cu at (58.2, -236.0)
- added C64: 100nC, Capacitor_SMD:C_0603_1608Metric, F.Cu at (58.2, -233.5)
- added C65: 100nC, Capacitor_SMD:C_0603_1608Metric, F.Cu at (58.2, -231.0)
- added C66: 100nC, Capacitor_SMD:C_0603_1608Metric, F.Cu at (152.1, -223.5)
- added C67: 100nC, Capacitor_SMD:C_0603_1608Metric, F.Cu at (152.1, -221.0)
- added C68: 100nC, Capacitor_SMD:C_0603_1608Metric, F.Cu at (152.1, -218.5)
- added C69: 100nC, Capacitor_SMD:C_0603_1608Metric, F.Cu at (235.1, -229.5)
- added C7: 100nC, Capacitor_SMD:C_0603_1608Metric, F.Cu at (589.6, -188.4)
- added C70: 100nC, Capacitor_SMD:C_0603_1608Metric, F.Cu at (235.1, -227.0)
- added C71: 100nC, Capacitor_SMD:C_0603_1608Metric, F.Cu at (235.1, -224.5)
- added C72: 100nC, Capacitor_SMD:C_0603_1608Metric, F.Cu at (322.1, -229.5)
- added C73: 100nC, Capacitor_SMD:C_0603_1608Metric, F.Cu at (322.1, -227.0)
- added C74: 100nC, Capacitor_SMD:C_0603_1608Metric, F.Cu at (322.1, -224.5)
- added C75: 47uC, Capacitor_SMD:CP_Elec_4x5.8, F.Cu at (-280.6, -211.4)
- added C76: 47uC, Capacitor_SMD:CP_Elec_4x5.8, F.Cu at (-280.6, -205.6)
- added C77: 100nC, Capacitor_SMD:C_0603_1608Metric, F.Cu at (-264.9, -204.3)
- added C78: 100nC, Capacitor_SMD:C_0603_1608Metric, F.Cu at (-264.9, -201.8)
- added C79: 100nC, Capacitor_SMD:C_0603_1608Metric, F.Cu at (-264.9, -199.2)
- added C8: 100nC, Capacitor_SMD:C_0603_1608Metric, F.Cu at (589.6, -185.9)
- added C80: 47uC, Capacitor_SMD:CP_Elec_4x5.8, F.Cu at (-280.6, -199.8)
- added C81: 47uC, Capacitor_SMD:CP_Elec_4x5.8, F.Cu at (-280.6, -193.9)
- added C82: 100nC, Capacitor_SMD:C_0603_1608Metric, F.Cu at (-264.9, -196.7)
- added C83: 100nC, Capacitor_SMD:C_0603_1608Metric, F.Cu at (-264.9, -194.2)
- added C84: 100nC, Capacitor_SMD:C_0603_1608Metric, F.Cu at (401.1, -232.4)
- added C85: 100nC, Capacitor_SMD:C_0603_1608Metric, F.Cu at (401.1, -229.9)
- added C86: 100nC, Capacitor_SMD:C_0603_1608Metric, F.Cu at (401.1, -227.3)
- added C87: 100nC, Capacitor_SMD:C_0603_1608Metric, F.Cu at (479.1, -237.4)
- added C88: 100nC, Capacitor_SMD:C_0603_1608Metric, F.Cu at (479.1, -234.9)
- added C89: 100nC, Capacitor_SMD:C_0603_1608Metric, F.Cu at (479.1, -232.3)
- added C9: 100nC, Capacitor_SMD:C_0603_1608Metric, F.Cu at (589.6, -183.4)
- added C90: 100nC, Capacitor_SMD:C_0603_1608Metric, F.Cu at (727.4, -184.4)
- added C91: 10uC, Capacitor_SMD:CP_Elec_4x5.4, F.Cu at (721.5, -182.8)
- added C92: 1000uC, Capacitor_SMD:CP_Elec_10x10.5, F.Cu at (704.8, -197.3)
- added C93: 100nC, Capacitor_SMD:C_1206_3216Metric, F.Cu at (714.8, -184.0)
- added C94: 1000uC, Capacitor_SMD:CP_Elec_10x10.5, F.Cu at (704.8, -185.3)
- added C95: 100nC, Capacitor_SMD:C_1206_3216Metric, F.Cu at (714.8, -180.7)
- added C96: 100nC, Capacitor_SMD:C_0603_1608Metric, F.Cu at (727.4, -181.9)
- added C97: 100nC, Capacitor_SMD:C_0603_1608Metric, F.Cu at (727.4, -179.4)
- added C98: 10uC, Capacitor_SMD:CP_Elec_4x5.4, F.Cu at (721.5, -176.9)
- added C99: 1000uC, Capacitor_SMD:CP_Elec_10x10.5, F.Cu at (704.8, -173.2)
- added D1: BZT52H-B6V8, Diode_SMD:D_SOD-123F, F.Cu at (-303.4, -100.6)
- added D10: BZT52H-B6V8, Diode_SMD:D_SOD-123F, F.Cu at (-218.4, -90.9)
- added D11: BZT52H-B6V8, Diode_SMD:D_SOD-123F, F.Cu at (-218.4, -87.5)
- added D12: BZT52H-B6V8, Diode_SMD:D_SOD-123F, F.Cu at (-218.4, -84.2)
- added D13: BZT52H-C3V3, Diode_SMD:D_SOD-123F, F.Cu at (-218.4, -80.8)
- added D14: LED, LED_THT:LED_D5.0mm, F.Cu at (-203.9, -95.5)
- added D15: BZT52H-B6V8, Diode_SMD:D_SOD-123F, F.Cu at (-132.4, -97.6)
- added D16: BZT52H-B6V8, Diode_SMD:D_SOD-123F, F.Cu at (-132.4, -94.2)
- added D17: BZT52H-B6V8, Diode_SMD:D_SOD-123F, F.Cu at (-132.4, -90.9)
- added D18: BZT52H-B6V8, Diode_SMD:D_SOD-123F, F.Cu at (-132.4, -87.5)
- added D19: BZT52H-B6V8, Diode_SMD:D_SOD-123F, F.Cu at (-132.4, -84.2)
- added D2: BZT52H-B6V8, Diode_SMD:D_SOD-123F, F.Cu at (-303.4, -97.2)
- added D20: BZT52H-C3V3, Diode_SMD:D_SOD-123F, F.Cu at (-132.4, -80.8)
- added D21: LED, LED_THT:LED_D5.0mm, F.Cu at (-117.9, -95.5)
- added D22: BZT52H-B6V8, Diode_SMD:D_SOD-123F, F.Cu at (-52.4, -96.6)
- added D23: BZT52H-B6V8, Diode_SMD:D_SOD-123F, F.Cu at (-52.4, -93.2)
- added D24: BZT52H-B6V8, Diode_SMD:D_SOD-123F, F.Cu at (-52.4, -89.9)
- added D25: BZT52H-B6V8, Diode_SMD:D_SOD-123F, F.Cu at (-52.4, -86.5)
- added D26: BZT52H-B6V8, Diode_SMD:D_SOD-123F, F.Cu at (-52.4, -83.2)
- added D27: BZT52H-C3V3, Diode_SMD:D_SOD-123F, F.Cu at (-52.4, -79.8)
- added D28: LED, LED_THT:LED_D5.0mm, F.Cu at (-37.9, -94.5)
- added D29: BZT52H-B6V8, Diode_SMD:D_SOD-123F, F.Cu at (30.6, -94.6)
- added D3: BZT52H-B6V8, Diode_SMD:D_SOD-123F, F.Cu at (-303.4, -93.9)
- added D30: BZT52H-B6V8, Diode_SMD:D_SOD-123F, F.Cu at (30.6, -91.2)
- added D31: BZT52H-B6V8, Diode_SMD:D_SOD-123F, F.Cu at (30.6, -87.9)
- added D32: BZT52H-B6V8, Diode_SMD:D_SOD-123F, F.Cu at (30.6, -84.5)
- added D33: BZT52H-B6V8, Diode_SMD:D_SOD-123F, F.Cu at (30.6, -81.2)
- added D34: BZT52H-C3V3, Diode_SMD:D_SOD-123F, F.Cu at (30.6, -77.8)
- added D35: LED, LED_THT:LED_D5.0mm, F.Cu at (45.1, -92.5)
- added D36: BZT52H-B6V8, Diode_SMD:D_SOD-123F, F.Cu at (118.6, -93.6)
- added D37: BZT52H-B6V8, Diode_SMD:D_SOD-123F, F.Cu at (118.6, -90.2)
- added D38: BZT52H-B6V8, Diode_SMD:D_SOD-123F, F.Cu at (118.6, -86.9)
- added D39: BZT52H-B6V8, Diode_SMD:D_SOD-123F, F.Cu at (118.6, -83.5)
- added D4: BZT52H-B6V8, Diode_SMD:D_SOD-123F, F.Cu at (-303.4, -90.5)
- added D40: BZT52H-B6V8, Diode_SMD:D_SOD-123F, F.Cu at (118.6, -80.2)
- added D41: BZT52H-C3V3, Diode_SMD:D_SOD-123F, F.Cu at (118.6, -76.8)
- added D42: LED, LED_THT:LED_D5.0mm, F.Cu at (133.1, -91.5)
- added D43: BZT52H-B6V8, Diode_SMD:D_SOD-123F, F.Cu at (200.6, -91.6)
- added D44: BZT52H-B6V8, Diode_SMD:D_SOD-123F, F.Cu at (200.6, -88.2)
- added D45: BZT52H-B6V8, Diode_SMD:D_SOD-123F, F.Cu at (200.6, -84.9)
- added D46: BZT52H-B6V8, Diode_SMD:D_SOD-123F, F.Cu at (200.6, -81.5)
- added D47: BZT52H-B6V8, Diode_SMD:D_SOD-123F, F.Cu at (200.6, -78.2)
- added D48: BZT52H-C3V3, Diode_SMD:D_SOD-123F, F.Cu at (200.6, -74.8)
- added D49: LED, LED_THT:LED_D5.0mm, F.Cu at (215.1, -89.5)
- added D5: BZT52H-B6V8, Diode_SMD:D_SOD-123F, F.Cu at (-303.4, -87.2)
- added D50: BZT52H-B6V8, Diode_SMD:D_SOD-123F, F.Cu at (289.6, -89.6)
- added D51: BZT52H-B6V8, Diode_SMD:D_SOD-123F, F.Cu at (289.6, -86.2)
- added D52: BZT52H-B6V8, Diode_SMD:D_SOD-123F, F.Cu at (289.6, -82.9)
- added D53: BZT52H-B6V8, Diode_SMD:D_SOD-123F, F.Cu at (289.6, -79.5)
- added D54: BZT52H-B6V8, Diode_SMD:D_SOD-123F, F.Cu at (289.6, -76.2)
- added D55: BZT52H-C3V3, Diode_SMD:D_SOD-123F, F.Cu at (289.6, -72.8)
- added D56: LED, LED_THT:LED_D5.0mm, F.Cu at (304.1, -87.5)
- added D57: BZT52H-B6V8, Diode_SMD:D_SOD-123F, F.Cu at (370.6, -88.6)
- added D58: BZT52H-B6V8, Diode_SMD:D_SOD-123F, F.Cu at (370.6, -85.2)
- added D59: BZT52H-B6V8, Diode_SMD:D_SOD-123F, F.Cu at (370.6, -81.9)
- added D6: BZT52H-C3V3, Diode_SMD:D_SOD-123F, F.Cu at (-303.4, -83.8)
- added D60: BZT52H-B6V8, Diode_SMD:D_SOD-123F, F.Cu at (370.6, -78.5)
- added D61: BZT52H-B6V8, Diode_SMD:D_SOD-123F, F.Cu at (370.6, -75.2)
- added D62: BZT52H-C3V3, Diode_SMD:D_SOD-123F, F.Cu at (370.6, -71.8)
- added D63: LED, LED_THT:LED_D5.0mm, F.Cu at (385.1, -86.5)
- added D64: BZT52H-B6V8, Diode_SMD:D_SOD-123F, F.Cu at (459.6, -84.6)
- added D65: BZT52H-B6V8, Diode_SMD:D_SOD-123F, F.Cu at (459.6, -81.2)
- added D66: BZT52H-B6V8, Diode_SMD:D_SOD-123F, F.Cu at (459.6, -77.9)
- added D67: BZT52H-B6V8, Diode_SMD:D_SOD-123F, F.Cu at (459.6, -74.5)
- added D68: BZT52H-B6V8, Diode_SMD:D_SOD-123F, F.Cu at (459.6, -71.2)
- added D69: BZT52H-C3V3, Diode_SMD:D_SOD-123F, F.Cu at (459.6, -67.8)
- added D7: LED, LED_THT:LED_D5.0mm, F.Cu at (-288.9, -98.5)
- added D70: LED, LED_THT:LED_D5.0mm, F.Cu at (474.1, -82.5)
- added D71: BAS16H, Diode_SMD:D_SOD-123F, F.Cu at (-281.2, -156.6)
- added D72: BAS16H, Diode_SMD:D_SOD-123F, F.Cu at (719.9, -160.4)
- added D73: BAS16H, Diode_SMD:D_SOD-123F, F.Cu at (-204.6, -156.2)
- added D74: BAS16H, Diode_SMD:D_SOD-123F, F.Cu at (-109.9, -151.8)
- added D75: BAS16H, Diode_SMD:D_SOD-123F, F.Cu at (-32.1, -139.8)
- added D76: BAS16H, Diode_SMD:D_SOD-123F, F.Cu at (41.8, -145.7)
- added D77: BAS16H, Diode_SMD:D_SOD-123F, F.Cu at (136.9, -140.3)
- added D78: BAS16H, Diode_SMD:D_SOD-123F, F.Cu at (216.4, -144.2)
- added D79: BAS16H, Diode_SMD:D_SOD-123F, F.Cu at (308.1, -145.0)
- added D8: BZT52H-B6V8, Diode_SMD:D_SOD-123F, F.Cu at (-218.4, -97.6)
- added D80: BAS16H, Diode_SMD:D_SOD-123F, F.Cu at (384.7, -141.9)
- added D81: BAS16H, Diode_SMD:D_SOD-123F, F.Cu at (469.7, -134.9)
- added D9: BZT52H-B6V8, Diode_SMD:D_SOD-123F, F.Cu at (-218.4, -94.2)
- added H1: MountingHole, MountingHole:MountingHole_3.2mm_M3, F.Cu at (25.0, 25.0)
- added H2: MountingHole, MountingHole:MountingHole_3.2mm_M3, F.Cu at (25.0, 155.0)
- added H3: MountingHole, MountingHole:MountingHole_3.2mm_M3, F.Cu at (122.0, 177.1)
- added H4: MountingHole, MountingHole:MountingHole_3.2mm_M3, F.Cu at (122.0, 185.0)
- added H5: MountingHole, MountingHole:MountingHole_3.2mm_M3, F.Cu at (130.0, 177.1)
- added H6: MountingHole, MountingHole:MountingHole_3.2mm_M3, F.Cu at (130.0, 185.0)
- added H7: MountingHole, MountingHole:MountingHole_3.2mm_M3, F.Cu at (265.0, 25.0)
- added H8: MountingHole, MountingHole:MountingHole_3.2mm_M3, F.Cu at (265.0, 155.0)
- added J1: SCART-F, Connector_SCART:SCART-F, F.Cu at (41.5, 58.0)
- added J10: SCART-F, Connector_SCART:SCART-F, F.Cu at (179.6, 58.0)
- added J11: SCART-F, Connector_SCART:SCART-F, F.Cu at (202.6, 58.0)
- added J12: SCART-F, Connector_SCART:SCART-F, F.Cu at (225.6, 58.0)
- added J13: SCART-F, Connector_SCART:SCART-F, F.Cu at (248.6, 58.0)
- added J14: Conn_01x06, Connector_PinSocket_2.54mm:PinSocket_1x06_P2.54mm_Horizontal, F.Cu at (862.4, -155.1)
- added J2: RCA Left, Connector_RCA:RCA_Vertical, F.Cu at (667.4, -79.7)
- added J3: RCA Right, Connector_RCA:RCA_Vertical, F.Cu at (678.7, -79.7)
- added J4: SCART-F, Connector_SCART:SCART-F, F.Cu at (695.9, -94.5)
- added J5: SCART-F, Connector_SCART:SCART-F, F.Cu at (64.5, 58.0)
- added J6: SCART-F, Connector_SCART:SCART-F, F.Cu at (87.5, 58.0)
- added J7: SCART-F, Connector_SCART:SCART-F, F.Cu at (110.5, 58.0)
- added J8: SCART-F, Connector_SCART:SCART-F, F.Cu at (133.6, 58.0)
- added J9: SCART-F, Connector_SCART:SCART-F, F.Cu at (156.6, 58.0)
- added Q1: BC847, Package_TO_SOT_SMD:SOT-23, F.Cu at (-293.8, -100.0)
- added Q10: BC847, Package_TO_SOT_SMD:SOT-23, F.Cu at (-42.8, -96.0)
- added Q11: BC847, Package_TO_SOT_SMD:SOT-23, F.Cu at (-42.8, -91.6)
- added Q12: BC847, Package_TO_SOT_SMD:SOT-23, F.Cu at (40.2, -94.0)
- added Q13: BC847, Package_TO_SOT_SMD:SOT-23, F.Cu at (40.2, -89.6)
- added Q14: BC847, Package_TO_SOT_SMD:SOT-23, F.Cu at (128.2, -93.0)
- added Q15: BC847, Package_TO_SOT_SMD:SOT-23, F.Cu at (128.2, -88.6)
- added Q16: BC847, Package_TO_SOT_SMD:SOT-23, F.Cu at (210.2, -91.0)
- added Q17: BC847, Package_TO_SOT_SMD:SOT-23, F.Cu at (210.2, -86.6)
- added Q18: BC847, Package_TO_SOT_SMD:SOT-23, F.Cu at (299.2, -89.0)
- added Q19: BC847, Package_TO_SOT_SMD:SOT-23, F.Cu at (299.2, -84.6)
- added Q2: BC847, Package_TO_SOT_SMD:SOT-23, F.Cu at (-293.8, -95.6)
- added Q20: BC847, Package_TO_SOT_SMD:SOT-23, F.Cu at (380.2, -88.0)
- added Q21: BC847, Package_TO_SOT_SMD:SOT-23, F.Cu at (380.2, -83.6)
- added Q22: BC847, Package_TO_SOT_SMD:SOT-23, F.Cu at (469.2, -84.0)
- added Q23: BC847, Package_TO_SOT_SMD:SOT-23, F.Cu at (469.2, -79.6)
- added Q24: BC847, Package_TO_SOT_SMD:SOT-23, F.Cu at (-276.1, -156.1)
- added Q25: BC847, Package_TO_SOT_SMD:SOT-23, F.Cu at (-276.1, -151.6)
- added Q26: 2SK209, Package_TO_SOT_SMD:SC-59, F.Cu at (-259.9, -157.0)
- added Q27: 2SK209, Package_TO_SOT_SMD:SC-59, F.Cu at (-259.9, -152.3)
- added Q28: BC857, Package_TO_SOT_SMD:SOT-23, F.Cu at (727.8, -175.9)
- added Q29: BC847, Package_TO_SOT_SMD:SOT-23, F.Cu at (-199.5, -155.6)
- added Q3: BC847, Package_TO_SOT_SMD:SOT-23, F.Cu at (691.2, -83.1)
- added Q30: BC847, Package_TO_SOT_SMD:SOT-23, F.Cu at (-199.5, -151.2)
- added Q31: 2SK209, Package_TO_SOT_SMD:SC-59, F.Cu at (-183.3, -156.6)
- added Q32: 2SK209, Package_TO_SOT_SMD:SC-59, F.Cu at (-183.3, -151.9)
- added Q33: BC847, Package_TO_SOT_SMD:SOT-23, F.Cu at (-104.8, -151.3)
- added Q34: BC847, Package_TO_SOT_SMD:SOT-23, F.Cu at (-104.8, -146.8)
- added Q35: 2SK209, Package_TO_SOT_SMD:SC-59, F.Cu at (-88.6, -152.2)
- added Q36: 2SK209, Package_TO_SOT_SMD:SC-59, F.Cu at (-88.6, -147.6)
- added Q37: BC847, Package_TO_SOT_SMD:SOT-23, F.Cu at (-27.0, -139.3)
- added Q38: BC847, Package_TO_SOT_SMD:SOT-23, F.Cu at (-27.0, -134.8)
- added Q39: 2SK209, Package_TO_SOT_SMD:SC-59, F.Cu at (-10.8, -140.2)
- added Q4: BC857, Package_TO_SOT_SMD:SOT-23, F.Cu at (691.2, -78.7)
- added Q40: 2SK209, Package_TO_SOT_SMD:SC-59, F.Cu at (-10.8, -135.6)
- added Q41: BC847, Package_TO_SOT_SMD:SOT-23, F.Cu at (47.0, -145.1)
- added Q42: BC847, Package_TO_SOT_SMD:SOT-23, F.Cu at (47.0, -140.7)
- added Q43: 2SK209, Package_TO_SOT_SMD:SC-59, F.Cu at (63.1, -146.1)
- added Q44: 2SK209, Package_TO_SOT_SMD:SC-59, F.Cu at (63.1, -141.4)
- added Q45: BC847, Package_TO_SOT_SMD:SOT-23, F.Cu at (142.0, -139.8)
- added Q46: BC847, Package_TO_SOT_SMD:SOT-23, F.Cu at (142.0, -135.3)
- added Q47: 2SK209, Package_TO_SOT_SMD:SC-59, F.Cu at (158.2, -140.7)
- added Q48: 2SK209, Package_TO_SOT_SMD:SC-59, F.Cu at (158.2, -136.1)
- added Q49: BC847, Package_TO_SOT_SMD:SOT-23, F.Cu at (221.5, -143.6)
- added Q5: BC847, Package_TO_SOT_SMD:SOT-23, F.Cu at (594.1, -195.0)
- added Q50: BC847, Package_TO_SOT_SMD:SOT-23, F.Cu at (221.5, -139.2)
- added Q51: 2SK209, Package_TO_SOT_SMD:SC-59, F.Cu at (237.7, -144.6)
- added Q52: 2SK209, Package_TO_SOT_SMD:SC-59, F.Cu at (237.7, -139.9)
- added Q53: BC847, Package_TO_SOT_SMD:SOT-23, F.Cu at (313.2, -144.4)
- added Q54: BC847, Package_TO_SOT_SMD:SOT-23, F.Cu at (313.2, -140.0)
- added Q55: 2SK209, Package_TO_SOT_SMD:SC-59, F.Cu at (329.4, -145.4)
- added Q56: 2SK209, Package_TO_SOT_SMD:SC-59, F.Cu at (329.4, -140.8)
- added Q57: BC847, Package_TO_SOT_SMD:SOT-23, F.Cu at (389.8, -141.4)
- added Q58: BC847, Package_TO_SOT_SMD:SOT-23, F.Cu at (389.8, -136.9)
- added Q59: 2SK209, Package_TO_SOT_SMD:SC-59, F.Cu at (406.0, -142.3)
- added Q6: BC847, Package_TO_SOT_SMD:SOT-23, F.Cu at (-208.8, -97.0)
- added Q60: 2SK209, Package_TO_SOT_SMD:SC-59, F.Cu at (406.0, -137.7)
- added Q61: BC847, Package_TO_SOT_SMD:SOT-23, F.Cu at (474.8, -134.4)
- added Q62: BC847, Package_TO_SOT_SMD:SOT-23, F.Cu at (474.8, -129.9)
- added Q63: 2SK209, Package_TO_SOT_SMD:SC-59, F.Cu at (491.0, -135.3)
- added Q64: 2SK209, Package_TO_SOT_SMD:SC-59, F.Cu at (491.0, -130.7)
- added Q7: BC847, Package_TO_SOT_SMD:SOT-23, F.Cu at (-208.8, -92.6)
- added Q8: BC847, Package_TO_SOT_SMD:SOT-23, F.Cu at (-122.8, -97.0)
- added Q9: BC847, Package_TO_SOT_SMD:SOT-23, F.Cu at (-122.8, -92.6)
- added R1: 10kR, Resistor_SMD:R_0805_2012Metric, F.Cu at (-298.4, -100.8)
- added R10: 100R, Resistor_SMD:R_0805_2012Metric, F.Cu at (686.5, -72.1)
- added R100: 220kR, Resistor_SMD:R_0805_2012Metric, F.Cu at (-277.4, -162.7)
- added R101: 100kR, Resistor_SMD:R_0805_2012Metric, F.Cu at (-277.4, -159.8)
- added R102: 100kR, Resistor_SMD:R_0805_2012Metric, F.Cu at (-273.0, -171.6)
- added R103: 20kR, Resistor_SMD:R_0805_2012Metric, F.Cu at (-273.0, -168.6)
- added R104: 20kR, Resistor_SMD:R_0805_2012Metric, F.Cu at (-273.0, -165.7)
- added R105: 75R, Resistor_SMD:R_1210_3225Metric, F.Cu at (-273.9, -212.3)
- added R106: 75R, Resistor_SMD:R_1210_3225Metric, F.Cu at (-273.9, -208.1)
- added R107: 100kR, Resistor_SMD:R_0805_2012Metric, F.Cu at (-268.9, -212.9)
- added R108: 100kR, Resistor_SMD:R_0805_2012Metric, F.Cu at (-268.9, -209.9)
- added R109: 75R, Resistor_SMD:R_1210_3225Metric, F.Cu at (-273.9, -203.8)
- added R11: 100kR, Resistor_SMD:R_0805_2012Metric, F.Cu at (581.2, -206.0)
- added R110: 1kR, Resistor_SMD:R_0805_2012Metric, F.Cu at (-268.9, -207.0)
- added R111: 1kR, Resistor_SMD:R_0805_2012Metric, F.Cu at (-264.5, -212.9)
- added R112: 10kR, Resistor_SMD:R_0805_2012Metric, F.Cu at (-264.5, -209.9)
- added R113: 75R, Resistor_SMD:R_1210_3225Metric, F.Cu at (-273.9, -199.6)
- added R114: 75R, Resistor_SMD:R_1210_3225Metric, F.Cu at (-273.9, -195.4)
- added R115: 100kR, Resistor_SMD:R_0805_2012Metric, F.Cu at (-264.5, -207.0)
- added R116: 100kR, Resistor_SMD:R_0805_2012Metric, F.Cu at (-260.1, -212.9)
- added R117: 1kR, Resistor_SMD:R_0805_2012Metric, F.Cu at (-260.1, -209.9)
- added R118: 1kR, Resistor_SMD:R_0805_2012Metric, F.Cu at (-260.1, -207.0)
- added R119: 4k7R, Resistor_SMD:R_0805_2012Metric, F.Cu at (714.2, -201.9)
- added R12: 100kR, Resistor_SMD:R_0805_2012Metric, F.Cu at (581.2, -203.0)
- added R120: 1kR, Resistor_SMD:R_0805_2012Metric, F.Cu at (714.2, -198.9)
- added R121: 1kR, Resistor_SMD:R_0805_2012Metric, F.Cu at (714.2, -196.0)
- added R122: 1kR, Resistor_SMD:R_0805_2012Metric, F.Cu at (714.2, -193.1)
- added R123: 1kR, Resistor_SMD:R_0805_2012Metric, F.Cu at (714.2, -190.1)
- added R124: 4k7R, Resistor_SMD:R_0805_2012Metric, F.Cu at (714.2, -187.2)
- added R125: 2kR, Resistor_SMD:R_0805_2012Metric, F.Cu at (718.6, -201.9)
- added R126: 2kR, Resistor_SMD:R_0805_2012Metric, F.Cu at (718.6, -198.9)
- added R127: 10kR, Resistor_SMD:R_0805_2012Metric, F.Cu at (718.6, -196.0)
- added R128: 100kR, Resistor_SMD:R_0805_2012Metric, F.Cu at (718.6, -193.1)
- added R129: 100R, Resistor_SMD:R_0805_2012Metric, F.Cu at (718.6, -190.1)
- added R13: 10kR, Resistor_SMD:R_0805_2012Metric, F.Cu at (581.2, -200.1)
- added R130: 75R, Resistor_SMD:R_1210_3225Metric, F.Cu at (728.0, -201.3)
- added R131: 75R, Resistor_SMD:R_1210_3225Metric, F.Cu at (728.0, -197.1)
- added R132: 1kR, Resistor_SMD:R_0805_2012Metric, F.Cu at (718.6, -187.2)
- added R133: 1kR, Resistor_SMD:R_0805_2012Metric, F.Cu at (723.0, -201.9)
- added R134: 1kR, Resistor_SMD:R_0805_2012Metric, F.Cu at (723.0, -198.9)
- added R135: 1kR, Resistor_SMD:R_0805_2012Metric, F.Cu at (723.0, -196.0)
- added R136: 2kR, Resistor_SMD:R_0805_2012Metric, F.Cu at (723.0, -193.1)
- added R137: 2kR, Resistor_SMD:R_0805_2012Metric, F.Cu at (723.0, -190.1)
- added R138: 75R, Resistor_SMD:R_1210_3225Metric, F.Cu at (728.0, -192.8)
- added R139: 75R, Resistor_SMD:R_1210_3225Metric, F.Cu at (728.0, -188.6)
- added R14: 4k7R, Resistor_SMD:R_0805_2012Metric, F.Cu at (581.2, -197.1)
- added R140: 75R, Resistor_SMD:R_1210_3225Metric, F.Cu at (-191.9, -210.4)
- added R141: 75R, Resistor_SMD:R_1210_3225Metric, F.Cu at (-191.9, -206.2)
- added R142: 100kR, Resistor_SMD:R_0805_2012Metric, F.Cu at (-186.9, -211.0)
- added R143: 100kR, Resistor_SMD:R_0805_2012Metric, F.Cu at (-186.9, -208.1)
- added R144: 75R, Resistor_SMD:R_1210_3225Metric, F.Cu at (-191.9, -201.9)
- added R145: 1kR, Resistor_SMD:R_0805_2012Metric, F.Cu at (-186.9, -205.1)
- added R146: 1kR, Resistor_SMD:R_0805_2012Metric, F.Cu at (-182.5, -211.0)
- added R147: 10kR, Resistor_SMD:R_0805_2012Metric, F.Cu at (-182.5, -208.1)
- added R148: 75R, Resistor_SMD:R_1210_3225Metric, F.Cu at (-191.9, -197.7)
- added R149: 75R, Resistor_SMD:R_1210_3225Metric, F.Cu at (-191.9, -193.5)
- added R15: 100kR, Resistor_SMD:R_0805_2012Metric, F.Cu at (581.2, -194.2)
- added R150: 100kR, Resistor_SMD:R_0805_2012Metric, F.Cu at (-182.5, -205.1)
- added R151: 100kR, Resistor_SMD:R_0805_2012Metric, F.Cu at (-178.1, -211.0)
- added R152: 1kR, Resistor_SMD:R_0805_2012Metric, F.Cu at (-178.1, -208.1)
- added R153: 1kR, Resistor_SMD:R_0805_2012Metric, F.Cu at (-178.1, -205.1)
- added R154: 10kR, Resistor_SMD:R_0805_2012Metric, F.Cu at (-205.2, -171.1)
- added R155: 4k7R, Resistor_SMD:R_0805_2012Metric, F.Cu at (-205.2, -168.2)
- added R156: 10kR, Resistor_SMD:R_0805_2012Metric, F.Cu at (-205.2, -165.2)
- added R157: 220kR, Resistor_SMD:R_0805_2012Metric, F.Cu at (-205.2, -162.3)
- added R158: 4k7R, Resistor_SMD:R_0805_2012Metric, F.Cu at (-205.2, -159.3)
- added R159: 100R, Resistor_SMD:R_0805_2012Metric, F.Cu at (-200.8, -171.1)
- added R16: 100kR, Resistor_SMD:R_0805_2012Metric, F.Cu at (581.2, -191.2)
- added R160: 100R, Resistor_SMD:R_0805_2012Metric, F.Cu at (-200.8, -168.2)
- added R161: 220kR, Resistor_SMD:R_0805_2012Metric, F.Cu at (-200.8, -165.2)
- added R162: 220kR, Resistor_SMD:R_0805_2012Metric, F.Cu at (-200.8, -162.3)
- added R163: 100kR, Resistor_SMD:R_0805_2012Metric, F.Cu at (-200.8, -159.3)
- added R164: 100kR, Resistor_SMD:R_0805_2012Metric, F.Cu at (-196.4, -171.1)
- added R165: 20kR, Resistor_SMD:R_0805_2012Metric, F.Cu at (-196.4, -168.2)
- added R166: 20kR, Resistor_SMD:R_0805_2012Metric, F.Cu at (-196.4, -165.2)
- added R167: 75R, Resistor_SMD:R_1210_3225Metric, F.Cu at (-103.5, -207.3)
- added R168: 75R, Resistor_SMD:R_1210_3225Metric, F.Cu at (-103.5, -203.1)
- added R169: 100kR, Resistor_SMD:R_0805_2012Metric, F.Cu at (-98.5, -207.9)
- added R17: 100kR, Resistor_SMD:R_0805_2012Metric, F.Cu at (581.2, -188.3)
- added R170: 100kR, Resistor_SMD:R_0805_2012Metric, F.Cu at (-98.5, -205.0)
- added R171: 75R, Resistor_SMD:R_1210_3225Metric, F.Cu at (-103.5, -198.9)
- added R172: 1kR, Resistor_SMD:R_0805_2012Metric, F.Cu at (-98.5, -202.1)
- added R173: 1kR, Resistor_SMD:R_0805_2012Metric, F.Cu at (-94.1, -207.9)
- added R174: 10kR, Resistor_SMD:R_0805_2012Metric, F.Cu at (-94.1, -205.0)
- added R175: 75R, Resistor_SMD:R_1210_3225Metric, F.Cu at (-103.5, -194.7)
- added R176: 75R, Resistor_SMD:R_1210_3225Metric, F.Cu at (-103.5, -190.5)
- added R177: 100kR, Resistor_SMD:R_0805_2012Metric, F.Cu at (-94.1, -202.1)
- added R178: 100kR, Resistor_SMD:R_0805_2012Metric, F.Cu at (-89.7, -207.9)
- added R179: 1kR, Resistor_SMD:R_0805_2012Metric, F.Cu at (-89.7, -205.0)
- added R18: 100kR, Resistor_SMD:R_0805_2012Metric, F.Cu at (581.2, -185.3)
- added R180: 1kR, Resistor_SMD:R_0805_2012Metric, F.Cu at (-89.7, -202.1)
- added R181: 10kR, Resistor_SMD:R_0805_2012Metric, F.Cu at (-110.5, -166.8)
- added R182: 4k7R, Resistor_SMD:R_0805_2012Metric, F.Cu at (-110.5, -163.8)
- added R183: 10kR, Resistor_SMD:R_0805_2012Metric, F.Cu at (-110.5, -160.9)
- added R184: 220kR, Resistor_SMD:R_0805_2012Metric, F.Cu at (-110.5, -157.9)
- added R185: 4k7R, Resistor_SMD:R_0805_2012Metric, F.Cu at (-110.5, -155.0)
- added R186: 100R, Resistor_SMD:R_0805_2012Metric, F.Cu at (-106.1, -166.8)
- added R187: 100R, Resistor_SMD:R_0805_2012Metric, F.Cu at (-106.1, -163.8)
- added R188: 220kR, Resistor_SMD:R_0805_2012Metric, F.Cu at (-106.1, -160.9)
- added R189: 220kR, Resistor_SMD:R_0805_2012Metric, F.Cu at (-106.1, -157.9)
- added R19: 10kR, Resistor_SMD:R_0805_2012Metric, F.Cu at (-213.4, -97.8)
- added R190: 100kR, Resistor_SMD:R_0805_2012Metric, F.Cu at (-106.1, -155.0)
- added R191: 100kR, Resistor_SMD:R_0805_2012Metric, F.Cu at (-101.7, -166.8)
- added R192: 20kR, Resistor_SMD:R_0805_2012Metric, F.Cu at (-101.7, -163.8)
- added R193: 20kR, Resistor_SMD:R_0805_2012Metric, F.Cu at (-101.7, -160.9)
- added R194: 75R, Resistor_SMD:R_1210_3225Metric, F.Cu at (-24.3, -203.3)
- added R195: 75R, Resistor_SMD:R_1210_3225Metric, F.Cu at (-24.3, -199.1)
- added R196: 100kR, Resistor_SMD:R_0805_2012Metric, F.Cu at (-19.3, -203.9)
- added R197: 100kR, Resistor_SMD:R_0805_2012Metric, F.Cu at (-19.3, -200.9)
- added R198: 75R, Resistor_SMD:R_1210_3225Metric, F.Cu at (-24.3, -194.8)
- added R199: 1kR, Resistor_SMD:R_0805_2012Metric, F.Cu at (-19.3, -198.0)
- added R2: 220kR, Resistor_SMD:R_0805_2012Metric, F.Cu at (-298.4, -97.8)
- added R20: 220kR, Resistor_SMD:R_0805_2012Metric, F.Cu at (-213.4, -94.8)
- added R200: 1kR, Resistor_SMD:R_0805_2012Metric, F.Cu at (-14.9, -203.9)
- added R201: 10kR, Resistor_SMD:R_0805_2012Metric, F.Cu at (-14.9, -200.9)
- added R202: 75R, Resistor_SMD:R_1210_3225Metric, F.Cu at (-24.3, -190.6)
- added R203: 75R, Resistor_SMD:R_1210_3225Metric, F.Cu at (-24.3, -186.4)
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Other:
- copper layers 2 -> 4

Commit message: Progressed ECAD.
Parts:
- C112, C113, C114, C115, C116, C117, C127, C128, C129, C130, C131, C132, C142, C143, C144, C145, C146, C147, C157, C158, C159, C160, C161, C162, C172, C173, C174, C175, C176, C177, C187, C188, C189, C190, C191, C192, C202, C203, C204, C205, C206, C207, C217, C218, C219, C220, C221, C222, C232, C233, C234, C235, C236, C237, C45, C46, C47, C48, C49, C50, D71, D73, D74, D75, D76, D77, D78, D79, D80, D81, Q24, Q25, Q26, Q27, Q29, Q30, Q31, Q32, Q33, Q34, Q35, Q36, Q37, Q38, Q39, Q40, Q41, Q42, Q43, Q44, Q45, Q46, Q47, Q48, Q49, Q50, Q51, Q52, Q53, Q54, Q55, Q56, Q57, Q58, Q59, Q60, Q61, Q62, Q63, Q64, R100, R101, R102, R103, R104, R154, R155, R156, R157, R158, R159, R160, R161, R162, R163, R164, R165, R166, R181, R182, R183, R184, R185, R186, R187, R188, R189, R190, R191, R192, R193, R208, R209, R210, R211, R212, R213, R214, R215, R216, R217, R218, R219, R220, R235, R236, R237, R238, R239, R240, R241, R242, R243, R244, R245, R246, R247, R262, R263, R264, R265, R266, R267, R268, R269, R270, R271, R272, R273, R274, R289, R290, R291, R292, R293, R294, R295, R296, R297, R298, R299, R300, R301, R316, R317, R318, R319, R320, R321, R322, R323, R324, R325, R326, R327, R328, R343, R344, R345, R346, R347, R348, R349, R350, R351, R352, R353, R354, R355, R370, R371, R372, R373, R374, R375, R376, R377, R378, R379, R380, R381, R382, R92, R93, R94, R95, R96, R97, R98, R99, U100, U101, U107, U108, U114, U115, U121, U122, U128, U129, U135, U136, U34, U35, U79, U80, U86, U87, U93, U94: moved to B.Cu
- moved J3 601.8 mm to (87.0, 30.0), turned to 180 degrees
- moved J2 577.9 mm to (100.0, 30.0), turned to 180 degrees
- moved J4 564.8 mm to (145.0, 30.1), turned to 180 degrees
- moved D7 377.5 mm to (40.5, 86.0)
- moved D14 323.1 mm to (63.5, 86.0)
- moved D70 282.4 mm to (247.5, 86.0)
- moved D21 273.3 mm to (86.5, 86.0)
- moved D63 235.7 mm to (224.5, 86.0)
- moved D28 233.0 mm to (109.5, 86.0)
- moved D56 201.6 mm to (201.5, 86.0)
- moved D35 198.7 mm to (132.5, 86.0)
- moved D49 179.3 mm to (178.5, 86.0)
- moved D42 178.9 mm to (155.5, 86.0)
- moved D64 119.0 mm to (452.6, -203.4)
- moved D65 119.0 mm to (452.6, -200.1)
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