File: ECAD/SCART_switcher/SCART_switcher.kicad_pcb (KiCad board)
At the start: 4 copper layers, 250 x 140 mm, 922 parts, among them J1 SCART-F, J10 SCART-F, J11 SCART-F, J12 SCART-F, J13 SCART-F, J14 Conn_01x06, J2 RCA Left, J3 RCA Right, J4 SCART-F, J5 SCART-F, J6 SCART-F, J7 SCART-F, J8 SCART-F, J9 SCART-F, Q1 BC847, Q10 BC847, Q11 BC847, Q12 BC847, Q13 BC847, Q14 BC847, Q15 BC847, Q16 BC847, Q17 BC847, Q18 BC847, Q19 BC847, Q2 BC847, Q20 BC847, Q21 BC847, Q22 BC847, Q23 BC847, Q24 BC847, Q25 BC847, Q26 2SK209, Q27 2SK209, Q28 BC857, Q29 BC847, Q3 BC847, Q30 BC847, Q31 2SK209, Q32 2SK209, Q33 BC847, Q34 BC847, Q35 2SK209, Q36 2SK209, Q37 BC847, Q38 BC847, Q39 2SK209, Q4 BC857, Q40 2SK209, Q41 BC847, Q42 BC847, Q43 2SK209, Q44 2SK209, Q45 BC847, Q46 BC847, Q47 2SK209, Q48 2SK209, Q49 BC847, Q5 BC847, Q50 BC847, Q51 2SK209, Q52 2SK209, Q53 BC847, Q54 BC847, Q55 2SK209, Q56 2SK209, Q57 BC847, Q58 BC847, Q59 2SK209, Q6 BC847, Q60 2SK209, Q61 BC847, Q62 BC847, Q63 2SK209, Q64 2SK209, Q7 BC847, Q8 BC847, Q9 BC847, U1 74LVC1G14, U10 74LVC1G3157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

Commit message: Progressed ECAD
Connections:
- net /SCART input 1/FUNCTION renamed /SCART input 1/FUNCTION_SCART_IN
- net /SCART input 10/FUNCTION renamed /SCART input 10/FUNCTION_SCART_IN
- net /SCART input 2/FUNCTION renamed /SCART input 2/FUNCTION_SCART_IN
- net /SCART input 3/FUNCTION renamed /SCART input 3/FUNCTION_SCART_IN
- net /SCART input 4/FUNCTION renamed /SCART input 4/FUNCTION_SCART_IN
- net /SCART input 5/FUNCTION renamed /SCART input 5/FUNCTION_SCART_IN
- net /SCART input 6/FUNCTION renamed /SCART input 6/FUNCTION_SCART_IN
- net /SCART input 7/FUNCTION renamed /SCART input 7/FUNCTION_SCART_IN
- net /SCART input 8/FUNCTION renamed /SCART input 8/FUNCTION_SCART_IN
- net /SCART input 9/FUNCTION renamed /SCART input 9/FUNCTION_SCART_IN
- C103 pad 2: /GREEN -> /SCART input 2/GREEN_SCART_IN
- C104 pad 2: /RED -> /SCART input 2/RED_SCART_IN
- C108 pad 2: /BLUE -> /SCART input 2/BLUE_SCART_IN
- C109 pad 2: /VIDEO_RGB_SYNC -> /SCART input 2/VIDEO_RGB_SYNC_SCART_IN
- C118 pad 2: /GREEN -> /SCART input 3/GREEN_SCART_IN
- C119 pad 2: /RED -> /SCART input 3/RED_SCART_IN
- C123 pad 2: /BLUE -> /SCART input 3/BLUE_SCART_IN
- C124 pad 2: /VIDEO_RGB_SYNC -> /SCART input 3/VIDEO_RGB_SYNC_SCART_IN
- C133 pad 2: /GREEN -> /SCART input 4/GREEN_SCART_IN
- C134 pad 2: /RED -> /SCART input 4/RED_SCART_IN
- C138 pad 2: /BLUE -> /SCART input 4/BLUE_SCART_IN
- C139 pad 2: /VIDEO_RGB_SYNC -> /SCART input 4/VIDEO_RGB_SYNC_SCART_IN
- C148 pad 2: /GREEN -> /SCART input 5/GREEN_SCART_IN
- C149 pad 2: /RED -> /SCART input 5/RED_SCART_IN
- C153 pad 2: /BLUE -> /SCART input 5/BLUE_SCART_IN
- C154 pad 2: /VIDEO_RGB_SYNC -> /SCART input 5/VIDEO_RGB_SYNC_SCART_IN
- C163 pad 2: /GREEN -> /SCART input 6/GREEN_SCART_IN
- C164 pad 2: /RED -> /SCART input 6/RED_SCART_IN
- C168 pad 2: /BLUE -> /SCART input 6/BLUE_SCART_IN
- C169 pad 2: /VIDEO_RGB_SYNC -> /SCART input 6/VIDEO_RGB_SYNC_SCART_IN
- C178 pad 2: /GREEN -> /SCART input 7/GREEN_SCART_IN
- C179 pad 2: /RED -> /SCART input 7/RED_SCART_IN
- C183 pad 2: /BLUE -> /SCART input 7/BLUE_SCART_IN
- C184 pad 2: /VIDEO_RGB_SYNC -> /SCART input 7/VIDEO_RGB_SYNC_SCART_IN
- C193 pad 2: /GREEN -> /SCART input 8/GREEN_SCART_IN
- C194 pad 2: /RED -> /SCART input 8/RED_SCART_IN
- C198 pad 2: /BLUE -> /SCART input 8/BLUE_SCART_IN
- C199 pad 2: /VIDEO_RGB_SYNC -> /SCART input 8/VIDEO_RGB_SYNC_SCART_IN
- C208 pad 2: /GREEN -> /SCART input 9/GREEN_SCART_IN
- C209 pad 2: /RED -> /SCART input 9/RED_SCART_IN
- C213 pad 2: /BLUE -> /SCART input 9/BLUE_SCART_IN
- C214 pad 2: /VIDEO_RGB_SYNC -> /SCART input 9/VIDEO_RGB_SYNC_SCART_IN
- C223 pad 2: /GREEN -> /SCART input 10/GREEN_SCART_IN
- C224 pad 2: /RED -> /SCART input 10/RED_SCART_IN
- C228 pad 2: /BLUE -> /SCART input 10/BLUE_SCART_IN
- C229 pad 2: /VIDEO_RGB_SYNC -> /SCART input 10/VIDEO_RGB_SYNC_SCART_IN
- C75 pad 2: /GREEN -> /SCART input 1/GREEN_SCART_IN
- C76 pad 2: /RED -> /SCART input 1/RED_SCART_IN
- C80 pad 2: /BLUE -> /SCART input 1/BLUE_SCART_IN
- C81 pad 2: /VIDEO_RGB_SYNC -> /SCART input 1/VIDEO_RGB_SYNC_SCART_IN
- D1 pad 1: /RED -> /SCART input 1/RED_SCART_IN
- D10 pad 1: /BLUE -> /SCART input 2/BLUE_SCART_IN
- D11 pad 1: /VIDEO_RGB_SYNC -> /SCART input 2/VIDEO_RGB_SYNC_SCART_IN
- D12 pad 1: /BLANKING -> /SCART input 2/BLANKING_SCART_IN
- D15 pad 1: /RED -> /SCART input 3/RED_SCART_IN
- D16 pad 1: /GREEN -> /SCART input 3/GREEN_SCART_IN
- D17 pad 1: /BLUE -> /SCART input 3/BLUE_SCART_IN
- D18 pad 1: /VIDEO_RGB_SYNC -> /SCART input 3/VIDEO_RGB_SYNC_SCART_IN
- D19 pad 1: /BLANKING -> /SCART input 3/BLANKING_SCART_IN
- D2 pad 1: /GREEN -> /SCART input 1/GREEN_SCART_IN
- D22 pad 1: /RED -> /SCART input 4/RED_SCART_IN
- D23 pad 1: /GREEN -> /SCART input 4/GREEN_SCART_IN
- D24 pad 1: /BLUE -> /SCART input 4/BLUE_SCART_IN
- D25 pad 1: /VIDEO_RGB_SYNC -> /SCART input 4/VIDEO_RGB_SYNC_SCART_IN
- D26 pad 1: /BLANKING -> /SCART input 4/BLANKING_SCART_IN
- D29 pad 1: /RED -> /SCART input 5/RED_SCART_IN
- D3 pad 1: /BLUE -> /SCART input 1/BLUE_SCART_IN
- D30 pad 1: /GREEN -> /SCART input 5/GREEN_SCART_IN
- D31 pad 1: /BLUE -> /SCART input 5/BLUE_SCART_IN
- D32 pad 1: /VIDEO_RGB_SYNC -> /SCART input 5/VIDEO_RGB_SYNC_SCART_IN
- D33 pad 1: /BLANKING -> /SCART input 5/BLANKING_SCART_IN
- D36 pad 1: /RED -> /SCART input 6/RED_SCART_IN
- D37 pad 1: /GREEN -> /SCART input 6/GREEN_SCART_IN
- D38 pad 1: /BLUE -> /SCART input 6/BLUE_SCART_IN
- D39 pad 1: /VIDEO_RGB_SYNC -> /SCART input 6/VIDEO_RGB_SYNC_SCART_IN
- D4 pad 1: /VIDEO_RGB_SYNC -> /SCART input 1/VIDEO_RGB_SYNC_SCART_IN
- D40 pad 1: /BLANKING -> /SCART input 6/BLANKING_SCART_IN
- D43 pad 1: /RED -> /SCART input 7/RED_SCART_IN
- D44 pad 1: /GREEN -> /SCART input 7/GREEN_SCART_IN
- D45 pad 1: /BLUE -> /SCART input 7/BLUE_SCART_IN
- D46 pad 1: /VIDEO_RGB_SYNC -> /SCART input 7/VIDEO_RGB_SYNC_SCART_IN
- D47 pad 1: /BLANKING -> /SCART input 7/BLANKING_SCART_IN
- D5 pad 1: /BLANKING -> /SCART input 1/BLANKING_SCART_IN
- D50 pad 1: /RED -> /SCART input 8/RED_SCART_IN
- D51 pad 1: /GREEN -> /SCART input 8/GREEN_SCART_IN
- D52 pad 1: /BLUE -> /SCART input 8/BLUE_SCART_IN
- D53 pad 1: /VIDEO_RGB_SYNC -> /SCART input 8/VIDEO_RGB_SYNC_SCART_IN
- D54 pad 1: /BLANKING -> /SCART input 8/BLANKING_SCART_IN
- D57 pad 1: /RED -> /SCART input 9/RED_SCART_IN
- D58 pad 1: /GREEN -> /SCART input 9/GREEN_SCART_IN
- D59 pad 1: /BLUE -> /SCART input 9/BLUE_SCART_IN
- D60 pad 1: /VIDEO_RGB_SYNC -> /SCART input 9/VIDEO_RGB_SYNC_SCART_IN
- D61 pad 1: /BLANKING -> /SCART input 9/BLANKING_SCART_IN
- D64 pad 1: /RED -> /SCART input 10/RED_SCART_IN
- D65 pad 1: /GREEN -> /SCART input 10/GREEN_SCART_IN
- D66 pad 1: /BLUE -> /SCART input 10/BLUE_SCART_IN
- D67 pad 1: /VIDEO_RGB_SYNC -> /SCART input 10/VIDEO_RGB_SYNC_SCART_IN
- D68 pad 1: /BLANKING -> /SCART input 10/BLANKING_SCART_IN
- D8 pad 1: /RED -> /SCART input 2/RED_SCART_IN
- D9 pad 1: /GREEN -> /SCART input 2/GREEN_SCART_IN
- J1 pad 11: /GREEN -> /SCART input 1/GREEN_SCART_IN
- J1 pad 15: /RED -> /SCART input 1/RED_SCART_IN
- J1 pad 16: /BLANKING -> /SCART input 1/BLANKING_SCART_IN
- J1 pad 2: /AUDIO_RIGHT -> /SCART input 1/AUDIO_RIGHT_SCART_IN
- J1 pad 20: /VIDEO_RGB_SYNC -> /SCART input 1/VIDEO_RGB_SYNC_SCART_IN
- J1 pad 6: /AUDIO_LEFT -> /SCART input 1/AUDIO_LEFT_SCART_IN
- J1 pad 7: /BLUE -> /SCART input 1/BLUE_SCART_IN
- J10 pad 11: /GREEN -> /SCART input 7/GREEN_SCART_IN
- J10 pad 15: /RED -> /SCART input 7/RED_SCART_IN
- J10 pad 16: /BLANKING -> /SCART input 7/BLANKING_SCART_IN
- J10 pad 2: /AUDIO_RIGHT -> /SCART input 7/AUDIO_RIGHT_SCART_IN
- J10 pad 20: /VIDEO_RGB_SYNC -> /SCART input 7/VIDEO_RGB_SYNC_SCART_IN
- J10 pad 6: /AUDIO_LEFT -> /SCART input 7/AUDIO_LEFT_SCART_IN
- J10 pad 7: /BLUE -> /SCART input 7/BLUE_SCART_IN
- J11 pad 11: /GREEN -> /SCART input 8/GREEN_SCART_IN
- J11 pad 15: /RED -> /SCART input 8/RED_SCART_IN
- J11 pad 16: /BLANKING -> /SCART input 8/BLANKING_SCART_IN
- J11 pad 2: /AUDIO_RIGHT -> /SCART input 8/AUDIO_RIGHT_SCART_IN
- J11 pad 20: /VIDEO_RGB_SYNC -> /SCART input 8/VIDEO_RGB_SYNC_SCART_IN
- J11 pad 6: /AUDIO_LEFT -> /SCART input 8/AUDIO_LEFT_SCART_IN
- J11 pad 7: /BLUE -> /SCART input 8/BLUE_SCART_IN
- J12 pad 11: /GREEN -> /SCART input 9/GREEN_SCART_IN
- J12 pad 15: /RED -> /SCART input 9/RED_SCART_IN
- J12 pad 16: /BLANKING -> /SCART input 9/BLANKING_SCART_IN
- J12 pad 2: /AUDIO_RIGHT -> /SCART input 9/AUDIO_RIGHT_SCART_IN
- J12 pad 20: /VIDEO_RGB_SYNC -> /SCART input 9/VIDEO_RGB_SYNC_SCART_IN
- J12 pad 6: /AUDIO_LEFT -> /SCART input 9/AUDIO_LEFT_SCART_IN
- J12 pad 7: /BLUE -> /SCART input 9/BLUE_SCART_IN
- J13 pad 11: /GREEN -> /SCART input 10/GREEN_SCART_IN
- J13 pad 15: /RED -> /SCART input 10/RED_SCART_IN
- J13 pad 16: /BLANKING -> /SCART input 10/BLANKING_SCART_IN
- J13 pad 2: /AUDIO_RIGHT -> /SCART input 10/AUDIO_RIGHT_SCART_IN
- J13 pad 20: /VIDEO_RGB_SYNC -> /SCART input 10/VIDEO_RGB_SYNC_SCART_IN
- J13 pad 6: /AUDIO_LEFT -> /SCART input 10/AUDIO_LEFT_SCART_IN
- J13 pad 7: /BLUE -> /SCART input 10/BLUE_SCART_IN
- J5 pad 11: /GREEN -> /SCART input 2/GREEN_SCART_IN
- J5 pad 15: /RED -> /SCART input 2/RED_SCART_IN
- J5 pad 16: /BLANKING -> /SCART input 2/BLANKING_SCART_IN
- J5 pad 2: /AUDIO_RIGHT -> /SCART input 2/AUDIO_RIGHT_SCART_IN
- J5 pad 20: /VIDEO_RGB_SYNC -> /SCART input 2/VIDEO_RGB_SYNC_SCART_IN
- J5 pad 6: /AUDIO_LEFT -> /SCART input 2/AUDIO_LEFT_SCART_IN
- J5 pad 7: /BLUE -> /SCART input 2/BLUE_SCART_IN
- J6 pad 11: /GREEN -> /SCART input 3/GREEN_SCART_IN
- J6 pad 15: /RED -> /SCART input 3/RED_SCART_IN
- J6 pad 16: /BLANKING -> /SCART input 3/BLANKING_SCART_IN
- J6 pad 2: /AUDIO_RIGHT -> /SCART input 3/AUDIO_RIGHT_SCART_IN
- J6 pad 20: /VIDEO_RGB_SYNC -> /SCART input 3/VIDEO_RGB_SYNC_SCART_IN
- J6 pad 6: /AUDIO_LEFT -> /SCART input 3/AUDIO_LEFT_SCART_IN
- J6 pad 7: /BLUE -> /SCART input 3/BLUE_SCART_IN
- J7 pad 11: /GREEN -> /SCART input 4/GREEN_SCART_IN
- J7 pad 15: /RED -> /SCART input 4/RED_SCART_IN
- J7 pad 16: /BLANKING -> /SCART input 4/BLANKING_SCART_IN
- J7 pad 2: /AUDIO_RIGHT -> /SCART input 4/AUDIO_RIGHT_SCART_IN
- J7 pad 20: /VIDEO_RGB_SYNC -> /SCART input 4/VIDEO_RGB_SYNC_SCART_IN
- J7 pad 6: /AUDIO_LEFT -> /SCART input 4/AUDIO_LEFT_SCART_IN
- J7 pad 7: /BLUE -> /SCART input 4/BLUE_SCART_IN
- J8 pad 11: /GREEN -> /SCART input 5/GREEN_SCART_IN
- J8 pad 15: /RED -> /SCART input 5/RED_SCART_IN
- J8 pad 16: /BLANKING -> /SCART input 5/BLANKING_SCART_IN
- J8 pad 2: /AUDIO_RIGHT -> /SCART input 5/AUDIO_RIGHT_SCART_IN
- J8 pad 20: /VIDEO_RGB_SYNC -> /SCART input 5/VIDEO_RGB_SYNC_SCART_IN
- J8 pad 6: /AUDIO_LEFT -> /SCART input 5/AUDIO_LEFT_SCART_IN
- J8 pad 7: /BLUE -> /SCART input 5/BLUE_SCART_IN
- J9 pad 11: /GREEN -> /SCART input 6/GREEN_SCART_IN
- J9 pad 15: /RED -> /SCART input 6/RED_SCART_IN
- J9 pad 16: /BLANKING -> /SCART input 6/BLANKING_SCART_IN
- J9 pad 2: /AUDIO_RIGHT -> /SCART input 6/AUDIO_RIGHT_SCART_IN
- J9 pad 20: /VIDEO_RGB_SYNC -> /SCART input 6/VIDEO_RGB_SYNC_SCART_IN
- J9 pad 6: /AUDIO_LEFT -> /SCART input 6/AUDIO_LEFT_SCART_IN
- J9 pad 7: /BLUE -> /SCART input 6/BLUE_SCART_IN
- R105 pad 1: /GREEN -> /SCART input 1/GREEN_SCART_IN
- R106 pad 1: /RED -> /SCART input 1/RED_SCART_IN
- R109 pad 1: /BLANKING -> /SCART input 1/BLANKING_SCART_IN
- R113 pad 1: /BLUE -> /SCART input 1/BLUE_SCART_IN
- R114 pad 1: /VIDEO_RGB_SYNC -> /SCART input 1/VIDEO_RGB_SYNC_SCART_IN
- R140 pad 1: /GREEN -> /SCART input 2/GREEN_SCART_IN
- R141 pad 1: /RED -> /SCART input 2/RED_SCART_IN
- R144 pad 1: /BLANKING -> /SCART input 2/BLANKING_SCART_IN
- R148 pad 1: /BLUE -> /SCART input 2/BLUE_SCART_IN
- R149 pad 1: /VIDEO_RGB_SYNC -> /SCART input 2/VIDEO_RGB_SYNC_SCART_IN
- R159 pad 1: /AUDIO_LEFT -> /SCART input 2/AUDIO_LEFT_SCART_IN
- R160 pad 1: /AUDIO_RIGHT -> /SCART input 2/AUDIO_RIGHT_SCART_IN
- R167 pad 1: /GREEN -> /SCART input 3/GREEN_SCART_IN
- R168 pad 1: /RED -> /SCART input 3/RED_SCART_IN
- R171 pad 1: /BLANKING -> /SCART input 3/BLANKING_SCART_IN
- R175 pad 1: /BLUE -> /SCART input 3/BLUE_SCART_IN
- R176 pad 1: /VIDEO_RGB_SYNC -> /SCART input 3/VIDEO_RGB_SYNC_SCART_IN
- R186 pad 1: /AUDIO_LEFT -> /SCART input 3/AUDIO_LEFT_SCART_IN
- R187 pad 1: /AUDIO_RIGHT -> /SCART input 3/AUDIO_RIGHT_SCART_IN
- R194 pad 1: /GREEN -> /SCART input 4/GREEN_SCART_IN
- R195 pad 1: /RED -> /SCART input 4/RED_SCART_IN
- R198 pad 1: /BLANKING -> /SCART input 4/BLANKING_SCART_IN
- R202 pad 1: /BLUE -> /SCART input 4/BLUE_SCART_IN
- R203 pad 1: /VIDEO_RGB_SYNC -> /SCART input 4/VIDEO_RGB_SYNC_SCART_IN
- R213 pad 1: /AUDIO_LEFT -> /SCART input 4/AUDIO_LEFT_SCART_IN
- R214 pad 1: /AUDIO_RIGHT -> /SCART input 4/AUDIO_RIGHT_SCART_IN
- R221 pad 1: /GREEN -> /SCART input 5/GREEN_SCART_IN
- R222 pad 1: /RED -> /SCART input 5/RED_SCART_IN
- R225 pad 1: /BLANKING -> /SCART input 5/BLANKING_SCART_IN
- R229 pad 1: /BLUE -> /SCART input 5/BLUE_SCART_IN
- R230 pad 1: /VIDEO_RGB_SYNC -> /SCART input 5/VIDEO_RGB_SYNC_SCART_IN
- R240 pad 1: /AUDIO_LEFT -> /SCART input 5/AUDIO_LEFT_SCART_IN
- R241 pad 1: /AUDIO_RIGHT -> /SCART input 5/AUDIO_RIGHT_SCART_IN
- R248 pad 1: /GREEN -> /SCART input 6/GREEN_SCART_IN
- R249 pad 1: /RED -> /SCART input 6/RED_SCART_IN
- R252 pad 1: /BLANKING -> /SCART input 6/BLANKING_SCART_IN
- R256 pad 1: /BLUE -> /SCART input 6/BLUE_SCART_IN
- R257 pad 1: /VIDEO_RGB_SYNC -> /SCART input 6/VIDEO_RGB_SYNC_SCART_IN
- R267 pad 1: /AUDIO_LEFT -> /SCART input 6/AUDIO_LEFT_SCART_IN
- R268 pad 1: /AUDIO_RIGHT -> /SCART input 6/AUDIO_RIGHT_SCART_IN
- R275 pad 1: /GREEN -> /SCART input 7/GREEN_SCART_IN
- R276 pad 1: /RED -> /SCART input 7/RED_SCART_IN
- R279 pad 1: /BLANKING -> /SCART input 7/BLANKING_SCART_IN
- R283 pad 1: /BLUE -> /SCART input 7/BLUE_SCART_IN
- R284 pad 1: /VIDEO_RGB_SYNC -> /SCART input 7/VIDEO_RGB_SYNC_SCART_IN
- R294 pad 1: /AUDIO_LEFT -> /SCART input 7/AUDIO_LEFT_SCART_IN
- R295 pad 1: /AUDIO_RIGHT -> /SCART input 7/AUDIO_RIGHT_SCART_IN
- R302 pad 1: /GREEN -> /SCART input 8/GREEN_SCART_IN
- R303 pad 1: /RED -> /SCART input 8/RED_SCART_IN
- R306 pad 1: /BLANKING -> /SCART input 8/BLANKING_SCART_IN
- R310 pad 1: /BLUE -> /SCART input 8/BLUE_SCART_IN
- R311 pad 1: /VIDEO_RGB_SYNC -> /SCART input 8/VIDEO_RGB_SYNC_SCART_IN
- R321 pad 1: /AUDIO_LEFT -> /SCART input 8/AUDIO_LEFT_SCART_IN
- R322 pad 1: /AUDIO_RIGHT -> /SCART input 8/AUDIO_RIGHT_SCART_IN
- R329 pad 1: /GREEN -> /SCART input 9/GREEN_SCART_IN
- R330 pad 1: /RED -> /SCART input 9/RED_SCART_IN
- R333 pad 1: /BLANKING -> /SCART input 9/BLANKING_SCART_IN
- R337 pad 1: /BLUE -> /SCART input 9/BLUE_SCART_IN
- R338 pad 1: /VIDEO_RGB_SYNC -> /SCART input 9/VIDEO_RGB_SYNC_SCART_IN
- R348 pad 1: /AUDIO_LEFT -> /SCART input 9/AUDIO_LEFT_SCART_IN
- R349 pad 1: /AUDIO_RIGHT -> /SCART input 9/AUDIO_RIGHT_SCART_IN
- R356 pad 1: /GREEN -> /SCART input 10/GREEN_SCART_IN
- R357 pad 1: /RED -> /SCART input 10/RED_SCART_IN
- R360 pad 1: /BLANKING -> /SCART input 10/BLANKING_SCART_IN
- R364 pad 1: /BLUE -> /SCART input 10/BLUE_SCART_IN
- R365 pad 1: /VIDEO_RGB_SYNC -> /SCART input 10/VIDEO_RGB_SYNC_SCART_IN
- R375 pad 1: /AUDIO_LEFT -> /SCART input 10/AUDIO_LEFT_SCART_IN
- R376 pad 1: /AUDIO_RIGHT -> /SCART input 10/AUDIO_RIGHT_SCART_IN
- R97 pad 1: /AUDIO_LEFT -> /SCART input 1/AUDIO_LEFT_SCART_IN
- R98 pad 1: /AUDIO_RIGHT -> /SCART input 1/AUDIO_RIGHT_SCART_IN
- U104 pad 4: /BLANKING -> /SCART input 6/BLANKING_SCART_IN
- U111 pad 4: /BLANKING -> /SCART input 7/BLANKING_SCART_IN
- U118 pad 4: /BLANKING -> /SCART input 8/BLANKING_SCART_IN
- U125 pad 4: /BLANKING -> /SCART input 9/BLANKING_SCART_IN
- U132 pad 4: /BLANKING -> /SCART input 10/BLANKING_SCART_IN
- U62 pad 4: /BLANKING -> /SCART input 1/BLANKING_SCART_IN
- U76 pad 4: /BLANKING -> /SCART input 2/BLANKING_SCART_IN
- U83 pad 4: /BLANKING -> /SCART input 3/BLANKING_SCART_IN
- U90 pad 4: /BLANKING -> /SCART input 4/BLANKING_SCART_IN
- U97 pad 4: /BLANKING -> /SCART input 5/BLANKING_SCART_IN

Commit message: Update SCART_switcher.kicad_pcb
Connections:
- net /SCART output/AUDIO_SCART_LEFT renamed /SCART output/AUDIO_SCART_OUT_LEFT
- net /SCART output/AUDIO_SCART_RIGHT renamed /SCART output/AUDIO_SCART_OUT_RIGHT
- net /SCART output/FUNCTION renamed /SCART output/FUNCTION_SCART_OUT
- J4 pad 11: /GREEN -> /SCART output/GREEN_SCART_OUT
- J4 pad 15: /RED -> /SCART output/RED_SCART_OUT
- J4 pad 16: /BLANKING -> /SCART output/BLANKING_SCART_OUT
- J4 pad 20: /VIDEO_RGB_SYNC -> /SCART output/VIDEO_RGB_SYNC_SCART_OUT
- J4 pad 7: /BLUE -> /SCART output/BLUE_SCART_OUT
- R129 pad 1: /BLANKING -> /SCART output/BLANKING_SCART_OUT
- R130 pad 2: /GREEN -> /SCART output/GREEN_SCART_OUT
- R131 pad 2: /RED -> /SCART output/RED_SCART_OUT
- R138 pad 2: /BLUE -> /SCART output/BLUE_SCART_OUT
- R139 pad 2: /VIDEO_RGB_SYNC -> /SCART output/VIDEO_RGB_SYNC_SCART_OUT
Changed lines of the file:
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@@
   (net 171 "/SCART output/AUDIO_RCA_RIGHT")
   (net 172 "unconnected-(J4-P1-Pad1)")
-  (net 173 "/SCART output/AUDIO_SCART_RIGHT")
+  (net 173 "/SCART output/AUDIO_SCART_OUT_RIGHT")
   (net 174 "unconnected-(J4-P3-Pad3)")
-  (net 175 "/SCART output/AUDIO_SCART_LEFT")
-  (net 176 "/SCART output/FUNCTION")
+  (net 175 "/SCART output/AUDIO_SCART_OUT_LEFT")
+  (net 176 "/SCART output/BLUE_SCART_OUT")
   (net 177 "unconnected-(J4-P10-Pad10)")
   (net 178 "unconnected-(J4-P12-Pad12)")
@@
   (net 535 "/SCART input 10/AUDIO_LEFT_SCART_IN")
   (net 536 "/SCART input 10/FUNCTION_SCART_IN")
+  (net 537 "/SCART output/FUNCTION_SCART_OUT")
+  (net 538 "/SCART output/GREEN_SCART_OUT")
+  (net 539 "/SCART output/RED_SCART_OUT")
+  (net 540 "/SCART output/BLANKING_SCART_OUT")
+  (net 541 "/SCART output/VIDEO_RGB_SYNC_SCART_OUT")
   (footprint "Package_TO_SOT_SMD:SOT-23-5" (layer "F.Cu")
     (at 714.5425 -159.84)
@@
       (net 35 "Net-(C101-Pad2)") (pintype "passive"))
     (pad "2" smd roundrect (at 1.4625 0) (size 1.125 2.65) (layers "F.Cu" "F.Paste" "F.Mask") (roundrect_rratio 0.222222)
-      (net 27 "/VIDEO_RGB_SYNC") (pintype "passive"))
+      (net 541 "/SCART output/VIDEO_RGB_SYNC_SCART_OUT") (pintype "passive"))
     (model "${KICAD6_3DMODEL_DIR}/Resistor_SMD.3dshapes/R_1210_3225Metric.wrl"
       (offset (xyz 0 0 0))
@@
       (net 11 "Net-(C42-Pad2)") (pintype "passive"))
     (pad "2" smd roundrect (at 0.9125 0) (size 1.025 1.4) (layers "F.Cu" "F.Paste" "F.Mask") (roundrect_rratio 0.243902)
-      (net 173 "/SCART output/AUDIO_SCART_RIGHT") (pintype "passive"))
+      (net 173 "/SCART output/AUDIO_SCART_OUT_RIGHT") (pintype "passive"))
     (model "${KICAD6_3DMODEL_DIR}/Resistor_SMD.3dshapes/R_0805_2012Metric.wrl"
       (offset (xyz 0 0 0))
@@
       (net 31 "Net-(C94-Pad2)") (pintype "passive"))
     (pad "2" smd roundrect (at 1.4625 0) (size 1.125 2.65) (layers "F.Cu" "F.Paste" "F.Mask") (roundrect_rratio 0.222222)
-      (net 23 "/RED") (pintype "passive"))
+      (net 539 "/SCART output/RED_SCART_OUT") (pintype "passive"))
     (model "${KICAD6_3DMODEL_DIR}/Resistor_SMD.3dshapes/R_1210_3225Metric.wrl"
       (offset (xyz 0 0 0))
@@
       (net 29 "Net-(C92-Pad2)") (pintype "passive"))
     (pad "2" smd roundrect (at 1.4625 0) (size 1.125 2.65) (layers "F.Cu" "F.Paste" "F.Mask") (roundrect_rratio 0.222222)
-      (net 21 "/GREEN") (pintype "passive"))
+      (net 538 "/SCART output/GREEN_SCART_OUT") (pintype "passive"))
     (model "${KICAD6_3DMODEL_DIR}/Resistor_SMD.3dshapes/R_1210_3225Metric.wrl"
       (offset (xyz 0 0 0))
@@
       (net 250 "Net-(Q4-C)") (pintype "passive"))
     (pad "2" smd roundrect (at 0.9125 0) (size 1.025 1.4) (layers "F.Cu" "F.Paste" "F.Mask") (roundrect_rratio 0.243902)
-      (net 176 "/SCART output/FUNCTION") (pintype "passive"))
+      (net 537 "/SCART output/FUNCTION_SCART_OUT") (pintype "passive"))
     (model "${KICAD6_3DMODEL_DIR}/Resistor_SMD.3dshapes/R_0805_2012Metric.wrl"
       (offset (xyz 0 0 0))
@@
       (stroke (width 0.1) (type solid)) (layer "F.Fab"))
     (pad "1" smd roundrect (at -0.9125 0) (size 1.025 1.4) (layers "F.Cu" "F.Paste" "F.Mask") (roundrect_rratio 0.243902)
-      (net 108 "/BLANKING") (pintype "passive"))
+      (net 540 "/SCART output/BLANKING_SCART_OUT") (pintype "passive"))
     (pad "2" smd roundrect (at 0.9125 0) (size 1.025 1.4) (layers "F.Cu" "F.Paste" "F.Mask") (roundrect_rratio 0.243902)
       (net 286 "Net-(Q28-C)") (pintype "passive"))
@@
       (net 33 "Net-(C100-Pad1)") (pintype "passive"))
     (pad "2" smd roundrect (at 1.4625 0) (size 1.125 2.65) (layers "F.Cu" "F.Paste" "F.Mask") (roundrect_rratio 0.222222)
-      (net 25 "/BLUE") (pintype "passive"))
+      (net 176 "/SCART output/BLUE_SCART_OUT") (pintype "passive"))
     (model "${KICAD6_3DMODEL_DIR}/Resistor_SMD.3dshapes/R_1210_3225Metric.wrl"
       (offset (xyz 0 0 0))
@@
       (net 172 "unconnected-(J4-P1-Pad1)") (pinfunction "P1") (pintype "passive+no_connect"))
     (pad "2" thru_hole oval (at -17.145 2.55 180) (size 2 3) (drill 1.3 (offset 0 0.5)) (layers "*.Cu" "*.Mask")
-      (net 173 "/SCART output/AUDIO_SCART_RIGHT") (pinfunction "P2") (pintype "passive"))
+      (net 173 "/SCART output/AUDIO_SCART_OUT_RIGHT") (pinfunction "P2") (pintype "passive"))
     (pad "3" thru_hole oval (at -15.24 -2.55 180) (size 2 3) (drill 1.3 (offset 0 -0.5)) (layers "*.Cu" "*.Mask")
       (net 174 "unconnected-(J4-P3-Pad3)") (pinfunction "P3") (pintype "passive+no_connect"))
@@
       (net 2 "GND") (pinfunction "P5") (pintype "passive"))
     (pad "6" thru_hole oval (at -9.525 2.55 180) (size 2 3) (drill 1.3 (offset 0 0.5)) (layers "*.Cu" "*.Mask")
-      (net 175 "/SCART output/AUDIO_SCART_LEFT") (pinfunction "P6") (pintype "passive"))
+      (net 175 "/SCART output/AUDIO_SCART_OUT_LEFT") (pinfunction "P6") (pintype "passive"))
     (pad "7" thru_hole oval (at -7.62 -2.55 180) (size 2 3) (drill 1.3 (offset 0 -0.5)) (layers "*.Cu" "*.Mask")
-      (net 25 "/BLUE") (pinfunction "P7") (pintype "passive"))
+      (net 176 "/SCART output/BLUE_SCART_OUT") (pinfunction "P7") (pintype "passive"))
     (pad "8" thru_hole oval (at -5.715 2.55 180) (size 2 3) (drill 1.3 (offset 0 0.5)) (layers "*.Cu" "*.Mask")
-      (net 176 "/SCART output/FUNCTION") (pinfunction "P8") (pintype "passive"))
+      (net 537 "/SCART output/FUNCTION_SCART_OUT") (pinfunction "P8") (pintype "passive"))
     (pad "9" thru_hole oval (at -3.81 -2.55 180) (size 2 3) (drill 1.3 (offset 0 -0.5)) (layers "*.Cu" "*.Mask")
       (net 2 "GND") (pinfunction "P9") (pintype "passive"))
@@
       (net 177 "unconnected-(J4-P10-Pad10)") (pinfunction "P10") (pintype "passive+no_connect"))
     (pad "11" thru_hole oval (at 0 -2.55 180) (size 2 3) (drill 1.3 (offset 0 -0.5)) (layers "*.Cu" "*.Mask")
-      (net 21 "/GREEN") (pinfunction "P11") (pintype "passive"))
+      (net 538 "/SCART output/GREEN_SCART_OUT") (pinfunction "P11") (pintype "passive"))
     (pad "12" thru_hole oval (at 1.905 2.55 180) (size 2 3) (drill 1.3 (offset 0 0.5)) (layers "*.Cu" "*.Mask")
       (net 178 "unconnected-(J4-P12-Pad12)") (pinfunction "P12") (pintype "passive+no_connect"))
@@
       (net 2 "GND") (pinfunction "P14") (pintype "passive"))
     (pad "15" thru_hole oval (at 7.62 -2.55 180) (size 2 3) (drill 1.3 (offset 0 -0.5)) (layers "*.Cu" "*.Mask")
-      (net 23 "/RED") (pinfunction "P15") (pintype "passive"))
+      (net 539 "/SCART output/RED_SCART_OUT") (pinfunction "P15") (pintype "passive"))
     (pad "16" thru_hole oval (at 9.525 2.55 180) (size 2 3) (drill 1.3 (offset 0 0.5)) (layers "*.Cu" "*.Mask")
-      (net 108 "/BLANKING") (pinfunction "P16") (pintype "passive"))
+      (net 540 "/SCART output/BLANKING_SCART_OUT") (pinfunction "P16") (pintype "passive"))
     (pad "17" thru_hole oval (at 11.43 -2.55 180) (size 2 3) (drill 1.3 (offset 0 -0.5)) (layers "*.Cu" "*.Mask")
       (net 179 "unconnected-(J4-P17-Pad17)") (pinfunction "P17") (pintype "passive+no_connect"))
@@
       (net 180 "unconnected-(J4-P19-Pad19)") (pinfunction "P19") (pintype "passive+no_connect"))
     (pad "20" thru_hole oval (at 17.145 2.55 180) (size 2 3) (drill 1.3 (offset 0 0.5)) (layers "*.Cu" "*.Mask")
-      (net 27 "/VIDEO_RGB_SYNC") (pinfunction "P20") (pintype "passive"))
+      (net 541 "/SCART output/VIDEO_RGB_SYNC_SCART_OUT") (pinfunction "P20") (pintype "passive"))
     (pad "21" thru_hole oval (at 19.05 -2.55 180) (size 2 3) (drill 1.3 (offset 0 -0.5)) (layers "*.Cu" "*.Mask")
       (net 2 "GND") (pinfunction "P21") (pintype "passive"))
@@
       (net 9 "Net-(C41-Pad2)") (pintype "passive"))
     (pad "2" smd roundrect (at 0.9125 0) (size 1.025 1.4) (layers "F.Cu" "F.Paste" "F.Mask") (roundrect_rratio 0.243902)
-      (net 175 "/SCART output/AUDIO_SCART_LEFT") (pintype "passive"))
+      (net 175 "/SCART output/AUDIO_SCART_OUT_LEFT") (pintype "passive"))
     (model "${KICAD6_3DMODEL_DIR}/Resistor_SMD.3dshapes/R_0805_2012Metric.wrl"
       (offset (xyz 0 0 0))
