File: ECAD/SCART_switcher/SCART_switcher.kicad_pcb (KiCad board)
At the start: 4 copper layers, 262 x 124.5 mm, 82 parts, among them J1 SCART-F, Q1 BC847, Q2 BC847, Q24 BC847, Q25 BC847, Q26 2SK209, Q27 2SK209, U137 74LVC1G14, U2 74LVC1G08, U34 74LVC1G08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

Commit message: Progressed ECAD.
Parts:
- moved C2 0.25 mm to (23.5, 52.8)
- moved C45 0.25 mm to (38.5, 55.0)
- moved D7 0.25 mm to (30.3, 68.8)
- moved D71 0.25 mm to (30.5, 150.5)
- moved J1 0.25 mm to (28.9, 111.4)
- moved Q2 0.25 mm to (23.3, 68.2)
- moved Q24 0.25 mm to (24.6, 150.4)
- moved Q25 0.25 mm to (34.6, 152.0)
- moved R112 0.25 mm to (37.5, 59.0)
- moved R3 0.25 mm to (20.0, 56.0)
- moved R4 0.25 mm to (38.5, 68.0)
- moved R5 0.25 mm to (35.0, 68.8)
- moved R68 0.25 mm to (15.5, 78.0)
- moved R73 0.25 mm to (15.5, 147.8)
- moved R92 0.25 mm to (21.5, 150.5)
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Routing:
- net GND: track 90.0 -> 98.4 mm, vias 45 -> 44
- net /SCART input 1/IN_ENABLE: track 64.1 -> 69.9 mm
- net +2V5: track 58.6 -> 61.2 mm
- net /SCART input 1/IN_ACTIVE: track 34.1 -> 32.1 mm
- net Net-(R92-Pad1): track 125.9 -> 127.4 mm
- net +5V: track 104.8 -> 105.6 mm
Other:
- board size 262 x 124.5 mm -> 262 x 125 mm

Commit message: Update SCART_switcher.kicad_pcb
Routing:
- net GND: track 98.4 -> 96.4 mm
- net +4V5: track 10.5 -> 12.1 mm
- net /SCART input 1/Audio input stage/AUDIO_OUT_ENABLE: track 18.7 -> 19.3 mm
- net Net-(Q1-C): track 70.5 -> 71.0 mm
