File: ECAD/SCART_switcher_input/SCART_input.kicad_sch (KiCad schematic)
At the start: 12 parts, among them Q1 BC847, Q2 BC847, U1 74LVC1G14

Commit message: Progressed ECAD.
Parts:
- removed C1: 100nC, Capacitor_SMD:C_0805_2012Metric, symbol Device:C
- removed U1: 74LVC1G14, Package_TO_SOT_SMD:SOT-353_SC-70-5, symbol 74xGxx:74AHCT1G14
- renumbered Q2 to Q1, Q1 to Q2, R4 to R3, R5 to R4, R3 to R5
Connections:
- net IN_ACTIVE: now also Q2.3 (C), R5.2
Other:
- moved on the sheet: D1, Q2, R2, R5, R?

Commit message: progressed ecad.
Connections:
- net IN_ACTIVE renamed ~{IN_ACTIVE}
Other:
- sheet Priority Level ports: added ~{IN_ACTIVE}; removed IN_ACTIVE
Changed lines of the file:
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@@
     (effects (font (size 1.27 1.27)) (justify left bottom))
   )
-  (label "IN_ACTIVE" (at 252.73 43.18 180) (fields_autoplaced)
+  (label "~{IN_ACTIVE}" (at 252.73 43.18 180) (fields_autoplaced)
     (effects (font (size 1.27 1.27)) (justify right bottom))
   )
-  (label "IN_ACTIVE" (at 203.2 88.9 0) (fields_autoplaced)
+  (label "~{IN_ACTIVE}" (at 203.2 88.9 0) (fields_autoplaced)
     (effects (font (size 1.27 1.27)) (justify left bottom))
   )
@@
       (effects (font (size 1.27 1.27)) (justify right))
     )
-    (pin "IN_ACTIVE" input (at 213.36 88.9 180)
-      (effects (font (size 1.27 1.27)) (justify left))
-    )
+    (pin "~{IN_ACTIVE}" input (at 213.36 88.9 180)
+      (effects (font (size 1.27 1.27)) (justify left))
+    )

Commit message: progressed ecad
Parts:
- gave numbers to parts that had none: 2
Changed lines of the file:
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@@
       )
       (project "SCART_switcher_input"
-        (path "/8cd08eb5-4755-4ef5-8eeb-77fd9974b180/19b1c794-1d68-480b-a4cd-c99f5e9ef1e6"
-          (reference "D?") (unit 1)
-        )
         (path "/8cd08eb5-4755-4ef5-8eeb-77fd9974b180/6e53f4c9-ed59-4c5d-ac8d-a66f0d353ca7"
           (reference "D2") (unit 1)
@@
   (symbol (lib_id "Connector:SCART-F") (at 90.17 71.12 0) (unit 1)
     (in_bom yes) (on_board yes) (dnp no) (fields_autoplaced)
-    (property "Reference" "J?" (at 90.17 33.02 0)
+    (property "Reference" "J16" (at 90.17 33.02 0)
       (effects (font (size 1.27 1.27)))
     )
@@
     (instances
       (project "SCART_switcher_input"
-        (path "/8cd08eb5-4755-4ef5-8eeb-77fd9974b180"
-          (reference "J?") (unit 1)
-        )
         (path "/8cd08eb5-4755-4ef5-8eeb-77fd9974b180/6e53f4c9-ed59-4c5d-ac8d-a66f0d353ca7"
           (reference "J16") (unit 1)
@@
   (symbol (lib_id "power:+12V") (at 229.87 120.65 0) (unit 1)
     (in_bom yes) (on_board yes) (dnp no) (fields_autoplaced)
-    (property "Reference" "#PWR?" (at 229.87 124.46 0)
+    (property "Reference" "#PWR025" (at 229.87 124.46 0)
       (effects (font (size 1.27 1.27)) hide)
     )
@@
     (instances
       (project "SCART_switcher_input"
-        (path "/8cd08eb5-4755-4ef5-8eeb-77fd9974b180/19b1c794-1d68-480b-a4cd-c99f5e9ef1e6"
-          (reference "#PWR?") (unit 1)
-        )
         (path "/8cd08eb5-4755-4ef5-8eeb-77fd9974b180/6e53f4c9-ed59-4c5d-ac8d-a66f0d353ca7"
           (reference "#PWR025") (unit 1)
@@
         (path "/8cd08eb5-4755-4ef5-8eeb-77fd9974b180/272a4677-3ef2-418e-abc5-b29f59e726f9"
           (reference "#PWR051") (unit 1)
-        )
-        (path "/8cd08eb5-4755-4ef5-8eeb-77fd9974b180/6e53f4c9-ed59-4c5d-ac8d-a66f0d353ca7/0117abb0-e8aa-4002-a68c-61b92aed6fa0"
-          (reference "#PWR?") (unit 1)
-        )
-        (path "/8cd08eb5-4755-4ef5-8eeb-77fd9974b180/8ea6db35-25d0-43bc-9de5-3ca23502dcdc/0117abb0-e8aa-4002-a68c-61b92aed6fa0"
-          (reference "#PWR?") (unit 1)
-        )
-        (path "/8cd08eb5-4755-4ef5-8eeb-77fd9974b180/272a4677-3ef2-418e-abc5-b29f59e726f9/0117abb0-e8aa-4002-a68c-61b92aed6fa0"
-          (reference "#PWR?") (unit 1)
         )
       )
@@
           (reference "R12") (unit 1)
         )
-        (path "/8cd08eb5-4755-4ef5-8eeb-77fd9974b180/6e53f4c9-ed59-4c5d-ac8d-a66f0d353ca7/8a52048d-21a1-4895-a4b6-c190738f75a0"
-          (reference "R?") (unit 1)
-        )
-        (path "/8cd08eb5-4755-4ef5-8eeb-77fd9974b180/8ea6db35-25d0-43bc-9de5-3ca23502dcdc/8a52048d-21a1-4895-a4b6-c190738f75a0"
-          (reference "R?") (unit 1)
-        )
-        (path "/8cd08eb5-4755-4ef5-8eeb-77fd9974b180/272a4677-3ef2-418e-abc5-b29f59e726f9/8a52048d-21a1-4895-a4b6-c190738f75a0"
-          (reference "R?") (unit 1)
-        )
       )
     )
@@
   (symbol (lib_id "Device:R") (at 215.9 36.83 0) (unit 1)
     (in_bom yes) (on_board yes) (dnp no) (fields_autoplaced)
-    (property "Reference" "R?" (at 218.44 35.56 0)
+    (property "Reference" "R1" (at 218.44 35.56 0)
       (effects (font (size 1.27 1.27)) (justify left))
     )
@@
     (instances
       (project "SCART_switcher_input"
-        (path "/8cd08eb5-4755-4ef5-8eeb-77fd9974b180/6e53f4c9-ed59-4c5d-ac8d-a66f0d353ca7/8a52048d-21a1-4895-a4b6-c190738f75a0"
-          (reference "R?") (unit 1)
-        )
-        (path "/8cd08eb5-4755-4ef5-8eeb-77fd9974b180/8ea6db35-25d0-43bc-9de5-3ca23502dcdc/8a52048d-21a1-4895-a4b6-c190738f75a0"
-          (reference "R?") (unit 1)
-        )
-        (path "/8cd08eb5-4755-4ef5-8eeb-77fd9974b180/272a4677-3ef2-418e-abc5-b29f59e726f9/8a52048d-21a1-4895-a4b6-c190738f75a0"
-          (reference "R?") (unit 1)
-        )
         (path "/8cd08eb5-4755-4ef5-8eeb-77fd9974b180/6e53f4c9-ed59-4c5d-ac8d-a66f0d353ca7"
           (reference "R1") (unit 1)

Commit message: progressed ecad
Parts:
- renumbered J16 to J3
