File: ECAD/SCART_switcher_input/SCART_switcher_input.kicad_sch (KiCad schematic)
At the start: 19 parts, among them J1 Conn_01x02, J10 Conn_Coaxial, J11 Conn_Coaxial, J12 Conn_Coaxial, J13 Conn_Coaxial, J14 Conn_Coaxial, J15 Conn_01x02, J2 Conn_01x02, J3 Conn_01x03, J4 Conn_Coaxial, J5 Conn_Coaxial, J6 Conn_Coaxial, J7 Conn_Coaxial, J8 Conn_Coaxial, J9 Conn_01x03

Commit message: progressed ecad
Parts:
- removed J1, J15, J2: Conn_01x02, Connector_JST:JST_PH_S2B-PH-K_1x02_P2.00mm_Horizontal, symbol Connector_Generic:Conn_01x02
- removed J10, J11, J12, J13, J14, J4, J5, J6, J7, J8: Conn_Coaxial, Connector_Coaxial:U.FL_Hirose_U.FL-R-SMT-1_Vertical, symbol Connector:Conn_Coaxial
- removed J3, J9: Conn_01x03, Connector_JST:JST_PH_S3B-PH-K_1x03_P2.00mm_Horizontal, symbol Connector_Generic:Conn_01x03
- added J1: Bus in, Connector_FFC-FPC:Hirose_FH12-24S-0.5SH_1x24-1MP_P0.50mm_Horizontal, symbol Connector_Generic:Conn_01x24
- added J2: Bus out, Connector_FFC-FPC:Hirose_FH12-24S-0.5SH_1x24-1MP_P0.50mm_Horizontal, symbol Connector_Generic:Conn_01x24
Connections:
- net +12V: now also J1.1 (Pin_1), J1.2 (Pin_2), J2.23 (Pin_23), J2.24 (Pin_24)
- net AUDIO_LEFT: now also J1.6 (Pin_6), J2.19 (Pin_19)
- net AUDIO_RIGHT: now also J1.8 (Pin_8), J2.17 (Pin_17)
- net BLANKING: now also J1.23 (Pin_23), J2.2 (Pin_2)
- net BLUE: now also J1.14 (Pin_14), J2.11 (Pin_11)
- net GND: now also J1.10 (Pin_10), J1.12 (Pin_12), J1.13 (Pin_13), J1.15 (Pin_15), J1.16 (Pin_16), J1.18 (Pin_18), J1.19 (Pin_19), J1.21 (Pin_21), J1.22 (Pin_22), J1.24 (Pin_24), J1.3 (Pin_3), J1.5 (Pin_5), J1.7 (Pin_7), J1.9 (Pin_9), J2.1 (Pin_1), J2.10 (Pin_10), J2.12 (Pin_12), J2.13 (Pin_13), J2.15 (Pin_15), J2.16 (Pin_16), J2.18 (Pin_18), J2.20 (Pin_20), J2.22 (Pin_22), J2.3 (Pin_3), J2.4 (Pin_4), J2.6 (Pin_6), J2.7 (Pin_7), J2.9 (Pin_9)
- net GREEN: now also J1.17 (Pin_17), J2.8 (Pin_8)
- net RED: now also J1.11 (Pin_11), J2.14 (Pin_14)
- net SCART input 1/CARRY_IN: now also J1.4 (Pin_4)
- net SCART input 3/CARRY_OUT: now also J2.21 (Pin_21)
- net VIDEO_RGB_SYNC: now also J1.20 (Pin_20), J2.5 (Pin_5)
