File: ECAD/SCART_switcher_input/audio_in.kicad_sch (KiCad schematic)
At the start: 28 parts, among them Q8 BC857

Commit message: Progressed ECAD.
Parts:
- C?: footprint Capacitor_SMD:C_0805_2012Metric -> Capacitor_SMD:C_0603_1608Metric; MPN CL21B104KBCNNNC -> (none)
- renumbered C21 to C15, C22 to C16, D8 to D7, Q8 to Q23, R25 to R48, R26 to R49, R27 to R50, R28 to R51, R29 to R52

Commit message: Progressed ECAD.
Parts:
- removed R48, R50: 47kR, Resistor_SMD:R_0805_2012Metric, symbol Device:R
- removed R49, R52: 10kR, Resistor_SMD:R_0805_2012Metric, symbol Device:R
- added R42, R43: 10kR, Resistor_SMD:R_0805_2012Metric, symbol Device:R
- added R? (x2): 4k7R, Resistor_SMD:R_0805_2012Metric, symbol Device:R
- renumbered Q23 to Q20, R51 to R45
Connections:
- net +9V: now also R?.1
- net AUDIO_OUT_ENABLE: now also R?.1
- net ENABLE: now also R42.1
- net GND: now also R?.2
- net at D7.3 (K), Q?.3 (C): now also R43.1, R?.2
- net at Q20.1 (B): now also R43.2
- net at Q?.1 (B): now also R42.2

Commit message: progressed ecad.
Parts:
- renumbered Q20 to Q29, R42 to R60, R43 to R62, R45 to R63

Commit message: progressed ecad
Parts:
- removed Q29: BC857, Package_TO_SOT_SMD:SOT-23, symbol Transistor_BJT:BC857
- removed R?: 4k7R, Resistor_SMD:R_0805_2012Metric, symbol Device:R
- added Q29: BC847, Package_TO_SOT_SMD:SOT-23, symbol Transistor_BJT:BC847
- added R64: 4k7R, Resistor_SMD:R_0805_2012Metric, symbol Device:R
- gave numbers to parts that had none: 16
Connections:
- net +9V: now also R64.1
- net AUDIO_OUT_ENABLE: now also Q29.3 (C), R64.2
- net GND: now also Q29.2 (E)
- net at R62.2: now also Q29.1 (B)
Other:
- moved on the sheet: R62

Commit message: Progressed ECAD.
Changed lines of the file:
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@@
-    )
-  )
-  (symbol (lib_id "Transistor_FET:MMBFJ111") (at 194.31 106.68 0) (unit 1)
-    (in_bom yes) (on_board yes) (dnp no)
-    (property "Reference" "Q31" (at 186.69 109.22 0)
-      (effects (font (size 1.27 1.27)) (justify left))
-    )
-    (property "Value" "2SK209" (at 184.15 111.76 0)
-      (effects (font (size 1.27 1.27)) (justify left))
-    )
-    (property "Footprint" "Package_TO_SOT_SMD:SC-59" (at 199.39 108.585 0)
-      (effects (font (size 1.27 1.27) italic) (justify left) hide)
-    )
-    (property "Datasheet" "https://datasheet.lcsc.com/lcsc/1810271708_TOSHIBA-2SK209-GR-TE85L-F_C61792.pdf" (at 194.31 106.68 0)
-      (effects (font (size 1.27 1.27)) (justify left) hide)
-    )
-    (property "MPN" "2SK209-GR(TE85L,F)" (at 194.31 106.68 0)
-      (effects (font (size 1.27 1.27)) hide)
-    )
-    (property "Status" "OK" (at 194.31 106.68 0)
-      (effects (font (size 1.27 1.27)) hide)
-    )
-    (pin "1")
-    (pin "2")
-    (pin "3")
-    (instances
-      (project "SCART_switcher_input"
-        (path "/8cd08eb5-4755-4ef5-8eeb-77fd9974b180/6e53f4c9-ed59-4c5d-ac8d-a66f0d353ca7/8a52048d-21a1-4895-a4b6-c190738f75a0"
-          (reference "Q31") (unit 1)
-        )
-        (path "/8cd08eb5-4755-4ef5-8eeb-77fd9974b180/8ea6db35-25d0-43bc-9de5-3ca23502dcdc/8a52048d-21a1-4895-a4b6-c190738f75a0"
-          (reference "Q39") (unit 1)
-        )
-        (path "/8cd08eb5-4755-4ef5-8eeb-77fd9974b180/272a4677-3ef2-418e-abc5-b29f59e726f9/8a52048d-21a1-4895-a4b6-c190738f75a0"
-          (reference "Q45") (unit 1)
-        )
-      )
     )
   )
@@
         (path "/8cd08eb5-4755-4ef5-8eeb-77fd9974b180/272a4677-3ef2-418e-abc5-b29f59e726f9/8a52048d-21a1-4895-a4b6-c190738f75a0"
           (reference "#PWR0291") (unit 1)
+        )
+      )
+    )
+  )
+  (symbol (lib_name "MMBFJ111_1") (lib_id "Transistor_FET:MMBFJ111") (at 194.31 106.68 0) (unit 1)
+    (in_bom yes) (on_board yes) (dnp no) (fields_autoplaced)
+    (property "Reference" "Q31" (at 199.39 105.41 0)
+      (effects (font (size 1.27 1.27)) (justify left))
+    )
+    (property "Value" "2SK209" (at 199.39 107.95 0)
+      (effects (font (size 1.27 1.27)) (justify left))
+    )
+    (property "Footprint" "Package_TO_SOT_SMD:SC-59" (at 199.39 108.585 0)
+      (effects (font (size 1.27 1.27) italic) (justify left) hide)
+    )
+    (property "Datasheet" "https://datasheet.lcsc.com/lcsc/1810271708_TOSHIBA-2SK209-GR-TE85L-F_C61792.pdf" (at 199.39 110.49 0)
+      (effects (font (size 1.27 1.27)) (justify left) hide)
+    )
+    (property "MPN" "2SK209-GR(TE85L,F)" (at 194.31 106.68 0)
+      (effects (font (size 1.27 1.27)) hide)
+    )
+    (property "Status" "OK" (at 194.31 106.68 0)
+      (effects (font (size 1.27 1.27)) hide)
+    )
+    (pin "2")
+    (pin "3")
+    (pin "1")
+    (instances
+      (project "SCART_switcher_input"
+        (path "/8cd08eb5-4755-4ef5-8eeb-77fd9974b180/6e53f4c9-ed59-4c5d-ac8d-a66f0d353ca7/8a52048d-21a1-4895-a4b6-c190738f75a0"
+          (reference "Q31") (unit 1)
+        )
+        (path "/8cd08eb5-4755-4ef5-8eeb-77fd9974b180/8ea6db35-25d0-43bc-9de5-3ca23502dcdc/8a52048d-21a1-4895-a4b6-c190738f75a0"
+          (reference "Q39") (unit 1)
+        )
+        (path "/8cd08eb5-4755-4ef5-8eeb-77fd9974b180/272a4677-3ef2-418e-abc5-b29f59e726f9/8a52048d-21a1-4895-a4b6-c190738f75a0"
+          (reference "Q45") (unit 1)
         )
       )
@@
     )
   )
-  (symbol (lib_id "Transistor_FET:MMBFJ111") (at 194.31 60.96 0) (unit 1)
-    (in_bom yes) (on_board yes) (dnp no)
-    (property "Reference" "Q30" (at 186.69 63.5 0)
-      (effects (font (size 1.27 1.27)) (justify left))
-    )
-    (property "Value" "2SK209" (at 184.15 66.04 0)
+  (symbol (lib_name "MMBFJ111_1") (lib_id "Transistor_FET:MMBFJ111") (at 194.31 60.96 0) (unit 1)
+    (in_bom yes) (on_board yes) (dnp no) (fields_autoplaced)
+    (property "Reference" "Q30" (at 199.39 59.69 0)
+      (effects (font (size 1.27 1.27)) (justify left))
+    )
+    (property "Value" "2SK209" (at 199.39 62.23 0)
       (effects (font (size 1.27 1.27)) (justify left))
     )
@@
       (effects (font (size 1.27 1.27) italic) (justify left) hide)
     )
-    (property "Datasheet" "https://datasheet.lcsc.com/lcsc/1810271708_TOSHIBA-2SK209-GR-TE85L-F_C61792.pdf" (at 194.31 60.96 0)
+    (property "Datasheet" "https://datasheet.lcsc.com/lcsc/1810271708_TOSHIBA-2SK209-GR-TE85L-F_C61792.pdf" (at 199.39 64.77 0)
       (effects (font (size 1.27 1.27)) (justify left) hide)
     )
@@
       (effects (font (size 1.27 1.27)) hide)
     )
-    (pin "1")
     (pin "2")
     (pin "3")
-    (instances
-      (project "SCART_switcher_input"
+    (pin "1")
+    (instances
+      (project "SCART_switcher_input"
