File: ECAD/SCART_switcher_input/power.kicad_sch (KiCad schematic)
At the start: 26 parts, among them U13 L7805, U14 L7809, U15 RC4580, U16 RC4580

Commit message: Progressed ECAD.
Parts:
- removed D?: LED, LED_THT:LED_D5.0mm, symbol Device:LED
- removed R?: 1kR, Resistor_SMD:R_1210_3225Metric, symbol Device:R
- C? (x6): footprint Capacitor_SMD:C_0805_2012Metric -> Capacitor_SMD:C_0603_1608Metric; MPN CL21B104KBCNNNC -> (none)
- renumbered C16 to C10, C15 to C9, U13 to U1, U14 to U2, U15 to U3, U16 to U4
Other:
- note removed: "0.3W min"
- note removed: "Power indicator"

Commit message: progressed ecad
Parts:
- gave numbers to parts that had none: 14
