File: ECAD/SCART_switcher_input/video_in.kicad_sch (KiCad schematic)
At the start: 32 parts, among them U18 74LVC1G3157, U19 74LVC1G3157, U22 74LVC1G3157, U23 74LVC1G3157

Commit message: Progressed ECAD.
Parts:
- added C?: 100nC, Capacitor_SMD:C_0603_1608Metric, symbol Device:C
- added U?: 74LVC1G14, Package_TO_SOT_SMD:SOT-353_SC-70-5, symbol 74xGxx:74AHCT1G14
- C? (x6): footprint Capacitor_SMD:C_0805_2012Metric -> Capacitor_SMD:C_0603_1608Metric; MPN CL21B104KBCNNNC -> (none)
- renumbered U22 to U11, U23 to U12, U18 to U7, U19 to U8
Connections:
- net +5V: now also C?.1, U?.5 (VCC)
- net ENABLE: now also U?.2, U?.4
- net GND: now also C?.2, U?.3 (GND)

Commit message: Progressed ECAD.
Parts:
- removed C? (x2): 100nC, Capacitor_SMD:C_0603_1608Metric, symbol Device:C
- removed R?: 10kR, Resistor_SMD:R_0805_2012Metric, symbol Device:R
- removed U?: 74LVC1G126, Package_TO_SOT_SMD:SOT-353_SC-70-5, symbol 74xGxx:74AHC1G126
- removed U?: 74LVC1G14, Package_TO_SOT_SMD:SOT-353_SC-70-5, symbol 74xGxx:74AHCT1G14
- added C?: 100nC, Capacitor_SMD:C_0603_1608Metric, symbol Device:C
- added R?: 4k7R, Resistor_SMD:R_0805_2012Metric, symbol Device:R
- added U9: 74LVC1G3157, Package_TO_SOT_SMD:SOT-363_SC-70-6, symbol Analog_Switch:TS5A63157DBV
- renumbered U11 to U10, U12 to U11
Connections:
- net +2V5: now also U9.3
- net +5V: now also C?.1, R?.1, U9.5 (V+)
- net BLANKING_OUT: now also U9.1
- net ENABLE: now also U9.6
- net GND: now also C?.2, U9.2 (GND)
- net at Q?.3 (C): now also R?.2, U9.4
Other:
- note added: "(*3)"
- note added: "(*3) As per standard EN 50049-1, the input's DC component is within 0 V and +2 V. Considering that the input is AC coupled to a DC level of +2.5 V, the usage of a polarized input capacitor is safe."

Commit message: progressed ecad
Parts:
- removed U?: 74LVC1G14, Package_TO_SOT_SMD:SOT-353_SC-70-5, symbol 74xGxx:74AHCT1G14
- added U26: 74LVC1G17, Package_TO_SOT_SMD:SOT-353_SC-70-5, symbol 74xGxx:74LVC1G17
- gave numbers to parts that had none: 26
Connections:
- net +5V: now also U26.5 (VCC)
- net ENABLE: now also U26.2, U26.4
- net GND: now also U26.3 (GND)

Commit message: Progressed ECAD.
Parts:
- removed U26: 74LVC1G17, Package_TO_SOT_SMD:SOT-353_SC-70-5, symbol 74xGxx:74LVC1G17
- added Q32: BC847, Package_TO_SOT_SMD:SOT-23, symbol Transistor_BJT:BC847
- added R75: 10kR, Resistor_SMD:R_0805_2012Metric, symbol Device:R
- added R78: 4k7R, Resistor_SMD:R_0805_2012Metric, symbol Device:R
- added U8: 74LVC1G14, Package_TO_SOT_SMD:SOT-353_SC-70-5, symbol 74xGxx:74AHC1G14
- renumbered Q32 to Q33, R75 to R76, R76 to R77, R77 to R79, R78 to R80, R79 to R81, R80 to R82, R81 to R83, R82 to R84, R83 to R85, R84 to R86, R85 to R87, R86 to R88, R87 to R89, U7 to U6, U8 to U7
Connections:
- net +5V: now also R78.1, U8.5 (VCC)
- net ENABLE: now also R75.2, U8.4
- net GND: now also Q32.2 (E), U8.3 (GND)
- new net: Q32.1 (B), R75.1
- new net: Q32.3 (C), R78.2, U8.2
Other:
- moved on the sheet: C20, C23, Q33, R81, R82, R83, U9A, U9B
