File: ECAD/Power_supply/Power_supply.kicad_sch (KiCad schematic)
At the start: 36 parts, among them J1 Conn_01x06, J2 Barrel_Jack_Switch, Q1 DMP3037LSS-13, SW1 SW_Push_DPDT, U1 LM317_TO-220, U2 LM317_TO-220

Commit message: Update Power_supply.kicad_sch
Parts:
- added C13: 1000uC, Capacitor_SMD:CP_Elec_10x10.5, symbol Device:C_Polarized
- added C14: 100uC, Capacitor_SMD:CP_Elec_6.3x5.4, symbol Device:C_Polarized
- added C15: 10uC, Capacitor_SMD:CP_Elec_6.3x5.4, symbol Device:C_Polarized
- added C16: 1uC, Capacitor_SMD:C_0805_2012Metric, symbol Device:C
- added C17: 100nC, Capacitor_SMD:C_0805_2012Metric, symbol Device:C
- added C18: 10nC, Capacitor_SMD:C_0805_2012Metric, symbol Device:C
- added C19: 1nC, Capacitor_SMD:C_0805_2012Metric, symbol Device:C
- added L1, L2: 100uL, symbol Device:L_Ferrite
- added L3, L4: 10uL, symbol Device:L_Ferrite
- added R7: 100kR, Resistor_SMD:R_0805_2012Metric, symbol Device:R
- renumbered D4 to D3, D5 to D4, D6 to D5, D7 to D6, D3 to D7, J2 to J1, J1 to J2, R3 to R2, R4 to R3, R5 to R4, R6 to R5, R2 to R6
Connections:
- net +12V: now also C13.1, C14.1, C15.1, C16.1, C17.1, C18.1, C19.1, L3.2, R7.1; no longer FL3.3
- net GND: now also C13.2, C14.2, C15.2, C16.2, C17.2, C18.2, C19.2, L4.2, R7.2; no longer FL2.4, FL3.2
- net +12P: no longer names the net of D2.3 (K), FL1.1, Q1.1 (S), Q1.2 (S), Q1.3 (S)
- new net: L1.2, L3.1
- new net: FL2.4, FL3.2, L2.1
- new net: FL3.3, L1.1
- new net: L2.2, L4.1
Other:
- note added: "Power output connector"
- note removed: "Power output"
- moved on the sheet: C1, C10, C11, C12, C2, C3, C4, C5, C6, C7, C8, C9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

Commit message: Progressed ECAD.
Parts:
- removed C1, C2: 10uC, Capacitor_SMD:CP_Elec_6.3x5.4, symbol Device:C_Polarized
- FL2: value Filter_EMI_LL_1423 -> SRF0905-202Y; footprint (none) -> Filter:Filter_Bourns_SRF0905_6.0x9.2mm; MPN (none) -> SRF0905-202Y
Other:
- note added: "Power ON indicator"
- note removed: "Power indicator"
- moved on the sheet: C10, C11, C12, C13, C14, C15, C16, C17, C18, C19, C3, C4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

Commit message: Progressed ECAD.
Other:
- note added: "0.6mA rated"
- moved on the sheet: C7, C8
Changed lines of the file:
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@@
   (junction (at 182.88 58.42) (diameter 0) (color 0 0 0 0)
   )
+  (junction (at 106.68 118.11) (diameter 0) (color 0 0 0 0)
+  )
   (junction (at 102.87 53.34) (diameter 0) (color 0 0 0 0)
   )
@@
   (junction (at 121.92 163.83) (diameter 0) (color 0 0 0 0)
   )
-  (junction (at 101.6 118.11) (diameter 0) (color 0 0 0 0)
-  )
   (junction (at 95.25 163.83) (diameter 0) (color 0 0 0 0)
   )
   (junction (at 82.55 173.99) (diameter 0) (color 0 0 0 0)
   )
-  (junction (at 101.6 173.99) (diameter 0) (color 0 0 0 0)
-  )
   (junction (at 91.44 163.83) (diameter 0) (color 0 0 0 0)
   )
@@
   )
   (junction (at 106.68 163.83) (diameter 0) (color 0 0 0 0)
+  )
+  (junction (at 106.68 173.99) (diameter 0) (color 0 0 0 0)
   )
   (junction (at 257.81 48.26) (diameter 0) (color 0 0 0 0)
@@
     (stroke (width 0) (type default))
   )
-  (wire (pts (xy 101.6 118.11) (xy 95.25 118.11))
-    (stroke (width 0) (type default))
-  )
   (wire (pts (xy 163.83 58.42) (xy 167.64 58.42))
     (stroke (width 0) (type default))
@@
     (stroke (width 0) (type default))
   )
-  (wire (pts (xy 106.68 173.99) (xy 101.6 173.99))
-    (stroke (width 0) (type default))
-  )
   (wire (pts (xy 196.85 48.26) (xy 196.85 49.53))
     (stroke (width 0) (type default))
@@
     (stroke (width 0) (type default))
   )
-  (wire (pts (xy 106.68 118.11) (xy 101.6 118.11))
+  (wire (pts (xy 95.25 118.11) (xy 106.68 118.11))
     (stroke (width 0) (type default))
   )
@@
     (stroke (width 0) (type default))
   )
-  (wire (pts (xy 101.6 173.99) (xy 95.25 173.99))
-    (stroke (width 0) (type default))
-  )
   (wire (pts (xy 44.45 163.83) (xy 48.26 163.83))
     (stroke (width 0) (type default))
@@
   )
   (wire (pts (xy 138.43 53.34) (xy 138.43 58.42))
+    (stroke (width 0) (type default))
+  )
+  (wire (pts (xy 95.25 173.99) (xy 106.68 173.99))
     (stroke (width 0) (type default))
   )
@@
     (effects (font (size 1.27 1.27)) (justify left bottom))
   )
+  (text "0.6mA rated" (at 114.3 57.15 0)
+    (effects (font (size 1.27 1.27)) (justify left bottom))
+  )
   (text "0.3W min" (at 256.54 110.49 0)
     (effects (font (size 1.27 1.27)) (justify left bottom))
@@
     )
   )
-  (symbol (lib_id "power:GND") (at 101.6 181.61 0) (unit 1)
-    (in_bom yes) (on_board yes) (dnp no) (fields_autoplaced)
-    (property "Reference" "#PWR017" (at 101.6 187.96 0)
-      (effects (font (size 1.27 1.27)) hide)
-    )
-    (property "Value" "GND" (at 101.6 186.69 0)
-      (effects (font (size 1.27 1.27)))
-    )
-    (property "Footprint" "" (at 101.6 181.61 0)
-      (effects (font (size 1.27 1.27)) hide)
-    )
-    (property "Datasheet" "" (at 101.6 181.61 0)
+  (symbol (lib_id "power:GND") (at 106.68 181.61 0) (unit 1)
+    (in_bom yes) (on_board yes) (dnp no) (fields_autoplaced)
+    (property "Reference" "#PWR017" (at 106.68 187.96 0)
+      (effects (font (size 1.27 1.27)) hide)
+    )
+    (property "Value" "GND" (at 106.68 186.69 0)
+      (effects (font (size 1.27 1.27)))
+    )
+    (property "Footprint" "" (at 106.68 181.61 0)
+      (effects (font (size 1.27 1.27)) hide)
+    )
+    (property "Datasheet" "" (at 106.68 181.61 0)
       (effects (font (size 1.27 1.27)) hide)
     )
@@
     )
   )
-  (symbol (lib_id "Device:C_Polarized") (at 101.6 121.92 0) (unit 1)
-    (in_bom yes) (on_board yes) (dnp no) (fields_autoplaced)
-    (property "Reference" "C7" (at 105.41 119.761 0)
-      (effects (font (size 1.27 1.27)) (justify left))
-    )
-    (property "Value" "10uC" (at 105.41 122.301 0)
-      (effects (font (size 1.27 1.27)) (justify left))
-    )
-    (property "Footprint" "Capacitor_SMD:CP_Elec_6.3x5.4" (at 102.5652 125.73 0)
-      (effects (font (size 1.27 1.27)) hide)
-    )
-    (property "Datasheet" "https://datasheet.lcsc.com/lcsc/2304140030_Nichicon-UWX1H100MCL1GB_C134237.pdf" (at 101.6 121.92 0)
-      (effects (font (size 1.27 1.27)) hide)
-    )
-    (property "MPN" "UWX1H100MCL1GB" (at 101.6 121.92 0)
-      (effects (font (size 1.27 1.27)) hide)
-    )
-    (property "Status" "OK" (at 101.6 121.92 0)
+  (symbol (lib_id "Device:C_Polarized") (at 106.68 121.92 0) (unit 1)
+    (in_bom yes) (on_board yes) (dnp no) (fields_autoplaced)
+    (property "Reference" "C7" (at 110.49 119.761 0)
+      (effects (font (size 1.27 1.27)) (justify left))
+    )
+    (property "Value" "10uC" (at 110.49 122.301 0)
+      (effects (font (size 1.27 1.27)) (justify left))
+    )
+    (property "Footprint" "Capacitor_SMD:CP_Elec_6.3x5.4" (at 107.6452 125.73 0)
+      (effects (font (size 1.27 1.27)) hide)
+    )
+    (property "Datasheet" "https://datasheet.lcsc.com/lcsc/2304140030_Nichicon-UWX1H100MCL1GB_C134237.pdf" (at 106.68 121.92 0)
+      (effects (font (size 1.27 1.27)) hide)
+    )
+    (property "MPN" "UWX1H100MCL1GB" (at 106.68 121.92 0)
+      (effects (font (size 1.27 1.27)) hide)
+    )
+    (property "Status" "OK" (at 106.68 121.92 0)
       (effects (font (size 1.27 1.27)) hide)
     )
@@
     )
   )
-  (symbol (lib_id "Device:C_Polarized") (at 101.6 177.8 0) (unit 1)
-    (in_bom yes) (on_board yes) (dnp no) (fields_autoplaced)
-    (property "Reference" "C8" (at 105.41 175.641 0)
-      (effects (font (size 1.27 1.27)) (justify left))
-    )
-    (property "Value" "10uC" (at 105.41 178.181 0)
-      (effects (font (size 1.27 1.27)) (justify left))
-    )
-    (property "Footprint" "Capacitor_SMD:CP_Elec_6.3x5.4" (at 102.5652 181.61 0)
-      (effects (font (size 1.27 1.27)) hide)
-    )
-    (property "Datasheet" "https://datasheet.lcsc.com/lcsc/2304140030_Nichicon-UWX1H100MCL1GB_C134237.pdf" (at 101.6 177.8 0)
-      (effects (font (size 1.27 1.27)) hide)
-    )
-    (property "MPN" "UWX1H100MCL1GB" (at 101.6 177.8 0)
-      (effects (font (size 1.27 1.27)) hide)
-    )
-    (property "Status" "OK" (at 101.6 177.8 0)
+  (symbol (lib_id "Device:C_Polarized") (at 106.68 177.8 0) (unit 1)
+    (in_bom yes) (on_board yes) (dnp no) (fields_autoplaced)
+    (property "Reference" "C8" (at 110.49 175.641 0)
+      (effects (font (size 1.27 1.27)) (justify left))
+    )
+    (property "Value" "10uC" (at 110.49 178.181 0)
+      (effects (font (size 1.27 1.27)) (justify left))
+    )
+    (property "Footprint" "Capacitor_SMD:CP_Elec_6.3x5.4" (at 107.6452 181.61 0)
+      (effects (font (size 1.27 1.27)) hide)
+    )
+    (property "Datasheet" "https://datasheet.lcsc.com/lcsc/2304140030_Nichicon-UWX1H100MCL1GB_C134237.pdf" (at 106.68 177.8 0)
+      (effects (font (size 1.27 1.27)) hide)
+    )
+    (property "MPN" "UWX1H100MCL1GB" (at 106.68 177.8 0)
+      (effects (font (size 1.27 1.27)) hide)
+    )
+    (property "Status" "OK" (at 106.68 177.8 0)
       (effects (font (size 1.27 1.27)) hide)
     )
@@
     )
   )
-  (symbol (lib_id "power:GND") (at 101.6 125.73 0) (unit 1)
-    (in_bom yes) (on_board yes) (dnp no) (fields_autoplaced)
-    (property "Reference" "#PWR016" (at 101.6 132.08 0)
-      (effects (font (size 1.27 1.27)) hide)
-    )
-    (property "Value" "GND" (at 101.6 130.81 0)
-      (effects (font (size 1.27 1.27)))
-    )
-    (property "Footprint" "" (at 101.6 125.73 0)
-      (effects (font (size 1.27 1.27)) hide)
-    )
-    (property "Datasheet" "" (at 101.6 125.73 0)
-      (effects (font (size 1.27 1.27)) hide)
-    )
+  (symbol (lib_id "power:GND") (at 106.68 125.73 0) (unit 1)
+    (in_bom yes) (on_board yes) (dnp no) (fields_autoplaced)
+    (property "Reference" "#PWR016" (at 106.68 132.08 0)
+      (effects (font (size 1.27 1.27)) hide)
+    )
+    (property "Value" "GND" (at 106.68 130.81 0)
+      (effects (font (size 1.27 1.27)))
+    )
+    (property "Footprint" "" (at 106.68 125.73 0)
+      (effects (font (size 1.27 1.27)) hide)
+    )
+    (property "Datasheet" "" (at 106.68 125.73 0)
+      (effects (font (size 1.27 1.27)) hide)
+    )

Commit message: Progressed ECAD.
Parts:
- J2: footprint (none) -> Connector_PinHeader_2.54mm:PinHeader_1x06_P2.54mm_Horizontal; MPN (none) -> PZ254-1-06-W-8.5; Status (none) -> OK
Changed lines of the file:
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@@
       (effects (font (size 1.27 1.27)) (justify left))
     )
-    (property "Footprint" "" (at 189.23 111.76 0)
+    (property "Footprint" "Connector_PinHeader_2.54mm:PinHeader_1x06_P2.54mm_Horizontal" (at 189.23 111.76 0)
       (effects (font (size 1.27 1.27)) hide)
     )
-    (property "Datasheet" "~" (at 189.23 111.76 0)
+    (property "Datasheet" "https://datasheet.lcsc.com/lcsc/2306091006_HCTL-PZ254-1-06-W-8-5_C2894948.pdf" (at 189.23 111.76 0)
       (effects (font (size 1.27 1.27)) hide)
     )
+    (property "MPN" "PZ254-1-06-W-8.5" (at 189.23 111.76 0)
+      (effects (font (size 1.27 1.27)) hide)
+    )
+    (property "Status" "OK" (at 189.23 111.76 0)
+      (effects (font (size 1.27 1.27)) hide)
+    )

Commit message: Update Power_supply.kicad_sch
Parts:
- removed FL1, FL3: Filter_EMI_LCL, symbol Device:Filter_EMI_LCL
- renumbered C3 to C1, C12 to C10, C13 to C11, C14 to C12, C15 to C13, C16 to C14, C17 to C15, C18 to C16, C19 to C17, C4 to C2, C5 to C3, C6 to C4, C7 to C5, C8 to C6, C9 to C7, C10 to C8, C11 to C9, D3 to D2, D4 to D3, D2 to D4, FL2 to FL1, R2 to R1, R3 to R2, R1 to R3, R7 to R6, R6 to R7
Connections:
- net at FL1.3: now also L1.1
- net at D4.3 (K), Q1.1 (S), Q1.2 (S)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: now also FL1.2
Other:
- moved on the sheet: C11, C12, C13, C14, C15, C16, C17, D1, D4, FL1, J1, L1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

Commit message: Update Power_supply.kicad_sch
Parts:
- removed C1, C10, C13, C2, C5, C6, C7, C8, C9: 10uC, Capacitor_SMD:CP_Elec_6.3x5.4, symbol Device:C_Polarized
- added C1, C13, C18, C2, C5, C6, C7, C8, C9: 10uC, Capacitor_SMD:C_1206_3216Metric, symbol Device:C
Connections:
- net +12V: now also C1.1, C13.1, C18.1
- net +5V: now also C2.1, C5.1
- net +9V: now also C6.1, C7.1
- net GND: now also C1.2, C13.2, C18.2, C2.2, C5.2, C6.2, C7.2, C8.2, C9.2
- net at D6.2 (A), R2.1, R5.2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: now also C8.1
- net at D5.2 (A), R1.1, R4.2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: now also C9.1
Other:
- moved on the sheet: R1, R2

Commit message: Update Power_supply.kicad_sch
Parts:
- L1, L2: footprint (none) -> Inductor_SMD:L_Taiyo-Yuden_NR-60xx; MPN (none) -> NRS6045T101MMGK; Status (none) -> OK
- L3, L4: footprint (none) -> Inductor_SMD:L_Taiyo-Yuden_NR-30xx; MPN (none) -> NR3015T100M; Status (none) -> OK
Changed lines of the file:
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@@
       (effects (font (size 1.27 1.27)))
     )
-    (property "Footprint" "" (at 151.13 48.26 0)
-      (effects (font (size 1.27 1.27)) hide)
-    )
-    (property "Datasheet" "~" (at 151.13 48.26 0)
+    (property "Footprint" "Inductor_SMD:L_Taiyo-Yuden_NR-30xx" (at 151.13 48.26 0)
+      (effects (font (size 1.27 1.27)) hide)
+    )
+    (property "Datasheet" "https://datasheet.lcsc.com/lcsc/2304140030_Taiyo-Yuden-NR3015T100M_C87168.pdf" (at 151.13 48.26 0)
+      (effects (font (size 1.27 1.27)) hide)
+    )
+    (property "MPN" "NR3015T100M" (at 151.13 48.26 0)
+      (effects (font (size 1.27 1.27)) hide)
+    )
+    (property "Status" "OK" (at 151.13 48.26 0)
       (effects (font (size 1.27 1.27)) hide)
     )
@@
       (effects (font (size 1.27 1.27)))
     )
-    (property "Footprint" "" (at 142.24 58.42 0)
-      (effects (font (size 1.27 1.27)) hide)
-    )
-    (property "Datasheet" "~" (at 142.24 58.42 0)
+    (property "Footprint" "Inductor_SMD:L_Taiyo-Yuden_NR-60xx" (at 142.24 58.42 0)
+      (effects (font (size 1.27 1.27)) hide)
+    )
+    (property "Datasheet" "https://datasheet.lcsc.com/lcsc/2108160930_Taiyo-Yuden-NRS6045T101MMGK_C223018.pdf" (at 142.24 58.42 0)
+      (effects (font (size 1.27 1.27)) hide)
+    )
+    (property "MPN" "NRS6045T101MMGK" (at 142.24 58.42 0)
+      (effects (font (size 1.27 1.27)) hide)
+    )
+    (property "Status" "OK" (at 142.24 58.42 0)
       (effects (font (size 1.27 1.27)) hide)
     )
@@
       (effects (font (size 1.27 1.27)))
     )
-    (property "Footprint" "" (at 151.13 58.42 0)
-      (effects (font (size 1.27 1.27)) hide)
-    )
-    (property "Datasheet" "~" (at 151.13 58.42 0)
+    (property "Footprint" "Inductor_SMD:L_Taiyo-Yuden_NR-30xx" (at 151.13 58.42 0)
+      (effects (font (size 1.27 1.27)) hide)
+    )
+    (property "Datasheet" "https://datasheet.lcsc.com/lcsc/2304140030_Taiyo-Yuden-NR3015T100M_C87168.pdf" (at 151.13 58.42 0)
+      (effects (font (size 1.27 1.27)) hide)
+    )
+    (property "MPN" "NR3015T100M" (at 151.13 58.42 0)
+      (effects (font (size 1.27 1.27)) hide)
+    )
+    (property "Status" "OK" (at 151.13 58.42 0)
       (effects (font (size 1.27 1.27)) hide)
     )
@@
       (effects (font (size 1.27 1.27)))
     )
-    (property "Footprint" "" (at 142.24 48.26 0)
-      (effects (font (size 1.27 1.27)) hide)
-    )
-    (property "Datasheet" "~" (at 142.24 48.26 0)
-      (effects (font (size 1.27 1.27)) hide)
-    )
+    (property "Footprint" "Inductor_SMD:L_Taiyo-Yuden_NR-60xx" (at 142.24 48.26 0)
+      (effects (font (size 1.27 1.27)) hide)
+    )
+    (property "Datasheet" "https://datasheet.lcsc.com/lcsc/2108160930_Taiyo-Yuden-NRS6045T101MMGK_C223018.pdf" (at 142.24 48.26 0)
+      (effects (font (size 1.27 1.27)) hide)
+    )
+    (property "MPN" "NRS6045T101MMGK" (at 142.24 48.26 0)
+      (effects (font (size 1.27 1.27)) hide)
+    )
+    (property "Status" "OK" (at 142.24 48.26 0)
+      (effects (font (size 1.27 1.27)) hide)
+    )

Commit message: Update Power_supply.kicad_sch
Parts:
- removed L2: 100uL, Inductor_SMD:L_Taiyo-Yuden_NR-60xx, symbol Device:L_Ferrite
- removed L4: 10uL, Inductor_SMD:L_Taiyo-Yuden_NR-30xx, symbol Device:L_Ferrite
- renumbered C18 to C1, C6 to C10, C1 to C2, C9 to C5, C8 to C6, C2 to C7, C7 to C8, C5 to C9, L3 to L2
Connections:
- net GND: now also FL1.4
