File: ECAD/Power_supply/Power_supply.kicad_sch (KiCad schematic)
At the start: 42 parts, among them J1 Barrel_Jack_Switch, J2 Conn_01x06, Q1 DMP3037LSS-13, SW1 SW_Push_DPDT, U1 LM317_TO-220, U2 LM317_TO-220

Commit message: Update Power_supply.kicad_sch
Parts:
- removed C1, C2: 10uC, Capacitor_SMD:C_1206_3216Metric, symbol Device:C
- C1: renamed from C3; footprint Capacitor_SMD:C_0805_2012Metric -> Capacitor_SMD:C_1206_3216Metric; MPN (none) -> CC1206KRX7R9BB104; Status (none) -> OK
- C12: renamed from C14; footprint Capacitor_SMD:C_0805_2012Metric -> Capacitor_SMD:C_1206_3216Metric; MPN (none) -> CC1206KKX7R0BB105; Status (none) -> OK
- C13: renamed from C15; footprint Capacitor_SMD:C_0805_2012Metric -> Capacitor_SMD:C_1206_3216Metric; MPN (none) -> CC1206KRX7R9BB104; Status (none) -> OK
- C14: renamed from C16; footprint Capacitor_SMD:C_0805_2012Metric -> Capacitor_SMD:C_1206_3216Metric; MPN (none) -> CC1206KKX7RCBB103; Status (none) -> OK
- C15: renamed from C17; footprint Capacitor_SMD:C_0805_2012Metric -> Capacitor_SMD:C_1206_3216Metric; MPN (none) -> CC1206KKX7RDBB102; Status (none) -> OK
- C2: renamed from C4; footprint Capacitor_SMD:C_0805_2012Metric -> Capacitor_SMD:C_1206_3216Metric; MPN (none) -> CC1206KRX7R9BB104; Status (none) -> OK
- D2, D3, D5, D6: value SM4001 -> S1A-13-F; footprint Diode_SMD:D_MELF -> Diode_SMD:D_SMA; MPN (none) -> S1A-13-F; Status (none) -> OK
- renumbered C12 to C10, C13 to C11, C5 to C3, C6 to C4, C7 to C5, C8 to C6, C9 to C7, C10 to C8, C11 to C9

Commit message: Update Power_supply.kicad_sch
Parts:
- C10: footprint Capacitor_SMD:CP_Elec_6.3x5.4 -> Capacitor_SMD:CP_Elec_8x10; MPN (none) -> UWT1H101MNL1GS; Status (none) -> OK
- C9: MPN EEEFT1C102AP -> EEEFT1E102UP; Status (none) -> OK
- FL1, Q1: Status (none) -> OK
- U1, U2: MPN (none) -> LM317KCS; Status (none) -> OK
Changed lines of the file:
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@@
       (effects (font (size 1.27 1.27) italic) hide)
     )
-    (property "Datasheet" "http://www.ti.com/lit/ds/symlink/lm317.pdf" (at 82.55 163.83 0)
+    (property "Datasheet" "https://datasheet.lcsc.com/lcsc/2003172043_Texas-Instruments-LM317KCS_C496105.pdf" (at 82.55 163.83 0)
+      (effects (font (size 1.27 1.27)) hide)
+    )
+    (property "MPN" "LM317KCS" (at 82.55 163.83 0)
+      (effects (font (size 1.27 1.27)) hide)
+    )
+    (property "Status" "OK" (at 82.55 163.83 0)
       (effects (font (size 1.27 1.27)) hide)
     )
@@
       (effects (font (size 1.27 1.27)) hide)
     )
+    (property "Status" "OK" (at 91.44 50.8 0)
+      (effects (font (size 1.27 1.27)) hide)
+    )
     (pin "8")
     (pin "2")
@@
       (effects (font (size 1.27 1.27)) (justify left))
     )
-    (property "Footprint" "Capacitor_SMD:CP_Elec_6.3x5.4" (at 174.9552 57.15 0)
-      (effects (font (size 1.27 1.27)) hide)
-    )
-    (property "Datasheet" "" (at 173.99 53.34 0)
-      (effects (font (size 1.27 1.27)) hide)
-    )
-    (property "MPN" "" (at 173.99 53.34 0)
-      (effects (font (size 1.27 1.27)) hide)
-    )
-    (property "Status" "" (at 173.99 53.34 0)
+    (property "Footprint" "Capacitor_SMD:CP_Elec_8x10" (at 174.9552 57.15 0)
+      (effects (font (size 1.27 1.27)) hide)
+    )
+    (property "Datasheet" "https://datasheet.lcsc.com/lcsc/2304140030_Nichicon-UWT1H101MNL1GS_C445063.pdf" (at 173.99 53.34 0)
+      (effects (font (size 1.27 1.27)) hide)
+    )
+    (property "MPN" "UWT1H101MNL1GS" (at 173.99 53.34 0)
+      (effects (font (size 1.27 1.27)) hide)
+    )
+    (property "Status" "OK" (at 173.99 53.34 0)
       (effects (font (size 1.27 1.27)) hide)
     )
@@
       (effects (font (size 1.27 1.27)) hide)
     )
-    (property "Datasheet" "https://datasheet.lcsc.com/lcsc/2304140030_PANASONIC-EEEFT1C102AP_C178587.pdf" (at 158.75 53.34 0)
-      (effects (font (size 1.27 1.27)) hide)
-    )
-    (property "MPN" "EEEFT1C102AP" (at 158.75 53.34 0)
+    (property "Datasheet" "https://datasheet.lcsc.com/lcsc/1912111437_PANASONIC-EEEFT1E102UP_C401766.pdf" (at 158.75 53.34 0)
+      (effects (font (size 1.27 1.27)) hide)
+    )
+    (property "MPN" "EEEFT1E102UP" (at 158.75 53.34 0)
+      (effects (font (size 1.27 1.27)) hide)
+    )
+    (property "Status" "OK" (at 158.75 53.34 0)
       (effects (font (size 1.27 1.27)) hide)
     )
@@
       (effects (font (size 1.27 1.27)) hide)
     )
+    (property "Status" "OK" (at 125.73 53.34 0)
+      (effects (font (size 1.27 1.27)) hide)
+    )
     (pin "3")
     (pin "4")
@@
       (effects (font (size 1.27 1.27) italic) hide)
     )
-    (property "Datasheet" "http://www.ti.com/lit/ds/symlink/lm317.pdf" (at 82.55 107.95 0)
-      (effects (font (size 1.27 1.27)) hide)
-    )
+    (property "Datasheet" "https://datasheet.lcsc.com/lcsc/2003172043_Texas-Instruments-LM317KCS_C496105.pdf" (at 82.55 107.95 0)
+      (effects (font (size 1.27 1.27)) hide)
+    )
+    (property "MPN" "LM317KCS" (at 82.55 107.95 0)
+      (effects (font (size 1.27 1.27)) hide)
+    )
+    (property "Status" "OK" (at 82.55 107.95 0)
+      (effects (font (size 1.27 1.27)) hide)
+    )

Commit message: Progressed ECAD.
Parts:
- R1: MPN (none) -> 0805W8F7150T5E; Status (none) -> OK
- R2: MPN (none) -> RC0805FR-071K5L; Status (none) -> OK
- R3: MPN RC0805FR-0710KL -> AC0805FR-0710KL; Status (none) -> OK
- R4, R5: MPN (none) -> RC0805FR-07240RL; Status (none) -> OK
- R6: footprint Resistor_SMD:R_0805_2012Metric -> Resistor_SMD:R_1210_3225Metric; MPN (none) -> RC0805FR-07100KL; Status (none) -> OK
- R7: MPN (none) -> 1210W2F1001T5E; Status (none) -> OK
Changed lines of the file:
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@@
       (effects (font (size 1.27 1.27)) hide)
     )
-    (property "Datasheet" "" (at 95.25 113.03 0)
-      (effects (font (size 1.27 1.27)) hide)
-    )
-    (property "MPN" "" (at 95.25 113.03 0)
-      (effects (font (size 1.27 1.27)) hide)
-    )
-    (property "Status" "" (at 95.25 113.03 0)
+    (property "Datasheet" "https://datasheet.lcsc.com/lcsc/2304140030_YAGEO-RC0805FR-07240RL_C185292.pdf" (at 95.25 113.03 0)
+      (effects (font (size 1.27 1.27)) hide)
+    )
+    (property "MPN" "RC0805FR-07240RL" (at 95.25 113.03 0)
+      (effects (font (size 1.27 1.27)) hide)
+    )
+    (property "Status" "OK" (at 95.25 113.03 0)
       (effects (font (size 1.27 1.27)) hide)
     )
@@
       (effects (font (size 1.27 1.27)) hide)
     )
-    (property "Datasheet" "" (at 82.55 123.19 0)
-      (effects (font (size 1.27 1.27)) hide)
-    )
-    (property "MPN" "" (at 82.55 123.19 0)
-      (effects (font (size 1.27 1.27)) hide)
-    )
-    (property "Status" "" (at 82.55 123.19 0)
+    (property "Datasheet" "https://datasheet.lcsc.com/lcsc/2205311830_UNI-ROYAL-Uniroyal-Elec-0805W8F7150T5E_C17813.pdf" (at 82.55 123.19 0)
+      (effects (font (size 1.27 1.27)) hide)
+    )
+    (property "MPN" "0805W8F7150T5E" (at 82.55 123.19 0)
+      (effects (font (size 1.27 1.27)) hide)
+    )
+    (property "Status" "OK" (at 82.55 123.19 0)
       (effects (font (size 1.27 1.27)) hide)
     )
@@
       (effects (font (size 1.27 1.27)) hide)
     )
-    (property "Datasheet" "" (at 95.25 168.91 0)
-      (effects (font (size 1.27 1.27)) hide)
-    )
-    (property "MPN" "" (at 95.25 168.91 0)
-      (effects (font (size 1.27 1.27)) hide)
-    )
-    (property "Status" "" (at 95.25 168.91 0)
+    (property "Datasheet" "https://datasheet.lcsc.com/lcsc/2304140030_YAGEO-RC0805FR-07240RL_C185292.pdf" (at 95.25 168.91 0)
+      (effects (font (size 1.27 1.27)) hide)
+    )
+    (property "MPN" "RC0805FR-07240RL" (at 95.25 168.91 0)
+      (effects (font (size 1.27 1.27)) hide)
+    )
+    (property "Status" "OK" (at 95.25 168.91 0)
       (effects (font (size 1.27 1.27)) hide)
     )
@@
       (effects (font (size 1.27 1.27)) hide)
     )
-    (property "Datasheet" "https://datasheet.lcsc.com/lcsc/1810201611_YAGEO-RC0805FR-0710KL_C84376.pdf" (at 91.44 59.69 0)
-      (effects (font (size 1.27 1.27)) hide)
-    )
-    (property "MPN" "RC0805FR-0710KL" (at 91.44 59.69 0)
-      (effects (font (size 1.27 1.27)) hide)
-    )
-    (property "Status" "" (at 91.44 59.69 0)
+    (property "Datasheet" "https://datasheet.lcsc.com/lcsc/2304140030_YAGEO-AC0805FR-0710KL_C140868.pdf" (at 91.44 59.69 0)
+      (effects (font (size 1.27 1.27)) hide)
+    )
+    (property "MPN" "AC0805FR-0710KL" (at 91.44 59.69 0)
+      (effects (font (size 1.27 1.27)) hide)
+    )
+    (property "Status" "OK" (at 91.44 59.69 0)
       (effects (font (size 1.27 1.27)) hide)
     )
@@
       (effects (font (size 1.27 1.27)) hide)
     )
-    (property "Datasheet" "" (at 248.92 109.22 0)
-      (effects (font (size 1.27 1.27)) hide)
-    )
-    (property "MPN" "" (at 248.92 109.22 0)
-      (effects (font (size 1.27 1.27)) hide)
-    )
-    (property "Status" "" (at 248.92 109.22 0)
+    (property "Datasheet" "https://datasheet.lcsc.com/lcsc/2206010000_UNI-ROYAL-Uniroyal-Elec-1210W2F1001T5E_C52444.pdf" (at 248.92 109.22 0)
+      (effects (font (size 1.27 1.27)) hide)
+    )
+    (property "MPN" "1210W2F1001T5E" (at 248.92 109.22 0)
+      (effects (font (size 1.27 1.27)) hide)
+    )
+    (property "Status" "OK" (at 248.92 109.22 0)
       (effects (font (size 1.27 1.27)) hide)
     )
@@
       (effects (font (size 1.27 1.27)) hide)
     )
-    (property "Datasheet" "" (at 82.55 179.07 0)
-      (effects (font (size 1.27 1.27)) hide)
-    )
-    (property "MPN" "" (at 82.55 179.07 0)
-      (effects (font (size 1.27 1.27)) hide)
-    )
-    (property "Status" "" (at 82.55 179.07 0)
+    (property "Datasheet" "https://datasheet.lcsc.com/lcsc/2304140030_YAGEO-RC0805FR-071K5L_C114555.pdf" (at 82.55 179.07 0)
+      (effects (font (size 1.27 1.27)) hide)
+    )
+    (property "MPN" "RC0805FR-071K5L" (at 82.55 179.07 0)
+      (effects (font (size 1.27 1.27)) hide)
+    )
+    (property "Status" "OK" (at 82.55 179.07 0)
       (effects (font (size 1.27 1.27)) hide)
     )
@@
       (effects (font (size 1.27 1.27)) (justify left))
     )
-    (property "Footprint" "Resistor_SMD:R_0805_2012Metric" (at 247.142 53.34 90)
-      (effects (font (size 1.27 1.27)) hide)
-    )
-    (property "Datasheet" "~" (at 248.92 53.34 0)
-      (effects (font (size 1.27 1.27)) hide)
-    )
-    (property "Status" "" (at 248.92 53.34 0)
-      (effects (font (size 1.27 1.27)) hide)
-    )
+    (property "Footprint" "Resistor_SMD:R_1210_3225Metric" (at 247.142 53.34 90)
+      (effects (font (size 1.27 1.27)) hide)
+    )
+    (property "Datasheet" "https://datasheet.lcsc.com/lcsc/2304140030_YAGEO-RC0805FR-07100KL_C96346.pdf" (at 248.92 53.34 0)
+      (effects (font (size 1.27 1.27)) hide)
+    )
+    (property "Status" "OK" (at 248.92 53.34 0)
+      (effects (font (size 1.27 1.27)) hide)
+    )
+    (property "MPN" "RC0805FR-07100KL" (at 248.92 53.34 0)
+      (effects (font (size 1.27 1.27)) hide)
+    )

Commit message: Update Power_supply.kicad_sch
Parts:
- HS1, HS2: footprint Heatsink:Heatsink_Fischer_SK129-STS_42x25mm_2xDrill2.5mm -> Heatsink:Heatsink_Fischer_SK104-STC-STIC_35x13mm_2xDrill2.5mm
Changed lines of the file:
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@@
       (effects (font (size 1.27 1.27)) (justify left))
     )
-    (property "Footprint" "Heatsink:Heatsink_Fischer_SK129-STS_42x25mm_2xDrill2.5mm" (at 65.0748 185.42 0)
+    (property "Footprint" "Heatsink:Heatsink_Fischer_SK104-STC-STIC_35x13mm_2xDrill2.5mm" (at 65.0748 185.42 0)
       (effects (font (size 1.27 1.27)) hide)
     )
@@
       (effects (font (size 1.27 1.27)) (justify left))
     )
-    (property "Footprint" "Heatsink:Heatsink_Fischer_SK129-STS_42x25mm_2xDrill2.5mm" (at 65.0748 129.54 0)
+    (property "Footprint" "Heatsink:Heatsink_Fischer_SK104-STC-STIC_35x13mm_2xDrill2.5mm" (at 65.0748 129.54 0)
       (effects (font (size 1.27 1.27)) hide)
     )

Commit message: Progressed ECAD.
Connections:
- net at D1.2 (A2), Q1.5 (D), Q1.6 (D)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: now also SW1.3 (C), SW1.6 (C); no longer SW1.1 (A), SW1.4 (A)

Commit message: Thermal calculations.
Connections:
- net +12V: now also J2.3 (Pin_3); no longer J2.1 (Pin_1)
- net +5V: now also J2.1 (Pin_1); no longer J2.5 (Pin_5)
- net +9V: now also J2.5 (Pin_5); no longer J2.3 (Pin_3)
Other:
- note added: "I_{5V max} = 300mA"
- note added: "I_{9V max} = 100mA"
- note added: "Junction-to-case (bottom) thermal resistance: 0.1 °C/W"
- note added: "Thermal calculations U1 power dissipation: PD = PI - PO = (VI - VO)*IO = (12 - 5)*0.3 = 2.1 W Thermal resistances: θJA = θJC + θCS + θSA = 0.1 + 0.4 + 14 = 14.5 °C/W Junction temperature rise: (TJ-TA)/PD = θJA TJ = θJA*PD + TA TJ = 14.5*2.1 + 25 TJ = 41.6 °C TJmax = 125 °C"
- note added: "Thermal calculations U1 power dissipation: PD = PI - PO = (VI - VO)*IO = (12 - 9)*0.1 = 0.3 W Thermal resistances: θJA = θJC + θCS + θSA = 0.1 + 0.4 + 14 = 14.5 °C/W Junction temperature rise: (TJ-TA)/PD = θJA TJ = θJA*PD + TA TJ = 14.5*0.3 + 25 TJ = 29.35 °C TJmax = 125 °C"
- note added: "Thermal resistance: 14 °C/W"
Changed lines of the file:
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@@
 	)
 	(junction
+		(at 242.57 48.26)
+		(diameter 0)
+		(color 0 0 0 0)
+	)
+	(junction
 		(at 200.66 58.42)
 		(diameter 0)
@@
 	)
 	(junction
-		(at 196.85 106.68)
-		(diameter 0)
-		(color 0 0 0 0)
-	)
-	(junction
 		(at 95.25 173.99)
 		(diameter 0)
@@
 	(wire
 		(pts
-			(xy 196.85 106.68) (xy 205.74 106.68)
+			(xy 194.31 106.68) (xy 205.74 106.68)
 		)
 		(stroke
@@
 		)
 	)
+	(polyline
+		(pts
+			(xy 90.17 101.6) (xy 95.25 97.79)
+		)
+		(stroke
+			(width 0)
+			(type default)
+		)
+	)
 	(wire
 		(pts
@@
 	(wire
 		(pts
+			(xy 242.57 48.26) (xy 248.92 48.26)
+		)
+		(stroke
+			(width 0)
+			(type default)
+		)
+	)
+	(wire
+		(pts
 			(xy 194.31 116.84) (xy 218.44 116.84)
 		)
@@
 		)
 	)
+	(polyline
+		(pts
+			(xy 90.17 157.48) (xy 95.25 153.67)
+		)
+		(stroke
+			(width 0)
+			(type default)
+		)
+	)
 	(wire
 		(pts
@@
 	(wire
 		(pts
-			(xy 238.76 48.26) (xy 248.92 48.26)
-		)
-		(stroke
-			(width 0)
-			(type default)
-		)
-	)
-	(wire
-		(pts
-			(xy 194.31 106.68) (xy 196.85 106.68)
+			(xy 238.76 48.26) (xy 242.57 48.26)
 		)
 		(stroke
@@
 		)
 	)
+	(text "I_{5V max} = 300mA"
+		(exclude_from_sim no)
+		(at 106.68 105.41 0)
+		(effects
+			(font
+				(size 1.27 1.27)
+			)
+			(justify left bottom)
+		)
+	)
 	(text "5V power supply"
 		(exclude_from_sim no)
@@
 		)
 	)
+	(text "I_{9V max} = 100mA"
+		(exclude_from_sim no)
+		(at 107.442 160.782 0)
+		(effects
+			(font
+				(size 1.27 1.27)
+			)
+			(justify left bottom)
+		)
+	)
 	(text "Reverse polarity\nprotection"
 		(exclude_from_sim no)
@@
 		)
 	)
+	(text "Junction-to-case (bottom)\nthermal resistance: 0.1 °C/W"
+		(exclude_from_sim no)
+		(at 109.982 96.012 0)
+		(effects
+			(font
+				(size 1.27 1.27)
+			)
+		)
+	)
+	(text "Thermal resistance: 14 °C/W"
+		(exclude_from_sim no)
+		(at 64.77 133.858 0)
+		(effects
+			(font
+				(size 1.27 1.27)
+			)
+		)
+	)
 	(text "EMI filter"
 		(exclude_from_sim no)
@@
 		)
 	)
+	(text "Thermal calculations\n\nU1 power dissipation:\nPD = PI - PO = (VI - VO)*IO\n= (12 - 9)*0.1\n= 0.3 W\n\nThermal resistances:\nθJA = θJC + θCS + θSA\n= 0.1 + 0.4 + 14\n= 14.5 °C/W\n\nJunction temperature rise:\n(TJ-TA)/PD = θJA\nTJ = θJA*PD + TA\nTJ = 14.5*0.3 + 25\nTJ = 29.35 °C\n\nTJmax = 125 °C"
+		(exclude_from_sim no)
+		(at 15.748 169.418 0)
+		(effects
+			(font
+				(size 1.27 1.27)
+			)
+			(justify left)
+		)
+	)
 	(text "9V power supply"
 		(exclude_from_sim no)
@@
 		)
 	)
+	(text "Thermal resistance: 14 °C/W"
+		(exclude_from_sim no)
+		(at 65.024 189.738 0)
+		(effects
+			(font
+				(size 1.27 1.27)
+			)
+		)
+	)
+	(text "Junction-to-case (bottom)\nthermal resistance: 0.1 °C/W"
+		(exclude_from_sim no)
+		(at 109.982 151.892 0)
+		(effects
+			(font
+				(size 1.27 1.27)
+			)
+		)
+	)
+	(text "Thermal calculations\n\nU1 power dissipation:\nPD = PI - PO = (VI - VO)*IO\n= (12 - 5)*0.3\n= 2.1 W\n\nThermal resistances:\nθJA = θJC + θCS + θSA\n= 0.1 + 0.4 + 14\n= 14.5 °C/W\n\nJunction temperature rise:\n(TJ-TA)/PD = θJA\nTJ = θJA*PD + TA\nTJ = 14.5*2.1 + 25\nTJ = 41.6 °C\n\nTJmax = 125 °C"
+		(exclude_from_sim no)
+		(at 16.002 113.538 0)
+		(effects
+			(font
+				(size 1.27 1.27)
+			)
+			(justify left)
+		)
+	)
 	(text "Transient\novervoltage\nprotection"
 		(exclude_from_sim no)
@@
 	(symbol
 		(lib_id "power:+5V")
-		(at 218.44 115.57 0)
+		(at 205.74 105.41 0)
 		(unit 1)
 		(exclude_from_sim no)
@@
 		(fields_autoplaced yes)
 		(property "Reference" "#PWR023"
-			(at 218.44 119.38 0)
+			(at 205.74 109.22 0)
 			(effects
 				(font
@@
 		)
 		(property "Value" "+5V"
-			(at 218.44 110.49 0)
+			(at 205.74 100.33 0)
 			(effects
 				(font
@@
 		)
 		(property "Footprint" ""
-			(at 218.44 115.57 0)
+			(at 205.74 105.41 0)
 			(effects
 				(font
@@
 		)
 		(property "Datasheet" ""
-			(at 218.44 115.57 0)
+			(at 205.74 105.41 0)
 			(effects
 				(font
@@
 		)
 		(property "Description" "Power symbol creates a global label with name \"+5V\""
-			(at 218.44 115.57 0)
+			(at 205.74 105.41 0)
 			(effects
 				(font
@@
 	)
 	(symbol
-		(lib_id "power:PWR_FLAG")
-		(at 196.85 106.68 0)
-		(unit 1)
-		(exclude_from_sim no)
-		(in_bom yes)
-		(on_board yes)
-		(dnp no)
-		(fields_autoplaced yes)
-		(property "Reference" "#FLG02"
-			(at 196.85 104.775 0)
-			(effects
-				(font
-					(size 1.27 1.27)
-				)
-				(hide yes)
-			)
-		)
-		(property "Value" "PWR_FLAG"
-			(at 196.85 101.6 0)
-			(effects
-				(font
-					(size 1.27 1.27)
-				)
-			)
-		)
-		(property "Footprint" ""
-			(at 196.85 106.68 0)
-			(effects
-				(font
-					(size 1.27 1.27)
-				)
-				(hide yes)
-			)
-		)
-		(property "Datasheet" "~"
-			(at 196.85 106.68 0)
-			(effects
-				(font
-					(size 1.27 1.27)
-				)
-				(hide yes)
-			)
-		)
-		(property "Description" "Special symbol for telling ERC where power comes from"
-			(at 196.85 106.68 0)
-			(effects
-				(font
-					(size 1.27 1.27)
-				)
-				(hide yes)
-			)
-		)
-		(pin "1"
-		)
-		(instances
-			(project "Power_supply"
-				(path "/edc8412f-0483-47e1-aeb9-21064b18cc9b"
-					(reference "#FLG02")
-					(unit 1)
-				)
-			)
-		)
-	)
-	(symbol
 		(lib_id "Device:C")
 		(at 62.23 168.91 0)
@@
 	)
 	(symbol
+		(lib_id "power:PWR_FLAG")
+		(at 242.57 48.26 0)
+		(unit 1)
+		(exclude_from_sim no)
+		(in_bom yes)
+		(on_board yes)
+		(dnp no)
+		(fields_autoplaced yes)
+		(property "Reference" "#FLG02"
+			(at 242.57 46.355 0)
+			(effects
+				(font
+					(size 1.27 1.27)
+				)
+				(hide yes)
+			)
+		)
+		(property "Value" "PWR_FLAG"
+			(at 242.57 43.18 0)
+			(effects
+				(font
+					(size 1.27 1.27)
+				)
+			)
+		)
+		(property "Footprint" ""
+			(at 242.57 48.26 0)
+			(effects
+				(font
+					(size 1.27 1.27)
+				)
+				(hide yes)
+			)
+		)
+		(property "Datasheet" "~"
+			(at 242.57 48.26 0)
+			(effects
+				(font
+					(size 1.27 1.27)
+				)
+				(hide yes)
+			)
+		)
+		(property "Description" "Special symbol for telling ERC where power comes from"
+			(at 242.57 48.26 0)
+			(effects
+				(font
+					(size 1.27 1.27)
+				)
+				(hide yes)
+			)
+		)
+		(pin "1"
+		)
+		(instances
+			(project "Power_supply"
+				(path "/edc8412f-0483-47e1-aeb9-21064b18cc9b"
+					(reference "#FLG02")
+					(unit 1)
+				)
+			)
+		)
+	)
+	(symbol
 		(lib_id "power:GND")
 		(at 254 60.96 0)
@@
 	(symbol
 		(lib_id "power:+12V")
-		(at 205.74 105.41 0)
+		(at 212.09 110.49 0)
 		(unit 1)
 		(exclude_from_sim no)
@@
 		(fields_autoplaced yes)
 		(property "Reference" "#PWR021"
-			(at 205.74 109.22 0)
+			(at 212.09 114.3 0)
 			(effects
 				(font
@@
 		)
 		(property "Value" "+12V"
-			(at 205.74 100.584 0)
+			(at 212.09 105.664 0)
 			(effects
 				(font
@@
 		)
 		(property "Footprint" ""
-			(at 205.74 105.41 0)
+			(at 212.09 110.49 0)
 			(effects
 				(font
@@
 		)
 		(property "Datasheet" ""
-			(at 205.74 105.41 0)
+			(at 212.09 110.49 0)
 			(effects
 				(font
@@
 		)
 		(property "Description" "Power symbol creates a global label with name \"+12V\""
-			(at 205.74 105.41 0)
+			(at 212.09 110.49 0)
 			(effects
 				(font
@@
 	(symbol
 		(lib_id "power:+9V")
-		(at 212.09 110.49 0)
+		(at 218.44 115.57 0)
 		(unit 1)
 		(exclude_from_sim no)
@@
 		(fields_autoplaced yes)
 		(property "Reference" "#PWR022"
-			(at 212.09 114.3 0)
+			(at 218.44 119.38 0)
 			(effects
 				(font
@@
 		)
 		(property "Value" "+9V"
-			(at 212.09 105.41 0)
+			(at 218.44 110.49 0)
 			(effects
 				(font
@@
 		)
 		(property "Footprint" ""
-			(at 212.09 110.49 0)
+			(at 218.44 115.57 0)
 			(effects
 				(font
@@
 		)
 		(property "Datasheet" ""
-			(at 212.09 110.49 0)
+			(at 218.44 115.57 0)
 			(effects
 				(font
@@
 		)
 		(property "Description" "Power symbol creates a global label with name \"+9V\""
-			(at 212.09 110.49 0)
+			(at 218.44 115.57 0)
 			(effects
 				(font

Commit message: Progressed PCB layout.
Parts:
- J2: footprint Connector_PinHeader_2.54mm:PinHeader_1x06_P2.54mm_Horizontal -> Connector_PinSocket_2.54mm:PinSocket_1x06_P2.54mm_Vertical; Status OK -> (none)
Changed lines of the file:
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@@
 			)
 		)
-		(property "Footprint" "Connector_PinHeader_2.54mm:PinHeader_1x06_P2.54mm_Horizontal"
+		(property "Footprint" "Connector_PinSocket_2.54mm:PinSocket_1x06_P2.54mm_Vertical"
 			(at 189.23 111.76 0)
 			(effects
@@
 			)
 		)
-		(property "Status" "OK"
+		(property "Status" ""
 			(at 189.23 111.76 0)
 			(effects

Commit message: Updated the schematic.
Parts:
- added C16, C18: 100nC, Capacitor_SMD:C_1206_3216Metric, symbol Device:C
- added C17: 10uC, Capacitor_SMD:C_1206_3216Metric, symbol Device:C
- added C19: 100pC, Capacitor_SMD:C_0805_2012Metric, symbol Device:C
- added D8, D9: S1A-13-F, Diode_SMD:D_SMA, symbol Diode:SM4001
- added H1: MountingHole, symbol Mechanical:MountingHole
- added HS3: Heatsink, Heatsink:Heatsink_Fischer_SK104-STC-STIC_35x13mm_2xDrill2.5mm, symbol Mechanical:Heatsink_Pad
- added R8: 340R, Resistor_SMD:R_0805_2012Metric, symbol Device:R
- added R9: 240R, Resistor_SMD:R_0805_2012Metric, symbol Device:R
- added U3: LM317_TO-220, Package_TO_SOT_THT:TO-220-3_Vertical, symbol Regulator_Linear:LM317_TO-220
- C1: value 100nC -> 10uC; MPN CC1206KRX7R9BB104 -> CL31A106KBHNNNE
Connections:
- net +12V: now also C16.1, D9.1 (K), U3.3 (VI); no longer C1.1, D2.1 (K), U1.3 (VI)
- net +5V: now also C19.2, R8.2
- net GND: now also C16.2, C17.2, C18.2
- new net: C17.1, C19.1, D8.2 (A), R8.1, R9.2, U3.1 (ADJ)
- new net +8V: C1.1, C18.1, D2.1 (K), D8.1 (K), D9.2 (A), R9.1, U1.3 (VI), U3.2 (VO)
- no-connect marks 4 -> 5
Other:
- note added: "Thermal calculations U1 power dissipation: PD = PI - PO = (VI - VO)*IO = (12 - 8)*0.3 = 1.2 W Thermal resistances: θJA = θJC + θCS + θSA = 0.1 + 0.4 + 14 = 14.5 °C/W Junction temperature rise: (TJ-TA)/PD = θJA TJ = θJA*PD + TA TJ = 14.5*1.2 + 25 TJ = 42.4 °C TJmax = 125 °C"
- note added: "Thermal calculations U1 power dissipation: PD = PI - PO = (VI - VO)*IO = (8 - 5)*0.3 = 0.9 W Thermal resistances: θJA = θJC + θCS + θSA = 0.1 + 0.4 + 14 = 14.5 °C/W Junction temperature rise: (TJ-TA)/PD = θJA TJ = θJA*PD + TA TJ = 14.5*0.9 + 25 TJ = 38.5 °C TJmax = 125 °C"
- note added: "Tracking Preregulator"
- note removed: "Thermal calculations U1 power dissipation: PD = PI - PO = (VI - VO)*IO = (12 - 5)*0.3 = 2.1 W Thermal resistances: θJA = θJC + θCS + θSA = 0.1 + 0.4 + 14 = 14.5 °C/W Junction temperature rise: (TJ-TA)/PD = θJA TJ = θJA*PD + TA TJ = 14.5*2.1 + 25 TJ = 41.6 °C TJmax = 125 °C"
- moved on the sheet: C10, C11, C12, C13, C14, C15, C2, C3, C4, C5, C6, C7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
