File: ECAD/Power_supply/Power_supply.kicad_sch (KiCad schematic)
At the start: 51 parts, among them J1 Barrel_Jack_Switch, J2 Conn_01x06, Q1 DMP3037LSS-13, SW1 SW_Push_DPDT, U1 LM317_TO-220, U2 LM317_TO-220, U3 LM317_TO-220

Commit message: Progressed PCB.
Parts:
- added H2, H3, H4: MountingHole, MountingHole:MountingHole_3.2mm_M3, symbol Mechanical:MountingHole
- H1: footprint (none) -> MountingHole:MountingHole_3.2mm_M3
Connections:
- net +5V: now also HS1.1
- net +8V: now also HS3.1
- net +9V: now also HS2.1
- no-connect marks 5 -> 2
Other:
- moved on the sheet: HS1, HS2, HS3

Commit message: Progressed PCB.
Changed lines of the file:
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@@
+		)
+	)
+	(polyline
+		(pts
+			(xy 227.33 125.73) (xy 227.33 95.25)
+		)
+		(stroke
+			(width 0)
+			(type dash)
 		)
 	)
@@
 		)
 	)
+	(polyline
+		(pts
+			(xy 224.79 95.25) (xy 227.33 95.25)
+		)
+		(stroke
+			(width 0)
+			(type dash)
+		)
+	)
 	(wire
 		(pts
@@
 		)
 	)
+	(polyline
+		(pts
+			(xy 87.63 123.19) (xy 87.63 125.73)
+		)
+		(stroke
+			(width 0)
+			(type dash)
+		)
+	)
 	(wire
 		(pts
@@
 		)
 	)
+	(polyline
+		(pts
+			(xy 87.63 125.73) (xy 227.33 125.73)
+		)
+		(stroke
+			(width 0)
+			(type dash)
+		)
+	)
 	(wire
 		(pts
@@
 		)
 	)
+	(polyline
+		(pts
+			(xy 87.63 123.19) (xy 88.9 124.46)
+		)
+		(stroke
+			(width 0)
+			(type dash)
+		)
+	)
 	(wire
 		(pts
@@
 		)
 	)
+	(polyline
+		(pts
+			(xy 86.36 124.46) (xy 87.63 123.19)
+		)
+		(stroke
+			(width 0)
+			(type dash)
+		)
+	)

Commit message: Progressed PCB.
Parts:
- removed C1, C5, C6, C7, C8: 10uC, Capacitor_SMD:C_1206_3216Metric, symbol Device:C
- removed C18: 100nC, Capacitor_SMD:C_1206_3216Metric, symbol Device:C
- added C1, C20, C5: 22uC, Capacitor_SMD:CP_Elec_5x5.4, symbol Device:C_Polarized
Connections:
- net +12V: now also U1.3 (VI); no longer U2.3 (VI)
- net +5V: now also HS2.1, U2.2 (VO), C20.1; no longer HS1.1, U1.2 (VO)
- net +8V: now also U2.3 (VI), C1.1; no longer U1.3 (VI)
- net +9V: now also HS1.1, U1.2 (VO), C5.1; no longer HS2.1, U2.2 (VO)
- net GND: now also C1.2, C20.2, C5.2
- net ADJ_9V: now reaches C4.1, D6.2 (A), R2.1, R5.2
- net ADJ_9V: now also U1.1 (ADJ); no longer U2.1 (ADJ)
- net at C3.1, D5.2 (A), R1.1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: now also U2.1 (ADJ); no longer U1.1 (ADJ)
Other:
- moved on the sheet: HS1, HS2, U1, U2

Commit message: Updated schematic
Parts:
- added C6: 100nC, Capacitor_SMD:C_1206_3216Metric, symbol Device:C
Connections:
- net +8V: now also C6.1
- net GND: now also C6.2
- net ADJ_PRE: now reaches C17.1, C19.1, D8.2 (A), R8.1, R9.2, U3.1 (ADJ)
- net ADJ_5V: now reaches C3.1, D5.2 (A), R1.1, R4.2, U2.1 (ADJ)
Changed lines of the file:
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@@
 	)
 	(junction
+		(at 144.78 97.79)
+		(diameter 0)
+		(color 0 0 0 0)
+	)
+	(junction
 		(at 74.93 33.02)
 		(diameter 0)
@@
 	(wire
 		(pts
+			(xy 144.78 97.79) (xy 154.94 97.79)
+		)
+		(stroke
+			(width 0)
+			(type default)
+		)
+	)
+	(wire
+		(pts
 			(xy 207.01 151.13) (xy 231.14 151.13)
 		)
@@
 	(wire
 		(pts
-			(xy 139.7 97.79) (xy 154.94 97.79)
+			(xy 139.7 97.79) (xy 144.78 97.79)
 		)
 		(stroke
@@
 	(wire
 		(pts
+			(xy 144.78 97.79) (xy 144.78 99.06)
+		)
+		(stroke
+			(width 0)
+			(type default)
+		)
+	)
+	(wire
+		(pts
 			(xy 248.92 33.02) (xy 248.92 34.29)
 		)
@@
 		)
 	)
+	(label "ADJ_5V"
+		(at 166.37 107.95 0)
+		(effects
+			(font
+				(size 1.27 1.27)
+			)
+			(justify left bottom)
+		)
+	)
 	(label "ADJ_9V"
 		(at 90.17 163.83 0)
@@
 		)
 	)
+	(label "ADJ_PRE"
+		(at 88.9 107.95 0)
+		(effects
+			(font
+				(size 1.27 1.27)
+			)
+			(justify left bottom)
+		)
+	)
 	(symbol
 		(lib_id "Mechanical:Heatsink_Pad")
@@
 	)
 	(symbol
+		(lib_id "power:GND")
+		(at 144.78 106.68 0)
+		(unit 1)
+		(exclude_from_sim no)
+		(in_bom yes)
+		(on_board yes)
+		(dnp no)
+		(fields_autoplaced yes)
+		(property "Reference" "#PWR016"
+			(at 144.78 113.03 0)
+			(effects
+				(font
+					(size 1.27 1.27)
+				)
+				(hide yes)
+			)
+		)
+		(property "Value" "GND"
+			(at 144.78 111.76 0)
+			(effects
+				(font
+					(size 1.27 1.27)
+				)
+			)
+		)
+		(property "Footprint" ""
+			(at 144.78 106.68 0)
+			(effects
+				(font
+					(size 1.27 1.27)
+				)
+				(hide yes)
+			)
+		)
+		(property "Datasheet" ""
+			(at 144.78 106.68 0)
+			(effects
+				(font
+					(size 1.27 1.27)
+				)
+				(hide yes)
+			)
+		)
+		(property "Description" "Power symbol creates a global label with name \"GND\" , ground"
+			(at 144.78 106.68 0)
+			(effects
+				(font
+					(size 1.27 1.27)
+				)
+				(hide yes)
+			)
+		)
+		(pin "1"
+		)
+		(instances
+			(project "Power_supply"
+				(path "/edc8412f-0483-47e1-aeb9-21064b18cc9b"
+					(reference "#PWR016")
+					(unit 1)
+				)
+			)
+		)
+	)
+	(symbol
 		(lib_id "Diode:BZX84Cxx")
 		(at 96.52 36.83 270)
@@
 					(unit 1)
 				)
+			)
+		)
+	)
+	(symbol
+		(lib_id "Device:C")
+		(at 144.78 102.87 0)
+		(unit 1)
+		(exclude_from_sim no)
+		(in_bom yes)
+		(on_board yes)
+		(dnp no)
+		(fields_autoplaced yes)
+		(property "Reference" "C6"
+			(at 148.336 101.6 0)
+			(effects
+				(font
+					(size 1.27 1.27)
+				)
+				(justify left)
+			)
+		)
+		(property "Value" "100nC"
+			(at 148.336 104.14 0)
+			(effects
+				(font
+					(size 1.27 1.27)
+				)
+				(justify left)
+			)
+		)
+		(property "Footprint" "Capacitor_SMD:C_1206_3216Metric"
+			(at 145.7452 106.68 0)
+			(effects
+				(font
+					(size 1.27 1.27)
+				)
+				(hide yes)
+			)
+		)
+		(property "Datasheet" "https://datasheet.lcsc.com/lcsc/2304140030_YAGEO-CC1206KRX7R9BB104_C82601.pdf"
+			(at 144.78 102.87 0)
+			(effects
+				(font
+					(size 1.27 1.27)
+				)
+				(hide yes)
+			)
+		)
+		(property "Description" ""
+			(at 144.78 102.87 0)
+			(effects
+				(font
+					(size 1.27 1.27)
+				)
+				(hide yes)
+			)
+		)
+		(property "MPN" "CC1206KRX7R9BB104"
+			(at 144.78 102.87 0)
+			(effects
+				(font
+					(size 1.27 1.27)
+				)
+				(hide yes)
+			)
+		)
+		(property "Status" "OK"
+			(at 144.78 102.87 0)
+			(effects
+				(font
+					(size 1.27 1.27)
+				)
+				(hide yes)
+			)
+		)
+		(pin "1"
+		)
+		(pin "2"
+		)
+		(instances
+			(project "Power_supply"
+				(path "/edc8412f-0483-47e1-aeb9-21064b18cc9b"
+					(reference "C6")
+					(unit 1)
+				)

Commit message: Progressed ECAD.
Connections:
- net SW_IN: now reaches J1.1, SW1.2 (B), SW1.5 (B)
- net SW_OUT: now reaches D1.2 (A2), Q1.5 (D), Q1.6 (D), Q1.7 (D), Q1.8 (D), SW1.3 (C), SW1.6 (C)
Changed lines of the file:
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@@
+		)
+	)
+	(label "SW_OUT"
+		(at 76.2 33.02 0)
+		(effects
+			(font
+				(size 1.27 1.27)
+			)
+			(justify left bottom)
+		)
+	)
+	(label "SW_IN"
+		(at 50.8 33.02 0)
+		(effects
+			(font
+				(size 1.27 1.27)
+			)
+			(justify left bottom)
 		)
 	)

Commit message: Progressed PCB
Connections:
- net PRE_FILTER: now reaches D4.3 (K), FL1.2, Q1.1 (S), Q1.2 (S), Q1.3 (S)
Changed lines of the file:
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@@
+		)
+	)
+	(label "PRE_FILTER"
+		(at 102.87 33.02 0)
+		(effects
+			(font
+				(size 1.27 1.27)
+			)
+			(justify left bottom)
 		)
 	)

Commit message: Added heatsink 3D model.
Parts:
- HS1, HS2, HS3: footprint Heatsink:Heatsink_Fischer_SK104-STC-STIC_35x13mm_2xDrill2.5mm -> Heatsink_custom:Heatsink_Fischer_SK104-STC-STIC_35x13mm_2xDrill2.5mm
Changed lines of the file:
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@@
 			)
 		)
-		(property "Footprint" "Heatsink:Heatsink_Fischer_SK104-STC-STIC_35x13mm_2xDrill2.5mm"
+		(property "Footprint" "Heatsink_custom:Heatsink_Fischer_SK104-STC-STIC_35x13mm_2xDrill2.5mm"
 			(at 101.9048 95.25 0)
 			(effects
@@
 			)
 		)
-		(property "Footprint" "Heatsink:Heatsink_Fischer_SK104-STC-STIC_35x13mm_2xDrill2.5mm"
+		(property "Footprint" "Heatsink_custom:Heatsink_Fischer_SK104-STC-STIC_35x13mm_2xDrill2.5mm"
 			(at 178.1048 95.25 0)
 			(effects
@@
 			)
 		)
-		(property "Footprint" "Heatsink:Heatsink_Fischer_SK104-STC-STIC_35x13mm_2xDrill2.5mm"
+		(property "Footprint" "Heatsink_custom:Heatsink_Fischer_SK104-STC-STIC_35x13mm_2xDrill2.5mm"
 			(at 101.9048 151.13 0)
 			(effects

Commit message: Progressed PCB.
Connections:
- net L2: now reaches L1.2, L2.1
- net L1: now reaches FL1.3, L1.1
Other:
- moved on the sheet: L2
Changed lines of the file:
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@@
 	(wire
 		(pts
-			(xy 154.94 33.02) (xy 158.75 33.02)
+			(xy 157.48 33.02) (xy 158.75 33.02)
 		)
 		(stroke
@@
 	(wire
 		(pts
-			(xy 146.05 33.02) (xy 147.32 33.02)
+			(xy 146.05 33.02) (xy 149.86 33.02)
 		)
 		(stroke
@@
 	(label "PRE_FILTER"
 		(at 102.87 33.02 0)
+		(effects
+			(font
+				(size 1.27 1.27)
+			)
+			(justify left bottom)
+		)
+	)
+	(label "L1"
+		(at 134.62 33.02 0)
+		(effects
+			(font
+				(size 1.27 1.27)
+			)
+			(justify left bottom)
+		)
+	)
+	(label "L2"
+		(at 146.05 33.02 0)
 		(effects
 			(font
@@
 	(symbol
 		(lib_id "Device:L_Ferrite")
-		(at 151.13 33.02 90)
+		(at 153.67 33.02 90)
 		(unit 1)
 		(exclude_from_sim no)
@@
 		(fields_autoplaced yes)
 		(property "Reference" "L2"
-			(at 151.13 26.67 90)
+			(at 153.67 26.67 90)
 			(effects
 				(font
@@
 		)
 		(property "Value" "10uL"
-			(at 151.13 29.21 90)
+			(at 153.67 29.21 90)
 			(effects
 				(font
@@
 		)
 		(property "Footprint" "Inductor_SMD:L_Taiyo-Yuden_NR-30xx"
-			(at 151.13 33.02 0)
+			(at 153.67 33.02 0)
 			(effects
 				(font
@@
 		)
 		(property "Datasheet" "https://datasheet.lcsc.com/lcsc/2304140030_Taiyo-Yuden-NR3015T100M_C87168.pdf"
-			(at 151.13 33.02 0)
+			(at 153.67 33.02 0)
 			(effects
 				(font
@@
 		)
 		(property "Description" ""
-			(at 151.13 33.02 0)
+			(at 153.67 33.02 0)
 			(effects
 				(font
@@
 		)
 		(property "MPN" "NR3015T100M"
-			(at 151.13 33.02 0)
+			(at 153.67 33.02 0)
 			(effects
 				(font
@@
 		)
 		(property "Status" "OK"
-			(at 151.13 33.02 0)
-			(effects
-				(font
+			(at 153.67 33.02 0)
+			(effects
+				(font
