File: ECAD/Power_supply/Power_supply.kicad_pcb (KiCad board)
At the start: 2 copper layers, 40 parts, among them J1 Barrel_Jack_Switch, J2 Conn_01x06, Q1 DMP3037LSS-13, SW1 SW_Push_DPDT, U1 LM317_TO-220, U2 LM317_TO-220

Commit message: Progressed PCB layout.
Parts:
- J2: footprint Connector_PinHeader_2.54mm:PinHeader_1x06_P2.54mm_Horizontal -> Connector_PinSocket_2.54mm:PinSocket_1x06_P2.54mm_Vertical
- moved J1 88.9 mm to (180.0, 48.0), turned to 180 degrees
- moved SW1 86.7 mm to (186.4, 62.0)
- moved FL1 86.1 mm to (149.0, 45.0)
- moved L1 78.6 mm to (137.0, 44.0)
- moved Q1 75.5 mm to (161.0, 45.4)
- moved R6 74.9 mm to (117.8, 44.0)
- moved D1 67.9 mm to (171.0, 44.0)
- moved R2 67.9 mm to (155.0, 138.2)
- moved R5 67.9 mm to (155.0, 147.0)
- moved C10 65.9 mm to (115.8, 57.0)
- moved D7 62.2 mm to (182.0, 75.0)
- moved R7 62.2 mm to (189.8, 77.5)
- moved C2 56.8 mm to (158.0, 124.8)
- moved C6 56.8 mm to (163.6, 121.4)
- moved C4 56.8 mm to (158.0, 131.4)
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Connections:
- J2 pad 1: +12V -> +5V
- J2 pad 3: +9V -> +12V
- J2 pad 5: +5V -> +9V
Other:
- board outline added: 104 x 127 mm

Commit message: Updated the schematic.
Parts:
- added C1: 10uC, Capacitor_SMD:C_1206_3216Metric, F.Cu at (257.2, 152.8)
- added C16: 100nC, Capacitor_SMD:C_1206_3216Metric, F.Cu at (250.1, 149.2)
- added C17: 10uC, Capacitor_SMD:C_1206_3216Metric, F.Cu at (257.2, 156.1)
- added C18: 100nC, Capacitor_SMD:C_1206_3216Metric, F.Cu at (250.2, 156.1)
- added C19: 100pC, Capacitor_SMD:C_0805_2012Metric, F.Cu at (249.6, 159.2)
- added D8: S1A-13-F, Diode_SMD:D_SMA, F.Cu at (238.9, 149.8)
- added D9: S1A-13-F, Diode_SMD:D_SMA, F.Cu at (238.9, 154.3)
- added HS3: Heatsink, Heatsink:Heatsink_Fischer_SK104-STC-STIC_35x13mm_2xDrill2.5mm, F.Cu at (241.5, 140.2)
- added R8: 720R, Resistor_SMD:R_0805_2012Metric, F.Cu at (245.1, 149.0)
- added R8: 340R, Resistor_SMD:R_0805_2012Metric, F.Cu at (256.6, 159.2)
- added R9: 240R, Resistor_SMD:R_0805_2012Metric, F.Cu at (245.1, 151.9)
- added U3: LM317_TO-220, Package_TO_SOT_THT:TO-220-3_Vertical, F.Cu at (226.5, 151.4)
- moved C6 132.2 mm to (264.9, 36.4)
- moved C8 132.2 mm to (264.9, 43.1)
- moved HS2 132.2 mm to (235.3, 44.0)
- moved R2 132.2 mm to (256.3, 53.1)
- moved R5 132.2 mm to (256.3, 62.0)
- moved C2 132.2 mm to (259.3, 39.8)
- moved C4 132.2 mm to (259.3, 46.5)
- moved D3 132.2 mm to (245.5, 62.6)
- moved U2 132.2 mm to (232.8, 40.9)
- moved D6 131.3 mm to (234.0, 61.0)
- moved C1 101.8 mm to (254.4, 85.4)
- moved C3 101.8 mm to (254.4, 92.1)
- moved C5 101.8 mm to (254.4, 98.8)
- moved C7 101.8 mm to (260.1, 88.8)
- moved HS1 101.8 mm to (233.3, 91.0)
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Connections:
- C1 pad 1: +12V -> Net-(D2-K)
- D2 pad 1: +12V -> +8V
- U1 pad 3: +12V -> +8V
Routing:
- added copper zone on B.Cu, net GND

Commit message: Progressed PCB.
Parts:
- removed the C1 at (254.4, 85.4)
- removed the R8 at (245.1, 149.0)
- added H1: MountingHole, MountingHole:MountingHole_3.2mm_M3, F.Cu at (95.8, 41.8)
- added H2: MountingHole, MountingHole:MountingHole_3.2mm_M3, F.Cu at (190.0, 39.8)
- added H3: MountingHole, MountingHole:MountingHole_3.2mm_M3, F.Cu at (96.2, 157.2)
- added H4: MountingHole, MountingHole:MountingHole_3.2mm_M3, F.Cu at (189.0, 157.8)
- added REF**: Symbol_Barrel_Polarity, Symbol:Symbol_Barrel_Polarity, F.Cu at (185.5, 67.8)
- added REF**: Polarity_Center_Positive_6mm_SilkScreen, Symbol:Polarity_Center_Positive_6mm_SilkScreen, F.Cu at (179.5, 82.0)
- added REF**: KiCad-Logo2_5mm_SilkScreen, Symbol:KiCad-Logo2_5mm_SilkScreen, F.Cu at (185.0, 72.2)
- D9: moved to B.Cu
- moved R8 140.2 mm to (121.8, 120.8), turned to -90 degrees
- moved C19 135.6 mm to (119.5, 120.8), turned to -90 degrees
- moved C17 134.2 mm to (126.0, 128.0)
- moved R9 123.3 mm to (126.0, 119.8), turned to 180 degrees
- moved C1 123.3 mm to (137.2, 124.2)
- moved C18 121.7 mm to (130.5, 134.0)
- moved C16 121.6 mm to (132.1, 120.0)
- moved D3 120.8 mm to (129.4, 95.9)
- moved D6 120.8 mm to (117.9, 94.2)
- moved R5 120.8 mm to (140.2, 95.2)
- moved HS3 117.9 mm to (127.3, 111.0)
- moved D9 117.8 mm to (129.3, 111.0), turned to 180 degrees
- moved C3 117.6 mm to (148.7, 143.6)
- moved C5 117.6 mm to (148.7, 150.3)
- moved C7 117.6 mm to (154.3, 140.2)
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Connections:
- HS1 pad 1: unconnected-(HS1-Pad1)_1 -> +5V
- HS2 pad 1: unconnected-(HS2-Pad1)_1 -> +9V
- HS3 pad 1: unconnected-(HS3-Pad1) -> +8V

Commit message: Progressed PCB.
Parts:
- moved C11 141.6 mm to (234.9, 97.7)
- moved C12 141.6 mm to (234.9, 101.0)
- moved C9 141.6 mm to (233.8, 108.8)
- moved D1 141.6 mm to (302.9, 95.8)
- moved FL1 141.6 mm to (280.9, 96.8)
- moved L1 141.6 mm to (268.9, 95.8)
- moved L2 141.6 mm to (260.6, 95.8)
- moved Q1 141.6 mm to (292.9, 97.1)
- moved R3 141.6 mm to (292.3, 103.8)
- moved C10 141.6 mm to (247.6, 108.8)
- moved D4 141.6 mm to (292.3, 109.7)
- moved R6 141.6 mm to (249.6, 95.8)
- moved C13 141.6 mm to (241.5, 93.7)
- moved C14 141.6 mm to (241.5, 97.0)
- moved C15 141.6 mm to (241.5, 100.3)
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
Commit message: Progressed PCB.
Parts:
- removed C18: 100nC, Capacitor_SMD:C_1206_3216Metric
- removed C6, C7, C8: 10uC, Capacitor_SMD:C_1206_3216Metric
- removed REF**: Symbol_Barrel_Polarity, Symbol:Symbol_Barrel_Polarity
- removed REF**: Polarity_Center_Positive_6mm_SilkScreen, Symbol:Polarity_Center_Positive_6mm_SilkScreen
- removed REF**: KiCad-Logo2_5mm_SilkScreen, Symbol:KiCad-Logo2_5mm_SilkScreen
- added C20: 22uC, Capacitor_SMD:CP_Elec_5x5.4, F.Cu at (146.5, 59.5)
- C1, C5: value 10uC -> 22uC; footprint Capacitor_SMD:C_1206_3216Metric -> Capacitor_SMD:CP_Elec_5x5.4
- moved C2 112.5 mm to (147.3, 156.0), turned to -90 degrees
- moved C4 109.7 mm to (138.9, 158.2), turned to -90 degrees
- moved R2 102.9 mm to (136.4, 158.1), turned to -90 degrees
- moved D6 95.2 mm to (132.6, 154.4)
- moved R5 91.8 mm to (134.6, 150.4), turned to -90 degrees
- moved C3 91.3 mm to (151.8, 52.4)
- moved D2 91.3 mm to (133.7, 67.8)
- moved D5 91.3 mm to (132.7, 60.2)
- moved R1 91.3 mm to (157.8, 55.4)
- moved R4 91.3 mm to (157.8, 64.2)
- moved D3 84.6 mm to (136.1, 145.3), turned to 180 degrees
- moved C5 32.3 mm to (116.8, 155.9), turned to -90 degrees
- moved HS1 19.4 mm to (134.9, 136.4), turned to 0 degrees
- moved U1 12.4 mm to (132.3, 140.7), turned to 0 degrees
- moved C1 8.68 mm to (147.5, 105.0)
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Connections:
- C4 pad 1: Net-(D6-A) -> /ADJ_9V
- C5 pad 1: +5V -> +9V
- D6 pad 2: Net-(D6-A) -> /ADJ_9V
- HS1 pad 1: +5V -> +9V
- HS2 pad 1: +9V -> +5V
- R2 pad 1: Net-(D6-A) -> /ADJ_9V
- R5 pad 2: Net-(D6-A) -> /ADJ_9V
- U1 pad 1: Net-(D5-A) -> /ADJ_9V
- U1 pad 2: +5V -> +9V
- U1 pad 3: +8V -> +12V
- U2 pad 1: Net-(D6-A) -> Net-(D5-A)
- U2 pad 2: +9V -> +5V
- U2 pad 3: +12V -> +8V
Routing:
- net /ADJ_9V: track 0.00 -> 14.3 mm, vias 0 -> 1
- net GND: vias 0 -> 4
- added copper zone on F.Cu, net +12V
- added copper zone on F.Cu, net +9V
- added copper zone on F.Cu, net /ADJ_9V
- added copper zone on F.Cu, net GND

Commit message: Progressed PCB layout.
Parts:
- added C6: 100nC, Capacitor_SMD:C_1206_3216Metric, F.Cu at (142.7, 90.2)
- D9: moved to F.Cu
- moved C5 64.4 mm to (52.5, 154.7)
- moved R5 64.4 mm to (70.2, 149.2)
- moved C2 64.4 mm to (82.9, 154.8)
- moved D6 64.4 mm to (68.2, 153.2)
- moved R2 64.4 mm to (72.0, 156.9)
- moved C4 64.4 mm to (74.5, 157.1)
- moved R8 59.3 mm to (162.8, 54.2)
- moved C1 59.3 mm to (174.3, 52.1)
- moved C16 59.3 mm to (161.1, 44.6)
- moved C17 59.3 mm to (155.1, 52.6)
- moved C19 59.3 mm to (158.8, 56.1)
- moved R9 59.3 mm to (155.1, 44.3)
- moved R1 46.6 mm to (160.9, 101.9)
- moved C20 46.6 mm to (149.6, 106.0)
- moved D5 46.6 mm to (135.8, 106.8)
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Connections:
- net Net-(D5-A) renamed /ADJ_5V
- net Net-(D8-A) renamed /ADJ_PRE
Routing:
- net /ADJ_PRE: track 0.00 -> 18.4 mm, vias 0 -> 1
- net /ADJ_5V: track 0.00 -> 18.4 mm, vias 0 -> 1
- net /ADJ_9V: track 14.3 -> 18.4 mm
- net GND: vias 4 -> 0
- removed copper zone on F.Cu, net +12V
- removed copper zone on F.Cu, net +9V
- removed copper zone on F.Cu, net /ADJ_9V

Commit message: Progressed PCB.
Parts:
- moved C1 36.4 mm to (141.0, 66.7)
- moved R9 23.8 mm to (134.6, 56.5), turned to 0 degrees
- moved R8 22.4 mm to (141.0, 59.1), turned to 0 degrees
- moved C16 21.5 mm to (141.0, 52.1)
- moved C19 18.7 mm to (141.0, 61.6), turned to 0 degrees
- moved C17 14.7 mm to (141.0, 56.5)
- moved D8 4.45 mm to (134.6, 61.6)
Routing:
- net /ADJ_PRE: track 18.4 -> 13.3 mm
- net GND: vias 0 -> 6
- added copper zone on F.Cu, net +12V
- added copper zone on F.Cu, net +8V
- added copper zone on F.Cu, net /ADJ_PRE
- removed copper zone on B.Cu, net GND
- removed copper zone on F.Cu, net GND

Commit message: Progressed PCB.
Parts:
- moved R4 28.5 mm to (134.6, 99.7)
- moved R1 19.9 mm to (141.0, 102.2)
- moved C20 15.7 mm to (134.6, 110.5)
- moved C3 14.0 mm to (141.0, 99.7)
- moved C6 9.87 mm to (134.6, 95.9)
- moved C16 7.85 mm to (133.3, 50.2), turned to 90 degrees
- moved C1 6.38 mm to (134.6, 67.3)
- moved D5 2.33 mm to (134.6, 104.8)
Routing:
- net /ADJ_5V: track 18.4 -> 13.3 mm
- net GND: vias 6 -> 14
- net +5V: vias 0 -> 1
- added copper zone on B.Cu, net +5V
- added copper zone on F.Cu, net +5V
- added copper zone on F.Cu, net +9V
- added copper zone on F.Cu, net /ADJ_5V
- added copper zone on B.Cu, net GND
- added copper zone on F.Cu, net GND
